File: DSO_Hardware/Digital Interface/FPGA.sch (KiCad schematic (older format))
At the start: 45 parts, among them Q1 DMN62D0UW, SW1 SW_Push, U7 EEPROM, U8 XC6SLX9-2TQG144C, X1 ASE-xxxMHz

Commit message: Digital Interface Breakout WIP
Also added programming issue warning (M1 pin being used twice) to digital interface schematic.
Other:
- note added: "Pin 60 is Duplicated\nBoth M1 & D2A+ on same pin\nUsed 1k pulldown on Rev.1"
Changed lines of the file:
@@
 Text Notes 7650 800  0    60   ~ 0
 TMS & TDO Swapped in Rev1
+Text Notes 9050 3600 0    60   ~ 0
+Pin 60 is Duplicated\nBoth M1 & D2A+ on same pin\nUsed 1k pulldown on Rev.1
 $EndSCHEMATC
