File: DSO_Hardware/Digital Interface/Breakout_Board/DI_Breakout/DI_Breakout.kicad_pcb (KiCad board)
At the start: 2 copper layers, 63 x 21 mm, 20 parts, among them J1 Conn_02x14_Odd_Even, J2 FX18-80P-0.8SH, U1 LP2980-3.3

Commit message: Finished DI_Breakout
Parts:
- removed H3, H4: MountingHole, MountingHole:MountingHole_2.7mm_M2.5_ISO14580_Pad
- moved R3 14.0 mm to (120.6, 117.3), turned to 180 degrees
- moved R8 14.0 mm to (123.1, 117.3), turned to 180 degrees
- moved R9 11.4 mm to (138.3, 117.3), turned to 180 degrees
- moved R10 11.3 mm to (133.2, 117.3), turned to 180 degrees
- moved R4 11.3 mm to (135.8, 117.3), turned to 180 degrees
- moved R5 11.3 mm to (130.8, 117.3), turned to 180 degrees
- moved R2 1.91 mm to (140.9, 117.3), turned to 180 degrees
- moved C2 1.81 mm to (156.8, 117.5)
- moved U1 1.81 mm to (156.8, 120.6)
- moved R1 1.64 mm to (148.5, 117.3), turned to 180 degrees
- moved R6 1.64 mm to (151.0, 117.3), turned to 180 degrees
- moved R7 1.61 mm to (145.4, 117.3)
- moved R11 1.58 mm to (143.4, 117.3), turned to 180 degrees
- moved C1 1.46 mm to (156.6, 123.7)
- moved J1 1.22 mm to (152.8, 120.0)
Connections:
- J1 pad 14: /FE_SDA -> /~PGA_CS_4
- J1 pad 16: /FE_SCL -> /~PGA_CS_3
- J1 pad 18: /FE_SCLK -> /~PGA_CS_2
- J1 pad 20: /FE_SDIO -> /~PGA_CS_1
- J1 pad 22: /~PGA_CS_4 -> /FE_SCLK
- J1 pad 24: /~PGA_CS_3 -> /FE_SDIO
- J1 pad 26: /~PGA_CS_2 -> /FE_SDA
- J1 pad 28: /~PGA_CS_1 -> /FE_SCL
Routing:
- net +3V3: track 0.00 -> 49.5 mm
- net GND: track 2.97 -> 29.4 mm, vias 0 -> 8
- net +5V: track 0.00 -> 22.5 mm
- net /~PGA_CS_4: track 5.59 -> 24.9 mm, vias 0 -> 1
- net /~PGA_CS_3: track 5.66 -> 24.5 mm, vias 0 -> 1
- net /FE_SDIO: track 13.6 -> 6.60 mm
- net /FE_SCLK: track 15.2 -> 8.34 mm
- net /FE_SDA: track 28.6 -> 23.2 mm, vias 1 -> 0
- net /FE_SCL: track 26.9 -> 22.7 mm, vias 1 -> 0
- net /~PGA_CS_1: track 20.1 -> 23.8 mm, vias 0 -> 1
- net /~PGA_CS_2: track 20.7 -> 24.1 mm, vias 0 -> 1
- net /~PLL_LE: track 30.4 -> 27.9 mm
- net /~ADC_CS: track 31.2 -> 29.7 mm
- net /ADC_PLL_SDIO: track 26.1 -> 24.6 mm
- net /ADC_PLL_SCLK: track 27.7 -> 26.3 mm
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- added copper zone on B.Cu, net GND
Other:
- board size 63 x 21 mm -> 63 x 19 mm
- net class Default: clearance 0.1524 -> 0.1778
- net class PWR added: clearance 0.1778, trace_width 0.2032, via_dia 0.508, via_drill 0.254
- rule trace_clearance: 0.1524 -> 0.1778
- board text added: "ADC"
- board text added: "FE"
- board text added: "GND"
- board text added: "I2C"
- board text added: "PD"
- board text added: "PLL ADC SPI"
- board text added: "SCK"
- board text added: "SCL"
- board text added: "SCLK"
- board text added: "SDA"
- board text added: "SDIO"
- board text added: "SDO"
- board text added: "SPI"
- board text added: "~A_CS"
- board text added: "~CS1"
- board text added: "~CS2"
- board text added: "~CS3"
- board text added: "~CS4"
- board text added: "~P_LE"
- board text added: "~RST"
