File: DSO_Hardware/FE/FFE Rev3/FFE_REV3.sch (KiCad schematic (older format))
At the start: 75 parts, among them J1 BNC, J2 SMA, J3 Conn_02x07_Odd_Even, K1 FTR-B3GA, Q1 CPH3910, Q2 2N3904, Q3 DMN62D0UW, U1 OP07, U2 CPC1014, U3 OP07, U4 LM27761

Commit message: Final FFE Rev.3 Commit
Parts:
- C8: Voltage (none) -> 100V; Voltage Rating 100V -> (none)
- R26: value 300 -> 300k
Changed lines of the file:
@@
 P 9900 4350
 F 0 "R26" V 9980 4350 50  0000 C CNN
-F 1 "300" V 9900 4350 50  0000 C CNN
+F 1 "300k" V 9900 4350 50  0000 C CNN
 F 2 "Resistor_SMD:R_0402_1005Metric" V 9830 4350 50  0001 C CNN
 F 3 "" H 9900 4350 50  0001 C CNN
@@
 F 2 "Capacitor_SMD:C_0603_1608Metric" H 2038 1550 50  0001 C CNN
 F 3 "" H 2000 1700 50  0001 C CNN
-F 4 "100V" H 2115 1655 50  0000 L CNN "Voltage Rating"
+F 4 "100V" H 2115 1655 50  0000 L CNN "Voltage"
 F 5 "0603" H 2115 1564 50  0000 L CNN "Package"
 	1    2000 1700
