File: Hardware/KiCad/FPGA_Module_Rev2/FPGA_CFG.kicad_sch (KiCad schematic)
At the start: 19 parts, among them Q1 DMN62D0UW, U1 IC FPGA XC7A50T-2CSG325C, U2 MX25U6432FZNI02, U3 TXB0104RUTR

Commit message: Adding the KiCad Design for the FPGA Module Board with no DRC errors
Other:
- note added: "8MB"
- note added: "CONFIGURATION SPI FLASH"
- note added: "FPGA CONFIGURATION BANK"
- note added: "FPGA_CFG"
- moved on the sheet: C1, C2, C3, FB2, Q1, R12, R13, R14, R15, TP1, TP10, TP11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
