File: Hardware/KiCad/FPGA_Module_Rev2/FPGA_PWR.kicad_sch (KiCad schematic)
At the start: 45 parts, among them U1 IC FPGA XC7A50T-2CSG325C

Commit message: Adding the KiCad Design for the FPGA Module Board with no DRC errors
Other:
- note added: "FPGA_POWER"
- note added: "GND"
- moved on the sheet: C29, C30, C31, C32, C33, C34, C35, C36, C37, C38, C39, C40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
