File: Hardware/KiCad/FPGA_Module_Rev2/TS_FPGA_Module_Rev2.kicad_sch (KiCad schematic)
At the start: 0 parts

Commit message: Adding the KiCad Design for the FPGA Module Board with no DRC errors
Parts:
- added FID1, FID2, FID3, FID4, FID5, FID6, FID7, FID8: PCB, DSO.PcbLib:GEN_FID, symbol scratch-altium-import:root_0_FID 1mm
- added JM1, JM2: LSHM-150-04.0-L-DV-A-S-K-TR, DSO.PcbLib:SAM_LSHM-150-XX.X-XX-DV-A-S, symbol scratch-altium-import:root_0_mirrored_CONN LSHM-150-04.0-L-DV-A-S-K-TR
- added JM3: LSHM-130-04.0-L-DV-A-S-K-TR, DSO.PcbLib:SAM_LSHM-130-XX.X-XX-DV-A-S, symbol scratch-altium-import:root_0_CONN LSHM-130-04.0-L-DV-A-S-K-TR
- added MH1, MH2, MH3, MH4: M3, Custom_Footprints:MH M3, symbol scratch-altium-import:root_0_MH M3
- added Q2: DMN62D0UW, DSO.PcbLib:GEN_SOT_323, symbol scratch-altium-import:root_0_mirrored_NMOS DMN62D0UW
- added R59: 4.7K, DSO.PcbLib:GEN_R_0201, symbol scratch-altium-import:root_3_RES 4.7K OHM 1% 1/20W 0201
- added R62: 100, DSO.PcbLib:GEN_R_0201, symbol scratch-altium-import:root_2_RES 100 OHM 1% 1/20W 0201
Connections:
- new net +1V8: JM2.91
- new net +3V3_IN: JM1.1, JM1.13, JM1.15, JM1.3, JM1.5
- new net ACQ_EN: JM2.51
- new net ADC_CSn: JM2.65
- new net ADC_PD: JM2.61
- new net ADC_PG: JM2.67
- new net ADC_RSTn: JM2.63
- new net ADC_SCLK: JM2.41
- new net ADC_SDATA: JM2.43
- new net ATTEN_1: JM2.38
- new net ATTEN_2: JM2.48
- new net ATTEN_3: JM2.56
- new net ATTEN_4: JM2.64
- new net D1A_N: JM1.58
- new net D1A_P: JM1.56
- new net D1B_N: JM1.62
- new net D1B_P: JM1.60
- new net D2A_N: JM1.68
- new net D2A_P: JM1.66
- new net D2B_N: JM1.72
- new net D2B_P: JM1.70
- new net D3A_N: JM1.82
- new net D3A_P: JM1.80
- new net D3B_N: JM1.88
- new net D3B_P: JM1.86
- new net D4A_N: JM1.96
- new net D4A_P: JM1.94
- new net D4B_N: JM1.100
- new net D4B_P: JM1.98
- new net DC_CPL_1: JM2.42
- new net DC_CPL_2: JM2.52
- new net DC_CPL_3: JM2.58
- new net DC_CPL_4: JM2.66
- new net FCLK_N: JM1.77
- new net FCLK_P: JM1.75
- new net FE_EN: JM2.53
- new net FE_PG: JM2.45
- new net GND: JM1.101, JM1.102, JM1.2, JM1.20, JM1.26, JM1.29, JM1.34, JM1.44, JM1.53, JM1.54, JM1.63, JM1.64, JM1.73, JM1.74, JM1.8, JM1.84, JM1.90, JM2.101, JM2.102, JM2.20, JM2.30, JM2.39, JM2.40, JM2.49, JM2.50, JM2.59, JM2.60, JM2.69, JM2.70, JM2.79, JM2.80, JM2.90, JM3.11, JM3.12, JM3.17, JM3.18, JM3.23, JM3.24, JM3.29, JM3.30, JM3.35, JM3.36, JM3.45, JM3.46, JM3.5, JM3.6, JM3.61, JM3.62, MH1.1, MH2.1, MH3.1, MH4.1, Q2.3 (S), R59.2
- new net LCLK_N: JM1.61
- new net LCLK_P: JM1.59
- new net LED: R62.1
- new net LED_3V3: JM1.95, Q2.1 (D)
- new net MGT_CLK1_N: JM3.31
- new net MGT_CLK1_P: JM3.33
- new net MGT_RX0_N: JM3.8
- new net MGT_RX0_P: JM3.10
- new net MGT_RX1_N: JM3.14
- new net MGT_RX1_P: JM3.16
- new net MGT_RX2_N: JM3.20
- new net MGT_RX2_P: JM3.22
- new net MGT_RX3_N: JM3.26
- new net MGT_RX3_P: JM3.28
- new net MGT_TX0_N: JM3.7
- new net MGT_TX0_P: JM3.9
- new net MGT_TX1_N: JM3.13
- new net MGT_TX1_P: JM3.15
- new net MGT_TX2_N: JM3.19
- new net MGT_TX2_P: JM3.21
- new net MGT_TX3_N: JM3.25
- new net MGT_TX3_P: JM3.27
- new net NetQ2_2: Q2.2 (G), R59.1, R62.2
- new net OSC_OE: JM2.47
- new net PERST#: JM3.59
- new net PGA_CSn_1: JM2.36
- new net PGA_CSn_2: JM2.46
- new net PGA_CSn_3: JM2.54
- new net PGA_CSn_4: JM2.62
- new net PGA_SCLK: JM2.34
- new net PGA_SDIO: JM2.32
- new net PROBE_COMP: JM2.44
- new net SCL: JM2.57
- new net SDA: JM2.55
- new net SYNC: JM1.93
- new net TCK: JM2.99
- new net TDI: JM2.95
- new net TDO: JM2.97
- new net TMS: JM2.93
- no-connect marks 0 -> 140
Other:
- sheet FPGA_Bank_IO renamed FPGA_Bank_34_IO
- sheet FPGA_Banks_DDR3 renamed FPGA_Banks_14_15_DDR3
- sheet PWR renamed Board_PWR
- removed sheet Connectors
- sheet Board_PWR: file PWR.kicad_sch -> Board_PWR.kicad_sch
- sheet FPGA_Bank_34_IO: file FPGA_Bank_IO.kicad_sch -> FPGA_Bank_34_IO.kicad_sch
- sheet FPGA_Bank_34_IO ports: added ACQ_EN, ADC_CSn, ADC_PD, ADC_PG, ADC_RSTn, ADC_SCLK, ADC_SDATA, ATTEN_1, ATTEN_2, ATTEN_3, ATTEN_4, D1A_N, D1A_P, D1B_N, D1B_P, D2A_N, D2A_P, D2B_N, D2B_P, D3A_N, D3A_P, D3B_N, D3B_P, D4A_N, D4A_P, D4B_N, D4B_P, DC_CPL_1, DC_CPL_2, DC_CPL_3, DC_CPL_4, FCLK_N, FCLK_P, FE_EN, FE_PG, LCLK_N, LCLK_P, OSC_OE, PERST#, PGA_CSn_1, PGA_CSn_2, PGA_CSn_3, PGA_CSn_4, PGA_SCLK, PGA_SDIO, PROBE_COMP, SCL, SDA, SYNC; removed none
- sheet FPGA_Banks_14_15_DDR3: file FPGA_Banks_DDR3.kicad_sch -> FPGA_Banks_14_15_DDR3.kicad_sch
- sheet FPGA_Banks_14_15_DDR3 ports: added LED, SPI_CS_1V35, SPI_DQ0_1V35, SPI_DQ1_1V35, SPI_DQ2_1V35, SPI_DQ3_1V35; removed none
- sheet FPGA_CFG ports: added SPI_CS_1V35, SPI_DQ0_1V35, SPI_DQ1_1V35, SPI_DQ2_1V35, SPI_DQ3_1V35, TCK, TDI, TDO, TMS; removed none
- sheet FPGA_MGT ports: added MGT_CLK1_N, MGT_CLK1_P, MGT_RX0_N, MGT_RX0_P, MGT_RX1_N, MGT_RX1_P, MGT_RX2_N, MGT_RX2_P, MGT_RX3_N, MGT_RX3_P, MGT_TX0_N, MGT_TX0_P, MGT_TX1_N, MGT_TX1_P, MGT_TX2_N, MGT_TX2_P, MGT_TX3_N, MGT_TX3_P; removed none
- note added: "256MB"
- note added: "3.3VIN"
- note added: "ADC"
- note added: "ADC Diff Pairs on JM1"
- note added: "ARTIX 50T"
- note added: "B13_L13_N"
- note added: "B15_L10_N"
- note added: "B15_L10_P"
- note added: "B15_L11_N"
- note added: "B15_L11_P"
- note added: "B15_L12_N"
- note added: "B15_L12_P"
- note added: "B15_L13_N"
- note added: "B15_L13_P"
- note added: "B15_L14_N"
- note added: "B15_L14_P"
- note added: "B15_L16_N"
- note added: "B15_L16_P"
- note added: "B15_L17_N"
- note added: "B15_L17_P"
- note added: "B15_L18_P"
- note added: "B15_L19_N"
- note added: "B15_L19_P"
- note added: "B15_L23_N"
- note added: "B15_L23_P"
- note added: "B15_L3_N"
- note added: "B15_L3_P"
- note added: "B15_L7_N"
- note added: "B15_L7_P"
- note added: "B15_L8_N"
- note added: "B15_L8_P"
- note added: "B15_L9_N"
- note added: "B15_L9_P"
- note added: "BOARD POWER"
- note added: "CLK"
- note added: "CONFIG"
- note added: "FE CH"
- note added: "FIDUCIALS AND MOUNTING HOLES"
- note added: "I2C"
- note added: "INTER-BOARD CONNECTORS"
- note added: "JTAG"
- note added: "JTAG_VREF"
- note added: "LED"
- note added: "MISC"
- note added: "Other IO on JM2"
- note added: "THUNDERSCOPE FPGA MODULE Rev2"
- note added: "These connectors are hermaphroditic. Odd pin numbers on the module are connected to even pin numbers on the baseboard and vice versa."
