File: Hardware/KiCad/HMCAD1520_Impedence_Checker/HMCAD1520_Impedence_Checker.kicad_sch (KiCad schematic)
At the start: 21 parts, among them J1 Conn_01x01, J2 Conn_01x20, J3 Conn_01x20, J4 Conn_01x01, K1 EE2-5NU, K2 EE2-5NU, K3 EE2-5NU, Q1 DMN61D8LQ, Q2 DMN61D8LQ, Q3 DMN61D8LQ

Commit message: Finished HMCAD1520 Impedance Checker
Parts:
- removed J2, J3: Conn_01x20, Connector_PinSocket_2.54mm:PinSocket_1x20_P2.54mm_Vertical, symbol Connector_Generic:Conn_01x20
- added D5, D6, D7, D8: ESD9B5.0ST5G, Diode_SMD:D_SOD-923, symbol Diode:ESD9B5.0ST5G
- added U2: Pico, MCU_RaspberryPi_and_Boards:RPi_Pico_SMD_TH, symbol MCU_RaspberryPi_and_Boards:Pico
- J1, J4: footprint (none) -> ThunderScope:CT3151
- U1: value ~ -> HMCAD1520; footprint (none) -> ThunderScope:3M_248-5205-01; symbol EEVengers:HMCAD1520 -> ThunderScope:HMCAD1520
Connections:
- net +5V: now also U2.39 (VSYS), U2.40 (VBUS)
- net AVDD: now also D5.2 (A2)
- net AVDD2: now also D6.2 (A2)
- net DVDD: now also D8.2 (A2)
- net GND: now also D5.1 (A1), D6.1 (A1), D7.1 (A1), D8.1 (A1), U2.13 (GND), U2.18 (GND), U2.23 (GND), U2.28 (GND), U2.3 (GND), U2.38 (GND), U2.42 (GND), U2.8 (GND)
- net OVDD: now also D7.2 (A2)
- net SEL0: now also U2.22 (GPIO17)
- net SEL1: now also U2.21 (GPIO16)
- net SEL2: now also U2.20 (GPIO15)
- no-connect marks 45 -> 75
Other:
- moved on the sheet: D1, D2, D3, D4, J1, J4, K1, K2, K3, Q1, Q2, Q3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
