File: Hardware/KiCad/Thunderscope_Rev5/PWR.kicad_sch (KiCad schematic)
At the start: 74 parts, among them J10 009155002852006, J9 B2B-PH-K-S(LF)(SN), U12 TPS7A9101, U13 LM27761, U14 TPS7A9101, U15 TPS7A9101, U16 TPS7A2033, U17 TPS61023

Commit message: Linked PCB to Schematic
Connections:
- no-connect marks 1 -> 0
Other:
- moved on the sheet: TP22

Commit message: Added WIP Mech Model and Interposer
Also reworked rev5 power tree
Parts:
- removed C113: ${ALTIUM_VALUE}, GEN_C_0402, symbol Thunderscope_Rev5:CAP 100nF 16V X7R 0402
- removed J10: 009155002852006, KYO_009155002852006, symbol Thunderscope_Rev5:CONN SPRING 2 PIN
- removed J9: B2B-PH-K-S(LF)(SN), JST_B2B-PH-K-S(LF)(SN), symbol Thunderscope_Rev5:CONN JST PH 2 Pin TH
- removed R55: ${ALTIUM_VALUE}, GEN_R_0603, symbol Thunderscope_Rev5:RES 0.01 OHM 1% 1/4W 0603
- removed R92: ${ALTIUM_VALUE}, GEN_R_0402, symbol Thunderscope_Rev5:RES 10K OHM 1% 1/10W 0402
- removed R95: ${ALTIUM_VALUE}, GEN_R_0402, symbol Thunderscope_Rev5:RES 4.7K OHM 1% 1/10W 0402
- removed TP23: 5015, KEY_5015, symbol Thunderscope_Rev5:TP KEYSTONE 5015
- removed U12: TPS7A9101, TI_WSON10_DSK0010A, symbol Thunderscope_Rev5:IC LDO TPS7A9101
- added C?: ${ALTIUM_VALUE}, GEN_C_0402, symbol Thunderscope_Rev5:CAP 1uF 25V X5R 0402
- added U?: TPS7A2033, GEN_SOT23_5_950_2900X1600X1450, symbol Thunderscope_Rev5:IC LDO TPS7A2033
- TP26, TP27, TP28, TP29, TP30, TP31, TP32, TP33, TP34, TP35, TP36, TP37, TP38, TP39, TP40: now left out of the parts list
Connections:
- net +3V3 is gone; now on net +VUSB: R89.1, TP30.1
- net +3V3_PGA: now also C?.1
- net GND: now also C?.2, U?.2 (GND)
- net at C107.2, C108.2, R89.2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: now also U?.1 (IN)
- net +2V5_ACQ renamed +3V3_ACQ
- net +3V3_ACQ: now also U?.5 (OUT)
- net +2V5_ACQ_EN renamed +3V3_ACQ_EN
- net +3V3_ACQ_EN: now also U?.3 (EN)
Other:
- note added: "3.3/5 = 66.7% efficiency"
- note added: "TODO: Hook up power good"
- note removed: "2.5/3.3 = 75.7% efficiency"
- note removed: "Vout = 0.8 * (10/4.7 +1)"
- note removed: "Vout = 2.50V"
- moved on the sheet: C106, C107, C108, C109, C110, C111, C112, C114, C127, C128, L1, R108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
