File: Hardware/KiCad/Thunderscope_Rev5/FPGA_CFG.kicad_sch (KiCad schematic)
At the start: 7 parts, among them U18 IC FPGA XC7A50T-2CSG325C

Commit message: Added WIP Mech Model and Interposer
Also reworked rev5 power tree
Parts:
- TP43, TP44, TP45: now left out of the parts list
Connections:
- net +2V5 renamed +3V3

Commit message: Schematic WIP
Parts:
- FB11: footprint GEN_R_0402 -> Thunderscope_Rev5:GEN_R_0402
- R113, R114: value ${ALTIUM_VALUE} -> 4.7K; footprint GEN_R_0402 -> Thunderscope_Rev5:GEN_R_0402; ALTIUM_VALUE 4.7K -> (none)
- TP43, TP44, TP45: footprint GEN_TP_PCB -> Thunderscope_Rev5:GEN_TP_PCB
- U18: footprint XILINX_XC7A50T-2CSG325C -> Thunderscope_Rev5:XILINX_XC7A50T-2CSG325C
Other:
- note added: "FPGA Configuration"
Changed lines of the file:
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@@
 (kicad_sch
-	(version 20241004)
+	(version 20241209)
 	(generator "eeschema")
 	(generator_version "8.99")
@@
 		(company "EEVengers")
 	)
+	(text "FPGA Configuration"
+		(exclude_from_sim no)
+		(at 15.24 15.24 0)
+		(effects
+			(font
+				(size 1.905 1.905)
+				(thickness 0.381)
+				(bold yes)
+			)
+			(justify left top)
+		)
+	)
 	(text "M[2:0] = 001"
 		(exclude_from_sim no)
@@
 	(label "TMS"
 		(at 154.94 76.2 0)
-		(fields_autoplaced yes)
 		(effects
 			(font
@@
 	(label "TCK"
 		(at 154.94 73.66 0)
-		(fields_autoplaced yes)
 		(effects
 			(font
@@
 	(label "TDO"
 		(at 154.94 71.12 0)
-		(fields_autoplaced yes)
 		(effects
 			(font
@@
 	(label "QSPI_CLK"
 		(at 154.94 81.28 0)
-		(fields_autoplaced yes)
 		(effects
 			(font
@@
 	(label "TDI"
 		(at 154.94 68.58 0)
-		(fields_autoplaced yes)
 		(effects
 			(font
@@
 		(shape input)
 		(at 165.1 76.2 0)
-		(fields_autoplaced yes)
 		(effects
 			(font
@@
 		(shape output)
 		(at 193.04 81.28 0)
-		(fields_autoplaced yes)
 		(effects
 			(font
@@
 		(shape input)
 		(at 165.1 73.66 0)
-		(fields_autoplaced yes)
 		(effects
 			(font
@@
 		(shape output)
 		(at 165.1 71.12 0)
-		(fields_autoplaced yes)
 		(effects
 			(font
@@
 		(shape input)
 		(at 165.1 68.58 0)
-		(fields_autoplaced yes)
 		(effects
 			(font
@@
 			)
 		)
-		(property "Value" "${ALTIUM_VALUE}"
+		(property "Value" "4.7K"
 			(at 162.56 96.52 0)
 			(effects
@@
 			)
 		)
-		(property "Footprint" "GEN_R_0402"
+		(property "Footprint" "Thunderscope_Rev5:GEN_R_0402"
 			(at 162.56 96.52 0)
 			(effects
@@
 			)
 		)
-		(property "ALTIUM_VALUE" "4.7K"
-			(at 156.972 95.464 0)
+		(property "HOUSE PART NUMBER" ""
+			(at 153.736 93.98 0)
 			(effects
 				(font
@@
 			)
 		)
-		(property "HOUSE PART NUMBER" ""
+		(property "MANUFACTURER" "Panasonic"
 			(at 153.736 93.98 0)
 			(effects
@@
 			)
 		)
-		(property "MANUFACTURER" "Panasonic"
+		(property "MANUFACTURER PART NUMBER" "ERJ-2RKF4701X"
 			(at 153.736 93.98 0)
 			(effects
@@
 			)
 		)
-		(property "MANUFACTURER PART NUMBER" "ERJ-2RKF4701X"
-			(at 153.736 93.98 0)
+		(property "ALTIUM_VALUE" ""
+			(at 162.56 96.52 0)
 			(effects
 				(font
 					(size 1.27 1.27)
 				)
-				(justify left bottom)
-				(hide yes)
 			)
 		)
@@
 			)
 		)
-		(property "Footprint" "GEN_TP_PCB"
+		(property "Footprint" "Thunderscope_Rev5:GEN_TP_PCB"
 			(at 177.8 93.98 0)
 			(effects
@@
 			)
 		)
+		(property "ALTIUM_VALUE" ""
+			(at 177.8 93.98 0)
+			(effects
+				(font
+					(size 1.27 1.27)
+				)
+			)
+		)
 		(pin "1"
 		)
@@
 			)
 		)
-		(property "Footprint" "GEN_R_0402"
+		(property "Footprint" "Thunderscope_Rev5:GEN_R_0402"
 			(at 162.56 134.62 0)
 			(effects
@@
 			)
 		)
+		(property "ALTIUM_VALUE" ""
+			(at 162.56 134.62 0)
+			(effects
+				(font
+					(size 1.27 1.27)
+				)
+			)
+		)
 		(pin "2"
 		)
@@
 			)
 		)
-		(property "Footprint" "GEN_TP_PCB"
+		(property "Footprint" "Thunderscope_Rev5:GEN_TP_PCB"
 			(at 180.34 81.28 0)
 			(effects
@@
 			)
 		)
+		(property "ALTIUM_VALUE" ""
+			(at 180.34 81.28 0)
+			(effects
+				(font
+					(size 1.27 1.27)
+				)
+			)
+		)
 		(pin "1"
 		)
@@
 					(size 1.27 1.27)
 				)
+				(hide yes)
 			)
 		)
@@
 					(size 1.27 1.27)
 				)
+				(hide yes)
 			)
 		)
-		(property "Description" ""
+		(property "Description" "Power symbol creates a global label with name '+3V3'"
 			(at 180.34 88.9 0)
 			(effects
@@
 					(size 1.27 1.27)
 				)
+				(hide yes)
 			)
 		)
@@
 			)
 		)
-		(property "Footprint" "GEN_TP_PCB"
+		(property "Footprint" "Thunderscope_Rev5:GEN_TP_PCB"
 			(at 180.34 109.22 0)
 			(effects
@@
 			)
 		)
+		(property "ALTIUM_VALUE" ""
+			(at 180.34 109.22 0)
+			(effects
+				(font
+					(size 1.27 1.27)
+				)
+			)
+		)
 		(pin "1"
 		)
@@
 			)
 		)
-		(property "Footprint" "XILINX_XC7A50T-2CSG325C"
+		(property "Footprint" "Thunderscope_Rev5:XILINX_XC7A50T-2CSG325C"
 			(at 144.78 66.04 0)
 			(effects
@@
 			)
 		)
+		(property "ALTIUM_VALUE" ""
+			(at 144.78 66.04 0)
+			(effects
+				(font
+					(size 1.27 1.27)
+				)
+			)
+		)
 		(pin "K1"
 		)
@@
 			)
 		)
-		(property "Value" "${ALTIUM_VALUE}"
+		(property "Value" "4.7K"
 			(at 162.56 101.6 0)
 			(effects
@@
 			)
 		)
-		(property "Footprint" "GEN_R_0402"
+		(property "Footprint" "Thunderscope_Rev5:GEN_R_0402"
 			(at 162.56 101.6 0)
 			(effects
@@
 			)
 		)
-		(property "ALTIUM_VALUE" "4.7K"
-			(at 156.972 100.544 0)
+		(property "HOUSE PART NUMBER" ""
+			(at 153.808 99.06 0)
 			(effects
 				(font
@@
 			)
 		)
-		(property "HOUSE PART NUMBER" ""
+		(property "MANUFACTURER" "Panasonic"
 			(at 153.808 99.06 0)
 			(effects
@@
 			)
 		)
-		(property "MANUFACTURER" "Panasonic"
+		(property "MANUFACTURER PART NUMBER" "ERJ-2RKF4701X"
 			(at 153.808 99.06 0)
 			(effects
@@
 			)
 		)
-		(property "MANUFACTURER PART NUMBER" "ERJ-2RKF4701X"
-			(at 153.808 99.06 0)
+		(property "ALTIUM_VALUE" ""
+			(at 162.56 101.6 0)
 			(effects
 				(font
 					(size 1.27 1.27)
 				)
-				(justify left bottom)
-				(hide yes)
 			)
 		)

Commit message: Schematic cleanup and RGB status LED
Other:
- moved on the sheet: TP43, TP44, TP45
Changed lines of the file:
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@@
 	)
 	(junction
-		(at 175.26 96.52)
+		(at 177.8 96.52)
 		(diameter 0)
 		(color 0 0 0 0)
@@
 	)
 	(junction
-		(at 180.34 81.28)
+		(at 177.8 101.6)
 		(diameter 0)
 		(color 0 0 0 0)
 	)
 	(junction
-		(at 175.26 101.6)
+		(at 187.96 81.28)
 		(diameter 0)
 		(color 0 0 0 0)
@@
 	)
 	(junction
-		(at 175.26 88.9)
+		(at 177.8 83.82)
 		(diameter 0)
 		(color 0 0 0 0)
@@
 	(wire
 		(pts
-			(xy 152.4 71.12) (xy 165.1 71.12)
+			(xy 187.96 81.28) (xy 193.04 81.28)
 		)
 		(stroke
@@
 	(wire
 		(pts
-			(xy 154.94 119.38) (xy 154.94 116.84)
+			(xy 152.4 71.12) (xy 165.1 71.12)
 		)
 		(stroke
@@
 	(wire
 		(pts
-			(xy 175.26 101.6) (xy 167.64 101.6)
+			(xy 154.94 119.38) (xy 154.94 116.84)
 		)
 		(stroke
@@
 	(wire
 		(pts
-			(xy 170.18 88.9) (xy 152.4 88.9)
+			(xy 177.8 101.6) (xy 167.64 101.6)
 		)
 		(stroke
@@
 	(wire
 		(pts
-			(xy 152.4 119.38) (xy 154.94 119.38)
+			(xy 170.18 88.9) (xy 152.4 88.9)
 		)
 		(stroke
@@
 	(wire
 		(pts
-			(xy 180.34 88.9) (xy 175.26 88.9)
+			(xy 152.4 119.38) (xy 154.94 119.38)
 		)
 		(stroke
@@
 	(wire
 		(pts
-			(xy 175.26 83.82) (xy 152.4 83.82)
+			(xy 177.8 83.82) (xy 152.4 83.82)
 		)
 		(stroke
@@
 	(wire
 		(pts
-			(xy 167.64 96.52) (xy 175.26 96.52)
+			(xy 167.64 96.52) (xy 177.8 96.52)
 		)
 		(stroke
@@
 	(wire
 		(pts
-			(xy 180.34 81.28) (xy 193.04 81.28)
-		)
-		(stroke
-			(width 0)
-			(type default)
-		)
-	)
-	(wire
-		(pts
 			(xy 154.94 116.84) (xy 152.4 116.84)
 		)
@@
 	(wire
 		(pts
-			(xy 175.26 96.52) (xy 175.26 101.6)
+			(xy 177.8 96.52) (xy 177.8 101.6)
 		)
 		(stroke
@@
 	(wire
 		(pts
-			(xy 175.26 88.9) (xy 175.26 83.82)
+			(xy 177.8 78.74) (xy 177.8 83.82)
 		)
 		(stroke
@@
 	(wire
 		(pts
-			(xy 157.48 134.62) (xy 154.94 134.62)
+			(xy 177.8 83.82) (xy 177.8 96.52)
 		)
 		(stroke
@@
 	(wire
 		(pts
-			(xy 175.26 96.52) (xy 175.26 88.9)
+			(xy 157.48 134.62) (xy 154.94 134.62)
 		)
 		(stroke
@@
 	(wire
 		(pts
-			(xy 177.8 93.98) (xy 152.4 93.98)
+			(xy 182.88 93.98) (xy 152.4 93.98)
 		)
 		(stroke
@@
 	(wire
 		(pts
-			(xy 152.4 81.28) (xy 180.34 81.28)
+			(xy 152.4 81.28) (xy 187.96 81.28)
 		)
 		(stroke
@@
 	(wire
 		(pts
-			(xy 175.26 104.14) (xy 175.26 101.6)
+			(xy 177.8 104.14) (xy 177.8 101.6)
 		)
 		(stroke
@@
 	(wire
 		(pts
-			(xy 152.4 104.14) (xy 175.26 104.14)
+			(xy 152.4 104.14) (xy 177.8 104.14)
 		)
 		(stroke
@@
 	(symbol
 		(lib_id "Thunderscope_Rev5:TP PCB 1mm")
-		(at 177.8 93.98 0)
+		(at 182.88 93.98 0)
 		(unit 1)
 		(exclude_from_sim no)
@@
 		(dnp no)
 		(property "Reference" "TP44"
-			(at 183.5827 94.6296 0)
+			(at 188.6627 94.6296 0)
 			(effects
 				(font
@@
 		)
 		(property "Value" "PCB"
-			(at 177.292 92.71 0)
+			(at 182.372 92.71 0)
 			(effects
 				(font
@@
 		)
 		(property "Footprint" "Thunderscope_Rev5:GEN_TP_PCB"
-			(at 177.8 93.98 0)
+			(at 182.88 93.98 0)
 			(effects
 				(font
@@
 		)
 		(property "Datasheet" ""
-			(at 177.8 93.98 0)
+			(at 182.88 93.98 0)
 			(effects
 				(font
@@
 		)
 		(property "Description" ""
-			(at 177.8 93.98 0)
+			(at 182.88 93.98 0)
 			(effects
 				(font
@@
 		)
 		(property "HOUSE PART NUMBER" ""
-			(at 177.292 92.71 0)
+			(at 182.372 92.71 0)
 			(effects
 				(font
@@
 		)
 		(property "MANUFACTURER" ""
-			(at 177.292 92.71 0)
+			(at 182.372 92.71 0)
 			(effects
 				(font
@@
 		)
 		(property "MANUFACTURER PART NUMBER" ""
-			(at 177.292 92.71 0)
+			(at 182.372 92.71 0)
 			(effects
 				(font
@@
 		)
 		(property "ALTIUM_VALUE" ""
-			(at 177.8 93.98 0)
+			(at 182.88 93.98 0)
 			(effects
 				(font
@@
 	(symbol
 		(lib_id "Thunderscope_Rev5:TP PCB 1mm")
-		(at 180.34 81.28 90)
+		(at 187.96 81.28 90)
 		(unit 1)
 		(exclude_from_sim no)
@@
 		(dnp no)
 		(property "Reference" "TP43"
-			(at 182.772 74.2429 90)
+			(at 190.392 74.2429 90)
 			(effects
 				(font
@@
 		)
 		(property "Value" "PCB"
-			(at 175.26 82.55 0)
+			(at 182.88 82.55 0)
 			(effects
 				(font
@@
 		)
 		(property "Footprint" "Thunderscope_Rev5:GEN_TP_PCB"
-			(at 180.34 81.28 0)
+			(at 187.96 81.28 0)
 			(effects
 				(font
@@
 		)
 		(property "Datasheet" ""
-			(at 180.34 81.28 0)
+			(at 187.96 81.28 0)
 			(effects
 				(font
@@
 		)
 		(property "Description" ""
-			(at 180.34 81.28 0)
+			(at 187.96 81.28 0)
 			(effects
 				(font
@@
 		)
 		(property "HOUSE PART NUMBER" ""
-			(at 175.26 82.55 0)
+			(at 182.88 82.55 0)
 			(effects
 				(font
@@
 		)
 		(property "MANUFACTURER" ""
-			(at 175.26 82.55 0)
+			(at 182.88 82.55 0)
 			(effects
 				(font
@@
 		)
 		(property "MANUFACTURER PART NUMBER" ""
-			(at 175.26 82.55 0)
+			(at 182.88 82.55 0)
 			(effects
 				(font
@@
 		)
 		(property "ALTIUM_VALUE" ""
-			(at 180.34 81.28 0)
+			(at 187.96 81.28 0)
 			(effects
 				(font
@@
 	(symbol
 		(lib_id "Thunderscope_Rev5:+3V3_BAR")
-		(at 180.34 88.9 90)
+		(at 177.8 78.74 180)
 		(unit 1)
 		(exclude_from_sim no)
@@
 		(dnp no)
 		(property "Reference" "#PWR0279"
-			(at 180.34 88.9 0)
+			(at 177.8 78.74 0)
 			(effects
 				(font
@@
 		)
 		(property "Value" "+3V3"
-			(at 184.15 88.9 0)
+			(at 177.8 74.93 0)
 			(effects
 				(font
@@
 		)
 		(property "Footprint" ""
-			(at 180.34 88.9 0)
+			(at 177.8 78.74 0)
 			(effects
 				(font
@@
 		)
 		(property "Datasheet" ""
-			(at 180.34 88.9 0)
+			(at 177.8 78.74 0)
 			(effects
 				(font
@@
 		)
 		(property "Description" "Power symbol creates a global label with name '+3V3'"
-			(at 180.34 88.9 0)
+			(at 177.8 78.74 0)
 			(effects
 				(font
@@
 	(symbol
 		(lib_id "Thunderscope_Rev5:TP PCB 1mm")
-		(at 180.34 109.22 0)
+		(at 187.96 109.22 90)
 		(unit 1)
 		(exclude_from_sim no)
@@
 		(dnp no)
 		(property "Reference" "TP45"
-			(at 181.61 106.68 0)
+			(at 190.5 101.6 90)
 			(effects
 				(font
@@
 		)
 		(property "Value" "PCB"
-			(at 179.07 104.14 0)
+			(at 182.88 110.49 0)
 			(effects
 				(font
@@
 		)
 		(property "Footprint" "Thunderscope_Rev5:GEN_TP_PCB"
-			(at 180.34 109.22 0)
+			(at 187.96 109.22 0)
 			(effects
 				(font
@@
 		)
 		(property "Datasheet" ""
-			(at 180.34 109.22 0)
+			(at 187.96 109.22 0)
 			(effects
 				(font
@@
 		)
 		(property "Description" ""
-			(at 180.34 109.22 0)
+			(at 187.96 109.22 0)
 			(effects
 				(font
@@
 		)
 		(property "HOUSE PART NUMBER" ""
-			(at 177.8 101.6 0)
+			(at 180.34 111.76 0)
 			(effects
 				(font
@@
 		)
 		(property "MANUFACTURER" ""
-			(at 177.8 101.6 0)
+			(at 180.34 111.76 0)
 			(effects
 				(font
@@
 		)
 		(property "MANUFACTURER PART NUMBER" ""
-			(at 177.8 101.6 0)
+			(at 180.34 111.76 0)
 			(effects
 				(font
@@
 		)
 		(property "ALTIUM_VALUE" ""
-			(at 180.34 109.22 0)
+			(at 187.96 109.22 0)
 			(effects
 				(font
@@
 	(symbol
 		(lib_id "Thunderscope_Rev5:GND")
-		(at 180.34 109.22 0)
+		(at 187.96 109.22 0)
 		(unit 1)
 		(exclude_from_sim no)
@@
 		(dnp no)
 		(property "Reference" "#PWR0503"
-			(at 180.34 115.57 0)
+			(at 187.96 115.57 0)
 			(effects
 				(font
@@
 		)
 		(property "Value" "GND"
-			(at 180.34 113.03 0)
+			(at 187.96 113.03 0)
 			(effects
 				(font
@@
 		)
 		(property "Footprint" ""
-			(at 180.34 109.22 0)
+			(at 187.96 109.22 0)
 			(effects
 				(font
@@
 		)
 		(property "Datasheet" ""
-			(at 180.34 109.22 0)
+			(at 187.96 109.22 0)
 			(effects
 				(font
@@
 		)
 		(property "Description" "Power symbol creates a global label with name \"GND\" , ground"
-			(at 180.34 109.22 0)
+			(at 187.96 109.22 0)
 			(effects
 				(font
