File: Hardware/KiCad/Thunderscope_Rev5/User_IO.kicad_sch (KiCad schematic)
At the start: 18 parts, among them J1 BNC, J2 BNC, J3 1.27mm 6 Pin TH, J4 TSW-101-16-G-Q-RA, U1 SN74LVC1G17

Commit message: Linked PCB to Schematic
Connections:
- no-connect marks 1 -> 0
Changed lines of the file:
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@@
 		(color 0 0 0 0)
 	)
-	(no_connect
-		(at 53.34 175.26)
+	(junction
+		(at 40.64 177.8)
+		(diameter 0)
+		(color 0 0 0 0)
 	)
 	(wire
@@
 	(wire
 		(pts
-			(xy 205.74 111.76) (xy 231.14 111.76)
-		)
-		(stroke
-			(width 0)
-			(type default)
-		)
-	)
-	(wire
-		(pts
 			(xy 236.22 127) (xy 251.46 127)
 		)
@@
 	(wire
 		(pts
+			(xy 40.64 180.34) (xy 40.64 177.8)
+		)
+		(stroke
+			(width 0)
+			(type default)
+		)
+	)
+	(wire
+		(pts
 			(xy 233.68 111.76) (xy 231.14 111.76)
 		)
@@
 		(pts
 			(xy 233.68 116.84) (xy 231.14 116.84)
+		)
+		(stroke
+			(width 0)
+			(type default)
+		)
+	)
+	(wire
+		(pts
+			(xy 208.28 111.76) (xy 231.14 111.76)
 		)
 		(stroke
@@
 		)
 	)
-	(label "LED"
-		(at 91.44 147.32 180)
+	(label "REFINOUT1"
+		(at 238.76 144.78 0)
 		(fields_autoplaced yes)
 		(effects
@@
 				(size 1.27 1.27)
 			)
-			(justify right bottom)
-		)
-	)
-	(label "REFINOUT1"
-		(at 238.76 144.78 0)
+			(justify left bottom)
+		)
+	)
+	(label "REFINOUT2"
+		(at 180.34 147.32 0)
 		(fields_autoplaced yes)
 		(effects
@@
 		)
 	)
-	(label "REFINOUT2"
-		(at 180.34 147.32 0)
+	(label "SYNC1"
+		(at 261.62 144.78 0)
 		(fields_autoplaced yes)
 		(effects
@@
 	)
 	(label "SYNC1"
-		(at 261.62 144.78 0)
+		(at 254 111.76 180)
 		(fields_autoplaced yes)
 		(effects
@@
 				(size 1.27 1.27)
 			)
-			(justify left bottom)
-		)
-	)
-	(label "SYNC1"
-		(at 254 111.76 180)
+			(justify right bottom)
+		)
+	)
+	(label "REFINOUT"
+		(at 208.28 127 0)
 		(fields_autoplaced yes)
 		(effects
@@
 				(size 1.27 1.27)
 			)
-			(justify right bottom)
-		)
-	)
-	(label "REFINOUT"
-		(at 208.28 127 0)
+			(justify left bottom)
+		)
+	)
+	(label "SYNC2"
+		(at 254 116.84 180)
 		(fields_autoplaced yes)
 		(effects
@@
 				(size 1.27 1.27)
 			)
-			(justify left bottom)
-		)
-	)
-	(label "SYNC2"
-		(at 254 116.84 180)
+			(justify right bottom)
+		)
+	)
+	(label "SYNC"
+		(at 208.28 111.76 0)
 		(fields_autoplaced yes)
 		(effects
@@
 				(size 1.27 1.27)
 			)
-			(justify right bottom)
-		)
-	)
-	(label "SYNC"
-		(at 208.28 111.76 0)
+			(justify left bottom)
+		)
+	)
+	(label "REFINOUT1"
+		(at 251.46 127 180)
 		(fields_autoplaced yes)
 		(effects
@@
 				(size 1.27 1.27)
 			)
-			(justify left bottom)
-		)
-	)
-	(label "REFINOUT1"
-		(at 251.46 127 180)
+			(justify right bottom)
+		)
+	)
+	(label "LED"
+		(at 86.36 147.32 0)
 		(fields_autoplaced yes)
 		(effects
@@
 				(size 1.27 1.27)
 			)
-			(justify right bottom)
+			(justify left bottom)
 		)
 	)
@@
 	(symbol
 		(lib_id "Thunderscope_Rev5:GND")
-		(at 40.64 177.8 0)
+		(at 40.64 180.34 0)
 		(unit 1)
 		(exclude_from_sim no)
@@
 		(dnp no)
 		(property "Reference" "#PWR01"
+			(at 40.64 186.69 0)
+			(effects
+				(font
+					(size 1.27 1.27)
+				)
+				(hide yes)
+			)
+		)
+		(property "Value" "GND"
 			(at 40.64 184.15 0)
 			(effects
@@
 					(size 1.27 1.27)
 				)
-				(hide yes)
-			)
-		)
-		(property "Value" "GND"
-			(at 40.64 181.61 0)
-			(effects
-				(font
-					(size 1.27 1.27)
-				)
 			)
 		)
 		(property "Footprint" ""
-			(at 40.64 177.8 0)
+			(at 40.64 180.34 0)
 			(effects
 				(font
@@
 		)
 		(property "Datasheet" ""
-			(at 40.64 177.8 0)
+			(at 40.64 180.34 0)
 			(effects
 				(font
@@
 		)
 		(property "Description" "Power symbol creates a global label with name \"GND\" , ground"
-			(at 40.64 177.8 0)
+			(at 40.64 180.34 0)
 			(effects
 				(font
@@
 					(unit 1)
 				)
+			)
+		)
+	)
+	(symbol
+		(lib_id "power:PWR_FLAG")
+		(at 40.64 177.8 90)
+		(unit 1)
+		(exclude_from_sim no)
+		(in_bom yes)
+		(on_board yes)
+		(dnp no)
+		(fields_autoplaced yes)
+		(property "Reference" "#FLG026"
+			(at 38.735 177.8 0)
+			(effects
+				(font
+					(size 1.27 1.27)
+				)
+				(hide yes)
+			)
+		)
+		(property "Value" "PWR_FLAG"
+			(at 36.83 177.7999 90)
+			(effects
+				(font
+					(size 1.27 1.27)
+				)
+				(justify left)
+			)
+		)
+		(property "Footprint" ""
+			(at 40.64 177.8 0)
+			(effects
+				(font
+					(size 1.27 1.27)
+				)
+				(hide yes)
+			)
+		)
+		(property "Datasheet" "~"
+			(at 40.64 177.8 0)
+			(effects
+				(font
+					(size 1.27 1.27)
+				)
+				(hide yes)
+			)
+		)
+		(property "Description" "Special symbol for telling ERC where power comes from"
+			(at 40.64 177.8 0)
+			(effects
+				(font
+					(size 1.27 1.27)
+				)
+				(hide yes)
+			)
+		)
+		(pin "1"
+		)
+		(instances
+			(project ""
+				(path "/031d3e2c-42e0-4016-8c32-579d45c83e09/4fd15650-a4c4-4d94-afbf-a5fab92becb6"
+					(reference "#FLG026")
+					(unit 1)
+				)

Commit message: Added WIP Mech Model and Interposer
Also reworked rev5 power tree
Parts:
- added J10: 009155002852006, KYO_009155002852006, symbol Thunderscope_Rev5:CONN SPRING 2 PIN
Connections:
- net GND: now also J10.1
- new net +VUSB: J10.2

Commit message: Schematic WIP
Parts:
- removed J10: 009155002852006, KYO_009155002852006, symbol Thunderscope_Rev5:CONN SPRING 2 PIN
- added C78: 1uF, Thunderscope_Rev5:GEN_C_0402, symbol Thunderscope_Rev5:CAP 1uF 25V X5R 0402
- added C79: 10uF, Thunderscope_Rev5:GEN_C_0603, symbol Thunderscope_Rev5:CAP 10uF 10V X5R 0603
- added D?: APFA3010, LED_SMD:LED_Kingbright_APFA3010_3x1.5mm_Horizontal, symbol LED:APFA3010
- added J9: F300-1B7H1-11036-E100, Thunderscope_Rev5:AMPHENOL_F300-1B7H1-11036-E100, symbol Thunderscope_Rev5:CONN FFC BOTTOM 36POS 0.5MM RA
- added R60: 100, Thunderscope_Rev5:GEN_R_0402, symbol Thunderscope_Rev5:RES 100 OHM 1% 1/10W 0402
- added R61, R62: 10K, Thunderscope_Rev5:GEN_R_0402, symbol Thunderscope_Rev5:RES 10K OHM 1% 1/10W 0402
- added R63: 49.9, Thunderscope_Rev5:GEN_R_0402, symbol Thunderscope_Rev5:RES 49.9 OHM 1% 1/10W 0402
- added U10: FIN1019MTCX, Thunderscope_Rev5:GEN_TSSOP-14_4.4x5mm_P0.65mm, symbol Thunderscope_Rev5:IC LVDS XCVR FIN1019MTCX
- C1: value ${ALTIUM_VALUE} -> 1uF; footprint GEN_C_0402 -> Thunderscope_Rev5:GEN_C_0402; symbol Thunderscope_Rev5:CAP 100nF 16V X7R 0402 -> Thunderscope_Rev5:CAP 1uF 25V X5R 0402; ALTIUM_VALUE 100nF -> (none); HOUSE PART NUMBER C-100nF-0402-002 -> (none); MANUFACTURER PART NUMBER GCM155R71C104KA55D -> GRM155R61E105KA12D; SUPPLIER PART NUMBER 1 81-GCM155R71C104KA5D -> 81-GRM155R61E105KA2D; VOLTAGE RATING 16V -> 25V
- D1: footprint LED_0603_LTST-S270K -> Thunderscope_Rev5:LED_0603_LTST-S270K
- D2, D3, D4, D5: footprint TI_X1SON_DPY0002A -> Thunderscope_Rev5:TI_X1SON_DPY0002A
- J1, J2: footprint MOL_0731000105 -> Thunderscope_Rev5:MOL_0731000105
- J3: footprint GEN_1.27mm_2x5_Pin_TH_RA -> Thunderscope_Rev5:GEN_1.27mm_2x5_Pin_TH_RA
- J4: footprint GEN_5.08mm_1x2_Pin_TH_RA -> Thunderscope_Rev5:GEN_5.08mm_1x2_Pin_TH_RA
- R2, R3, R4, R5: value ${ALTIUM_VALUE} -> 0; footprint GEN_R_0402 -> Thunderscope_Rev5:GEN_R_0402; ALTIUM_VALUE 0 -> (none)
- R6: value ${ALTIUM_VALUE} -> 1K; footprint GEN_R_0402 -> Thunderscope_Rev5:GEN_R_0402; ALTIUM_VALUE 1K -> (none)
- R7: value ${ALTIUM_VALUE} -> 100; footprint GEN_R_0402 -> Thunderscope_Rev5:GEN_R_0402; ALTIUM_VALUE 100 -> (none)
- R8: value ${ALTIUM_VALUE} -> 10K; footprint GEN_R_0402 -> Thunderscope_Rev5:GEN_R_0402; ALTIUM_VALUE 10K -> (none)
- U1: footprint GEN_SC-70-5 -> Thunderscope_Rev5:GEN_SC-70-5
Connections:
- net +3V3: now also C78.1, C79.2, R61.1, U10.14 (VCC); no longer C1.2, U1.5 (VCC)
- net GND: now also C1.2, C78.2, C79.1, J9.1, J9.10, J9.13, J9.16, J9.19, J9.22, J9.25, J9.28, J9.31, J9.34, J9.4, J9.7, J9.SH1, J9.SH2, R62.2, U10.7 (GND); no longer C1.1
- net SYNC: now also R63.1, U10.2 (DI)
- net SYNC_IN_N: now also U10.11 (DO-)
- net SYNC_IN_P: now also U10.12 (DO+)
- net SYNC_OUT_N: now also R60.1, U10.9 (RI-)
- net SYNC_OUT_P: now also R60.2, U10.10 (RI+)
- new net: R63.2, U10.4 (RO)
- new net +3V3_PGA: C1.1, U1.5 (VCC)
- new net SYNC_DE: R62.1, U10.1 (DE)
- new net SYNC_REn: R61.2, U10.8 (~{RE})
- new net USRIO_10_N: J9.30
- new net USRIO_10_P: J9.29
- new net USRIO_11_N: J9.33
- new net USRIO_11_P: J9.32
- new net USRIO_12_N: J9.36
- new net USRIO_12_P: J9.35
- new net USRIO_1_N: J9.3
- new net USRIO_1_P: J9.2
- new net USRIO_2_N: J9.6
- new net USRIO_2_P: J9.5
- new net USRIO_3_N: J9.9
- new net USRIO_3_P: J9.8
- new net USRIO_4_N: J9.12
- new net USRIO_4_P: J9.11
- new net USRIO_5_N: J9.15
- new net USRIO_5_P: J9.14
- new net USRIO_6_N: J9.18
- new net USRIO_6_P: J9.17
- new net USRIO_7_N: J9.21
- new net USRIO_7_P: J9.20
- new net USRIO_8_N: J9.24
- new net USRIO_8_P: J9.23
- new net USRIO_9_N: J9.27
- new net USRIO_9_P: J9.26
Other:
- note added: "DONE: 36 pin FPC connector for LVDS"
- note added: "DONE: FIN1019MTCX LVDS XCVR for Sync"
- note added: "Probe Compensation"
- note added: "Reference Clock and Sync"
- note added: "Status LED"
- note added: "TODO: RGB LED"
- note added: "User IO FFC Connector"
- note removed: "Connectors for muti-scope connection"
- moved on the sheet: C1, D1, D2, D3, D4, D5, J1, J2, J3, J4, R2, R3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

Commit message: Schematic cleanup and RGB status LED
Parts:
- removed D1: GREEN, Thunderscope_Rev5:LED_0603_LTST-S270K, symbol Thunderscope_Rev5:LED GREEN 0603 LTST-S270K
- removed D?: APFA3010, LED_SMD:LED_Kingbright_APFA3010_3x1.5mm_Horizontal, symbol LED:APFA3010
- added D1: RGB, Thunderscope_Rev5:LED_Kingbright_APFA3010_3x1.5mm_Horizontal, symbol Thunderscope_Rev5:LED RGB 1204 APFA3010LSEKJ3ZGKQBC
- added R64, R65: 1K, Thunderscope_Rev5:GEN_R_0402, symbol Thunderscope_Rev5:RES 1K OHM 1% 1/10W 0402
Connections:
- net GND: now also D1.2 (A)
- net at R6.1: now also D1.3 (G)
- net LED renamed LED_G
- new net: D1.4 (B), R65.1
- new net: D1.1 (R), R64.1
- new net LED_B: R65.2
- new net LED_R: R64.2
Other:
- note added: "DONE: 36 pin FFC for LVDS"
- note added: "DONE: Change Status LED to RGB"
- note added: "TEST: LED resistor values on Mech Board"
- note added: "User IO Flat Flex Connector"
- note removed: "DONE: 36 pin FPC connector for LVDS"
- note removed: "TODO: RGB LED"
- note removed: "User IO FFC Connector"
- moved on the sheet: R6
