File: Hardware/KiCad/Thunderscope_Rev5/FE.kicad_sch (KiCad schematic)
At the start: 23 parts, among them Q1 DMN62D0UW, Q2 DMN62D0UW, U2 MCP4452-104E, U3 MCP4728, U4 REF2025, U5 OPA140AIDR

Commit message: Linked PCB to Schematic
Connections:
- net SCL_5V renamed TRIM_SCL_5V
- net SDA_5V renamed TRIM_SDA_5V
Other:
- moved on the sheet: C2, C3, R10, R11, R12, R9, TP6, TP7, TP9, U3

Commit message: Added WIP Mech Model and Interposer
Also reworked rev5 power tree
Parts:
- TP6, TP7, TP8, TP9: now left out of the parts list
Changed lines of the file:
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@@
 		(unit 1)
 		(exclude_from_sim no)
-		(in_bom yes)
+		(in_bom no)
 		(on_board yes)
 		(dnp no)
@@
 		(unit 1)
 		(exclude_from_sim no)
-		(in_bom yes)
+		(in_bom no)
 		(on_board yes)
 		(dnp no)
@@
 		(unit 1)
 		(exclude_from_sim no)
-		(in_bom yes)
+		(in_bom no)
 		(on_board yes)
 		(dnp no)
@@
 		(unit 1)
 		(exclude_from_sim no)
-		(in_bom yes)
-		(on_board yes)
-		(dnp no)
+		(in_bom no)
+		(on_board yes)
+		(dnp no)

Commit message: Schematic WIP
Parts:
- C11, C2, C3, C4, C5, C6, C7, C8: value ${ALTIUM_VALUE} -> 100nF; footprint GEN_C_0402 -> Thunderscope_Rev5:GEN_C_0402; ALTIUM_VALUE 100nF -> (none)
- Q1, Q2: footprint GEN_SOT_323 -> Thunderscope_Rev5:GEN_SOT_323
- R10, R11, R12, R9: value ${ALTIUM_VALUE} -> 10K; footprint GEN_R_0402 -> Thunderscope_Rev5:GEN_R_0402; ALTIUM_VALUE 10K -> (none)
- R13: value ${ALTIUM_VALUE} -> 10K; footprint GEN_R_2ARRAY_0606 -> Thunderscope_Rev5:GEN_R_2ARRAY_0606; ALTIUM_VALUE 10K -> (none)
- TP6, TP7, TP8, TP9: footprint GEN_TP_PCB -> Thunderscope_Rev5:GEN_TP_PCB
- U2: footprint MC_TSSOP14 -> Thunderscope_Rev5:MC_TSSOP14
- U3: footprint MC_MSOP10_UN -> Thunderscope_Rev5:MC_MSOP10_UN
- U4: footprint GEN_SOT23_5_950_2900X1600X1450 -> Thunderscope_Rev5:GEN_SOT23_5_950_2900X1600X1450; MANUFACTURER (none) -> Texas Instruments; MANUFACTURER PART NUMBER (none) -> REF2025AIDDCR
- U5: footprint TI_SOIC8_D0008A -> Thunderscope_Rev5:TI_SOIC8_D0008A

Commit message: Sent Mech Models Out to Fab
Changed lines of the file:
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@@
 			(font
 				(size 1.27 1.27)
-				(thickness 0.254)
-				(bold yes)
+				(thickness 0.1588)
 			)
 			(justify left bottom)
@@
 			(font
 				(size 1.27 1.27)
-				(thickness 0.254)
-				(bold yes)
+				(thickness 0.1588)
 			)
 			(justify left bottom)

Commit message: Refactored Schematic
Other:
- moved on the sheet: U3
Changed lines of the file:
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@@
 	(text "Default I2C address: 1100000"
 		(exclude_from_sim no)
-		(at 121.92 71.12 0)
+		(at 124.46 71.12 0)
 		(effects
 			(font
@@
 	)
 	(junction
-		(at 111.76 63.5)
+		(at 114.3 63.5)
 		(diameter 0)
 		(color 0 0 0 0)
@@
 	)
 	(no_connect
-		(at 114.3 58.42)
+		(at 116.84 58.42)
 	)
 	(no_connect
@@
 	(wire
 		(pts
-			(xy 114.3 63.5) (xy 111.76 63.5)
+			(xy 116.84 63.5) (xy 114.3 63.5)
 		)
 		(stroke
@@
 	(wire
 		(pts
-			(xy 88.9 43.18) (xy 114.3 43.18)
+			(xy 88.9 43.18) (xy 116.84 43.18)
 		)
 		(stroke
@@
 	(wire
 		(pts
-			(xy 154.94 55.88) (xy 162.56 55.88)
+			(xy 157.48 55.88) (xy 165.1 55.88)
 		)
 		(stroke
@@
 	(wire
 		(pts
-			(xy 114.3 55.88) (xy 111.76 55.88)
+			(xy 116.84 55.88) (xy 114.3 55.88)
 		)
 		(stroke
@@
 	(wire
 		(pts
-			(xy 99.06 48.26) (xy 114.3 48.26)
+			(xy 99.06 48.26) (xy 116.84 48.26)
 		)
 		(stroke
@@
 	(wire
 		(pts
-			(xy 154.94 50.8) (xy 162.56 50.8)
+			(xy 157.48 50.8) (xy 165.1 50.8)
 		)
 		(stroke
@@
 	(wire
 		(pts
-			(xy 154.94 60.96) (xy 162.56 60.96)
+			(xy 157.48 60.96) (xy 165.1 60.96)
 		)
 		(stroke
@@
 	(wire
 		(pts
-			(xy 111.76 63.5) (xy 111.76 66.04)
+			(xy 114.3 63.5) (xy 114.3 66.04)
 		)
 		(stroke
@@
 	(wire
 		(pts
-			(xy 101.6 50.8) (xy 114.3 50.8)
+			(xy 101.6 50.8) (xy 116.84 50.8)
 		)
 		(stroke
@@
 	(wire
 		(pts
-			(xy 111.76 55.88) (xy 111.76 63.5)
+			(xy 114.3 55.88) (xy 114.3 63.5)
 		)
 		(stroke
@@
 	(wire
 		(pts
-			(xy 154.94 45.72) (xy 162.56 45.72)
+			(xy 157.48 45.72) (xy 165.1 45.72)
 		)
 		(stroke
@@
 	)
 	(label "VOUT3"
-		(at 162.56 50.8 180)
+		(at 165.1 50.8 180)
 		(effects
 			(font
@@
 	)
 	(label "VOUT4"
-		(at 162.56 45.72 180)
+		(at 165.1 45.72 180)
 		(effects
 			(font
@@
 	)
 	(label "VOUT2"
-		(at 162.56 55.88 180)
+		(at 165.1 55.88 180)
 		(effects
 			(font
@@
 	)
 	(label "VOUT1"
-		(at 162.56 60.96 180)
+		(at 165.1 60.96 180)
 		(effects
 			(font
@@
 	(symbol
 		(lib_id "Thunderscope_Rev5:IC DAC QUAD MCP4728")
-		(at 134.62 53.34 0)
+		(at 137.16 53.34 0)
 		(unit 1)
 		(exclude_from_sim no)
@@
 		(dnp no)
 		(property "Reference" "U3"
-			(at 121.92 40.64 0)
+			(at 124.46 40.64 0)
 			(effects
 				(font
@@
 		)
 		(property "Value" "MCP4728"
-			(at 121.92 68.58 0)
+			(at 124.46 68.58 0)
 			(effects
 				(font
@@
 		)
 		(property "Footprint" "Thunderscope_Rev5:MC_MSOP10_UN"
-			(at 134.62 53.34 0)
+			(at 137.16 53.34 0)
 			(effects
 				(font
@@
 		)
 		(property "Datasheet" ""
-			(at 134.62 53.34 0)
+			(at 137.16 53.34 0)
 			(effects
 				(font
@@
 		)
 		(property "Description" ""
-			(at 134.62 53.34 0)
+			(at 137.16 53.34 0)
 			(effects
 				(font
@@
 		)
 		(property "SUPPLIER 1" "Mouser"
-			(at 133.35 52.07 0)
+			(at 135.89 52.07 0)
 			(effects
 				(font
@@
 		)
 		(property "SUPPLIER PART NUMBER 1" "579-MCP4728A1T-E/UN"
-			(at 133.35 52.07 0)
+			(at 135.89 52.07 0)
 			(effects
 				(font
@@
 		)
 		(property "HOUSE PART NUMBER" ""
-			(at 113.792 38.1 0)
+			(at 116.332 38.1 0)
 			(effects
 				(font
@@
 		)
 		(property "MANUFACTURER" "Microchip"
-			(at 113.792 38.1 0)
+			(at 116.332 38.1 0)
 			(effects
 				(font
@@
 		)
 		(property "MANUFACTURER PART NUMBER" "MCP4728"
-			(at 113.792 38.1 0)
+			(at 116.332 38.1 0)
 			(effects
 				(font
@@
 		)
 		(property "ALTIUM_VALUE" ""
-			(at 134.62 53.34 0)
+			(at 137.16 53.34 0)
 			(effects
 				(font
@@
 	(symbol
 		(lib_id "Thunderscope_Rev5:GND")
-		(at 111.76 66.04 0)
+		(at 114.3 66.04 0)
 		(unit 1)
 		(exclude_from_sim no)
@@
 		(dnp no)
 		(property "Reference" "#PWR0181"
-			(at 111.76 72.39 0)
+			(at 114.3 72.39 0)
 			(effects
 				(font
@@
 		)
 		(property "Value" "GND"
-			(at 111.76 69.85 0)
+			(at 114.3 69.85 0)
 			(effects
 				(font
@@
 		)
 		(property "Footprint" ""
-			(at 111.76 66.04 0)
+			(at 114.3 66.04 0)
 			(effects
 				(font
@@
 		)
 		(property "Datasheet" ""
-			(at 111.76 66.04 0)
+			(at 114.3 66.04 0)
 			(effects
 				(font
@@
 		)
 		(property "Description" "Power symbol creates a global label with name \"GND\" , ground"
-			(at 111.76 66.04 0)
+			(at 114.3 66.04 0)
 			(effects
 				(font
