File: Hardware/KiCad/Thunderscope_Rev5/CON_PCIe_X4.kicad_sch (KiCad schematic)
At the start: 40 parts, among them J3 1.27mm 6 Pin TH, P1 PCIeX4-GF-2D-1000-1K-O64, U11 TPS563203DRLR

Commit message: Schematic Ready For Review
Parts:
- added C85: 12pF, Thunderscope_Rev5:GEN_C_0402, symbol Thunderscope_Rev5:CAP 12pF 50V C0G 0402
- added R81: 10K, Thunderscope_Rev5:GEN_R_0402, symbol Thunderscope_Rev5:RES 10K OHM 1% 1/10W 0402
- C28, C29, C32, C33, C36, C37, C40, C41, C44, C45: footprint Thunderscope_Rev5:GEN_C_0201 -> Thunderscope_Rev5:GEN_C_0402; symbol Thunderscope_Rev5:CAP 100nF 6.3V X5R 0201 -> Thunderscope_Rev5:CAP 100nF 16V X7R 0402; HOUSE PART NUMBER C-100nF-0201-002 -> C-100nF-0402-002; MANUFACTURER PART NUMBER GRM033R60J104KE19D -> GCM155R71C104KA55D; PACKAGE 0201 -> 0402; SUPPLIER PART NUMBER 1 81-GRM033R60J104KE19 -> 81-GCM155R71C104KA5D; VOLTAGE RATING 6.3V -> 16V
- R25, R26, R29, R30, R33, R34, R37, R38: footprint Thunderscope_Rev5:GEN_R_0201 -> Thunderscope_Rev5:GEN_R_0402; symbol Thunderscope_Rev5:RES 0 OHM 1% 1/20W 0201 -> Thunderscope_Rev5:RES 0 OHM 1/16W 0402; MANUFACTURER Stackpole Electronics -> Yageo; MANUFACTURER PART NUMBER RMCF0201ZT0R00 -> RC0402JR-070RL; PACKAGE 0201 -> 0402; SUPPLIER PART NUMBER 1 708-RMCF0201ZT0R00 -> 603-RC0402JR-070RL; TOLERANCE 1% -> (none)
Connections:
- net +VUSB: now also C85.2
- net GND: now also R81.1
- net at R73.1, R74.1, U11.6 (FB): now also C85.1
- net MGT_CLK0_N renamed MGT_CLK1_N
- net MGT_CLK0_P renamed MGT_CLK1_P
- net PCIe_PERST#_R renamed PERST#
- new net VARIANT: R81.2
Other:
- note added: "Variant Pin Strap"
- moved on the sheet: C80, C81, C82, C83, C84, L6, R42, R73, R74, TP14, TP15, U11
