File: Hardware/KiCad/Thunderscope_Rev5/FPGA_PWR.kicad_sch (KiCad schematic)
At the start: 46 parts, among them U18 IC FPGA XC7A50T-2CSG325C

Commit message: Altium Param Import with Script
Connections:
- net +2V5: now also C145.2, C146.2, C147.2, C148.2, C149.2, C150.2, C151.2, U18.A16 (VCCO_15), U18.B13 (VCCO_15), U18.C10 (VCCO_15), U18.D17 (VCCO_15), U18.E14 (VCCO_15), U18.G18 (VCCO_15), U18.H15 (VCCO_15); no longer C138.2, C139.2, C140.2, C141.2, C142.2, C143.2, C144.2, U18.L16 (VCCO_14), U18.P17 (VCCO_14), U18.R14 (VCCO_14), U18.T11 (VCCO_14), U18.U18 (VCCO_14), U18.U8 (VCCO_14), U18.V15 (VCCO_14)
- net +3V3: now also C138.2, C139.2, C140.2, C141.2, C142.2, C143.2, C144.2, U18.L16 (VCCO_14), U18.P17 (VCCO_14), U18.R14 (VCCO_14), U18.T11 (VCCO_14), U18.U18 (VCCO_14), U18.U8 (VCCO_14), U18.V15 (VCCO_14); no longer C145.2, C146.2, C147.2, C148.2, C149.2, C150.2, C151.2, U18.A16 (VCCO_15), U18.B13 (VCCO_15), U18.C10 (VCCO_15), U18.D17 (VCCO_15), U18.E14 (VCCO_15), U18.G18 (VCCO_15), U18.H15 (VCCO_15)
Changed lines of the file:
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@@
 	)
 	(symbol
+		(lib_id "Thunderscope_Rev5:+2V5_BAR")
+		(at 15.24 55.88 180)
+		(unit 1)
+		(exclude_from_sim no)
+		(in_bom yes)
+		(on_board yes)
+		(dnp no)
+		(property "Reference" "#PWR0263"
+			(at 15.24 55.88 0)
+			(effects
+				(font
+					(size 1.27 1.27)
+				)
+				(hide yes)
+			)
+		)
+		(property "Value" "+2V5"
+			(at 15.24 52.07 0)
+			(effects
+				(font
+					(size 1.27 1.27)
+				)
+			)
+		)
+		(property "Footprint" ""
+			(at 15.24 55.88 0)
+			(effects
+				(font
+					(size 1.27 1.27)
+				)
+			)
+		)
+		(property "Datasheet" ""
+			(at 15.24 55.88 0)
+			(effects
+				(font
+					(size 1.27 1.27)
+				)
+			)
+		)
+		(property "Description" ""
+			(at 15.24 55.88 0)
+			(effects
+				(font
+					(size 1.27 1.27)
+				)
+			)
+		)
+		(pin ""
+		)
+		(instances
+			(project "Thunderscope_Rev5"
+				(path "/031d3e2c-42e0-4016-8c32-579d45c83e09/0f922f52-a6e9-41f0-8991-df4889546a95/038472ca-999a-4bdd-b362-e2f5a3e05e32"
+					(reference "#PWR0263")
+					(unit 1)
+				)
+			)
+		)
+	)
+	(symbol
 		(lib_id "Thunderscope_Rev5:CAP 4.7uF 6.3V X5R 0402")
 		(at 33.02 116.84 0)
@@
 	)
 	(symbol
-		(lib_id "Thunderscope_Rev5:+3V3_BAR")
-		(at 15.24 55.88 180)
-		(unit 1)
-		(exclude_from_sim no)
-		(in_bom yes)
-		(on_board yes)
-		(dnp no)
-		(property "Reference" "#PWR0428"
-			(at 15.24 55.88 0)
-			(effects
-				(font
-					(size 1.27 1.27)
-				)
-				(hide yes)
-			)
-		)
-		(property "Value" "+3V3"
-			(at 15.24 52.07 0)
-			(effects
-				(font
-					(size 1.27 1.27)
-				)
-			)
-		)
-		(property "Footprint" ""
-			(at 15.24 55.88 0)
-			(effects
-				(font
-					(size 1.27 1.27)
-				)
-			)
-		)
-		(property "Datasheet" ""
-			(at 15.24 55.88 0)
-			(effects
-				(font
-					(size 1.27 1.27)
-				)
-			)
-		)
-		(property "Description" ""
-			(at 15.24 55.88 0)
-			(effects
-				(font
-					(size 1.27 1.27)
-				)
-			)
-		)
-		(pin ""
-		)
-		(instances
-			(project ""
-				(path "/031d3e2c-42e0-4016-8c32-579d45c83e09/0f922f52-a6e9-41f0-8991-df4889546a95/038472ca-999a-4bdd-b362-e2f5a3e05e32"
-					(reference "#PWR0428")
-					(unit 1)
-				)
-			)
-		)
-	)
-	(symbol
 		(lib_id "Thunderscope_Rev5:CAP 470nF 6.3V X5R 0201")
 		(at 96.52 93.98 0)
@@
 	)
 	(symbol
+		(lib_id "Thunderscope_Rev5:+3V3_BAR")
+		(at 243.84 27.94 180)
+		(unit 1)
+		(exclude_from_sim no)
+		(in_bom yes)
+		(on_board yes)
+		(dnp no)
+		(property "Reference" "#PWR0262"
+			(at 243.84 27.94 0)
+			(effects
+				(font
+					(size 1.27 1.27)
+				)
+				(hide yes)
+			)
+		)
+		(property "Value" "+3V3"
+			(at 243.84 24.13 0)
+			(effects
+				(font
+					(size 1.27 1.27)
+				)
+			)
+		)
+		(property "Footprint" ""
+			(at 243.84 27.94 0)
+			(effects
+				(font
+					(size 1.27 1.27)
+				)
+			)
+		)
+		(property "Datasheet" ""
+			(at 243.84 27.94 0)
+			(effects
+				(font
+					(size 1.27 1.27)
+				)
+			)
+		)
+		(property "Description" ""
+			(at 243.84 27.94 0)
+			(effects
+				(font
+					(size 1.27 1.27)
+				)
+			)
+		)
+		(pin ""
+		)
+		(instances
+			(project "Thunderscope_Rev5"
+				(path "/031d3e2c-42e0-4016-8c32-579d45c83e09/0f922f52-a6e9-41f0-8991-df4889546a95/038472ca-999a-4bdd-b362-e2f5a3e05e32"
+					(reference "#PWR0262")
+					(unit 1)
+				)
+			)
+		)
+	)
+	(symbol
 		(lib_id "Thunderscope_Rev5:GND")
 		(at 162.56 40.64 0)
@@
 					(unit 1)
 				)
-			)
-		)
-	)
-	(symbol
-		(lib_id "Thunderscope_Rev5:+2V5_BAR")
-		(at 243.84 27.94 180)
-		(unit 1)
-		(exclude_from_sim no)
-		(in_bom yes)
-		(on_board yes)
-		(dnp no)
-		(property "Reference" "#PWR0407"
-			(at 243.84 27.94 0)
-			(effects
-				(font
-					(size 1.27 1.27)
-				)
-				(hide yes)
-			)
-		)
-		(property "Value" "+2V5"
-			(at 243.84 24.13 0)
-			(effects
-				(font
-					(size 1.27 1.27)
-				)
-			)
-		)
-		(property "Footprint" ""
-			(at 243.84 27.94 0)
-			(effects
-				(font
-					(size 1.27 1.27)
-				)
-			)
-		)
-		(property "Datasheet" ""
-			(at 243.84 27.94 0)
-			(effects
-				(font
-					(size 1.27 1.27)
-				)
-			)
-		)
-		(property "Description" ""
-			(at 243.84 27.94 0)
-			(effects
-				(font
-					(size 1.27 1.27)
-				)
-			)
-		)
-		(pin ""
-		)
-		(instances
-			(project ""
-				(path "/031d3e2c-42e0-4016-8c32-579d45c83e09/0f922f52-a6e9-41f0-8991-df4889546a95/038472ca-999a-4bdd-b362-e2f5a3e05e32"
-					(reference "#PWR0407")
-					(unit 1)
-				)

Commit message: Linked PCB to Schematic
Connections:
- net GND: now also U18.L6 (VCCO_34), U18.M3 (VCCO_34), U18.P7 (VCCO_34), U18.R4 (VCCO_34), U18.T1 (VCCO_34), U18.V5 (VCCO_34)
- net +VIO: no longer names the net of C131.2, C132.2, C133.2, C134.2, C135.2, C136.2, C137.2
- net +VIO: no longer U18.L6 (VCCO_34), U18.M3 (VCCO_34), U18.P7 (VCCO_34), U18.R4 (VCCO_34), U18.T1 (VCCO_34), U18.V5 (VCCO_34)
Other:
- moved on the sheet: C131, C132, C133, C134, C135, C136, C137, C145, C146, C147, C148, C149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

Commit message: Added WIP Mech Model and Interposer
Also reworked rev5 power tree
Parts:
- removed C131: ${ALTIUM_VALUE}, GEN_C_0805, symbol Thunderscope_Rev5:CAP 47uF 6.3V X5R 0805
- removed C132, C133: ${ALTIUM_VALUE}, GEN_C_0402, symbol Thunderscope_Rev5:CAP 4.7uF 6.3V X5R 0402
- removed C134, C135, C136, C137: ${ALTIUM_VALUE}, GEN_C_0201, symbol Thunderscope_Rev5:CAP 470nF 6.3V X5R 0201
Connections:
- net +2V5: no longer C152.2, U18.E10 (VCCO_0), U18.R10 (VCCO_0)
- net +3V3: now also C152.2, U18.E10 (VCCO_0), U18.R10 (VCCO_0)

Commit message: Schematic WIP
Parts:
- C138, C139, C140, C141, C148, C149, C150, C151, C154, C155, C156, C157, C164, C165, C166, C167: value ${ALTIUM_VALUE} -> 470nF; footprint GEN_C_0201 -> Thunderscope_Rev5:GEN_C_0201; ALTIUM_VALUE 470nF -> (none)
- C142, C143, C146, C147, C158, C159, C162, C163, C168, C173: value ${ALTIUM_VALUE} -> 4.7uF; footprint GEN_C_0402 -> Thunderscope_Rev5:GEN_C_0402; ALTIUM_VALUE 4.7uF -> (none)
- C144, C145, C152, C153, C161: value ${ALTIUM_VALUE} -> 47uF; footprint GEN_C_0805 -> Thunderscope_Rev5:GEN_C_0805; ALTIUM_VALUE 47uF -> (none)
- C160: value ${ALTIUM_VALUE} -> 100uF; footprint GEN_C_1210 -> Thunderscope_Rev5:GEN_C_1210; ALTIUM_VALUE 100uF -> (none)
- C169, C170, C171, C172: value ${ALTIUM_VALUE} -> 100nF; footprint GEN_C_0201 -> Thunderscope_Rev5:GEN_C_0201; ALTIUM_VALUE 100nF -> (none)
- FB12, FB13: footprint GEN_R_0402 -> Thunderscope_Rev5:GEN_R_0402
- U18: footprint XILINX_XC7A50T-2CSG325C -> Thunderscope_Rev5:XILINX_XC7A50T-2CSG325C
Other:
- note added: "FPGA Power Inputs"

Commit message: Schematic Ready For Review
Parts:
- removed C160: 100uF, Thunderscope_Rev5:GEN_C_1210, symbol Thunderscope_Rev5:CAP 100uF 6.3V X5R 1210
- added C160, C86, C87: 47uF, Thunderscope_Rev5:GEN_C_0805, symbol Thunderscope_Rev5:CAP 47uF 6.3V X5R 0805
- C138, C139, C140, C141, C148, C149, C150, C151, C154, C155, C156, C157, C164, C165, C166, C167: value 470nF -> 1uF; footprint Thunderscope_Rev5:GEN_C_0201 -> Thunderscope_Rev5:GEN_C_0402; symbol Thunderscope_Rev5:CAP 470nF 6.3V X5R 0201 -> Thunderscope_Rev5:CAP 1uF 25V X5R 0402; HOUSE PART NUMBER C-470nF-0201-002 -> (none); MANUFACTURER PART NUMBER GRM033R60J474KE90D -> GRM155R61E105KA12D; PACKAGE 0201 -> 0402; SUPPLIER PART NUMBER 1 81-GRM33R60J474KE90D -> 81-GRM155R61E105KA2D; VOLTAGE RATING 6.3V -> 25V
- C142, C143, C146, C147, C158, C159, C162, C163, C168, C173: value 4.7uF -> 10uF; footprint Thunderscope_Rev5:GEN_C_0402 -> Thunderscope_Rev5:GEN_C_0603; symbol Thunderscope_Rev5:CAP 4.7uF 6.3V X5R 0402 -> Thunderscope_Rev5:CAP 10uF 10V X5R 0603; HOUSE PART NUMBER C-4.7uF-0402-002 -> C-10uF-0603-002; MANUFACTURER PART NUMBER GRM155R60J475ME47D -> GRM188R61A106ME69D; SUPPLIER PART NUMBER 1 81-GRM155R60J475ME7D -> 81-GRM188R61A106ME9D; VOLTAGE RATING 6.3V -> 10V
- C169, C170, C171, C172: footprint Thunderscope_Rev5:GEN_C_0201 -> Thunderscope_Rev5:GEN_C_0402; symbol Thunderscope_Rev5:CAP 100nF 6.3V X5R 0201 -> Thunderscope_Rev5:CAP 100nF 16V X7R 0402; HOUSE PART NUMBER C-100nF-0201-002 -> C-100nF-0402-002; MANUFACTURER PART NUMBER GRM033R60J104KE19D -> GCM155R71C104KA55D; PACKAGE 0201 -> 0402; SUPPLIER PART NUMBER 1 81-GRM033R60J104KE19 -> 81-GCM155R71C104KA5D; VOLTAGE RATING 6.3V -> 16V
Connections:
- net +1V0: now also C154.1, C155.1, C156.1, C157.1, C160.2, C86.2, C87.2; no longer C154.2, C155.2, C156.2, C157.2
- net +1V8: now also C164.1, C165.1, C166.1; no longer C164.2, C165.2, C166.2
- net +2V5: now also C148.1, C149.1, C150.1, C151.1; no longer C148.2, C149.2, C150.2, C151.2
- net +3V3: now also C138.1, C139.1, C140.1, C141.1; no longer C138.2, C139.2, C140.2, C141.2
- net AGND: now also C167.2; no longer C167.1
- net GND: now also C138.2, C139.2, C140.2, C141.2, C148.2, C149.2, C150.2, C151.2, C154.2, C155.2, C156.2, C157.2, C164.2, C165.2, C166.2, C160.1, C86.1, C87.1; no longer C138.1, C139.1, C140.1, C141.1, C148.1, C149.1, C150.1, C151.1, C154.1, C155.1, C156.1, C157.1, C164.1, C165.1, C166.1
- net at FB12.2, U18.J10 (VCCADC_0): now also C167.1; no longer C167.2
