File: Hardware/KiCad/Thunderscope_Rev5/M2_KEY_M.kicad_sch (KiCad schematic)
At the start: 4 parts, among them J8 M.2 Key M

Commit message: Added WIP Mech Model and Interposer
Also reworked rev5 power tree
Connections:
- net +3V3_IN renamed +VUSB
- net +3V3_M2 renamed +VUSB_M2
Other:
- note added: "Note that the TB/USB4 adaptor must be modified to give us VUSB instead of 3V3"
Changed lines of the file:
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@@
+		)
+	)
+	(text "Note that the TB/USB4 adaptor must be modified to give us VUSB instead of 3V3"
+		(exclude_from_sim no)
+		(at 137.16 162.56 0)
+		(effects
+			(font
+				(size 1.27 1.27)
+			)
 		)
 	)
@@
 		)
 	)
-	(label "+3V3_M2"
+	(label "+VUSB_M2"
 		(at 106.68 177.8 0)
 		(fields_autoplaced yes)
@@
 		)
 	)
-	(label "+3V3_M2"
+	(label "+VUSB_M2"
 		(at 139.7 43.18 180)
 		(fields_autoplaced yes)
@@
 	)
 	(symbol
-		(lib_id "Thunderscope_Rev5:+3V3_IN_BAR")
-		(at 165.1 175.26 180)
-		(unit 1)
-		(exclude_from_sim no)
-		(in_bom yes)
-		(on_board yes)
-		(dnp no)
-		(property "Reference" "#PWR0562"
-			(at 165.1 175.26 0)
-			(effects
-				(font
-					(size 1.27 1.27)
-				)
-				(hide yes)
-			)
-		)
-		(property "Value" "+3V3_IN"
-			(at 165.1 171.45 0)
-			(effects
-				(font
-					(size 1.27 1.27)
-				)
-			)
-		)
-		(property "Footprint" ""
-			(at 165.1 175.26 0)
-			(effects
-				(font
-					(size 1.27 1.27)
-				)
-			)
-		)
-		(property "Datasheet" ""
-			(at 165.1 175.26 0)
-			(effects
-				(font
-					(size 1.27 1.27)
-				)
-			)
-		)
-		(property "Description" ""
-			(at 165.1 175.26 0)
-			(effects
-				(font
-					(size 1.27 1.27)
-				)
-			)
-		)
-		(pin ""
-		)
-		(instances
-			(project ""
-				(path "/031d3e2c-42e0-4016-8c32-579d45c83e09/1740d22d-1854-48db-a246-157789f9c7e2"
-					(reference "#PWR0562")
-					(unit 1)
-				)
-			)
-		)
-	)
-	(symbol
 		(lib_id "Thunderscope_Rev5:GND")
 		(at 129.54 152.4 0)
@@
 					(unit 1)
 				)
+			)
+		)
+	)
+	(symbol
+		(lib_id "Thunderscope_Rev5:+VUSB")
+		(at 165.1 175.26 180)
+		(unit 1)
+		(exclude_from_sim no)
+		(in_bom yes)
+		(on_board yes)
+		(dnp no)
+		(property "Reference" "#PWR0302"
+			(at 165.1 175.26 0)
+			(effects
+				(font
+					(size 1.27 1.27)
+				)
+				(hide yes)
+			)
+		)
+		(property "Value" "+VUSB"
+			(at 165.1 171.45 0)
+			(effects
+				(font
+					(size 1.27 1.27)
+				)
+			)
+		)
+		(property "Footprint" ""
+			(at 165.1 175.26 0)
+			(effects
+				(font
+					(size 1.27 1.27)
+				)
+				(hide yes)
+			)
+		)
+		(property "Datasheet" ""
+			(at 165.1 175.26 0)
+			(effects
+				(font
+					(size 1.27 1.27)
+				)
+				(hide yes)
+			)
+		)
+		(property "Description" "Power symbol creates a global label with name '+VUSB'"
+			(at 165.1 175.26 0)
+			(effects
+				(font
+					(size 1.27 1.27)
+				)
+				(hide yes)
+			)
+		)
+		(pin ""
+		)
+		(instances
+			(project "Thunderscope_Rev5"
+				(path "/031d3e2c-42e0-4016-8c32-579d45c83e09/1740d22d-1854-48db-a246-157789f9c7e2"
+					(reference "#PWR0302")
+					(unit 1)
+				)

Commit message: Schematic WIP
Parts:
- added J10: 009155002852006, Thunderscope_Rev5:KYO_009155002852006, symbol Thunderscope_Rev5:CONN SPRING 2 PIN
- added J11: 7792, Thunderscope_Rev5:KEY_7792, symbol Thunderscope_Rev5:CONN M4 SCREW TERM KEYSTONE 7792
- J8: footprint TE_M2_KEYM_2199230 -> Thunderscope_Rev5:TE_M2_KEYM_2199230
- R54: value ${ALTIUM_VALUE} -> 0.01; footprint GEN_R_0603 -> Thunderscope_Rev5:GEN_R_0603; ALTIUM_VALUE 0.01 -> (none)
- TP19, TP20: footprint KEY_5015 -> Thunderscope_Rev5:KEY_5015
Connections:
- net +VUSB: now also J10.2
- net GND: now also J10.1, J11.1
Other:
- note added: "Fan Connector"
- note added: "Ground Lug"
- moved on the sheet: R54, TP19, TP20

Commit message: Schematic cleanup and RGB status LED
Other:
- note added: "NOTE: The TB/USB4 adaptor must be modified to give us VUSB instead of 3V3"
- note removed: "Note that the TB/USB4 adaptor must be modified to give us VUSB instead of 3V3"
Changed lines of the file:
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@@
 		)
 	)
-	(text "Note that the TB/USB4 adaptor must be modified to give us VUSB instead of 3V3"
+	(text "NOTE: The TB/USB4 adaptor must be modified to give us VUSB instead of 3V3"
 		(exclude_from_sim no)
 		(at 114.3 162.56 0)
@@
 			(font
 				(size 1.27 1.27)
+				(thickness 0.254)
+				(bold yes)
 			)
 		)

Commit message: Refactored Schematic
Parts:
- added C127, C128: 22uF, Thunderscope_Rev5:GEN_C_0805, symbol Thunderscope_Rev5:CAP 22uF 25V X5R 0805
- added C30, C31, C34, C35, C38, C39, C42, C43, C46, C47: 100nF, Thunderscope_Rev5:GEN_C_0201, symbol Thunderscope_Rev5:CAP 100nF 6.3V X5R 0201
- added D2, D3: TPD1E1B04, Thunderscope_Rev5:TI_X1SON_DPY0002A, symbol Thunderscope_Rev5:TVS TPD1E1B04
- added J1, J2: BNC, Thunderscope_Rev5:MOL_0731000105, symbol Thunderscope_Rev5:BNC JACK R/A
- added L1: 1uH, Thunderscope_Rev5:GEN_L_1210, symbol Thunderscope_Rev5:IND 1uH 5.5A 32 MOHM 1210
- added R109: 280K, Thunderscope_Rev5:GEN_R_0402, symbol Thunderscope_Rev5:RES 280K OHM 1% 1/16W 0402
- added R110: 35.7k, Thunderscope_Rev5:GEN_R_0402, symbol Thunderscope_Rev5:RES 35.7K OHM 1% 1/16W 0402
- added R14: 0.01, Thunderscope_Rev5:GEN_R_0603, symbol Thunderscope_Rev5:RES 0.01 OHM 1% 1/4W 0603
- added R2, R4: 0, Thunderscope_Rev5:GEN_R_0402, symbol Thunderscope_Rev5:RES 0 OHM 1/16W 0402
- added R24: 49.9, Thunderscope_Rev5:GEN_R_0402, symbol Thunderscope_Rev5:RES 49.9 OHM 1% 1/10W 0402
- added R27, R28, R31, R32, R35, R36, R39, R40: 0, Thunderscope_Rev5:GEN_R_0201, symbol Thunderscope_Rev5:RES 0 OHM 1% 1/20W 0201
- added R72: 10K, Thunderscope_Rev5:GEN_R_0402, symbol Thunderscope_Rev5:RES 10K OHM 1% 1/10W 0402
- added TP21, TP22: PCB, Thunderscope_Rev5:GEN_TP_PCB, symbol Thunderscope_Rev5:TP PCB 1mm
- added U17: TPS61023, Thunderscope_Rev5:TI_SOT563_DRL0006A, symbol Thunderscope_Rev5:IC BOOST TPS61023
Connections:
- net +VUSB: now also R14.1, TP21.1
- net GND: now also C127.1, C128.1, D2.2 (A), D3.2 (A), J1.2 (SHIELD), J2.2 (SHIELD), R110.2, U17.4 (GND)
- net M2_PER0_N: now also C42.1
- net M2_PER0_P: now also C43.1
- net M2_PER1_N: now also C38.1
- net M2_PER1_P: now also C39.1
- net M2_PER2_N: now also C34.1
- net M2_PER2_P: now also C35.1
- net M2_PER3_N: now also C30.1
- net M2_PER3_P: now also C31.1
- net M2_PERST#: now also R24.2
- net M2_PET0_N: now also R39.2
- net M2_PET0_P: now also R40.2
- net M2_PET1_N: now also R35.2
- net M2_PET1_P: now also R36.2
- net M2_PET2_N: now also R31.2
- net M2_PET2_P: now also R32.2
- net M2_PET3_N: now also R27.2
- net M2_PET3_P: now also R28.2
- net M2_REFCLK_N: now also C46.1
- net M2_REFCLK_P: now also C47.1
- new net: R72.1, U17.2 (EN)
- new net: C127.2, L1.1, R14.2, R72.2, TP22.1, U17.3 (VIN)
- new net: L1.2, U17.5 (SW)
- new net: R109.1, R110.1, U17.1 (FB)
- new net +5V2: C128.2, R109.2, U17.6 (VOUT)
- new net M2_PERST#_R: R24.1
- new net MGT_CLK1_N: C46.2
- new net MGT_CLK1_P: C47.2
- new net MGT_RX0_N: R27.1
- new net MGT_RX0_P: R28.1
- new net MGT_RX1_N: R31.1
- new net MGT_RX1_P: R32.1
- new net MGT_RX2_N: R35.1
- new net MGT_RX2_P: R36.1
- new net MGT_RX3_N: R39.1
- new net MGT_RX3_P: R40.1
- new net MGT_TX0_N: C30.2
- new net MGT_TX0_P: C31.2
- new net MGT_TX1_N: C34.2
- new net MGT_TX1_P: C35.2
- new net MGT_TX2_N: C38.2
- new net MGT_TX2_P: C39.2
- new net MGT_TX3_N: C42.2
- new net MGT_TX3_P: C43.2
- new net REFINOUT: R4.1
- new net REFINOUT1: D2.1 (K), J1.1 (Signal), R4.2
- new net SYNC: R2.1
- new net SYNC1: D3.1 (K), J2.1 (Signal), R2.2
Other:
- note added: "5V2: 1.05A pre-config, 0.807A post-config"
- note added: "AC Couple PER Lines with 100nF"
- note added: "AC Couple REFCLK Lines with 100nF"
- note added: "M.2 Key M Connector - Custom Pinout"
- note added: "Vout = (280/35.7+1)*0.6 = 5.31V"
- note removed: "Custom Pinout"
- note removed: "M.2 Key M Connector"
- note removed: "Main Board"
- moved on the sheet: J10, J11, J8, R54, TP19, TP20

Commit message: Schematic Rapidly Approaching Done
Still have to clear some new ERCs from the refactor
Other:
- note added: "5V2 Boost Converter"
- note added: "Refclock and Sync BNCs"
- moved on the sheet: C127, C128, C34, C35, C38, C39, C42, C43, C46, C47, D2, D3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

Commit message: Schematic Ready For Review
Parts:
- added J12, J13: 009155002852006, Thunderscope_Rev5:KYO_009155002852006, symbol Thunderscope_Rev5:CONN SPRING 2 PIN
- added R82: 10K, Thunderscope_Rev5:GEN_R_0402, symbol Thunderscope_Rev5:RES 10K OHM 1% 1/10W 0402
- C30, C31, C34, C35, C38, C39, C42, C43, C46, C47: footprint Thunderscope_Rev5:GEN_C_0201 -> Thunderscope_Rev5:GEN_C_0402; symbol Thunderscope_Rev5:CAP 100nF 6.3V X5R 0201 -> Thunderscope_Rev5:CAP 100nF 16V X7R 0402; HOUSE PART NUMBER C-100nF-0201-002 -> C-100nF-0402-002; MANUFACTURER PART NUMBER GRM033R60J104KE19D -> GCM155R71C104KA55D; PACKAGE 0201 -> 0402; SUPPLIER PART NUMBER 1 81-GRM033R60J104KE19 -> 81-GCM155R71C104KA5D; VOLTAGE RATING 6.3V -> 16V
- R27, R28, R31, R32, R35, R36, R39, R40: footprint Thunderscope_Rev5:GEN_R_0201 -> Thunderscope_Rev5:GEN_R_0402; symbol Thunderscope_Rev5:RES 0 OHM 1% 1/20W 0201 -> Thunderscope_Rev5:RES 0 OHM 1/16W 0402; MANUFACTURER Stackpole Electronics -> Yageo; MANUFACTURER PART NUMBER RMCF0201ZT0R00 -> RC0402JR-070RL; PACKAGE 0201 -> 0402; SUPPLIER PART NUMBER 1 708-RMCF0201ZT0R00 -> 603-RC0402JR-070RL; TOLERANCE 1% -> (none)
- TP21, TP22: now left out of the parts list
Connections:
- net GND: now also J12.1, J12.2, J13.1, J13.2
- net M2_PERST#_R renamed PERST#
- new net +3V3: R82.1
- new net VARIANT: R82.2
Other:
- note added: "EMI Spring Grounds"
- note added: "Variant Pin Strap"
- moved on the sheet: C127, C128, D2, D3, J1, J10, J11, J2, L1, R109, R110, R14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
