File: Hardware/KiCad/Thunderscope_Rev5/Thunderscope_Rev5.kicad_sch (KiCad schematic)
At the start: 34 parts, among them J1 BNC, J11 7792, J2 BNC, J3 1.27mm 6 Pin TH, J4 TSW-101-16-G-Q-RA, U1 SN74LVC1G17

Commit message: Altium Param Import with Script
Parts:
- removed C1: ${ALTIUM_VALUE}, GEN_C_0402, symbol Thunderscope_Rev5:CAP 100nF 16V X7R 0402
- removed D1: GREEN, LED_0603_LTST-S270K, symbol Thunderscope_Rev5:LED GREEN 0603 LTST-S270K
- removed D2, D3, D4, D5: TPD1E1B04, TI_X1SON_DPY0002A, symbol Thunderscope_Rev5:TVS TPD1E1B04
- removed J1, J2: BNC, MOL_0731000105, symbol Thunderscope_Rev5:BNC JACK R/A
- removed J3: 1.27mm 6 Pin TH, GEN_1.27mm_2x5_Pin_TH_RA, symbol Thunderscope_Rev5:CONN 1.27mm 2x5 Pin TH RA
- removed J4: TSW-101-16-G-Q-RA, GEN_5.08mm_1x2_Pin_TH_RA, symbol Thunderscope_Rev5:CONN 5.08mm 2 Pin TH RA
- removed R1, R8: ${ALTIUM_VALUE}, GEN_R_0402, symbol Thunderscope_Rev5:RES 10K OHM 1% 1/10W 0402
- removed R2, R3, R4, R5: ${ALTIUM_VALUE}, GEN_R_0402, symbol Thunderscope_Rev5:RES 0 OHM 1/16W 0402
- removed R6: ${ALTIUM_VALUE}, GEN_R_0402, symbol Thunderscope_Rev5:RES 1K OHM 1% 1/10W 0402
- removed R7: ${ALTIUM_VALUE}, GEN_R_0402, symbol Thunderscope_Rev5:RES 100 OHM 1% 1/10W 0402
- removed U1: SN74LVC1G17, GEN_SC-70-5, symbol Thunderscope_Rev5:IC BUFFER SN74LVC1G17
Connections:
- net FPGA/ACQ_EN renamed FPGA/+2V5_ACQ_EN
- no-connect marks 1 -> 0
Other:
- added sheet User IO (User_IO.kicad_sch)
- sheet FPGA ports: added +1V8_ACQ_EN, +2V5_ACQ_EN, ADC_SCLK, ADC_SDIO, PGA_SCLK, PGA_SDIO, PLL_SCL, PLL_SDA, SYNC_IN_N, SYNC_IN_P, SYNC_OUT_N, SYNC_OUT_P, TRIM_SCL, TRIM_SDA; removed ACQ_EN, SCL, SDA, SPI_SCLK, SPI_SDIO, SYNC
- sheet POWER ports: added +1V8_ACQ_EN, +2V5_ACQ_EN; removed ACQ_EN
- note removed: "*TE0712* 3V3IN: 1.381A (4.56W)"
- note removed: "3V3: 0.519A (1.71W)"
- note removed: "Connectors for muti-scope connection"
- note removed: "TODO: Seperate ADC SPI since it's now on 2V5"
- note removed: "TODO: Seperate PLL I2C since it's now on 2V5"
- moved on the sheet: FID1, FID2, FID3, FID4, FID5, FID6, FID7, FID8, J11, SHLD1, TP1, TP2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

Commit message: Added WIP Mech Model and Interposer
Also reworked rev5 power tree
Parts:
- FID1, FID2, FID3, FID4, FID5, FID6, FID7, FID8, TP1, TP4, TP5: now left out of the parts list
Connections:
- net FPGA/+2V5_ACQ_EN renamed FPGA/+3V3_ACQ_EN
Other:
- sheet FPGA ports: added +3V3_ACQ_EN; removed +2V5_ACQ_EN
- sheet POWER ports: added +3V3_ACQ_EN; removed +2V5_ACQ_EN
Changed lines of the file:
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@@
 		(unit 1)
 		(exclude_from_sim no)
-		(in_bom yes)
+		(in_bom no)
 		(on_board yes)
 		(dnp no)
@@
 		(unit 1)
 		(exclude_from_sim no)
-		(in_bom yes)
+		(in_bom no)
 		(on_board yes)
 		(dnp no)
@@
 		(unit 1)
 		(exclude_from_sim no)
-		(in_bom yes)
+		(in_bom no)
 		(on_board yes)
 		(dnp no)
@@
 		(unit 1)
 		(exclude_from_sim no)
-		(in_bom yes)
+		(in_bom no)
 		(on_board yes)
 		(dnp no)
@@
 		(unit 1)
 		(exclude_from_sim no)
-		(in_bom yes)
+		(in_bom no)
 		(on_board yes)
 		(dnp no)
@@
 		(unit 1)
 		(exclude_from_sim no)
-		(in_bom yes)
+		(in_bom no)
 		(on_board yes)
 		(dnp no)
@@
 		(unit 1)
 		(exclude_from_sim no)
-		(in_bom yes)
+		(in_bom no)
 		(on_board yes)
 		(dnp no)
@@
 		(unit 1)
 		(exclude_from_sim no)
-		(in_bom yes)
+		(in_bom no)
 		(on_board yes)
 		(dnp no)
@@
 		(unit 1)
 		(exclude_from_sim no)
-		(in_bom yes)
+		(in_bom no)
 		(on_board yes)
 		(dnp no)
@@
 		(unit 1)
 		(exclude_from_sim no)
-		(in_bom yes)
+		(in_bom no)
 		(on_board yes)
 		(dnp no)
@@
 		(unit 1)
 		(exclude_from_sim no)
-		(in_bom yes)
+		(in_bom no)
 		(on_board yes)
 		(dnp no)
@@
 			)
 		)
-		(pin "+2V5_ACQ_EN" output
+		(pin "+3V3_ACQ_EN" output
 			(at 208.28 40.64 0)
 			(effects
@@
 			(project "Thunderscope_Rev5"
 				(path "/031d3e2c-42e0-4016-8c32-579d45c83e09"
-					(page "18")
+					(page "15")
 				)
 			)
@@
 			)
 		)
-		(pin "+2V5_ACQ_EN" input
+		(pin "+3V3_ACQ_EN" input
 			(at 228.6 40.64 180)
 			(effects

Commit message: Schematic WIP
Parts:
- removed J11: 7792, KEY_7792, symbol Thunderscope_Rev5:CONN M4 SCREW TERM KEYSTONE 7792
- removed SHLD1: 9204, symbol Thunderscope_Rev5:PCIe IO Shield
- removed TP5: PCB, GEN_TP_PCB, symbol Thunderscope_Rev5:TP PCB 1mm
- FID1, FID2, FID3, FID4, FID5, FID6, FID7, FID8: footprint GEN_FID -> Thunderscope_Rev5:GEN_FID
- TP1, TP4: footprint GEN_TP_PCB -> Thunderscope_Rev5:GEN_TP_PCB
- TP2, TP3: footprint KEY_5019 -> Thunderscope_Rev5:KEY_5019
Connections:
- net FPGA/+3V3_ACQ_EN renamed ACQ and FE Voltage Regs/ACQ_EN
- net FPGA/FE_EN renamed ACQ and FE Voltage Regs/FE_EN
Other:
- sheet POWER renamed ACQ and FE Voltage Regs
- sheet ACQ and FE Voltage Regs: file PWR.kicad_sch -> ACQ_FE_VREG.kicad_sch
- sheet ACQ and FE Voltage Regs ports: added ACQ_EN, ACQ_PG, FE_PG; removed +1V8_ACQ_EN, +3V3_ACQ_EN
- sheet FPGA ports: added ACQ_EN, ACQ_PG, FE_PG, SYNC_DE, SYNC_REn, {USRIO}; removed +1V8_ACQ_EN, +3V3_ACQ_EN
- sheet User IO ports: added SYNC_DE, SYNC_REn, {USRIO}; removed none
- moved on the sheet: FID1, FID2, FID3, FID4, FID5, FID6, FID7, FID8, TP2, TP3

Commit message: Schematic cleanup and RGB status LED
Parts:
- removed TP1, TP4: PCB, Thunderscope_Rev5:GEN_TP_PCB, symbol Thunderscope_Rev5:TP PCB 1mm
Other:
- sheet FPGA ports: added {LED_RGB}; removed LED
- sheet User IO ports: added {LED_RGB}; removed LED

Commit message: Refactored Schematic
Other:
- removed sheet User IO
- sheet FPGA ports: added M2_PERST#_R, MGT_CLK0_N, MGT_CLK0_P, MGT_CLK1_N, MGT_CLK1_P, PCIe_PERST#_R, SYNC, {MGT_RX}, {MGT_TX}; removed M2_PERST#, M2_REFCLK_N, M2_REFCLK_P, PCIe_PERST#, PCIe_REFCLK_N, PCIe_REFCLK_P, PROBE_COMP, SYNC_DE, SYNC_IN_N, SYNC_IN_P, SYNC_OUT_N, SYNC_OUT_P, SYNC_REn, {LED_RGB}, {M2_RX}, {M2_TX}, {PCIe_RX}, {PCIe_TX}, {USRIO}
- sheet M.2_Key_M ports: added M2_PERST#_R, MGT_CLK1_N, MGT_CLK1_P, REFINOUT, SYNC, {MGT_RX}, {MGT_TX}; removed M2_PERST#, M2_REFCLK_N, M2_REFCLK_P, {M2_RX}, {M2_TX}
- sheet PCIe_x4 ports: added MGT_CLK0_N, MGT_CLK0_P, PCIe_PERST#_R, REFINOUT, SYNC, {MGT_RX}, {MGT_TX}; removed PCIe_PERST#, PCIe_REFCLK_N, PCIe_REFCLK_P, {PCIe_RX}, {PCIe_TX}

Commit message: Schematic Ready For Review
Other:
- sheet M.2_Key_M renamed TS-USB4 Components
- sheet PCIe_x4 renamed TS-PCIe Components
- sheet FPGA ports: added PERST#, VARIANT; removed M2_PERST#_R, MGT_CLK0_N, MGT_CLK0_P, PCIe_PERST#_R
- sheet TS-PCIe Components ports: added MGT_CLK1_N, MGT_CLK1_P, PERST#, VARIANT; removed MGT_CLK0_N, MGT_CLK0_P, PCIe_PERST#_R
- sheet TS-USB4 Components ports: added PERST#, VARIANT; removed M2_PERST#_R
Changed lines of the file:
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@@
 	(wire
 		(pts
+			(xy 223.52 83.82) (xy 236.22 83.82)
+		)
+		(stroke
+			(width 0)
+			(type default)
+		)
+	)
+	(wire
+		(pts
 			(xy 83.82 157.48) (xy 83.82 104.14)
 		)
@@
 	(wire
 		(pts
+			(xy 223.52 71.12) (xy 236.22 71.12)
+		)
+		(stroke
+			(width 0)
+			(type default)
+		)
+	)
+	(wire
+		(pts
 			(xy 147.32 142.24) (xy 160.02 142.24)
 		)
@@
 	(wire
 		(pts
+			(xy 215.9 139.7) (xy 236.22 139.7)
+		)
+		(stroke
+			(width 0)
+			(type default)
+		)
+	)
+	(wire
+		(pts
 			(xy 50.8 116.84) (xy 63.5 116.84)
 		)
@@
 	(wire
 		(pts
-			(xy 215.9 83.82) (xy 236.22 83.82)
-		)
-		(stroke
-			(width 0)
-			(type default)
-		)
-	)
-	(wire
-		(pts
 			(xy 71.12 71.12) (xy 71.12 88.9)
 		)
@@
 	(wire
 		(pts
-			(xy 50.8 175.26) (xy 63.5 175.26)
+			(xy 236.22 88.9) (xy 223.52 88.9)
 		)
 		(stroke
@@
 	(wire
 		(pts
-			(xy 215.9 91.44) (xy 236.22 91.44)
+			(xy 50.8 175.26) (xy 63.5 175.26)
 		)
 		(stroke
@@
 	(wire
 		(pts
-			(xy 215.9 88.9) (xy 236.22 88.9)
-		)
-		(stroke
-			(width 0)
-			(type default)
-		)
-	)
-	(wire
-		(pts
 			(xy 50.8 185.42) (xy 63.5 185.42)
 		)
@@
 	(wire
 		(pts
+			(xy 236.22 91.44) (xy 223.52 91.44)
+		)
+		(stroke
+			(width 0)
+			(type default)
+		)
+	)
+	(wire
+		(pts
 			(xy 50.8 73.66) (xy 63.5 73.66)
 		)
@@
 		)
 	)
+	(label "MGT_CLK1_N"
+		(at 223.52 119.38 0)
+		(effects
+			(font
+				(size 1.27 1.27)
+			)
+			(justify left bottom)
+		)
+	)
 	(label "PGA_SCLK"
 		(at 63.5 35.56 180)
@@
 		)
 	)
+	(label "PERST#"
+		(at 223.52 127 0)
+		(effects
+			(font
+				(size 1.27 1.27)
+			)
+			(justify left bottom)
+		)
+	)
 	(label "VCM"
 		(at 63.5 116.84 180)
@@
 		)
 	)
+	(label "PERST#"
+		(at 223.52 83.82 0)
+		(effects
+			(font
+				(size 1.27 1.27)
+			)
+			(justify left bottom)
+		)
+	)
 	(label "TERM_3"
 		(at 63.5 132.08 180)
@@
 		)
 	)
+	(label "MGT_CLK1_N"
+		(at 223.52 88.9 0)
+		(effects
+			(font
+				(size 1.27 1.27)
+			)
+			(justify left bottom)
+		)
+	)
+	(label "MGT_CLK1_P"
+		(at 223.52 121.92 0)
+		(effects
+			(font
+				(size 1.27 1.27)
+			)
+			(justify left bottom)
+		)
+	)
 	(label "TRIM_[4..1]"
 		(at 91.44 63.5 0)
@@
 		)
 	)
+	(label "MGT_CLK1_P"
+		(at 223.52 91.44 0)
+		(effects
+			(font
+				(size 1.27 1.27)
+			)
+			(justify left bottom)
+		)
+	)
 	(label "PGA_CSn_2"
 		(at 63.5 83.82 180)
@@
 		)
 	)
+	(label "VARIANT"
+		(at 223.52 71.12 0)
+		(effects
+			(font
+				(size 1.27 1.27)
+			)
+			(justify left bottom)
+		)
+	)
 	(label "CH4_P"
 		(at 63.5 154.94 180)
@@
 		)
 	)
+	(label "VARIANT"
+		(at 223.52 139.7 0)
+		(effects
+			(font
+				(size 1.27 1.27)
+			)
+			(justify left bottom)
+		)
+	)
 	(label "PGA_CSn_[4..1]"
 		(at 149.86 43.18 0)
@@
 			)
 		)
-		(pin "PCIe_PERST#_R" input
-			(at 215.9 83.82 0)
-			(effects
-				(font
-					(size 1.27 1.27)
-				)
-				(justify right)
-			)
-		)
-		(pin "M2_PERST#_R" input
+		(pin "PERST#" input
 			(at 215.9 127 0)
 			(effects
@@
 			)
 		)
-		(pin "MGT_CLK0_N" input
-			(at 215.9 88.9 0)
-			(effects
-				(font
-					(size 1.27 1.27)
-				)
-				(justify right)
-			)
-		)
-		(pin "MGT_CLK0_P" input
-			(at 215.9 91.44 0)
-			(effects
-				(font
-					(size 1.27 1.27)
-				)
-				(justify right)
-			)
-		)
 		(pin "MGT_CLK1_P" input
 			(at 215.9 119.38 0)
@@
 			)
 		)
+		(pin "VARIANT" input
+			(at 215.9 139.7 0)
+			(effects
+				(font
+					(size 1.27 1.27)
+				)
+				(justify right)
+			)
+		)
 		(instances
 			(project "Thunderscope_Rev5"
@@
 	(sheet
 		(at 236.22 109.22)
-		(size 27.94 27.94)
+		(size 27.94 33.02)
 		(exclude_from_sim no)
 		(in_bom yes)
@@
 			(color 0 0 0 0.0000)
 		)
-		(property "Sheetname" "M.2_Key_M"
+		(property "Sheetname" "TS-USB4 Components"
 			(at 236.22 108.5084 0)
 			(effects
@@
 		)
 		(property "Sheetfile" "M2_KEY_M.kicad_sch"
-			(at 236.22 137.7446 0)
+			(at 236.22 142.8246 0)
 			(effects
 				(font
@@
 			)
 		)
-		(pin "M2_PERST#_R" output
+		(pin "PERST#" output
 			(at 236.22 127 180)
 			(effects
@@
 			)
 		)
+		(pin "VARIANT" output
+			(at 236.22 139.7 180)
+			(effects
+				(font
+					(size 1.27 1.27)
+				)
+				(justify left)
+			)
+		)
 		(instances
 			(project "Thunderscope_Rev5"
@@
 			(project "Thunderscope_Rev5"
 				(path "/031d3e2c-42e0-4016-8c32-579d45c83e09"
-					(page "4")
+					(page "5")
 				)
 			)
@@
 	)
 	(sheet
-		(at 236.22 73.66)
-		(size 27.94 27.94)
+		(at 236.22 68.58)
+		(size 27.94 33.02)
 		(exclude_from_sim no)
 		(in_bom yes)
@@
 			(color 0 0 0 0.0000)
 		)
-		(property "Sheetname" "PCIe_x4"
-			(at 236.22 72.9484 0)
+		(property "Sheetname" "TS-PCIe Components"
+			(at 236.22 67.8684 0)
 			(effects
 				(font
@@
 			)
 		)
-		(pin "MGT_CLK0_P" output
-			(at 236.22 91.44 180)
+		(pin "PERST#" output
+			(at 236.22 83.82 180)
 			(effects
 				(font
@@
 			)
 		)
-		(pin "MGT_CLK0_N" output
-			(at 236.22 88.9 180)
+		(pin "REFINOUT" bidirectional
+			(at 236.22 78.74 180)
 			(effects
 				(font
@@
 			)
 		)
-		(pin "PCIe_PERST#_R" output
-			(at 236.22 83.82 180)
+		(pin "SYNC" bidirectional
+			(at 236.22 76.2 180)
 			(effects
 				(font
@@
 			)
 		)
-		(pin "REFINOUT" bidirectional
-			(at 236.22 78.74 180)
+		(pin "MGT_CLK1_N" output
+			(at 236.22 88.9 180)
 			(effects
 				(font
@@
 			)
 		)
-		(pin "SYNC" bidirectional
-			(at 236.22 76.2 180)
+		(pin "MGT_CLK1_P" output
+			(at 236.22 91.44 180)
+			(effects
+				(font
+					(size 1.27 1.27)
+				)
+				(justify left)
+			)
+		)
+		(pin "VARIANT" output
+			(at 236.22 71.12 180)
 			(effects
 				(font
@@
 			(project "Thunderscope_Rev5"
 				(path "/031d3e2c-42e0-4016-8c32-579d45c83e09"
-					(page "5")
+					(page "4")
 				)
 			)
