File: Hardware/KiCad/Thunderscope_Rev5/FPGA_VREG.kicad_sch (KiCad schematic)
At the start: 53 parts, among them U20 TPS62A02, U21 TPS62A02, U22 TPS7A9101, U23 TPS62A02, U8 TPS62A02

Commit message: Schematic cleanup and RGB status LED
Other:
- note added: "TODO: Replace FB Resistor"
- note removed: "TODO: Replace RB Resistor"
Changed lines of the file:
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@@
 		)
 	)
-	(text "TODO: Replace RB Resistor"
+	(text "TODO: Replace FB Resistor"
 		(exclude_from_sim no)
 		(at 215.9 121.92 0)
@@
 			(font
 				(size 1.27 1.27)
+				(thickness 0.254)
+				(bold yes)
 				(color 255 0 0 1)
 			)
@@
 			(font
 				(size 1.27 1.27)
-				(thickness 0.254)
-				(bold yes)
+				(thickness 0.1588)
 			)
 			(justify left bottom)

Commit message: Changed Relay & Flash + 1st pass BOM optimizations
Parts:
- removed R118: 66.5k, Thunderscope_Rev5:GEN_R_0402, symbol Thunderscope_Rev5:RES 66.5K OHM 1% 1/16W 0402
- removed R129, R55: 294K, Thunderscope_Rev5:GEN_R_0402, symbol Thunderscope_Rev5:RES 294K OHM 1% 1/16W 0402
- added R118, R129: 10K, Thunderscope_Rev5:GEN_R_0402, symbol Thunderscope_Rev5:RES 10K OHM 1% 1/10W 0402
- added R55: 90.9k, Thunderscope_Rev5:GEN_R_0402, symbol Thunderscope_Rev5:RES 90.9K OHM 1% 1/16W 0402
- added R69, R70: 4.7K, Thunderscope_Rev5:GEN_R_0402, symbol Thunderscope_Rev5:RES 4.7K OHM 1% 1/10W 0402
- C174, C178, C186, C74: value 39pF -> 100pF; symbol Thunderscope_Rev5:CAP 39pF 50V C0G 0402 -> Thunderscope_Rev5:CAP 100pF 50V C0G 0402; HOUSE PART NUMBER C-39pF-0402-002 -> (none); MANUFACTURER KEMET -> Murata; MANUFACTURER PART NUMBER C0402C390J5GACTU -> GCM1555C1H101FA16D; SUPPLIER PART NUMBER 1 80-C0402C390J5G -> 81-GCM1555C1H101FA6D
- R1, R117, R121, R128: value 100k -> 90.9k; symbol Thunderscope_Rev5:RES 100K OHM 1% 1/10W 0402 -> Thunderscope_Rev5:RES 90.9K OHM 1% 1/16W 0402; HOUSE PART NUMBER R-100K-0402-1%-001 -> (none); MANUFACTURER PART NUMBER RC0402FR-07100KL -> RC0402FR-0790K9L; SUPPLIER PART NUMBER 1 603-RC0402FR-07100KL -> 603-RC0402FR-0790K9L
- R119: value 100k -> 4.7K; symbol Thunderscope_Rev5:RES 100K OHM 1% 1/10W 0402 -> Thunderscope_Rev5:RES 4.7K OHM 1% 1/10W 0402; HOUSE PART NUMBER R-100K-0402-1%-001 -> (none); MANUFACTURER Yageo -> Panasonic; MANUFACTURER PART NUMBER RC0402FR-07100KL -> ERJ-2RKF4701X; SUPPLIER PART NUMBER 1 603-RC0402FR-07100KL -> 667-ERJ-2RKF4701X
- R122: value 200K -> 20k; symbol Thunderscope_Rev5:RES 200K OHM 1% 1/16W 0402 -> Thunderscope_Rev5:RES 20K OHM 1% 1/16W 0402; HOUSE PART NUMBER R-200K-0402-1%-001 -> (none); MANUFACTURER PART NUMBER RC0402FR-07200KL -> RC0402FR-0720KL; SUPPLIER PART NUMBER 1 603-RC0402FR-07200KL -> 603-RC0402FR-0720KL
- R124: value 100k -> 10K; symbol Thunderscope_Rev5:RES 100K OHM 1% 1/10W 0402 -> Thunderscope_Rev5:RES 10K OHM 1% 1/10W 0402; HOUSE PART NUMBER R-100K-0402-1%-001 -> (none); MANUFACTURER Yageo -> Panasonic; MANUFACTURER PART NUMBER RC0402FR-07100KL -> ERJ-2RKF1002X; SUPPLIER PART NUMBER 1 603-RC0402FR-07100KL -> 667-ERJ-2RKF1002X
- R130: value 90.9k -> 10K; symbol Thunderscope_Rev5:RES 90.9K OHM 1% 1/16W 0402 -> Thunderscope_Rev5:RES 10K OHM 1% 1/10W 0402; MANUFACTURER Yageo -> Panasonic; MANUFACTURER PART NUMBER RC0402FR-0790K9L -> ERJ-2RKF1002X; SUPPLIER PART NUMBER 1 603-RC0402FR-0790K9L -> 667-ERJ-2RKF1002X
- R56: value 90.9k -> 20k; symbol Thunderscope_Rev5:RES 90.9K OHM 1% 1/16W 0402 -> Thunderscope_Rev5:RES 20K OHM 1% 1/16W 0402; MANUFACTURER PART NUMBER RC0402FR-0790K9L -> RC0402FR-0720KL; SUPPLIER PART NUMBER 1 603-RC0402FR-0790K9L -> 603-RC0402FR-0720KL
Connections:
- net GND: now also R119.2, R56.1, R70.1; no longer R119.1, R56.2
- net at C74.1, U8.5 (FB): now also R56.2, R55.2; no longer R56.1
- net at C174.2, C176.2, C177.2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: now also R118.2, R69.2
- net at C74.2, C75.2, L5.2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: now also R55.1
- net at C174.1, U20.5 (FB): now also R119.1, R118.1, R69.1; no longer R119.2
- net at C186.1, R130.1, U23.5 (FB): now also R129.1, R70.2
- net at C186.2, C188.2, L4.2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: now also R129.2
Other:
- note added: "Vout = 0.6 * (10/3.197 + 1)"
- note added: "Vout = 0.6 * (20/10 + 1)"
- note added: "Vout = 0.6 * (3.197/4.7 + 1)"
- note added: "Vout = 0.6 * (90.9/20 + 1)"
- note added: "Vout = 0.6 * (R1/R2 + 1)"
- note added: "Vout = 1.008V"
- note added: "Vout = 1.2V"
- note added: "Vout = 1.8V"
- note added: "Vout = 2.477V"
- note added: "Vout = 3.327V"
- note removed: "R1 = 100 x (1.8/0.6 -1)"
- note removed: "R1 = 100 x (1/0.6 -1)"
- note removed: "R1 = 200k"
- note removed: "R1 = 287.85k"
- note removed: "R1 = 409.05k"
- note removed: "R1 = 66.67k"
- note removed: "R1 = 90.9 x (2.5/0.6 -1)"
- note removed: "R1 = R2 x (Vout/0.6 -1)"
- note removed: "TODO: Replace FB Resistor"
- note removed: "Vout = 1.79V"
- moved on the sheet: C176, C177, C186, R1, R116, R117, R119, R121, R124, R128, R56

Commit message: Refactored Schematic
Connections:
- net PG_+1V0 renamed PG_1V0
Changed lines of the file:
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@@
 		)
 	)
-	(label "PG_+1V0"
+	(label "PG_1V0"
 		(at 91.44 50.8 180)
 		(effects
@@
 		)
 	)
-	(label "PG_+1V0"
+	(label "PG_1V0"
 		(at 190.5 45.72 0)
 		(effects

Commit message: Rev 5 WIP
Added probe comp variants
Parts:
- C10, C175, C179, C181, C182, C183, C184, C187, C71, C72, C73, C9: symbol Thunderscope_Rev5:CAP 10uF 10V X5R 0603 -> Thunderscope_Rev5:CAP 10uF 25V X5R 0603; HOUSE PART NUMBER C-10uF-0603-002 -> (none); MANUFACTURER PART NUMBER GRM188R61A106ME69D -> GRM188R61E106MA73D; SUPPLIER PART NUMBER 1 81-GRM188R61A106ME9D -> 81-GRM188R61E106MA3D; VOLTAGE RATING 10V -> 25V
- U22: MANUFACTURER PART NUMBER TPS7A9101DSKT -> TPS7A9101DSKR; SUPPLIER 1 Digi-Key -> Texas Instruments; SUPPLIER PART NUMBER 1 296-45298-1-ND -> TPS7A9101DSKR
