File: Hardware/KiCad/Thunderscope_Rev5/ACQ_FE_VREG.kicad_sch (KiCad schematic)
At the start: 69 parts, among them U13 LM27761, U14 TPS7A9101, U15 TPS7A9101, U16 TPS7A2033, U17 TPS61023, U9 TPS7A2033

Commit message: Schematic cleanup and RGB status LED
Parts:
- added TP1, TP4: PCB, Thunderscope_Rev5:GEN_TP_PCB, symbol Thunderscope_Rev5:TP PCB 1mm
Connections:
- net ACQ_EN: now also TP1.1
- net FE_EN: now also TP4.1
Other:
- moved on the sheet: C107, C108, C109, C110, C115, C116, C117, C118, C123, C127, C77, R101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

Commit message: Changed Relay & Flash + 1st pass BOM optimizations
Parts:
- removed R108: 680K, Thunderscope_Rev5:GEN_R_0402, symbol Thunderscope_Rev5:RES 680K OHM 1% 1/16W 0402
- removed R109: 90.9k, Thunderscope_Rev5:GEN_R_0402, symbol Thunderscope_Rev5:RES 90.9K OHM 1% 1/16W 0402
- removed R93: 300K, Thunderscope_Rev5:GEN_R_0402, symbol Thunderscope_Rev5:RES 300K OHM 1% 1/10W 0402
- added R109, R93: 280K, Thunderscope_Rev5:GEN_R_0402, symbol Thunderscope_Rev5:RES 280K OHM 1% 1/16W 0402
- R110: value 100k -> 35.7k; symbol Thunderscope_Rev5:RES 100K OHM 1% 1/10W 0402 -> Thunderscope_Rev5:RES 35.7K OHM 1% 1/16W 0402; HOUSE PART NUMBER R-100K-0402-1%-001 -> (none); MANUFACTURER PART NUMBER RC0402FR-07100KL -> RC0402FR-0735K7L; SUPPLIER PART NUMBER 1 603-RC0402FR-07100KL -> 603-RC0402FR-0735K7L
- R96: value 100k -> 90.9k; symbol Thunderscope_Rev5:RES 100K OHM 1% 1/10W 0402 -> Thunderscope_Rev5:RES 90.9K OHM 1% 1/16W 0402; HOUSE PART NUMBER R-100K-0402-1%-001 -> (none); MANUFACTURER PART NUMBER RC0402FR-07100KL -> RC0402FR-0790K9L; SUPPLIER PART NUMBER 1 603-RC0402FR-07100KL -> 603-RC0402FR-0790K9L
Connections:
- net +5V2: now also R109.2
- net GND: now also R110.2; no longer R110.1
- net at C106.2, R91.1, TP29.1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: now also R93.2
- net at R96.2, U13.5 (VFB): now also R93.1
- net at U17.1 (FB): now also R110.1, R109.1; no longer R110.2
Other:
- note added: "The value for R2 must be no less than 50 kΩ."
- note added: "Vout = (280/35.7+1)*0.6 = 5.31V"
- note added: "Vout = -1.22*(280/90.9+1)= -4.98V"
- note added: "Vout = -1.22V*(R1+R2)/R2"
- note removed: "Vout = (771.9/100+1)*0.6= 5.23V"
- moved on the sheet: R110, R96

Commit message: Refactored Schematic
Parts:
- removed C127, C128: 22uF, Thunderscope_Rev5:GEN_C_0805, symbol Thunderscope_Rev5:CAP 22uF 25V X5R 0805
- removed L1: 1uH, Thunderscope_Rev5:GEN_L_1210, symbol Thunderscope_Rev5:IND 1uH 5.5A 32 MOHM 1210
- removed R109: 280K, Thunderscope_Rev5:GEN_R_0402, symbol Thunderscope_Rev5:RES 280K OHM 1% 1/16W 0402
- removed R110: 35.7k, Thunderscope_Rev5:GEN_R_0402, symbol Thunderscope_Rev5:RES 35.7K OHM 1% 1/16W 0402
- removed R14: 0.01, Thunderscope_Rev5:GEN_R_0603, symbol Thunderscope_Rev5:RES 0.01 OHM 1% 1/4W 0603
- removed TP21, TP22: 5015, Thunderscope_Rev5:KEY_5015, symbol Thunderscope_Rev5:TP KEYSTONE 5015
- removed U17: TPS61023, Thunderscope_Rev5:TI_SOT563_DRL0006A, symbol Thunderscope_Rev5:IC BOOST TPS61023
Connections:
- net FE_EN: now also U13.6 (EN), U15.7 (EN)
- net at C119.2, C120.2, R98.2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: no longer U15.7 (EN)
- net at C111.2, R90.2, TP28.1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: no longer U13.6 (EN)
Other:
- note removed: "5V2: 1.05A pre-config, 0.807A post-config"
- note removed: "Vout = (280/35.7+1)*0.6 = 5.31V"
- moved on the sheet: C106, C111, C112, C114, C119, C120, C121, C122, C124, C125, C126, C76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

Commit message: Rev 5 WIP
Added probe comp variants
Parts:
- C106, C107, C108, C109, C110, C111, C114, C115, C116, C117, C118, C119, C120, C121, C122: symbol Thunderscope_Rev5:CAP 10uF 10V X5R 0603 -> Thunderscope_Rev5:CAP 10uF 25V X5R 0603; HOUSE PART NUMBER C-10uF-0603-002 -> (none); MANUFACTURER PART NUMBER GRM188R61A106ME69D -> GRM188R61E106MA73D; SUPPLIER PART NUMBER 1 81-GRM188R61A106ME9D -> 81-GRM188R61E106MA3D; VOLTAGE RATING 10V -> 25V
- U14, U15: MANUFACTURER PART NUMBER TPS7A9101DSKT -> TPS7A9101DSKR; SUPPLIER 1 Digi-Key -> Texas Instruments; SUPPLIER PART NUMBER 1 296-45298-1-ND -> TPS7A9101DSKR

Commit message: Placement WIP
Connections:
- net +2V5_R_ACQ: now reaches C115.2, C116.2, R97.2, TP32.1, U14.10 (IN), U14.6 (SS_CTRL), U14.9 (IN)
- net +VUSB_R_ACQ: now reaches C107.2, C108.2, R89.2, TP26.1, U9.1 (IN)
Changed lines of the file:
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@@
+		)
+	)
+	(label "+VUSB_R_ACQ"
+		(at 60.96 33.02 0)
+		(effects
+			(font
+				(size 1.27 1.27)
+			)
+			(justify left bottom)
+		)
+	)
+	(label "+2V5_R_ACQ"
+		(at 180.34 33.02 0)
+		(effects
+			(font
+				(size 1.27 1.27)
+			)
+			(justify left bottom)
 		)
 	)
