File: Hardware/KiCad/Thunderscope_Rev5/ADC.kicad_sch (KiCad schematic)
At the start: 30 parts, among them U6 HMCAD1520

Commit message: Linked PCB to Schematic
Changed lines of the file:
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@@
 	)
 	(junction
+		(at 83.82 30.48)
+		(diameter 0)
+		(color 0 0 0 0)
+	)
+	(junction
 		(at 119.38 50.8)
 		(diameter 0)
@@
 	)
 	(junction
+		(at 190.5 30.48)
+		(diameter 0)
+		(color 0 0 0 0)
+	)
+	(junction
 		(at 147.32 50.8)
 		(diameter 0)
@@
 	(wire
 		(pts
+			(xy 83.82 30.48) (xy 78.74 30.48)
+		)
+		(stroke
+			(width 0)
+			(type default)
+		)
+	)
+	(wire
+		(pts
 			(xy 88.9 81.28) (xy 119.38 81.28)
 		)
@@
 	(wire
 		(pts
-			(xy 200.66 30.48) (xy 187.96 30.48)
+			(xy 200.66 30.48) (xy 190.5 30.48)
 		)
 		(stroke
@@
 	(wire
 		(pts
-			(xy 88.9 30.48) (xy 78.74 30.48)
+			(xy 88.9 30.48) (xy 83.82 30.48)
 		)
 		(stroke
@@
 	(wire
 		(pts
+			(xy 190.5 30.48) (xy 187.96 30.48)
+		)
+		(stroke
+			(width 0)
+			(type default)
+		)
+	)
+	(wire
+		(pts
 			(xy 195.58 152.4) (xy 182.88 152.4)
 		)
@@
 	)
 	(symbol
+		(lib_id "power:PWR_FLAG")
+		(at 83.82 30.48 0)
+		(unit 1)
+		(exclude_from_sim no)
+		(in_bom yes)
+		(on_board yes)
+		(dnp no)
+		(property "Reference" "#FLG07"
+			(at 83.82 28.575 0)
+			(effects
+				(font
+					(size 1.27 1.27)
+				)
+				(hide yes)
+			)
+		)
+		(property "Value" "PWR_FLAG"
+			(at 83.82 26.67 0)
+			(effects
+				(font
+					(size 1.27 1.27)
+				)
+			)
+		)
+		(property "Footprint" ""
+			(at 83.82 30.48 0)
+			(effects
+				(font
+					(size 1.27 1.27)
+				)
+				(hide yes)
+			)
+		)
+		(property "Datasheet" "~"
+			(at 83.82 30.48 0)
+			(effects
+				(font
+					(size 1.27 1.27)
+				)
+				(hide yes)
+			)
+		)
+		(property "Description" "Special symbol for telling ERC where power comes from"
+			(at 83.82 30.48 0)
+			(effects
+				(font
+					(size 1.27 1.27)
+				)
+				(hide yes)
+			)
+		)
+		(pin "1"
+		)
+		(instances
+			(project ""
+				(path "/031d3e2c-42e0-4016-8c32-579d45c83e09/9a43e052-ab3a-4eb2-8617-8e5430b531e4"
+					(reference "#FLG07")
+					(unit 1)
+				)
+			)
+		)
+	)
+	(symbol
 		(lib_id "Thunderscope_Rev5:RES 10K OHM 1% 1/10W 0402")
 		(at 93.98 68.58 90)
@@
 					(unit 1)
 				)
+			)
+		)
+	)
+	(symbol
+		(lib_id "power:PWR_FLAG")
+		(at 190.5 30.48 0)
+		(unit 1)
+		(exclude_from_sim no)
+		(in_bom yes)
+		(on_board yes)
+		(dnp no)
+		(property "Reference" "#FLG08"
+			(at 190.5 28.575 0)
+			(effects
+				(font
+					(size 1.27 1.27)
+				)
+				(hide yes)
+			)
+		)
+		(property "Value" "PWR_FLAG"
+			(at 190.5 26.67 0)
+			(effects
+				(font
+					(size 1.27 1.27)
+				)
+			)
+		)
+		(property "Footprint" ""
+			(at 190.5 30.48 0)
+			(effects
+				(font
+					(size 1.27 1.27)
+				)
+				(hide yes)
+			)
+		)
+		(property "Datasheet" "~"
+			(at 190.5 30.48 0)
+			(effects
+				(font
+					(size 1.27 1.27)
+				)
+				(hide yes)
+			)
+		)
+		(property "Description" "Special symbol for telling ERC where power comes from"
+			(at 190.5 30.48 0)
+			(effects
+				(font
+					(size 1.27 1.27)
+				)
+				(hide yes)
+			)
+		)
+		(pin "1"
+		)
+		(instances
+			(project ""
+				(path "/031d3e2c-42e0-4016-8c32-579d45c83e09/9a43e052-ab3a-4eb2-8617-8e5430b531e4"
+					(reference "#FLG08")
+					(unit 1)
+				)

Commit message: Added WIP Mech Model and Interposer
Also reworked rev5 power tree
Parts:
- TP10, TP11, TP12: now left out of the parts list
Connections:
- net +2V5_ACQ renamed +3V3_ACQ
Changed lines of the file:
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@@
 	(wire
 		(pts
+			(xy 198.12 48.26) (xy 198.12 50.8)
+		)
+		(stroke
+			(width 0)
+			(type default)
+		)
+	)
+	(wire
+		(pts
 			(xy 195.58 99.06) (xy 182.88 99.06)
 		)
@@
 	)
 	(symbol
-		(lib_id "Thunderscope_Rev5:+2V5_ACQ_BAR")
-		(at 88.9 58.42 180)
-		(unit 1)
-		(exclude_from_sim no)
-		(in_bom yes)
-		(on_board yes)
-		(dnp no)
-		(property "Reference" "#PWR0247"
-			(at 88.9 58.42 0)
-			(effects
-				(font
-					(size 1.27 1.27)
-				)
-				(hide yes)
-			)
-		)
-		(property "Value" "+2V5_ACQ"
-			(at 88.9 54.61 0)
-			(effects
-				(font
-					(size 1.27 1.27)
-				)
-			)
-		)
-		(property "Footprint" ""
-			(at 88.9 58.42 0)
-			(effects
-				(font
-					(size 1.27 1.27)
-				)
-			)
-		)
-		(property "Datasheet" ""
-			(at 88.9 58.42 0)
-			(effects
-				(font
-					(size 1.27 1.27)
-				)
-			)
-		)
-		(property "Description" ""
-			(at 88.9 58.42 0)
-			(effects
-				(font
-					(size 1.27 1.27)
-				)
-			)
-		)
-		(pin ""
-		)
-		(instances
-			(project "Thunderscope_Rev5"
-				(path "/031d3e2c-42e0-4016-8c32-579d45c83e09/9a43e052-ab3a-4eb2-8617-8e5430b531e4"
-					(reference "#PWR0247")
-					(unit 1)
-				)
-			)
-			(project ""
-				(path "/0b10f000-2eec-40e9-aede-51d71661a624"
-					(reference "#PWR?")
-					(unit 1)
-				)
-			)
-		)
-	)
-	(symbol
 		(lib_id "Thunderscope_Rev5:CAP 10nF 50V X7R 0402")
 		(at 167.64 35.56 0)
@@
 	)
 	(symbol
+		(lib_id "Thunderscope_Rev5:+3V3_ACQ_BAR")
+		(at 88.9 58.42 180)
+		(unit 1)
+		(exclude_from_sim no)
+		(in_bom yes)
+		(on_board yes)
+		(dnp no)
+		(property "Reference" "#PWR0247"
+			(at 88.9 58.42 0)
+			(effects
+				(font
+					(size 1.27 1.27)
+				)
+				(hide yes)
+			)
+		)
+		(property "Value" "+3V3_ACQ"
+			(at 88.9 54.61 0)
+			(effects
+				(font
+					(size 1.27 1.27)
+				)
+			)
+		)
+		(property "Footprint" ""
+			(at 88.9 58.42 0)
+			(effects
+				(font
+					(size 1.27 1.27)
+				)
+				(hide yes)
+			)
+		)
+		(property "Datasheet" ""
+			(at 88.9 58.42 0)
+			(effects
+				(font
+					(size 1.27 1.27)
+				)
+				(hide yes)
+			)
+		)
+		(property "Description" "Power symbol creates a global label with name '+3V3_ACQ'"
+			(at 88.9 58.42 0)
+			(effects
+				(font
+					(size 1.27 1.27)
+				)
+				(hide yes)
+			)
+		)
+		(pin ""
+		)
+		(instances
+			(project "Thunderscope_Rev5"
+				(path "/031d3e2c-42e0-4016-8c32-579d45c83e09/9a43e052-ab3a-4eb2-8617-8e5430b531e4"
+					(reference "#PWR0247")
+					(unit 1)
+				)
+			)
+		)
+	)
+	(symbol
 		(lib_id "Thunderscope_Rev5:GND")
 		(at 129.54 40.64 0)
@@
 	)
 	(symbol
-		(lib_id "Thunderscope_Rev5:+2V5_ACQ_BAR")
-		(at 198.12 50.8 90)
-		(unit 1)
-		(exclude_from_sim no)
-		(in_bom yes)
-		(on_board yes)
-		(dnp no)
-		(property "Reference" "#PWR0240"
-			(at 198.12 50.8 0)
-			(effects
-				(font
-					(size 1.27 1.27)
-				)
-				(hide yes)
-			)
-		)
-		(property "Value" "+2V5_ACQ"
-			(at 201.93 50.8 90)
-			(effects
-				(font
-					(size 1.27 1.27)
-				)
-				(justify right)
-			)
-		)
-		(property "Footprint" ""
-			(at 198.12 50.8 0)
-			(effects
-				(font
-					(size 1.27 1.27)
-				)
-			)
-		)
-		(property "Datasheet" ""
-			(at 198.12 50.8 0)
-			(effects
-				(font
-					(size 1.27 1.27)
-				)
-			)
-		)
-		(property "Description" ""
-			(at 198.12 50.8 0)
-			(effects
-				(font
-					(size 1.27 1.27)
-				)
-			)
-		)
-		(pin ""
-		)
-		(instances
-			(project "Thunderscope_Rev5"
-				(path "/031d3e2c-42e0-4016-8c32-579d45c83e09/9a43e052-ab3a-4eb2-8617-8e5430b531e4"
-					(reference "#PWR0240")
-					(unit 1)
-				)
-			)
-			(project ""
-				(path "/0b10f000-2eec-40e9-aede-51d71661a624"
-					(reference "#PWR?")
-					(unit 1)
-				)
-			)
-		)
-	)
-	(symbol
 		(lib_id "Thunderscope_Rev5:CAP 1nF 50V C0G 0402")
 		(at 129.54 35.56 0)
@@
 		(unit 1)
 		(exclude_from_sim no)
-		(in_bom yes)
+		(in_bom no)
 		(on_board yes)
 		(dnp no)
@@
 		(unit 1)
 		(exclude_from_sim no)
-		(in_bom yes)
+		(in_bom no)
 		(on_board yes)
 		(dnp no)
@@
 	)
 	(symbol
+		(lib_id "Thunderscope_Rev5:+3V3_ACQ_BAR")
+		(at 198.12 48.26 180)
+		(unit 1)
+		(exclude_from_sim no)
+		(in_bom yes)
+		(on_board yes)
+		(dnp no)
+		(property "Reference" "#PWR0240"
+			(at 198.12 48.26 0)
+			(effects
+				(font
+					(size 1.27 1.27)
+				)
+				(hide yes)
+			)
+		)
+		(property "Value" "+3V3_ACQ"
+			(at 198.12 44.45 0)
+			(effects
+				(font
+					(size 1.27 1.27)
+				)
+			)
+		)
+		(property "Footprint" ""
+			(at 198.12 48.26 0)
+			(effects
+				(font
+					(size 1.27 1.27)
+				)
+				(hide yes)
+			)
+		)
+		(property "Datasheet" ""
+			(at 198.12 48.26 0)
+			(effects
+				(font
+					(size 1.27 1.27)
+				)
+				(hide yes)
+			)
+		)
+		(property "Description" "Power symbol creates a global label with name '+3V3_ACQ'"
+			(at 198.12 48.26 0)
+			(effects
+				(font
+					(size 1.27 1.27)
+				)
+				(hide yes)
+			)
+		)
+		(pin ""
+		)
+		(instances
+			(project "Thunderscope_Rev5"
+				(path "/031d3e2c-42e0-4016-8c32-579d45c83e09/9a43e052-ab3a-4eb2-8617-8e5430b531e4"
+					(reference "#PWR0240")
+					(unit 1)
+				)
+			)
+		)
+	)
+	(symbol
 		(lib_id "Thunderscope_Rev5:RES 10K OHM 1% 1/10W 0402")
 		(at 88.9 68.58 90)
@@
 		(unit 1)
 		(exclude_from_sim no)
-		(in_bom yes)
+		(in_bom no)
 		(on_board yes)
 		(dnp no)

Commit message: Schematic WIP
Parts:
- added TP5: PCB, Thunderscope_Rev5:GEN_TP_PCB, symbol Thunderscope_Rev5:TP PCB 1mm
- C12, C13, C20, C21, C22, C26: value ${ALTIUM_VALUE} -> 1uF; footprint GEN_C_0402 -> Thunderscope_Rev5:GEN_C_0402; ALTIUM_VALUE 1uF -> (none)
- C14, C15, C18, C19, C23, C25: value ${ALTIUM_VALUE} -> 10nF; footprint GEN_C_0402 -> Thunderscope_Rev5:GEN_C_0402; ALTIUM_VALUE 10nF -> (none)
- C16, C17, C24: value ${ALTIUM_VALUE} -> 1nF; footprint GEN_C_0402 -> Thunderscope_Rev5:GEN_C_0402; ALTIUM_VALUE 1nF -> (none)
- C27: value ${ALTIUM_VALUE} -> 100nF; footprint GEN_C_0402 -> Thunderscope_Rev5:GEN_C_0402; ALTIUM_VALUE 100nF -> (none)
- FB1, FB2: footprint GEN_R_0402 -> Thunderscope_Rev5:GEN_R_0402
- R15, R16, R17: value ${ALTIUM_VALUE} -> 10K; footprint GEN_R_0402 -> Thunderscope_Rev5:GEN_R_0402; ALTIUM_VALUE 10K -> (none)
- R18, R19, R20, R21, R22: value ${ALTIUM_VALUE} -> 100; footprint GEN_R_0402 -> Thunderscope_Rev5:GEN_R_0402; ALTIUM_VALUE 100 -> (none)
- TP10, TP11, TP12: footprint GEN_TP_PCB -> Thunderscope_Rev5:GEN_TP_PCB
- U6: footprint AD_QFN48_LP7 -> Thunderscope_Rev5:AD_QFN48_LP7
Connections:
- net VCM: now also TP5.1
Other:
- moved on the sheet: C27

Commit message: Schematic cleanup and RGB status LED
Changed lines of the file:
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@@
 			(font
 				(size 1.27 1.27)
-				(thickness 0.254)
-				(bold yes)
+				(thickness 0.1588)
 			)
 			(justify left)
@@
 			(font
 				(size 1.27 1.27)
-				(thickness 0.254)
-				(bold yes)
+				(thickness 0.1588)
 			)
 			(justify left)
@@
 			(font
 				(size 1.27 1.27)
-				(thickness 0.254)
-				(bold yes)
+				(thickness 0.1588)
 			)
 			(justify left bottom)
@@
 			(font
 				(size 1.27 1.27)
-				(thickness 0.254)
-				(bold yes)
+				(thickness 0.1588)
 			)
 			(justify left bottom)

Commit message: Schematic Ready For Review
Parts:
- C14, C15, C18, C19, C23, C25: value 10nF -> 1uF; symbol Thunderscope_Rev5:CAP 10nF 50V X7R 0402 -> Thunderscope_Rev5:CAP 1uF 25V X5R 0402; HOUSE PART NUMBER C-10nF-0402-002 -> (none); MANUFACTURER PART NUMBER GRM155R71H103KA88J -> GRM155R61E105KA12D; SUPPLIER PART NUMBER 1 81-GRM155R71H103KA8J -> 81-GRM155R61E105KA2D; VOLTAGE RATING 50V -> 25V
- C16, C17, C24: value 1nF -> 1uF; symbol Thunderscope_Rev5:CAP 1nF 50V C0G 0402 -> Thunderscope_Rev5:CAP 1uF 25V X5R 0402; MANUFACTURER PART NUMBER GRM1555C1H102FA01D -> GRM155R61E105KA12D; SUPPLIER PART NUMBER 1 81-GRM1555C1H102FA1D -> 81-GRM155R61E105KA2D; VOLTAGE RATING 50V -> 25V
Connections:
- net +1V8A: now also C14.1, C15.1, C16.1, C17.1, C23.1, C24.1; no longer C14.2, C15.2, C16.2, C17.2, C23.2, C24.2
- net +1V8D: now also C18.1, C19.1; no longer C18.2, C19.2
- net +3V3_ACQ: now also C25.1; no longer C25.2
- net GND: now also C14.2, C15.2, C16.2, C17.2, C18.2, C19.2, C23.2, C24.2, C25.2; no longer C14.1, C15.1, C16.1, C17.1, C18.1, C19.1, C23.1, C24.1, C25.1
Changed lines of the file:
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@@
 	)
 	(symbol
-		(lib_id "Thunderscope_Rev5:CAP 1nF 50V C0G 0402")
+		(lib_id "Thunderscope_Rev5:CAP 1uF 25V X5R 0402")
 		(at 139.7 35.56 0)
 		(unit 1)
@@
 			)
 		)
-		(property "Value" "1nF"
+		(property "Value" "1uF"
 			(at 142.24 38.1 0)
 			(effects
@@
 			)
 		)
-		(property "VOLTAGE RATING" "50V"
+		(property "VOLTAGE RATING" "25V"
 			(at 137.446 29.972 0)
 			(effects
@@
 			)
 		)
-		(property "SUPPLIER PART NUMBER 1" "81-GRM1555C1H102FA1D"
+		(property "SUPPLIER PART NUMBER 1" "81-GRM155R61E105KA2D"
 			(at 137.446 29.972 0)
 			(effects
@@
 			)
 		)
-		(property "MANUFACTURER PART NUMBER" "GRM1555C1H102FA01D"
+		(property "MANUFACTURER PART NUMBER" "GRM155R61E105KA12D"
 			(at 137.446 29.972 0)
 			(effects
@@
 			)
 		)
-		(property "ALTIUM_VALUE" ""
-			(at 139.7 35.56 0)
-			(effects
-				(font
-					(size 1.27 1.27)
-				)
-			)
-		)
 		(pin "1"
 		)
@@
 	)
 	(symbol
-		(lib_id "Thunderscope_Rev5:CAP 10nF 50V X7R 0402")
+		(lib_id "Thunderscope_Rev5:CAP 1uF 25V X5R 0402")
 		(at 109.22 35.56 0)
 		(unit 1)
@@
 			)
 		)
-		(property "Value" "10nF"
+		(property "Value" "1uF"
 			(at 111.76 38.1 0)
 			(effects
@@
 			)
 		)
-		(property "VOLTAGE RATING" "50V"
+		(property "VOLTAGE RATING" "25V"
 			(at 106.966 29.972 0)
 			(effects
@@
 			)
 		)
-		(property "SUPPLIER PART NUMBER 1" "81-GRM155R71H103KA8J"
+		(property "SUPPLIER PART NUMBER 1" "81-GRM155R61E105KA2D"
 			(at 106.966 29.972 0)
 			(effects
@@
 			)
 		)
-		(property "HOUSE PART NUMBER" "C-10nF-0402-002"
+		(property "HOUSE PART NUMBER" ""
 			(at 106.966 29.972 0)
 			(effects
@@
 			)
 		)
-		(property "MANUFACTURER PART NUMBER" "GRM155R71H103KA88J"
+		(property "MANUFACTURER PART NUMBER" "GRM155R61E105KA12D"
 			(at 106.966 29.972 0)
 			(effects
@@
 			)
 		)
-		(property "ALTIUM_VALUE" ""
-			(at 109.22 35.56 0)
-			(effects
-				(font
-					(size 1.27 1.27)
-				)
-			)
-		)
 		(pin "1"
 		)
@@
 	)
 	(symbol
-		(lib_id "Thunderscope_Rev5:CAP 10nF 50V X7R 0402")
+		(lib_id "Thunderscope_Rev5:CAP 1uF 25V X5R 0402")
 		(at 167.64 55.88 0)
 		(unit 1)
@@
 			)
 		)
-		(property "Value" "10nF"
+		(property "Value" "1uF"
 			(at 170.18 58.42 0)
 			(effects
@@
 			)
 		)
-		(property "VOLTAGE RATING" "50V"
+		(property "VOLTAGE RATING" "25V"
 			(at 168.14 60.88 0)
 			(effects
@@
 			)
 		)
-		(property "SUPPLIER PART NUMBER 1" "81-GRM155R71H103KA8J"
+		(property "SUPPLIER PART NUMBER 1" "81-GRM155R61E105KA2D"
 			(at 165.386 50.292 0)
 			(effects
@@
 			)
 		)
-		(property "HOUSE PART NUMBER" "C-10nF-0402-002"
+		(property "HOUSE PART NUMBER" ""
 			(at 165.386 50.292 0)
 			(effects
@@
 			)
 		)
-		(property "MANUFACTURER PART NUMBER" "GRM155R71H103KA88J"
+		(property "MANUFACTURER PART NUMBER" "GRM155R61E105KA12D"
 			(at 165.386 50.292 0)
 			(effects
@@
 			)
 		)
-		(property "ALTIUM_VALUE" ""
-			(at 167.64 55.88 0)
-			(effects
-				(font
-					(size 1.27 1.27)
-				)
-			)
-		)
 		(pin "2"
 		)
@@
 	)
 	(symbol
-		(lib_id "Thunderscope_Rev5:CAP 10nF 50V X7R 0402")
+		(lib_id "Thunderscope_Rev5:CAP 1uF 25V X5R 0402")
 		(at 119.38 35.56 0)
 		(unit 1)
@@
 			)
 		)
-		(property "Value" "10nF"
+		(property "Value" "1uF"
 			(at 121.92 38.1 0)
 			(effects
@@
 			)
 		)
-		(property "VOLTAGE RATING" "50V"
+		(property "VOLTAGE RATING" "25V"
 			(at 117.126 29.972 0)
 			(effects
@@
 			)
 		)
-		(property "SUPPLIER PART NUMBER 1" "81-GRM155R71H103KA8J"
+		(property "SUPPLIER PART NUMBER 1" "81-GRM155R61E105KA2D"
 			(at 117.126 29.972 0)
 			(effects
@@
 			)
 		)
-		(property "HOUSE PART NUMBER" "C-10nF-0402-002"
+		(property "HOUSE PART NUMBER" ""
 			(at 117.126 29.972 0)
 			(effects
@@
 			)
 		)
-		(property "MANUFACTURER PART NUMBER" "GRM155R71H103KA88J"
+		(property "MANUFACTURER PART NUMBER" "GRM155R61E105KA12D"
 			(at 117.126 29.972 0)
 			(effects
@@
 			)
 		)
-		(property "ALTIUM_VALUE" ""
-			(at 119.38 35.56 0)
-			(effects
-				(font
-					(size 1.27 1.27)
-				)
-			)
-		)
 		(pin "1"
 		)
@@
 	)
 	(symbol
-		(lib_id "Thunderscope_Rev5:CAP 10nF 50V X7R 0402")
+		(lib_id "Thunderscope_Rev5:CAP 1uF 25V X5R 0402")
 		(at 157.48 35.56 0)
 		(unit 1)
@@
 			)
 		)
-		(property "Value" "10nF"
+		(property "Value" "1uF"
 			(at 160.02 38.1 0)
 			(effects
@@
 			)
 		)
-		(property "VOLTAGE RATING" "50V"
+		(property "VOLTAGE RATING" "25V"
 			(at 157.98 40.56 0)
 			(effects
@@
 			)
 		)
-		(property "SUPPLIER PART NUMBER 1" "81-GRM155R71H103KA8J"
+		(property "SUPPLIER PART NUMBER 1" "81-GRM155R61E105KA2D"
 			(at 155.226 29.972 0)
 			(effects
@@
 			)
 		)
-		(property "HOUSE PART NUMBER" "C-10nF-0402-002"
+		(property "HOUSE PART NUMBER" ""
 			(at 155.226 29.972 0)
 			(effects
@@
 			)
 		)
-		(property "MANUFACTURER PART NUMBER" "GRM155R71H103KA88J"
+		(property "MANUFACTURER PART NUMBER" "GRM155R61E105KA12D"
 			(at 155.226 29.972 0)
 			(effects
@@
 			)
 		)
-		(property "ALTIUM_VALUE" ""
-			(at 157.48 35.56 0)
-			(effects
-				(font
-					(size 1.27 1.27)
-				)
-			)
-		)
 		(pin "2"
 		)
@@
 	)
 	(symbol
-		(lib_id "Thunderscope_Rev5:CAP 1nF 50V C0G 0402")
+		(lib_id "Thunderscope_Rev5:CAP 1uF 25V X5R 0402")
 		(at 129.54 55.88 0)
 		(unit 1)
@@
 			)
 		)
-		(property "Value" "1nF"
+		(property "Value" "1uF"
 			(at 132.08 58.42 0)
 			(effects
@@
 			)
 		)
-		(property "VOLTAGE RATING" "50V"
+		(property "VOLTAGE RATING" "25V"
 			(at 127.286 50.292 0)
 			(effects
@@
 			)
 		)
-		(property "SUPPLIER PART NUMBER 1" "81-GRM1555C1H102FA1D"
+		(property "SUPPLIER PART NUMBER 1" "81-GRM155R61E105KA2D"
 			(at 127.286 50.292 0)
 			(effects
@@
 			)
 		)
-		(property "MANUFACTURER PART NUMBER" "GRM1555C1H102FA01D"
+		(property "MANUFACTURER PART NUMBER" "GRM155R61E105KA12D"
 			(at 127.286 50.292 0)
 			(effects
@@
 			)
 		)
-		(property "ALTIUM_VALUE" ""
-			(at 129.54 55.88 0)
-			(effects
-				(font
-					(size 1.27 1.27)
-				)
-			)
-		)
 		(pin "1"
 		)
@@
 	)
 	(symbol
-		(lib_id "Thunderscope_Rev5:CAP 10nF 50V X7R 0402")
+		(lib_id "Thunderscope_Rev5:CAP 1uF 25V X5R 0402")
 		(at 167.64 35.56 0)
 		(unit 1)
@@
 			)
 		)
-		(property "Value" "10nF"
+		(property "Value" "1uF"
 			(at 170.18 38.1 0)
 			(effects
@@
 			)
 		)
-		(property "VOLTAGE RATING" "50V"
+		(property "VOLTAGE RATING" "25V"
 			(at 168.14 40.56 0)
 			(effects
@@
 			)
 		)
-		(property "SUPPLIER PART NUMBER 1" "81-GRM155R71H103KA8J"
+		(property "SUPPLIER PART NUMBER 1" "81-GRM155R61E105KA2D"
 			(at 165.386 29.972 0)
 			(effects
@@
 			)
 		)
-		(property "HOUSE PART NUMBER" "C-10nF-0402-002"
+		(property "HOUSE PART NUMBER" ""
 			(at 165.386 29.972 0)
 			(effects
@@
 			)
 		)
-		(property "MANUFACTURER PART NUMBER" "GRM155R71H103KA88J"
+		(property "MANUFACTURER PART NUMBER" "GRM155R61E105KA12D"
 			(at 165.386 29.972 0)
 			(effects
@@
 			)
 		)
-		(property "ALTIUM_VALUE" ""
-			(at 167.64 35.56 0)
-			(effects
-				(font
-					(size 1.27 1.27)
-				)
-			)
-		)
 		(pin "2"
 		)
@@
 	)
 	(symbol
-		(lib_id "Thunderscope_Rev5:CAP 1nF 50V C0G 0402")
+		(lib_id "Thunderscope_Rev5:CAP 1uF 25V X5R 0402")
 		(at 129.54 35.56 0)
 		(unit 1)
@@
 			)
 		)
-		(property "Value" "1nF"
+		(property "Value" "1uF"
 			(at 132.08 38.1 0)
 			(effects
@@
 			)
 		)
-		(property "VOLTAGE RATING" "50V"
+		(property "VOLTAGE RATING" "25V"
 			(at 127.286 29.972 0)
 			(effects
@@
 			)
 		)
-		(property "SUPPLIER PART NUMBER 1" "81-GRM1555C1H102FA1D"
+		(property "SUPPLIER PART NUMBER 1" "81-GRM155R61E105KA2D"
 			(at 127.286 29.972 0)
 			(effects
@@
 			)
 		)
-		(property "MANUFACTURER PART NUMBER" "GRM1555C1H102FA01D"
+		(property "MANUFACTURER PART NUMBER" "GRM155R61E105KA12D"
 			(at 127.286 29.972 0)
 			(effects
@@
 			)
 		)
-		(property "ALTIUM_VALUE" ""
-			(at 129.54 35.56 0)
-			(effects
-				(font
-					(size 1.27 1.27)
-				)
-			)
-		)
 		(pin "1"
 		)
@@
 	)
 	(symbol
-		(lib_id "Thunderscope_Rev5:CAP 10nF 50V X7R 0402")
+		(lib_id "Thunderscope_Rev5:CAP 1uF 25V X5R 0402")
 		(at 119.38 55.88 0)
 		(unit 1)
@@
 			)
 		)
-		(property "Value" "10nF"
+		(property "Value" "1uF"
 			(at 121.92 58.42 0)
 			(effects
@@
 			)
 		)
-		(property "VOLTAGE RATING" "50V"
+		(property "VOLTAGE RATING" "25V"
 			(at 117.126 50.292 0)
 			(effects
@@
 			)
 		)
-		(property "SUPPLIER PART NUMBER 1" "81-GRM155R71H103KA8J"
+		(property "SUPPLIER PART NUMBER 1" "81-GRM155R61E105KA2D"
 			(at 117.126 50.292 0)
 			(effects
@@
 			)
 		)
-		(property "HOUSE PART NUMBER" "C-10nF-0402-002"
+		(property "HOUSE PART NUMBER" ""
 			(at 117.126 50.292 0)
 			(effects
@@
 			)
 		)
-		(property "MANUFACTURER PART NUMBER" "GRM155R71H103KA88J"
+		(property "MANUFACTURER PART NUMBER" "GRM155R61E105KA12D"
 			(at 117.126 50.292 0)
 			(effects
@@
 			)
 		)
-		(property "ALTIUM_VALUE" ""
-			(at 119.38 55.88 0)
-			(effects
-				(font
-					(size 1.27 1.27)
-				)
-			)
-		)

Commit message: Misc WIP
Changed ADC decoupling, improved acq reg placement, etc.
Parts:
- removed C12, C13, C22: 1uF, Thunderscope_Rev5:GEN_C_0402, symbol Thunderscope_Rev5:CAP 1uF 25V X5R 0402
- C14, C15, C20, C21, C23, C26: value 1uF -> 10uF; footprint Thunderscope_Rev5:GEN_C_0402 -> Thunderscope_Rev5:GEN_C_0603; symbol Thunderscope_Rev5:CAP 1uF 25V X5R 0402 -> Thunderscope_Rev5:CAP 10uF 25V X5R 0603; MANUFACTURER PART NUMBER GRM155R61E105KA12D -> GRM188R61E106MA73D; SUPPLIER PART NUMBER 1 81-GRM155R61E105KA2D -> 81-GRM188R61E106MA3D
Connections:
- net +1V8A: now also C14.2, C15.2, C23.2; no longer C14.1, C15.1, C23.1
- net +1V8D: now also C20.2, C21.2; no longer C20.1, C21.1
- net +3V3_ACQ: now also C26.2; no longer C26.1
- net GND: now also C14.1, C15.1, C20.1, C21.1, C23.1, C26.1; no longer C14.2, C15.2, C20.2, C21.2, C23.2, C26.2
Other:
- moved on the sheet: C14, C15, C23, C24, FB1, FB2
