File: Hardware/KiCad/Thunderscope_Rev5/FE_Channel.kicad_sch (KiCad schematic)
At the start: 92 parts, among them J1002B1 BNC, J3B1 UFL, J4B1 UFL, K1000B1 FTR-B3SA4.5Z, K1001B1 FTR-B3SA4.5Z, Q1002B1 DMN62D0UW, Q1003B1 DMN62D0UW, Q1004B1 DMN62D0UW, U1008B1 LMH6518, U1009B1 BUF802, U1010B1 TS12A4516, U1011B1 OPA140AIDR

Commit message: Schematic Ready For Review
Parts:
- C1036B1: value 1nF -> 1uF; symbol Thunderscope_Rev5:CAP 1nF 50V C0G 0402 -> Thunderscope_Rev5:CAP 1uF 25V X5R 0402; MANUFACTURER PART NUMBER GRM1555C1H102FA01D -> GRM155R61E105KA12D; SUPPLIER PART NUMBER 1 81-GRM1555C1H102FA1D -> 81-GRM155R61E105KA2D; VOLTAGE RATING 50V -> 25V
- C1037B1: value 10nF -> 1uF; symbol Thunderscope_Rev5:CAP 10nF 50V X7R 0402 -> Thunderscope_Rev5:CAP 1uF 25V X5R 0402; HOUSE PART NUMBER C-10nF-0402-002 -> (none); MANUFACTURER PART NUMBER GRM155R71H103KA88J -> GRM155R61E105KA12D; SUPPLIER PART NUMBER 1 81-GRM155R71H103KA8J -> 81-GRM155R61E105KA2D; VOLTAGE RATING 50V -> 25V
- C1038B1: value 100nF -> 1uF; symbol Thunderscope_Rev5:CAP 100nF 16V X7R 0402 -> Thunderscope_Rev5:CAP 1uF 25V X5R 0402; HOUSE PART NUMBER C-100nF-0402-002 -> (none); MANUFACTURER PART NUMBER GCM155R71C104KA55D -> GRM155R61E105KA12D; SUPPLIER PART NUMBER 1 81-GCM155R71C104KA5D -> 81-GRM155R61E105KA2D; VOLTAGE RATING 16V -> 25V
- C1039B1, C1040B1: value 1uF -> 10uF; footprint Thunderscope_Rev5:GEN_C_0402 -> Thunderscope_Rev5:GEN_C_0603; symbol Thunderscope_Rev5:CAP 1uF 25V X5R 0402 -> Thunderscope_Rev5:CAP 10uF 10V X5R 0603; HOUSE PART NUMBER (none) -> C-10uF-0603-002; MANUFACTURER PART NUMBER GRM155R61E105KA12D -> GRM188R61A106ME69D; SUPPLIER PART NUMBER 1 81-GRM155R61E105KA2D -> 81-GRM188R61A106ME9D; VOLTAGE RATING 25V -> 10V
Connections:
- net +5V: now also C1040B1.2; no longer C1040B1.1
- net +VPGA: now also C1036B1.1, C1037B1.1, C1038B1.1, C1039B1.2; no longer C1036B1.2, C1037B1.2, C1038B1.2, C1039B1.1
- net GND: now also C1036B1.2, C1037B1.2, C1038B1.2, C1039B1.1, C1040B1.1; no longer C1036B1.1, C1037B1.1, C1038B1.1, C1039B1.2, C1040B1.2

Commit message: Rev 5 WIP
Added probe comp variants
Parts:
- removed R1023B1: 30, Thunderscope_Rev5:GEN_R_0603, symbol Thunderscope_Rev5:RES 30 OHM 1% 1/3W 0603
- added C1058A1: 12pF, Thunderscope_Rev5:GEN_C_0402, symbol Thunderscope_Rev5:CAP 12pF 50V C0G 0402
- added C1059A1: 2-6pF, EW_TRIMCAP, symbol Thunderscope_Rev5:CAP TRIMMER 2-6PF 100V
- added R1053A1: 0, Thunderscope_Rev5:GEN_R_0402, symbol Thunderscope_Rev5:RES 0 OHM 1/16W 0402
- C1022A1: renamed from C1022B1; value 8pF -> 5pF; symbol Thunderscope_Rev5:CAP 8pF 250V C0G 0603 -> Thunderscope_Rev5:CAP 5pF 250V C0G 0603; MANUFACTURER PART NUMBER CBR06C809BAGAC -> CBR06C509BAGAC; SUPPLIER PART NUMBER 1 80-CBR06C809BAGAC -> 80-CBR06C509BAGAC
- C1026A1: renamed from C1026B1; symbol Thunderscope_Rev5:CAP 10uF 10V X5R 0603 -> Thunderscope_Rev5:CAP 10uF 25V X5R 0603; HOUSE PART NUMBER C-10uF-0603-002 -> (none); MANUFACTURER PART NUMBER GRM188R61A106ME69D -> GRM188R61E106MA73D; SUPPLIER PART NUMBER 1 81-GRM188R61A106ME9D -> 81-GRM188R61E106MA3D; VOLTAGE RATING 10V -> 25V
- C1027A1: renamed from C1027B1; symbol Thunderscope_Rev5:CAP 10uF 10V X5R 0603 -> Thunderscope_Rev5:CAP 10uF 25V X5R 0603; HOUSE PART NUMBER C-10uF-0603-002 -> (none); MANUFACTURER PART NUMBER GRM188R61A106ME69D -> GRM188R61E106MA73D; SUPPLIER PART NUMBER 1 81-GRM188R61A106ME9D -> 81-GRM188R61E106MA3D; VOLTAGE RATING 10V -> 25V
- C1028A1: renamed from C1028B1; symbol Thunderscope_Rev5:CAP 10uF 10V X5R 0603 -> Thunderscope_Rev5:CAP 10uF 25V X5R 0603; HOUSE PART NUMBER C-10uF-0603-002 -> (none); MANUFACTURER PART NUMBER GRM188R61A106ME69D -> GRM188R61E106MA73D; SUPPLIER PART NUMBER 1 81-GRM188R61A106ME9D -> 81-GRM188R61E106MA3D; VOLTAGE RATING 10V -> 25V
- C1029A1: renamed from C1029B1; symbol Thunderscope_Rev5:CAP 10uF 10V X5R 0603 -> Thunderscope_Rev5:CAP 10uF 25V X5R 0603; HOUSE PART NUMBER C-10uF-0603-002 -> (none); MANUFACTURER PART NUMBER GRM188R61A106ME69D -> GRM188R61E106MA73D; SUPPLIER PART NUMBER 1 81-GRM188R61A106ME9D -> 81-GRM188R61E106MA3D; VOLTAGE RATING 10V -> 25V
- C1039A1: renamed from C1039B1; symbol Thunderscope_Rev5:CAP 10uF 10V X5R 0603 -> Thunderscope_Rev5:CAP 10uF 25V X5R 0603; HOUSE PART NUMBER C-10uF-0603-002 -> (none); MANUFACTURER PART NUMBER GRM188R61A106ME69D -> GRM188R61E106MA73D; SUPPLIER PART NUMBER 1 81-GRM188R61A106ME9D -> 81-GRM188R61E106MA3D; VOLTAGE RATING 10V -> 25V
- C1040A1: renamed from C1040B1; symbol Thunderscope_Rev5:CAP 10uF 10V X5R 0603 -> Thunderscope_Rev5:CAP 10uF 25V X5R 0603; HOUSE PART NUMBER C-10uF-0603-002 -> (none); MANUFACTURER PART NUMBER GRM188R61A106ME69D -> GRM188R61E106MA73D; SUPPLIER PART NUMBER 1 81-GRM188R61A106ME9D -> 81-GRM188R61E106MA3D; VOLTAGE RATING 10V -> 25V
- K1000A1: renamed from K1000B1; MANUFACTURER PART NUMBER FTR-B3SA4.5Z-B10 -> FTR-B3SA4.5Z; SUPPLIER 1 (none) -> Mouser; SUPPLIER PART NUMBER 1 (none) -> 817-FTR-B3SA4.5Z
- K1001A1: renamed from K1001B1; MANUFACTURER PART NUMBER FTR-B3SA4.5Z-B10 -> FTR-B3SA4.5Z; SUPPLIER 1 (none) -> Mouser; SUPPLIER PART NUMBER 1 (none) -> 817-FTR-B3SA4.5Z
- U1008A1: renamed from U1008B1; MANUFACTURER PART NUMBER LMH6518SQE/NOPB -> LMH6518SQX/NOPB
- renumbered C1021B1 to C1021A1, C1023B1 to C1023A1, C1024B1 to C1024A1, C1025B1 to C1025A1, C1030B1 to C1030A1, C1031B1 to C1031A1, C1032B1 to C1032A1, C1033B1 to C1033A1, C1034B1 to C1034A1, C1035B1 to C1035A1, C1036B1 to C1036A1, C1037B1 to C1037A1, C1038B1 to C1038A1, C1041B1 to C1041A1, C1042B1 to C1042A1, C1043B1 to C1043A1, C1044B1 to C1044A1, C1045B1 to C1045A1, C1046B1 to C1046A1, C1047B1 to C1047A1, C1048B1 to C1048A1, C1049B1 to C1049A1, C1050B1 to C1050A1, C1051B1 to C1051A1, C1052B1 to C1052A1, C1053B1 to C1053A1, C1054B1 to C1054A1, C1055B1 to C1055A1, C1056B1 to C1056A1, C1057B1 to C1057A1, D1000B1 to D1000A1, D1001B1 to D1001A1, FB1000B1 to FB1000A1, FB1001B1 to FB1001A1, J1002B1 to J1002A1, J3B1 to J3A1, J4B1 to J4A1, Q1002B1 to Q1002A1, Q1003B1 to Q1003A1, Q1004B1 to Q1004A1, R1021B1 to R1021A1, R1022B1 to R1022A1, R1024B1 to R1024A1, R1025B1 to R1025A1, R1026B1 to R1026A1, R1027B1 to R1027A1, R1028B1 to R1028A1, R1029B1 to R1029A1, R1030B1 to R1030A1, R1031B1 to R1031A1, R1032B1 to R1032A1, R1033B1 to R1033A1, R1035B1 to R1035A1, R1036B1 to R1036A1, R1037B1 to R1037A1, R1038B1 to R1038A1, R1039B1 to R1039A1, R1041B1 to R1041A1, R1042B1 to R1042A1, R1043B1 to R1043A1, R1044B1 to R1044A1, R1045B1 to R1045A1, R1046B1 to R1046A1, R1047B1 to R1047A1, R1048B1 to R1048A1, R1049B1 to R1049A1, R1050B1 to R1050A1, R1051B1 to R1051A1, R1052B1 to R1052A1, R52B1 to R52A1, R97B1 to R97A1, SHLD1000B1 to SHLD1000A1, SHLD1001B1 to SHLD1001A1, TP1014B1 to TP1014A1, TP1015B1 to TP1015A1, TP1016B1 to TP1016A1, TP1017B1 to TP1017A1, TP1018B1 to TP1018A1, U1009B1 to U1009A1, U1010B1 to U1010A1, U1011B1 to U1011A1
Connections:
- net GND: now also C1059A1.2
- net at K1000A1.4, R1021A1.1, R1025A1.2: now also C1058A1.2
- net at C1021A1.2, C1024A1.1, K1001A1.7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: now also C1059A1.1
- net at K1000A1.5, R1021A1.2: now also R1053A1.2
- net at K1000A1.7: now also C1022A1.1, R1022A1.1
- new net: C1058A1.1, R1053A1.1
Other:
- note added: "DONE: Change 8pF cap to 5pF"
- note added: "DONE: add cap + resistor across 30 Ohm resistor in 50Z path"
- note added: "TODO: Change Coupling Cap to 0805 C0G (GRM21B5C2A223JA01L)"
- note added: "TODO: Change second 12pF to something lower and add trimcap in parallel"
- moved on the sheet: C1021A1, C1022A1, C1035A1, K1000A1B, K1001A1B, R1021A1, R1022A1, R1025A1, R1026A1

Commit message: Finished all new schematic TODOs
Parts:
- C1021A1: value 12pF -> 8pF; symbol Thunderscope_Rev5:CAP 12pF 50V C0G 0402 -> Thunderscope_Rev5:CAP 8pF 50V C0G 0402; MANUFACTURER PART NUMBER CBR04C120F5GAC -> CBR04C809B5GAC; SUPPLIER PART NUMBER 1 80-CBR04C120F5G -> 80-CBR04C809B5GAC
- C1031A1: footprint Thunderscope_Rev5:GEN_C_0603 -> Thunderscope_Rev5:GEN_C_0805; symbol Thunderscope_Rev5:CAP 22nF 100V X7R 0603 -> Thunderscope_Rev5:CAP 22nF 100V C0G 0805; MANUFACTURER PART NUMBER GCM188R72A223KA37D -> GRM21B5C2A223JA01L; PACKAGE 0603 -> 0805; SUPPLIER PART NUMBER 1 81-GCM188R72A223KA7D -> 81-GRM21B5C2A223JA1L
- C1059A1: footprint EW_TRIMCAP -> Thunderscope_Rev5:EW_TRIMCAP
Other:
- note added: "DONE: Change Coupling Cap to 0805 C0G (GRM21B5C2A223JA01L)"
- note added: "DONE: Change second 12pF to something lower and add trimcap in parallel"
- note removed: "TODO: Change Coupling Cap to 0805 C0G (GRM21B5C2A223JA01L)"
- note removed: "TODO: Change second 12pF to something lower and add trimcap in parallel"
Changed lines of the file:
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@@
 		)
 	)
-	(text "TODO: Change Coupling Cap to 0805 C0G (GRM21B5C2A223JA01L)"
+	(text "DONE: Change Coupling Cap to 0805 C0G (GRM21B5C2A223JA01L)"
 		(exclude_from_sim no)
 		(at 25.4 220.98 0)
@@
 				(thickness 0.254)
 				(bold yes)
-				(color 255 0 0 1)
+				(color 0 194 194 1)
 			)
 			(justify left bottom)
@@
 		)
 	)
-	(text "TODO: Change second 12pF to something lower and add trimcap in parallel\n"
+	(text "DONE: Change second 12pF to something lower and add trimcap in parallel\n"
 		(exclude_from_sim no)
-		(at 302.26 68.58 0)
+		(at 293.37 67.31 0)
 		(effects
 			(font
@@
 				(thickness 0.254)
 				(bold yes)
-				(color 255 0 0 1)
+				(color 0 194 194 1)
 			)
 			(justify left)
@@
 			)
 		)
-		(property "Footprint" "EW_TRIMCAP"
+		(property "Footprint" "Thunderscope_Rev5:EW_TRIMCAP"
 			(at 323.088 46.99 0)
 			(effects
@@
 	)
 	(symbol
-		(lib_id "Thunderscope_Rev5:CAP 12pF 50V C0G 0402")
+		(lib_id "Thunderscope_Rev5:CAP 8pF 50V C0G 0402")
 		(at 304.8 50.8 0)
 		(unit 1)
@@
 			)
 		)
-		(property "Value" "12pF"
-			(at 311.15 53.34 90)
+		(property "Value" "8pF"
+			(at 311.15 50.8 90)
 			(effects
 				(font
 					(size 1.27 1.27)
 				)
-				(justify left bottom)
+				(justify bottom)
 			)
 		)
@@
 			)
 		)
-		(property "SUPPLIER PART NUMBER 1" "80-CBR04C120F5G"
+		(property "SUPPLIER PART NUMBER 1" "80-CBR04C809B5GAC"
 			(at 302.546 46.292 0)
 			(effects
@@
 			)
 		)
-		(property "MANUFACTURER PART NUMBER" "CBR04C120F5GAC"
+		(property "MANUFACTURER PART NUMBER" "CBR04C809B5GAC"
 			(at 302.546 45.212 0)
 			(effects
@@
 	)
 	(symbol
-		(lib_id "Thunderscope_Rev5:CAP 22nF 100V X7R 0603")
+		(lib_id "Thunderscope_Rev5:CAP 22nF 100V C0G 0805")
 		(at 68.58 182.88 0)
 		(unit 1)
@@
 			)
 		)
-		(property "Footprint" "Thunderscope_Rev5:GEN_C_0603"
+		(property "Footprint" "Thunderscope_Rev5:GEN_C_0805"
 			(at 68.58 182.88 0)
 			(effects
@@
 			)
 		)
-		(property "PACKAGE" "0603"
+		(property "PACKAGE" "0805"
 			(at 66.326 177.292 0)
 			(effects
@@
 			)
 		)
-		(property "SUPPLIER PART NUMBER 1" "81-GCM188R72A223KA7D"
+		(property "SUPPLIER PART NUMBER 1" "81-GRM21B5C2A223JA1L"
 			(at 66.326 177.292 0)
 			(effects
@@
 			)
 		)
-		(property "MANUFACTURER PART NUMBER" "GCM188R72A223KA37D"
+		(property "MANUFACTURER PART NUMBER" "GRM21B5C2A223JA01L"
 			(at 66.326 177.292 0)
 			(effects

Commit message: Placement WIP
Parts:
- removed C1051A1: 1uF, Thunderscope_Rev5:GEN_C_0402, symbol Thunderscope_Rev5:CAP 1uF 25V X5R 0402
Connections:
- net TERM_1M: now reaches K1000A1.2, R1022A1.2
- net BNC_IN: now reaches J1002A1.1 (Signal), K1000A1.3
- net TERM_50Z: now reaches C1058A1.2, K1000A1.4, R1021A1.1, R1025A1.2
- net BUF_IN_AUX: now reaches C1034A1.2, R1043A1.1, U1009A1.4 (IN_Aux)
- net OPA_OUT: now reaches C1035A1.1, R1043A1.2, U1011A1.6 (OUT)
- net DC_FB: now reaches C1035A1.2, R1041A1.2, R1042A1.2, R1044A1.1, U1011A1.2 (-)
- net SW_COM: now reaches C1031A1.2, R1047A1.1, U1010A1.1 (COM), U1011A1.3 (+)
- net PGA_BIAS: now reaches C1042A1.2, FB1001A1.2, R1045A1.2, R1046A1.2, TP1017A1.1, U1008A1.7 (IN_N)
- net BUF_OUT: now reaches R1037A1.1, R1041A1.1, U1009A1.11 (OUT)
- net BUF_OUT_R: now reaches R1037A1.2, U1008A1.6 (IN_P)
- net ATTEN_50X_R: now reaches C1021A1.2, C1024A1.1, C1059A1.1, K1001A1.7, R1024A1.2, R1026A1.2
- net TERM_50Z_R: now reaches K1000A1.5, R1021A1.2, R1053A1.2
- net BUF_R_BIAS: now reaches R1036A1.1, U1009A1.7 (R_Bias)
- net ATTEN_IN: now reaches K1000A1.6, K1001A1.3
- net TERM_1M_R: now reaches C1022A1.1, K1000A1.7, R1022A1.1
- net ATTEN_50X: now reaches C1023A1.2, K1001A1.2, R1024A1.1
- net ATTEN_OUT_R: now reaches C1030A1.2, R1035A1.2
- net DC_FB_TRIM: now reaches R1044A1.2, R1048A1.2, R1049A1.1, R1049A1.2
- net BUF_IN: now reaches C1030A1.1, R1038A1.2, U1009A1.2 (IN)
- net BUF_IN_BIAS: now reaches R1038A1.1, U1009A1.3 (IN_Bias)
- net SW_NO: now reaches C1031A1.1, R1039A1.2, U1010A1.2 (NO)
- net ATTEN_1X: now reaches K1001A1.4, K1001A1.5
Other:
- note added: "(GRM21B5C2A223JA01L)"
- note added: "DONE: Change Coupling Cap to 0805 C0G"
- note added: "DONE: change upper R to 976k"
- note removed: "DONE: Change Coupling Cap to 0805 C0G (GRM21B5C2A223JA01L)"
- note removed: "DONE: change to 976k"
- moved on the sheet: C1021A1, C1022A1, C1023A1, C1024A1, C1025A1, C1026A1, C1027A1, C1028A1, C1029A1, C1030A1, C1031A1, C1032A1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

Commit message: Got multi-channel routing working
Needed to change refdes on front end channel components
Parts:
- renumbered C1021A1 to C1021_1, C1022A1 to C1022_1, C1023A1 to C1023_1, C1024A1 to C1024_1, C1025A1 to C1025_1, C1026A1 to C1026_1, C1027A1 to C1027_1, C1028A1 to C1028_1, C1029A1 to C1029_1, C1030A1 to C1030_1, C1031A1 to C1031_1, C1032A1 to C1032_1, C1033A1 to C1033_1, C1034A1 to C1034_1, C1035A1 to C1035_1, C1036A1 to C1036_1, C1037A1 to C1037_1, C1038A1 to C1038_1, C1039A1 to C1039_1, C1040A1 to C1040_1, C1041A1 to C1041_1, C1042A1 to C1042_1, C1043A1 to C1043_1, C1044A1 to C1044_1, C1045A1 to C1045_1, C1046A1 to C1046_1, C1047A1 to C1047_1, C1048A1 to C1048_1, C1049A1 to C1049_1, C1050A1 to C1050_1, C1052A1 to C1052_1, C1053A1 to C1053_1, C1054A1 to C1054_1, C1055A1 to C1055_1, C1056A1 to C1056_1, C1057A1 to C1057_1, C1058A1 to C1058_1, C1059A1 to C1059_1, D1000A1 to D1000_1, D1001A1 to D1001_1, FB1000A1 to FB1000_1, FB1001A1 to FB1001_1, J1002A1 to J1002_1, J3A1 to J3_1, J4A1 to J4_1, K1000A1 to K1000_1, K1001A1 to K1001_1, Q1002A1 to Q1002_1, Q1003A1 to Q1003_1, Q1004A1 to Q1004_1, R1021A1 to R1021_1, R1022A1 to R1022_1, R1024A1 to R1024_1, R1025A1 to R1025_1, R1026A1 to R1026_1, R1027A1 to R1027_1, R1028A1 to R1028_1, R1029A1 to R1029_1, R1030A1 to R1030_1, R1031A1 to R1031_1, R1032A1 to R1032_1, R1033A1 to R1033_1, R1035A1 to R1035_1, R1036A1 to R1036_1, R1037A1 to R1037_1, R1038A1 to R1038_1, R1039A1 to R1039_1, R1041A1 to R1041_1, R1042A1 to R1042_1, R1043A1 to R1043_1, R1044A1 to R1044_1, R1045A1 to R1045_1, R1046A1 to R1046_1, R1047A1 to R1047_1, R1048A1 to R1048_1, R1049A1 to R1049_1, R1050A1 to R1050_1, R1051A1 to R1051_1, R1052A1 to R1052_1, R1053A1 to R1053_1, R52A1 to R52_1, R97A1 to R97_1, SHLD1000A1 to SHLD1000_1, SHLD1001A1 to SHLD1001_1, TP1014A1 to TP1014_1, TP1015A1 to TP1015_1, TP1016A1 to TP1016_1, TP1017A1 to TP1017_1, TP1018A1 to TP1018_1, U1008A1 to U1008_1, U1009A1 to U1009_1, U1010A1 to U1010_1, U1011A1 to U1011_1

Commit message: Misc WIP
Changed ADC decoupling, improved acq reg placement, etc.
Other:
- moved on the sheet: C1052_1, C1053_1, C1054_1, C1055_1, C1056_1, C1057_1

Commit message: Routing in progress, minor SCH changes
Stiffer I2C Pullups, more 100nF changed to 1uF
Parts:
- C1043_1: value 100nF -> 1uF; symbol Thunderscope_Rev5:CAP 100nF 16V X7R 0402 -> Thunderscope_Rev5:CAP 1uF 25V X5R 0402; HOUSE PART NUMBER C-100nF-0402-002 -> (none); MANUFACTURER PART NUMBER GCM155R71C104KA55D -> GRM155R61E105KA12D; SUPPLIER PART NUMBER 1 81-GCM155R71C104KA5D -> 81-GRM155R61E105KA2D; VOLTAGE RATING 16V -> 25V
Connections:
- net +3V3_PGA: now also C1043_1.1; no longer C1043_1.2
- net GND: now also C1043_1.2; no longer C1043_1.1
Other:
- moved on the sheet: C1036_1, C1037_1, C1038_1, C1039_1, C1040_1, C1043_1, FB1000_1

Commit message: Reversed Channel Order
In channel blocks, net labels, and reference designators
Parts:
- renumbered C1021_1 to C1021_4, C1022_1 to C1022_4, C1023_1 to C1023_4, C1024_1 to C1024_4, C1025_1 to C1025_4, C1026_1 to C1026_4, C1027_1 to C1027_4, C1028_1 to C1028_4, C1029_1 to C1029_4, C1030_1 to C1030_4, C1031_1 to C1031_4, C1032_1 to C1032_4, C1033_1 to C1033_4, C1034_1 to C1034_4, C1035_1 to C1035_4, C1036_1 to C1036_4, C1037_1 to C1037_4, C1038_1 to C1038_4, C1039_1 to C1039_4, C1040_1 to C1040_4, C1041_1 to C1041_4, C1042_1 to C1042_4, C1043_1 to C1043_4, C1044_1 to C1044_4, C1045_1 to C1045_4, C1046_1 to C1046_4, C1047_1 to C1047_4, C1048_1 to C1048_4, C1049_1 to C1049_4, C1050_1 to C1050_4, C1052_1 to C1052_4, C1053_1 to C1053_4, C1054_1 to C1054_4, C1055_1 to C1055_4, C1056_1 to C1056_4, C1057_1 to C1057_4, C1058_1 to C1058_4, C1059_1 to C1059_4, D1000_1 to D1000_4, D1001_1 to D1001_4, FB1000_1 to FB1000_4, FB1001_1 to FB1001_4, J1002_1 to J1002_4, J3_1 to J3_4, J4_1 to J4_4, K1000_1 to K1000_4, K1001_1 to K1001_4, Q1002_1 to Q1002_4, Q1003_1 to Q1003_4, Q1004_1 to Q1004_4, R1021_1 to R1021_4, R1022_1 to R1022_4, R1024_1 to R1024_4, R1025_1 to R1025_4, R1026_1 to R1026_4, R1027_1 to R1027_4, R1028_1 to R1028_4, R1029_1 to R1029_4, R1030_1 to R1030_4, R1031_1 to R1031_4, R1032_1 to R1032_4, R1033_1 to R1033_4, R1035_1 to R1035_4, R1036_1 to R1036_4, R1037_1 to R1037_4, R1038_1 to R1038_4, R1039_1 to R1039_4, R1041_1 to R1041_4, R1042_1 to R1042_4, R1043_1 to R1043_4, R1044_1 to R1044_4, R1045_1 to R1045_4, R1046_1 to R1046_4, R1047_1 to R1047_4, R1048_1 to R1048_4, R1049_1 to R1049_4, R1050_1 to R1050_4, R1051_1 to R1051_4, R1052_1 to R1052_4, R1053_1 to R1053_4, R52_1 to R52_4, R97_1 to R97_4, SHLD1000_1 to SHLD1000_4, SHLD1001_1 to SHLD1001_4, TP1014_1 to TP1014_4, TP1015_1 to TP1015_4, TP1016_1 to TP1016_4, TP1017_1 to TP1017_4, TP1018_1 to TP1018_4, U1008_1 to U1008_4, U1009_1 to U1009_4, U1010_1 to U1010_4, U1011_1 to U1011_4
