File: Hardware/KiCad/Thunderscope_Rev5/FPGA_Bank_IO.kicad_sch (KiCad schematic)
At the start: 10 parts, among them U18 IC FPGA XC7A50T-2CSG325C

Commit message: Routed ADC and Clock Gen
Connections:
- net DC_CPL_2: now also U18.N18 (IO_L10P_T1_D14_14); no longer U18.R17 (IO_L14N_T2_SRCC_14)
- net LED_R: now also U18.R16 (IO_L14P_T2_SRCC_14); no longer U18.K17 (IO_L4P_T0_D04_14)
- net PGA_CSn_2: now also U18.R17 (IO_L14N_T2_SRCC_14); no longer U18.R16 (IO_L14P_T2_SRCC_14)
- net TERM_2: now also U18.K17 (IO_L4P_T0_D04_14); no longer U18.N18 (IO_L10P_T1_D14_14)
Other:
- note added: "D2B Inversion!"
- note added: "FCLK Inversion!"
- note removed: "D1B Inversion!"
Changed lines of the file:
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@@
 		(comment 1 "Aleksa Bjelogrlic")
 	)
+	(text "FCLK Inversion!"
+		(exclude_from_sim no)
+		(at 205.74 71.12 0)
+		(effects
+			(font
+				(size 1.27 1.27)
+			)
+			(justify left)
+		)
+	)
 	(text "FPGA IO Banks"
 		(exclude_from_sim no)
@@
 		)
 	)
-	(text "D1B Inversion!"
+	(text "D2B Inversion!"
 		(exclude_from_sim no)
-		(at 205.74 41.91 0)
+		(at 205.74 55.88 0)
 		(effects
 			(font
@@
 	(wire
 		(pts
-			(xy 66.04 86.36) (xy 81.28 86.36)
-		)
-		(stroke
-			(width 0)
-			(type default)
-		)
-	)
-	(wire
-		(pts
 			(xy 66.04 147.32) (xy 83.82 147.32)
 		)
@@
 	(wire
 		(pts
+			(xy 66.04 106.68) (xy 83.82 106.68)
+		)
+		(stroke
+			(width 0)
+			(type default)
+		)
+	)
+	(wire
+		(pts
 			(xy 129.54 180.34) (xy 132.08 180.34)
 		)
@@
 	(wire
 		(pts
+			(xy 66.04 55.88) (xy 81.28 55.88)
+		)
+		(stroke
+			(width 0)
+			(type default)
+		)
+	)
+	(wire
+		(pts
 			(xy 99.06 127) (xy 109.22 127)
 		)
@@
 	(wire
 		(pts
-			(xy 66.04 106.68) (xy 81.28 106.68)
+			(xy 66.04 109.22) (xy 81.28 109.22)
 		)
 		(stroke
@@
 	(wire
 		(pts
-			(xy 66.04 55.88) (xy 83.82 55.88)
-		)
-		(stroke
-			(width 0)
-			(type default)
-		)
-	)
-	(wire
-		(pts
 			(xy 180.34 43.18) (xy 182.88 43.18)
 		)
@@
 		)
 	)
-	(wire
-		(pts
-			(xy 66.04 109.22) (xy 81.28 109.22)
-		)
-		(stroke
-			(width 0)
-			(type default)
-		)
-	)
 	(bus
 		(pts
@@
 	(wire
 		(pts
+			(xy 66.04 86.36) (xy 81.28 86.36)
+		)
+		(stroke
+			(width 0)
+			(type default)
+		)
+	)
+	(wire
+		(pts
 			(xy 88.9 185.42) (xy 91.44 185.42)
 		)
@@
 			"AEEAQQBDAEoAMQBBAEEAQQBBAEEAQQBBAEEATgBTAEoAQQBBAEQAZAAvAHcAQQBBAEIAMABFAEEA"
 			"QQBEAFEASABBAEEARABPAHMAdwBBAEEAeAB0AGMAQQBBAEIAVgBSAEEAQQBBAEEAQQBBAEEAQQBp"
-			"AFMAOABBAEEAUAAvAC8AQQBBAEEAQQBYAFEAQQBBAFgAUQBBAEEAQQBQAC8ALw=="
+			"AFMAOABBAEEAUAAvAC8AQQBBAEEAQQBYAFEAQQBBAFgAUQBBAEEAQQBQAC8ALwAvAC8AOABBAEEA"
+			"QQBCAGQAQQBBAEIAZABBAEEAQQBBAC8ALwA4AEEAQQBJAG4AVQBBAEEAQQBBAEEAQQBBAEEAQgB3"
+			"AEEAQQBBAEgAOQBMAEEAQQBEAEYAcQB3AEEAQQBuAGUASQBBAEEAQQBBAEgAQQBBAEMAZQBVAFEA"
+			"QQBBADQAZQBFAEEAQQBMAHoAWABBAEEAQQBIAE4AQQBBAEEAVQBRAGMAQQBBAFAALwB1AEEAQQBE"
+			"AGgANgBnAEEAQQBBAEYAUQBBAEEARgBRAEEAQQBBAEQAawA0AFEAQQBBADEAUABnAEEAQQBBAEEA"
+			"dgBBAEEAQwBKAEwAdwBBAEEALwAvADgAQQBBAEcAMgA5AEEAQQBBAEEAQQBBAEEAQQBsAFYARQBB"
+			"AEEATwBIAFgAQQBBAEMASgB2AEEAQQBBAEEAQgBVAEEAQQBHADAAVgBBAEEARAAvACsAQQBBAEEA"
+			"aQBkAFEAQQBBAEEAQQBBAEEAQQBBAFYAQQBBAEEAQQB4AHAAVQBBAEEATQA3AGgAQQBBAEEAVgBV"
+			"AFEAQQBBAEUAUQBBAEEAQQBQACsAOQBBAEEARAAvAC8AdwBBAEEALwAvADgAQQBBAFAALwAvAEEA"
+			"QQBEAC8ALwB3AEEAQQAvAC8AOABBAEEAUAAvAC8AQQBBAEQALwAvAHcAQQBBAC8ALwA4AEEAQQBQ"
+			"AC8ALwBBAFAALwAvAC8ALwAvAC8ALwAvAC8ALwAvAC8ALwAvAC8ALwAvAC8ALwAvAC8ALwAvAC8A"
+			"LwAvAC8ALwAvAC8ALwAvAC8ALwAvAC8ALwAvAC8ALwAvAC8ALwAvAC8ALwAvAC8ALwAvAC8ALwAv"
+			"AC8ALwAvAC8ALwAvAC8ALwAvAC8ALwAvAC8ALwAvAC8ALwAvAC8ALwAvAC8ALwAvAC8ALwAvAC8A"
+			"LwAvAC8ALwAvAC8ALwAvAC8ALwAvAC8ALwAvAC8ALwAvAC8ALwAvAC8ALwAvAC8ALwAvAC8ALwAv"
+			"AC8ALwAvAC8ALwAvAC8ALwAvAC8ALwAvAC8ALwAvAC8ALwAvAC8ALwAvAC8ALwAvAC8ALwAvAC8A"
+			"LwAvAC8ALwAvAC8ALwAvAC8ALwAvAC8ALwAvAC8ALwAvAC8ALwAvAC8ALwAvAC8ALwAvAC8ALwAv"
+			"AC8ALwAvAC8ALwAvAC8ALwAvAC8ALwAvAC8ALwAvAC8ALwAvAC8ALwAvAC8ALwAvAC8ALwAvAC8A"
+			"LwAvAC8ALwAvAC8ALwAvAC8ALwAvAC8ALwAvAC8ALwAvAC8ALwAvAC8ALwAvAC8ALwAvAC8ALwAv"
+			"AC8ALwAvAC8ALwAvAC8ALwAvAC8ALwAvAC8ALwAvAC8ALwAvAC8ALwAvAC8ALw=="
 		)
 	)
@@
 		)
 	)
-	(label "LED_R"
-		(at 81.28 55.88 180)
-		(effects
-			(font
-				(size 1.27 1.27)
-			)
-			(justify right bottom)
-		)
-	)
 	(label "ACQ_EN"
 		(at 81.28 152.4 180)
@@
 		)
 	)
+	(label "TERM_2"
+		(at 81.28 55.88 180)
+		(effects
+			(font
+				(size 1.27 1.27)
+			)
+			(justify right bottom)
+		)
+	)
 	(label "TERM_[4..1]"
 		(at 96.52 93.98 0)
@@
 	)
 	(label "PGA_CSn_2"
-		(at 81.28 106.68 180)
+		(at 81.28 109.22 180)
 		(effects
 			(font
@@
 		)
 	)
+	(label "DC_CPL_2"
+		(at 81.28 86.36 180)
+		(effects
+			(font
+				(size 1.27 1.27)
+			)
+			(justify right bottom)
+		)
+	)
 	(label "TRIM_SCL"
 		(at 81.28 76.2 180)
@@
 		)
 	)
+	(label "LED_R"
+		(at 81.28 106.68 180)
+		(effects
+			(font
+				(size 1.27 1.27)
+			)
+			(justify right bottom)
+		)
+	)
 	(label "PGA_CSn_[4..1]"
 		(at 96.52 96.52 0)
@@
 		)
 	)
-	(label "DC_CPL_2"
-		(at 81.28 109.22 180)
-		(effects
-			(font
-				(size 1.27 1.27)
-			)
-			(justify right bottom)
-		)
-	)
 	(label "D4A_N"
 		(at 198.12 93.98 180)
@@
 		)
 	)
-	(label "TERM_2"
-		(at 81.28 86.36 180)
-		(effects
-			(font
-				(size 1.27 1.27)
-			)
-			(justify right bottom)
-		)
-	)
 	(label "QSPI_DQ3"
 		(at 81.28 48.26 180)
@@
 		)
 	)
+	(hierarchical_label "LED_R"
+		(shape output)
+		(at 83.82 106.68 0)
+		(effects
+			(font
+				(size 1.27 1.27)
+			)
+			(justify left)
+		)
+	)
 	(hierarchical_label "PERST#"
 		(shape input)
@@
 		(effects
 			(font
-				(size 1.27 1.27)
-			)
-			(justify left)
-		)
-	)
-	(hierarchical_label "LED_R"
-		(shape output)
-		(at 83.82 55.88 0)
-		(effects
-			(font

Commit message: Final signal routing WIP
Connections:
- net ACQ_EN: now also U18.T17 (IO_L16P_T2_CSI_B_14); no longer U18.U11 (IO_L23P_T3_A03_D19_14)
- net ADC_CSn: now also U18.U17 (IO_L16N_T2_A15_D31_14); no longer U18.U14 (IO_L20P_T3_A08_D24_14)
- net ADC_SCLK: now also U18.U16 (IO_L17N_T2_A13_D29_14); no longer U18.V14 (IO_L20N_T3_A07_D23_14)
- net ADC_SDIO: now also U18.R16 (IO_L14P_T2_SRCC_14); no longer U18.V12 (IO_L21P_T3_DQS_14)
- net ATTEN_1: now also U18.V11 (IO_L23N_T3_A02_D18_14); no longer U18.P14 (IO_L12P_T1_MRCC_14)
- net ATTEN_3: now also U18.R15 (IO_L12N_T1_MRCC_14); no longer U18.U16 (IO_L17N_T2_A13_D29_14)
- net DC_CPL_1: now also U18.V12 (IO_L21P_T3_DQS_14); no longer U18.R15 (IO_L12N_T1_MRCC_14)
- net DC_CPL_3: now also U18.U14 (IO_L20P_T3_A08_D24_14); no longer U18.U17 (IO_L16N_T2_A15_D31_14)
- net DC_CPL_4: now also U18.P14 (IO_L12P_T1_MRCC_14); no longer U18.V11 (IO_L23N_T3_A02_D18_14)
- net FE_EN: now also U18.U15 (IO_L17P_T2_A14_D30_14); no longer U18.N16 (IO_L9P_T1_DQS_14)
- net LED_R: now also U18.N14 (IO_L8N_T1_D12_14); no longer U18.R16 (IO_L14P_T2_SRCC_14)
- net PGA_CSn_1: now also U18.U11 (IO_L23P_T3_A03_D19_14); no longer U18.P16 (IO_L11N_T1_SRCC_14)
- net PGA_CSn_3: now also U18.P16 (IO_L11N_T1_SRCC_14); no longer U18.T17 (IO_L16P_T2_CSI_B_14)
- net PLL_SCL: now also U18.T14 (IO_L13P_T2_MRCC_14); no longer U18.V13 (IO_L21N_T3_DQS_A06_D22_14)
- net TERM_1: now also U18.V13 (IO_L21N_T3_DQS_A06_D22_14); no longer U18.T14 (IO_L13P_T2_MRCC_14)
- net TERM_3: now also U18.N16 (IO_L9P_T1_DQS_14); no longer U18.U15 (IO_L17P_T2_A14_D30_14)
- net TRIM_SDA: now also U18.V14 (IO_L20N_T3_A07_D23_14); no longer U18.N14 (IO_L8N_T1_D12_14)

Commit message: Finished all signal routing
PWR, GND and Length Tuning remains
Connections:
- net ATTEN_3: now also U18.M16 (IO_L7P_T1_D09_14); no longer U18.R15 (IO_L12N_T1_MRCC_14)
- net ATTEN_4: now also U18.N17 (IO_L9N_T1_DQS_D13_14); no longer U18.T13 (IO_L19N_T3_A09_D25_VREF_14)
- net DC_CPL_3: now also U18.M15 (IO_L6N_T0_D08_VREF_14); no longer U18.U14 (IO_L20P_T3_A08_D24_14)
- net DC_CPL_4: now also U18.N16 (IO_L9P_T1_DQS_14); no longer U18.P14 (IO_L12P_T1_MRCC_14)
- net LED_B: now also U18.U14 (IO_L20P_T3_A08_D24_14); no longer U18.P15 (IO_L11P_T1_SRCC_14)
- net LED_G: now also U18.R13 (IO_L19P_T3_A10_D26_14); no longer U18.M17 (IO_L7N_T1_D10_14)
- net LED_R: now also U18.T14 (IO_L13P_T2_MRCC_14); no longer U18.N14 (IO_L8N_T1_D12_14)
- net OSC_OE: now also U18.P14 (IO_L12P_T1_MRCC_14); no longer U18.U12 (IO_L22N_T3_A04_D20_14)
- net PGA_CSn_3: now also U18.M17 (IO_L7N_T1_D10_14); no longer U18.P16 (IO_L11N_T1_SRCC_14)
- net PGA_CSn_4: now also U18.P16 (IO_L11N_T1_SRCC_14); no longer U18.N17 (IO_L9N_T1_DQS_D13_14)
- net PGA_SCLK: now also U18.R15 (IO_L12N_T1_MRCC_14); no longer U18.M16 (IO_L7P_T1_D09_14)
- net PGA_SDIO: now also U18.N14 (IO_L8N_T1_D12_14); no longer U18.K15 (IO_L5N_T0_D07_14)
- net PLL_SCL: now also U18.U12 (IO_L22N_T3_A04_D20_14); no longer U18.T14 (IO_L13P_T2_MRCC_14)
- net PROBE_COMP: now also U18.P15 (IO_L11P_T1_SRCC_14); no longer U18.M15 (IO_L6N_T0_D08_VREF_14)
- net TERM_3: now also U18.K15 (IO_L5N_T0_D07_14); no longer U18.N16 (IO_L9P_T1_DQS_14)
- net TERM_4: now also U18.M14 (IO_L8P_T1_D11_14); no longer U18.R13 (IO_L19P_T3_A10_D26_14)
- net TRIM_SCL: now also U18.T13 (IO_L19N_T3_A09_D25_VREF_14); no longer U18.M14 (IO_L8P_T1_D11_14)

Commit message: Increased trace spacing where possible
Connections:
- net PGA_SCLK: now also U18.P15 (IO_L11P_T1_SRCC_14); no longer U18.R15 (IO_L12N_T1_MRCC_14)
- net PROBE_COMP: now also U18.R15 (IO_L12N_T1_MRCC_14); no longer U18.P15 (IO_L11P_T1_SRCC_14)
Changed lines of the file:
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@@
 	(wire
 		(pts
+			(xy 66.04 91.44) (xy 83.82 91.44)
+		)
+		(stroke
+			(width 0)
+			(type default)
+		)
+	)
+	(wire
+		(pts
 			(xy 104.14 124.46) (xy 104.14 129.54)
 		)
@@
 	(wire
 		(pts
-			(xy 66.04 91.44) (xy 83.82 91.44)
-		)
-		(stroke
-			(width 0)
-			(type default)
-		)
-	)
-	(wire
-		(pts
 			(xy 66.04 144.78) (xy 81.28 144.78)
 		)
@@
 	(wire
 		(pts
+			(xy 66.04 99.06) (xy 83.82 99.06)
+		)
+		(stroke
+			(width 0)
+			(type default)
+		)
+	)
+	(wire
+		(pts
 			(xy 66.04 73.66) (xy 81.28 73.66)
 		)
@@
 		)
 	)
-	(wire
-		(pts
-			(xy 66.04 99.06) (xy 83.82 99.06)
-		)
-		(stroke
-			(width 0)
-			(type default)
-		)
-	)
 	(image
 		(at 107.95 38.6657)
@@
 			"AC8ALwAvAC8ALwAvAC8ALwAvAC8ALwAvAC8ALwAvAC8ALwAvAC8ALwAvAC8ALwAvAC8ALwAvAC8A"
 			"LwAvAC8ALwAvAC8ALwAvAC8ALwAvAC8ALwAvAC8ALwAvAC8ALwAvAC8ALwAvAC8ALwAvAC8ALwAv"
-			"AC8ALwAvAC8ALwAvAC8ALwAvAC8ALwAvAC8ALwAvAC8ALwAvAC8ALwAvAC8ALw=="
+			"AC8ALwAvAC8ALwAvAC8ALwAvAC8ALwAvAC8ALwAvAC8ALwAvAC8ALwAvAC8ALwAvAC8ALwArAE4A"
+			"SAAvACsAUAAvAC8ALwAwAEcAVQAyAGYAKwBKAE4AQQB2AC8ALwAvAGoAUgAvAC8ALwAvAC8ALwA5"
+			"AGQAcwBQAGoALwBBAEEAQQBIAC8ANQA1AFIARgBmAC8AaAA0AGMANwAvAFkANgBuAE8ALwB3AHMA"
+			"UABNAC8AOABBAEEAQQBEAC8ALwA3AEIAZAAvAC8ALwAvAC8ALwAvAE0ALwAvAC8ALwBBAEMATgAv"
+			"AC8AMgBvAHYAQQBQACsAcgBxADUALwAvAHEANgB1AHIALwA2AHUAcgBxAC8ALwBYAHgAcgBUAC8A"
+			"LwAvAFQAcQAvAC8ALwAvAC8ALwA5AGQAcwBQAC8ALwBBAEEAQQBBAC8ALwArAHcAWABmAC8ALwAv"
+			"AC8ALwAvAC8ALwAvAC8ALwA0AG4AVQAvAC8AOABBAEEAQwAvAC8AMQBJAGsAdgAvAC8ALwAvAC8A"
+			"LwAvAC8ALwAvAC8ALwAvAC8ALwAvAC8ALwAvAC8ALwAvAC8AaQAvAC8ALwAvAEEARQBHAFkALwB6"
+			"AFEASABBAFAALwAwAHoAWQBYAC8AbgB0AGYAMAAvAHgAcwB6AFgAUAA4AEEAQQBCAEgALwAxAEkA"
+			"awB2AC8ALwAvAC8ALwAvACsASgAxAFAALwAvAEEAQQBBAHYALwA5AFMASgBMAC8ALwAvAC8ALwAv"
+			"AC8ALwAvAC8ALwAvADcARAAvAC8ALwA4AEEAQQBGADMALwBzAEYAMABBAC8ALwAvAC8ALwAvAC8A"
+			"LwAvAC8ALwAvAC8ALwAvAC8ALwAvAC8ALwAvAC8ALwAvAC8ALwAvAC8ALwAvAC8ALwAvAHcAQgBk"
+			"AHMAUAA5AGQAQQBBAEQALwAvAC8AKwB3AC8ALwAvAC8ALwAvADkAZABzAFAALwAvAEEAQQBBAEEA"
+			"LwAvACsAdwBYAGYALwAvAC8ALwAvAC8ALwAvAC8ALwAvADQAbgBVAC8ALwA4AEEAQQBDAC8ALwAx"
+			"AEkAawB2AC8ALwAvAC8ALwAvACsAdwAvAC8ALwAvAEEAQQBCAGQALwB6AG8ATABBAFAALwBmAHYA"
+			"SAAvAC8AKwBQAC8AMAAvADMAcgBBADQALwA5AHkATQB6AC8ALwAvACsAaQA2AC8ALwAvAC8ALwAv"
+			"AC8ALwAvAC8ALwAvAFgAYgBEADQALwB3AEEAQQBCAC8AKwBlAFUAUgBYAC8ANABlAEgATwAvADIA"
+			"TwBwAHoAdgA4AEwARAB6AFAALwBBAEEAQQBBAC8ALwArAHcAWABmAC8ALwAvAC8ALwAvAHQAZgAv"
+			"AC8ALwB3AEEASABZAC8AKwBBAEwAdwBEAC8AeAB0AGYARgAvACsAUABJAHUAUA=="
 		)
 	)
@@
 		)
 	)
+	(label "PGA_SCLK"
+		(at 81.28 91.44 180)
+		(effects
+			(font
+				(size 1.27 1.27)
+			)
+			(justify right bottom)
+		)
+	)
 	(label "CLK25"
 		(at 81.28 104.14 180)
@@
 		)
 	)
-	(label "PGA_SDIO"
-		(at 81.28 78.74 180)
-		(effects
-			(font
-				(size 1.27 1.27)
-			)
-			(justify right bottom)
-		)
-	)
 	(label "FE_PG"
 		(at 81.28 127 180)
@@
 		)
 	)
+	(label "PROBE_COMP"
+		(at 81.28 99.06 180)
+		(effects
+			(font
+				(size 1.27 1.27)
+			)
+			(justify right bottom)
+		)
+	)
 	(label "PERST#"
 		(at 81.28 157.48 180)
@@
 		)
 	)
-	(label "PROBE_COMP"
-		(at 81.28 91.44 180)
-		(effects
-			(font
-				(size 1.27 1.27)
-			)
-			(justify right bottom)
-		)
-	)
 	(label "HWID0"
 		(at 81.28 114.3 180)
@@
 		)
 	)
-	(label "PGA_SCLK"
-		(at 81.28 99.06 180)
+	(label "PGA_SDIO"
+		(at 81.28 78.74 180)
 		(effects
 			(font
@@
 		)
 	)
-	(hierarchical_label "PROBE_COMP"
+	(hierarchical_label "TRIM_SCL"
 		(shape output)
-		(at 83.82 91.44 0)
+		(at 83.82 134.62 0)
 		(effects
 			(font
@@
 		)
 	)
-	(hierarchical_label "TRIM_SCL"
+	(hierarchical_label "PROBE_COMP"
 		(shape output)
-		(at 83.82 134.62 0)
+		(at 83.82 99.06 0)
 		(effects
 			(font
@@
 		)
 	)
-	(hierarchical_label "PGA_SCLK"
-		(shape output)
-		(at 83.82 99.06 0)
-		(effects
-			(font
-				(size 1.27 1.27)
-			)
-			(justify left)
-		)
-	)
 	(hierarchical_label "SYNC_IN_P"
 		(shape input)
@@
 		)
 	)
-	(hierarchical_label "OSC_OE"
+	(hierarchical_label "PGA_SCLK"
 		(shape output)
-		(at 83.82 96.52 0)
+		(at 83.82 91.44 0)
 		(effects
 			(font
@@
 		)
 	)
-	(hierarchical_label "PGA_SDIO"
+	(hierarchical_label "OSC_OE"
 		(shape output)
-		(at 83.82 78.74 0)
+		(at 83.82 96.52 0)
 		(effects
 			(font
@@
 		(effects
 			(font
+				(size 1.27 1.27)
+			)
+			(justify left)
+		)
+	)
+	(hierarchical_label "PGA_SDIO"
+		(shape output)
+		(at 83.82 78.74 0)
+		(effects
+			(font

Commit message: Reversed Channel Order
In channel blocks, net labels, and reference designators
Connections:
- net ATTEN_1: now also U18.N17 (IO_L9N_T1_DQS_D13_14); no longer U18.V11 (IO_L23N_T3_A02_D18_14)
- net ATTEN_2: now also U18.M16 (IO_L7P_T1_D09_14); no longer U18.L18 (IO_L4N_T0_D05_14)
- net ATTEN_3: now also U18.L18 (IO_L4N_T0_D05_14); no longer U18.M16 (IO_L7P_T1_D09_14)
- net ATTEN_4: now also U18.V11 (IO_L23N_T3_A02_D18_14); no longer U18.N17 (IO_L9N_T1_DQS_D13_14)
- net DC_CPL_1: now also U18.N16 (IO_L9P_T1_DQS_14); no longer U18.V12 (IO_L21P_T3_DQS_14)
- net DC_CPL_2: now also U18.M15 (IO_L6N_T0_D08_VREF_14); no longer U18.N18 (IO_L10P_T1_D14_14)
- net DC_CPL_3: now also U18.N18 (IO_L10P_T1_D14_14); no longer U18.M15 (IO_L6N_T0_D08_VREF_14)
- net DC_CPL_4: now also U18.V12 (IO_L21P_T3_DQS_14); no longer U18.N16 (IO_L9P_T1_DQS_14)
- net PGA_CSn_1: now also U18.P16 (IO_L11N_T1_SRCC_14); no longer U18.U11 (IO_L23P_T3_A03_D19_14)
- net PGA_CSn_2: now also U18.M17 (IO_L7N_T1_D10_14); no longer U18.R17 (IO_L14N_T2_SRCC_14)
- net PGA_CSn_3: now also U18.R17 (IO_L14N_T2_SRCC_14); no longer U18.M17 (IO_L7N_T1_D10_14)
- net PGA_CSn_4: now also U18.U11 (IO_L23P_T3_A03_D19_14); no longer U18.P16 (IO_L11N_T1_SRCC_14)
- net TERM_1: now also U18.M14 (IO_L8P_T1_D11_14); no longer U18.V13 (IO_L21N_T3_DQS_A06_D22_14)
- net TERM_2: now also U18.K15 (IO_L5N_T0_D07_14); no longer U18.K17 (IO_L4P_T0_D04_14)
- net TERM_3: now also U18.K17 (IO_L4P_T0_D04_14); no longer U18.K15 (IO_L5N_T0_D07_14)
- net TERM_4: now also U18.V13 (IO_L21N_T3_DQS_A06_D22_14); no longer U18.M14 (IO_L8P_T1_D11_14)
Changed lines of the file:
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@@
 			"AC8ALwAvAC8ALwAvAFgAYgBEADQALwB3AEEAQQBCAC8AKwBlAFUAUgBYAC8ANABlAEgATwAvADIA"
 			"TwBwAHoAdgA4AEwARAB6AFAALwBBAEEAQQBBAC8ALwArAHcAWABmAC8ALwAvAC8ALwAvAHQAZgAv"
-			"AC8ALwB3AEEASABZAC8AKwBBAEwAdwBEAC8AeAB0AGYARgAvACsAUABJAHUAUA=="
+			"AC8ALwB3AEEASABZAC8AKwBBAEwAdwBEAC8AeAB0AGYARgAvACsAUABJAHUAUAAvAC8ALwAvAC8A"
+			"LwAvAC8ALwAvAC8ALwAvAC8ALwAvAC8ALwAvAC8ALwAvAC8ALwAvAC8ALwAvAC8ALwAvAC8ALwAv"
+			"AC8ALwAvAC8ALwAvAC8ALwAvAC8ALwAvAC8ALwAvAC8ALwAvAC8ALwAvAC8ALwAvAC8ALwAvAC8A"
+			"LwAvAC8ALwAvAC8ALwAvAC8ALwAvAC8ALwAvAC8ALwAvAC8ALwAvAC8ALwAvAC8ALwAvAC8ALwAv"
+			"AC8ALwAvAC8ALwAvAC8ALwAvAC8ALwAvAC8ALwAvAC8ALwAvAC8ALwAvAC8ALwAvAC8ALwAvAC8A"
+			"LwAvAC8ALwAvAC8ALwAvAC8ALwAvAC8ALwAvAC8ALwAvAC8ALwAvAC8ALwAvAC8ALwAvAC8ALwAv"
+			"AC8ALwAvAC8ALwAvAC8ALwAvAC8ALwAvAC8ALwAvAC8ALwAvAC8ALwAvAC8ALwAvAC8ALwAvAC8A"
+			"LwAvAC8ALwAvAC8ALwAvAC8ALwAvAC8ALwAvAC8ALwAvAC8ALwAvAC8ALwAvAC8ALwAvAC8ALwAv"
+			"AC8ALwAvAC8ALwAvAC8ALwAvAC8ALwAvAC8ALwAvAC8ALwAvAC8ALwAvAC8ALwAvAC8ALwAvAC8A"
+			"LwAvAC8ALwAvAC8ALwAvAC8ALwAvAC8ALwAvAC8ALwAvAC8ALwAvAC8ALwAvAC8ALwAvAC8ALwAv"
+			"AC8ALwAvAC8ALwAvAC8ALwAvAC8ALwAvAC8ALwAvAC8ALwAvAC8ALwAvAC8ALwAvAC8ALwAvAC8A"
+			"LwAvAC8ALwAvAC8ALwAvAC8ALwAvAC8ALwAvAC8ALwAvAC8ALwAvAC8ALwAvAC8ALwAvAC8ALwAv"
+			"AC8ALwAvAC8ALwAvAC8ALwAvAC8ALwAvAC8ALwAvAC8ALwAvAC8ALwAvAC8ALwAvAC8ALwAvAC8A"
+			"LwAvAC8ALwAvAC8ALwAvAC8ALwAvAC8ALwAvAC8ALwAvAC8ALwAvAC8ALwAvAC8ALwAvAC8ALwAv"
+			"AC8ALwAvAC8ALwAvAC8ALwAvAC8ALwAvAC8ALwAvAC8ALwAvAC8ALwAvAC8ALwAvAC8ALwAvAC8A"
+			"LwAvAC8ALwAvAC8ALwAvAC8ALwAvAC8ALwAvAC8ALwAvAC8ALwAvAC8ALwAvAC8ALwAvAC8ALwAv"
+			"AC8ALwAvAC8ALwAvAC8ALwAvAC8ALwAvAC8ALwAvAC8ALwAvAC8ALwAvAC8ALwAvAC8ALwAvAC8A"
+			"LwAvAC8ALwAvAC8ALwAvAC8ALwAvAC8ALwAvAC8ALwAvAC8ALwAvAC8ALwAvAC8ALwAvAC8ALwAv"
+			"AC8ALwAvAC8ALwAvAC8ALwAvAC8ALwAvAC8ALwAvAC8ALwAvAC8ALwAvAC8ALwAAAAAAAAAAAAAA"
+			"AAAAAAAAAAAAAAAAAAAAAAAAAAAAAAAAAAAAAAAAAAAAAAAAAAAAAAAAAAAAAAAAAAAAAAAAAAAA"
+			"AAAAAAAAAAAAAAAAAAAAAAAAAAAAAAAAAAAAAAAAAAAAAAAAAAAAAAAAAAAAAAAAAAAAAAAAAAAA"
+			"AAAAAAAAAAAAAAAAAAAAAAAAAAAAAAAAAAAAAAAAAAAAAAAAAAAAAAAAAAAAAAAAAAAAAAAAAAAA"
+			"AAAAAAAAAAAAAAAAAAAAAAAAAAAAAAAAAAAAAAAAAAAAAAAAAAAAAAAAAAAAAAAAAAAAAAAAAAAA"
+			"AAAAAAAAAAAAAAAAAAAAAAAAAAAAAAAAAAAAAAAAAAAAAAAAAAAAAAAAAAAAAAAAAAAAAAAAAAAA"
+			"AAAAAAAAAAAAAAAAAAAAAAAAAAAAAAAAAAAAAAAAAAAAAAAAAAAAAAAAAAAAAAAAAAAAAAAAAAAA"
+			"AAAAAAAAAAAAAAAAAAAAAAAAAAAAAAAAAAAAAAAAAAAAAAAAAAAAAAAAAAAAAAAAAAAAAAAAAAAA"
+			"AAAAAAAAAAAAAAAAAAAAAAAAAAAAAAAAAAAAAAAAAAAAAAAAAAAAAAAAAAAAAAAAAAAAAAAAAAAA"
+			"AAAAAAAAAAAAAAAAAAAAAAAAAAAAAAAAAAAAAAAAAAAAAAAAAAAAAAAAAAAAAAAAAAAAAAAAAAAA"
+			"AAAAAAAAAAAAAAAAAAAAAAAAAAAAAAAAAAAAAAAAAAAAAAAAAAAAAAAAAAAAAAAAAAAAAAAAAAAA"
+			"AAAAAAAAAAAAAAAAAAAAAAAAAAAAAAAAAAAAAAAAAAAAAAAAAAAAAAAAAAAAAAAAAAAAAAAAAAAA"
+			"AAAAAAAAAAAAAAAAAAAAAAAAAAAAAAAAAAAAAAAAAAAAAAAAAAAAAAAAAAAAAAAAAAAAAAAAAAAA"
+			"AAAAAAAAAAAAAAAAAAAAAAAAAAAAAAAAAAAAAAAAAAAAAAAAAAAAAAAAAAAAAAAAAAAAAAAAAAAA"
+			"AAAAAAAAAAAAAAAAAAAAAAAAAAAAAAAAAAAAAAAAAAAAAAAAAAAAAAAAAAAAAAAAAAAAAAAAAAAA"
+			"AAAAAAAAAAAAAAAAAAAAAAAAAAAAAAAAAAAAAAAAAAAAAAAAAAAAAAAAAAAAAAAAAAAAAAAAAAAA"
+			"AAAAAAAAAAAAAAAAAAAAAAAAAAAAAAAAAAAAAAAAAAAAAAAAAAAAAAAAAAAAAAAAAAAAAAAAAAAA"
+			"AAAAAAAAAAAAAAAAAAAAAAAAAAAAAAAAAAAAAAAAAAAAAAAAAAAAAAAAAAAAAAAAAAAAAAAAAAAA"
+			"AAAAAAAAAAAAAAAAAAAAAAAAAAAAAAAAAAAAAAAAAAAAAAAAAAAAAAAAAAAAAACNAACNDH15AGA9"
+			"gtafAQAAcGFJ/J4BAAAAAAAAAAAAAAAAAAAAAAAAAAAAAAAAAAAAAAAAAAAAAAAAAAAAAAAAAAAA"
+			"AAAAAAAAAAAAAAAAAAAAAAAAAAAAAAAAAAAAAAAAAAAAAAAAAAAAAAAAAAAAAAAAAAAAAAAAAAAA"
+			"AAAAAAAAAAAAAAAAAAAAAAAAAAAAAAAAAAAAAAAAAAAAAAAAAAAAAAAAAAAAAAAAAAAAAAAAAAAA"
+			"AAAAAAAAAAAAAAAAAAAAAAAAAAAAAAAAAAAAAAAAAAAAAAAAAAAAAAAAAAAAAAAAAAAAAAAAAAAA"
+			"AAAAAAAAAAAAAAAAAAAAAAAAAAAAAAAAAAAAAAAAAAAAAAAAAAAAAAAAAAAAAAAAAAAAAAAAAAAA"
+			"AAAAAAAAAAAAAAAAAAAAAAAAAAAAAAAAAAAAAAAAAAAAAAAAAAAAAAAAAAAAAAAAAAAAAAAAAAAA"
+			"AAAAAAAAAAAAAAAAAAAAAAAAAAAAAAAAAAAAAAAAAAAAAAAAAAAAAAAAAAAAAAAAAAAAAAAAAAAA"
+			"AAAAAAAAAAAAAAAAAAAAAAAAAAAAAAAAAAAAAAAAAAAAAAAAAAAAAAAAAAAAAAAAAAAAAAAAAAAA"
+			"AAAAAAAAAAAAAAAAAAAAAAAAAAAAAAAAAAAAAAAAAAAAAAAAAAAAAAAAAAAAAAAAAAAAAAAAAAAA"
+			"AAAAAAAAAAAAAAAAAAAAAAAAAAAAAAAAAAAAAAAAAAAAAAAAAAAAAAAAAAAAAAAAAAAAAAAAAAAA"
+			"AAAAAAAAAAAAAAAAAAAAAAAAAAAAAAAAAAAAAAAAAAAAAAAAAAAAAAAAAAAAAAAAAAAAAAAAAAAA"
+			"AAAAAAAAAAAAAAAAAAAAAAAAAAAAAAAAAAAAAAAAAAAAAAAAAAAAAAAAAAAAAAAAAAAAAAAAAAAA"
+			"AAAAAAAAAAAAAAAAAAAAAAAAAAAAAAAAAAAAAAAAAAAAAAAAAAAAAAAAAAAAAAAAAAAAAAAAAAAA"
+			"AAAAAAAAAAAAAAAAAAAAAAAAAAAAAAAAAAAAAAAAAAAAAAAAAAAAAAAAAAAAAAAAAAAAAAAAAAAA"
+			"AAAAAAAAAAAAAAAAAAAAAAAAAAAAAAAAAAAAAAAAAAAAAAAAAAAAAAAAAAAAAAAAAAAAAAAAAAAA"
+			"AAAAAAAAAAAAAAAAAAAAAAAAAAAAAAAAAAAAAAAAAAAAAAAAAAAAAAAAAAAAAAAAAAAAAAAAAAAA"
+			"AAAAAAAAAAAAAAAAAAAAAAAAAAAAAAAAAAAAAAAAAAAAAAAAAAAAAAAAAAAAAAAAAAAAAAAAAAAA"
+			"AAAAAAAAAAAAAAAAAAAAAAAAAAAAAAAAAAAAAAAAAAAAAAAAAAAAAAAAAAAAAA=="
 		)
 	)
@@
 		)
 	)
-	(label "ATTEN_3"
+	(label "ATTEN_2"
 		(at 81.28 71.12 180)
 		(effects
@@
 		)
 	)
-	(label "DC_CPL_1"
+	(label "DC_CPL_4"
 		(at 81.28 142.24 180)
 		(effects
@@
 		)
 	)
+	(label "PGA_CSn_1"
+		(at 81.28 93.98 180)
+		(effects
+			(font
+				(size 1.27 1.27)
+			)
+			(justify right bottom)
+		)
+	)
 	(label "PGA_CSn_4"
-		(at 81.28 93.98 180)
-		(effects
-			(font
-				(size 1.27 1.27)
-			)
-			(justify right bottom)
-		)
-	)
-	(label "PGA_CSn_1"
 		(at 81.28 152.4 180)
 		(effects
@@
 		)
 	)
-	(label "TERM_2"
+	(label "TERM_3"
 		(at 81.28 55.88 180)
 		(effects
@@
 		)
 	)
-	(label "PGA_CSn_3"
+	(label "PGA_CSn_2"
 		(at 81.28 73.66 180)
 		(effects
@@
 		)
 	)
-	(label "ATTEN_4"
+	(label "ATTEN_1"
 		(at 81.28 83.82 180)
 		(effects
@@
 		)
 	)
-	(label "PGA_CSn_2"
+	(label "PGA_CSn_3"
 		(at 81.28 109.22 180)
 		(effects
@@
 		)
 	)
-	(label "DC_CPL_2"
+	(label "DC_CPL_3"
 		(at 81.28 86.36 180)
 		(effects
@@
 		)
 	)
-	(label "TERM_3"
+	(label "TERM_2"
 		(at 81.28 63.5 180)
 		(effects
@@
 		)
 	)
-	(label "DC_CPL_4"
+	(label "DC_CPL_1"
 		(at 81.28 81.28 180)
 		(effects
@@
 		)
 	)
-	(label "TERM_1"
+	(label "TERM_4"
 		(at 81.28 144.78 180)
 		(effects
@@
 		)
 	)
-	(label "TERM_4"
+	(label "TERM_1"
 		(at 81.28 76.2 180)
 		(effects
@@
 		)
 	)
-	(label "DC_CPL_3"
+	(label "DC_CPL_2"
 		(at 81.28 68.58 180)
 		(effects
@@
 		)
 	)
-	(label "ATTEN_1"
+	(label "ATTEN_4"
 		(at 81.28 154.94 180)
 		(effects
@@
 		)
 	)
-	(label "ATTEN_2"
+	(label "ATTEN_3"
 		(at 81.28 58.42 180)
 		(effects

Commit message: Added more test points
Everything on Bank 14 covered except HWIDs, VARIENT, and PUDC
Parts:
- added TP23, TP24, TP25, TP42: PCB, Thunderscope_Rev5:GEN_TP_PCB, symbol Thunderscope_Rev5:TP PCB 1mm
Connections:
- net ACQ_PG: now also TP24.1
- net FE_PG: now also TP23.1
- net PGA_SCLK: now also TP42.1
- net PGA_SDIO: now also TP25.1
- net ADC_SDIO renamed ADC_SDATA
- net OSC_OE renamed PLL_RSTn
