File: Hardware/KiCad/Thunderscope_Rev5/FPGA_CFG_MGT.kicad_sch (KiCad schematic)
At the start: 13 parts, among them U18 IC FPGA XC7A50T-2CSG325C, U19 MX25L6433FZNI-08G

Commit message: Routed ADC and Clock Gen
Parts:
- added TP46, TP47, TP48, TP52, TP53: PCB, Thunderscope_Rev5:GEN_TP_PCB, symbol Thunderscope_Rev5:TP PCB 1mm
Connections:
- net QSPI_CS: now also TP53.1
- net QSPI_DQ0: now also TP47.1
- net QSPI_DQ1: now also TP46.1
- net QSPI_DQ2: now also TP48.1
- net QSPI_DQ3: now also TP52.1
Other:
- moved on the sheet: C129, U19
