File: Hardware/KiCad/TS_Front_Endcap/TS_Front_Endcap.kicad_pcb (KiCad board)
At the start: 2 copper layers, 103 x 30.5 mm, 11 parts

Commit message: Added PN on Front Endcap Silkscreen
Other:
- board text added: "TS-USB4-ENDCAP-FRONT-V3"
