File: Hardware/KiCad/Thunderscope_Rev5_Mech_Model/Thunderscope_Rev5_Mech_Model.kicad_pcb (KiCad board)
At the start: 2 copper layers, 123 x 103.6 mm, 115 parts, among them J1 BNC, J10 009155002852006, J1002A1 BNC, J1002B1 BNC, J1002C1 BNC, J1002D1 BNC, J11 7792, J2 BNC, J3 1.27mm 6 Pin TH, J4 TSW-101-16-G-Q-RA, J5 2.54mm 6 Pin TH, J6 F300-1B7H1-11036-E100, J8 M.2 Key M, P1 PCIeX4-GF-2D-1000-1K-O64

Commit message: Moved Fan Board Edge Down 0.9mm
Parts:
- added H1: MountingHole, Adaptor_Board_JoneyTech:M.2 Mounting Hole, F.Cu at (97.0, 85.4)
- added H1: MountingHole, Adaptor_Board_JoneyTech:M.2 Mounting Hole, F.Cu at (97.0, 128.7)
- added J11: 009155002852006, Thunderscope_Rev5:KYO_009155002852006, F.Cu at (89.5, 85.4)
- added J12: 009155002852006, Thunderscope_Rev5:KYO_009155002852006, F.Cu at (89.5, 128.7)
- J10: moved to F.Cu
- turned J10 to 90 degrees
- renumbered J11 to J7
Routing:
- net +VUSB: track 33.6 -> 51.4 mm
Other:
- outline, holes or cut-outs redrawn

Commit message: Reduced Board Length from 123mm to 122.5mm
Parts:
- removed the ? at (209.4, 142.3)
- moved J1 0.50 mm to (201.0, 89.0)
- moved J10 0.50 mm to (206.9, 134.3)
- moved J2 0.50 mm to (201.0, 125.1)
- moved J5 0.50 mm to (199.4, 107.1)
- moved J6 0.50 mm to (206.8, 107.1)
- moved J7 0.40 mm to (202.2, 143.4)
Routing:
- net +VUSB: track 51.4 -> 49.9 mm
Other:
- board size 123 x 103.6 mm -> 122.5 x 103.6 mm

Commit message: Changed Mech Model to use M2 Mounting Hardware
Parts:
- removed ? (x95): , 
- J5: footprint DSO.PcbLib:GEN_2.54MM_6_PIN_TH_RA -> Thunderscope_Rev5:GEN_2.54MM_6_PIN_TH_RA
- SO1, SO2, SO3: renamed from H1; value MountingHole -> 2.5mm M2 SMT Standoff; footprint Adaptor_Board_JoneyTech:M.2 Mounting Hole -> ThunderScope:M2_SMT_Standoff_9774025243R; moved to B.Cu
- turned SO1 to 180 degrees
- turned SO2 to 180 degrees
- turned SO3 to 180 degrees
Connections:
- J11 pad 1: (no net) -> unconnected-(J11-Pad1)
- J11 pad 2: (no net) -> GND
- J12 pad 1: (no net) -> GND
- J12 pad 2: (no net) -> GND
