File: Hardware/KiCad/Thunderscope_Rev5_Mech_Model/Thunderscope_Rev5_Mech_Model.kicad_sch (KiCad schematic)
At the start: 15 parts, among them J11 7792

Commit message: Updated mech model schematic to match pcb
Parts:
- removed FID1, FID2, FID3, FID4, FID5, FID6, FID7, FID8: PCB, GEN_FID, symbol Thunderscope_Rev5:FID 1mm
- removed SHLD1: 9204, symbol Thunderscope_Rev5:PCIe IO Shield
- removed TP1, TP4, TP5: PCB, GEN_TP_PCB, symbol Thunderscope_Rev5:TP PCB 1mm
- removed TP2, TP3: 5019, KEY_5019, symbol Thunderscope_Rev5:TP KEYSTONE 5019
- added D1: GREEN, LED_0603_LTST-S270K, symbol Thunderscope_Rev5:LED GREEN 0603 LTST-S270K
- added H1: MountingHole, symbol Mechanical:MountingHole
- added J1, J1002A1, J1002B1, J1002C1, J1002D1, J2: BNC, MOL_0731000105, symbol Thunderscope_Rev5:BNC JACK R/A
- added J10: 009155002852006, KYO_009155002852006, symbol Thunderscope_Rev5:CONN SPRING 2 PIN
- added J3: 1.27mm 6 Pin TH, GEN_1.27mm_2x5_Pin_TH_RA, symbol Thunderscope_Rev5:CONN 1.27mm 2x5 Pin TH RA
- added J4: TSW-101-16-G-Q-RA, GEN_5.08mm_1x2_Pin_TH_RA, symbol Thunderscope_Rev5:CONN 5.08mm 2 Pin TH RA
- added J5: 2.54mm 6 Pin TH, GEN_2.54mm_6_Pin_TH_RA, symbol Thunderscope_Rev5:CONN 2.54mm 6 Pin TH RA
- added J6: Conn_01x36, symbol Connector_Generic:Conn_01x36
- added J8: M.2 Key M, TE_M2_KEYM_2199230, symbol Thunderscope_Rev5:CONN M.2 Key M FEMALE
- added P1: PCIeX4-GF-2D-1000-1K-O64, PCIeX4-GF-2D-1000-1K-O64, symbol Thunderscope_Rev5:PCIeX4-GF-2D-1000-1K-O64
Connections:
- net GND: now also J1.2 (SHIELD), J1002A1.2 (SHIELD), J1002B1.2 (SHIELD), J1002C1.2 (SHIELD), J1002D1.2 (SHIELD), J2.2 (SHIELD)
Other:
- removed sheet ADC
- removed sheet CH1
- removed sheet CH2
- removed sheet CH3
- removed sheet CH4
- removed sheet Clock Generator
- removed sheet FPGA
- removed sheet Front End Trim and Bias
- removed sheet M.2_Key_M
- removed sheet PCIe_x4
- removed sheet POWER
- removed sheet User IO
- moved on the sheet: J11

Commit message: Schematic WIP
Parts:
- D1: footprint LED_0603_LTST-S270K -> Thunderscope_Rev5:LED_Kingbright_APFA3010_3x1.5mm_Horizontal; symbol Thunderscope_Rev5:LED GREEN 0603 LTST-S270K -> Thunderscope_Rev5:LED RGB 1204 APFA3010LSEEZGKQBKC; MANUFACTURER Vishay Lite-On -> Kingbright; MANUFACTURER PART NUMBER LTST-S270KGKT -> APFA3010LSEEZGKQBKC; SUPPLIER PART NUMBER 1 859-LTST-S270KGKT -> 604-APFA3010LSEEZGKQ
- J6: value Conn_01x36 -> F300-1B7H1-11036-E100; footprint (none) -> Thunderscope_Rev5:AMPHENOL_F300-1B7H1-11036-E100; symbol Connector_Generic:Conn_01x36 -> Thunderscope_Rev5:CONN FFC BOTTOM 36POS 0.5MM RA; MANUFACTURER (none) -> Amphenol ICC; MANUFACTURER PART NUMBER (none) -> F300-1B7H1-11036-E100; SUPPLIER 1 (none) -> Mouser; SUPPLIER PART NUMBER 1 (none) -> 649-F3001B7H111036E1
Other:
- moved on the sheet: H1
Changed lines of the file:
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@@
 (kicad_sch
-	(version 20241004)
+	(version 20241209)
 	(generator "eeschema")
 	(generator_version "8.99")
@@
 	)
 	(symbol
-		(lib_id "Thunderscope_Rev5:LED GREEN 0603 LTST-S270K")
-		(at 25.4 104.14 90)
+		(lib_id "Thunderscope_Rev5:LED RGB 1204 APFA3010LSEEZGKQBKC")
+		(at 25.4 104.14 180)
 		(unit 1)
 		(exclude_from_sim no)
@@
 		(dnp no)
 		(property "Reference" "D1"
-			(at 19.812 108.458 0)
+			(at 25.4 93.98 0)
+			(effects
+				(font
+					(size 1.27 1.27)
+				)
+			)
+		)
+		(property "Value" "GREEN"
+			(at 29.718 98.806 0)
 			(effects
 				(font
@@
 				)
 				(justify left bottom)
-			)
-		)
-		(property "Value" "GREEN"
-			(at 30.734 108.458 0)
-			(effects
-				(font
-					(size 1.27 1.27)
-				)
-				(justify left bottom)
-				(hide yes)
-			)
-		)
-		(property "Footprint" "LED_0603_LTST-S270K"
-			(at 25.4 104.14 0)
+				(hide yes)
+			)
+		)
+		(property "Footprint" "Thunderscope_Rev5:LED_Kingbright_APFA3010_3x1.5mm_Horizontal"
+			(at 25.4 91.44 0)
 			(effects
 				(font
@@
 		)
 		(property "SUPPLIER 1" "Mouser"
-			(at 19.812 110.998 0)
-			(effects
-				(font
-					(size 1.27 1.27)
-				)
-				(justify left bottom)
-				(hide yes)
-			)
-		)
-		(property "SUPPLIER PART NUMBER 1" "859-LTST-S270KGKT"
-			(at 19.812 110.998 0)
-			(effects
-				(font
-					(size 1.27 1.27)
-				)
-				(justify left bottom)
+			(at 25.4 91.44 0)
+			(effects
+				(font
+					(size 1.27 1.27)
+				)
+				(hide yes)
+			)
+		)
+		(property "SUPPLIER PART NUMBER 1" "604-APFA3010LSEEZGKQ"
+			(at 25.4 91.44 0)
+			(effects
+				(font
+					(size 1.27 1.27)
+				)
 				(hide yes)
 			)
 		)
 		(property "HOUSE PART NUMBER" ""
-			(at 19.812 110.998 0)
-			(effects
-				(font
-					(size 1.27 1.27)
-				)
-				(justify left bottom)
-				(hide yes)
-			)
-		)
-		(property "MANUFACTURER" "Vishay Lite-On"
-			(at 19.812 110.998 0)
-			(effects
-				(font
-					(size 1.27 1.27)
-				)
-				(justify left bottom)
-				(hide yes)
-			)
-		)
-		(property "MANUFACTURER PART NUMBER" "LTST-S270KGKT"
-			(at 19.812 110.998 0)
-			(effects
-				(font
-					(size 1.27 1.27)
-				)
-				(justify left bottom)
+			(at 25.4 104.14 0)
+			(effects
+				(font
+					(size 1.27 1.27)
+				)
+				(hide yes)
+			)
+		)
+		(property "MANUFACTURER" "Kingbright"
+			(at 25.4 91.44 0)
+			(effects
+				(font
+					(size 1.27 1.27)
+				)
+				(hide yes)
+			)
+		)
+		(property "MANUFACTURER PART NUMBER" "APFA3010LSEEZGKQBKC"
+			(at 25.4 91.44 0)
+			(effects
+				(font
+					(size 1.27 1.27)
+				)
 				(hide yes)
 			)
@@
 		)
 		(pin "2"
+		)
+		(pin "3"
+		)
+		(pin "4"
 		)
 		(instances
@@
 	)
 	(symbol
-		(lib_id "Connector_Generic:Conn_01x36")
-		(at 246.38 99.06 0)
+		(lib_id "Thunderscope_Rev5:CONN FFC BOTTOM 36POS 0.5MM RA")
+		(at 226.06 53.34 0)
 		(unit 1)
 		(exclude_from_sim no)
@@
 		(on_board yes)
 		(dnp no)
-		(fields_autoplaced yes)
 		(property "Reference" "J6"
-			(at 248.92 99.0599 0)
-			(effects
-				(font
-					(size 1.27 1.27)
-				)
-				(justify left)
-			)
-		)
-		(property "Value" "Conn_01x36"
-			(at 248.92 101.5999 0)
-			(effects
-				(font
-					(size 1.27 1.27)
-				)
-				(justify left)
-			)
-		)
-		(property "Footprint" ""
-			(at 246.38 99.06 0)
+			(at 228.6 52.07 0)
+			(effects
+				(font
+					(size 1.27 1.27)
+				)
+			)
+		)
+		(property "Value" "F300-1B7H1-11036-E100"
+			(at 228.6 154.94 0)
+			(effects
+				(font
+					(size 1.27 1.27)
+				)
+			)
+		)
+		(property "Footprint" "Thunderscope_Rev5:AMPHENOL_F300-1B7H1-11036-E100"
+			(at 228.6 153.924 0)
 			(effects
 				(font
@@
 		)
 		(property "Datasheet" "~"
-			(at 246.38 99.06 0)
+			(at 226.06 53.34 0)
 			(effects
 				(font
@@
 		)
 		(property "Description" "Generic connector, single row, 01x36, script generated (kicad-library-utils/schlib/autogen/connector/)"
-			(at 246.38 99.06 0)
+			(at 226.06 53.34 0)
+			(effects
+				(font
+					(size 1.27 1.27)
+				)
+				(hide yes)
+			)
+		)
+		(property "SUPPLIER 1" "Mouser"
+			(at 228.6 153.924 0)
+			(effects
+				(font
+					(size 1.27 1.27)
+				)
+				(hide yes)
+			)
+		)
+		(property "SUPPLIER PART NUMBER 1" "649-F3001B7H111036E1 "
+			(at 228.6 153.924 0)
+			(effects
+				(font
+					(size 1.27 1.27)
+				)
+				(hide yes)
+			)
+		)
+		(property "HOUSE PART NUMBER" ""
+			(at 226.06 53.34 0)
+			(effects
+				(font
+					(size 1.27 1.27)
+				)
+				(hide yes)
+			)
+		)
+		(property "MANUFACTURER" "Amphenol ICC"
+			(at 228.6 153.924 0)
+			(effects
+				(font
+					(size 1.27 1.27)
+				)
+				(hide yes)
+			)
+		)
+		(property "MANUFACTURER PART NUMBER" "F300-1B7H1-11036-E100"
+			(at 228.6 153.924 0)
 			(effects
 				(font
@@
 		)
 		(pin "31"
+		)
+		(pin "SH1"
+		)
+		(pin "SH2"
 		)
 		(instances
@@
 	(symbol
 		(lib_id "Mechanical:MountingHole")
-		(at 177.8 40.64 0)
+		(at 177.8 30.48 0)
 		(unit 1)
 		(exclude_from_sim yes)
@@
 		(fields_autoplaced yes)
 		(property "Reference" "H1"
-			(at 180.34 39.3699 0)
+			(at 180.34 29.2099 0)
 			(effects
 				(font
@@
 		)
 		(property "Value" "MountingHole"
-			(at 180.34 41.9099 0)
+			(at 180.34 31.7499 0)
 			(effects
 				(font
@@
 		)
 		(property "Footprint" ""
-			(at 177.8 40.64 0)
+			(at 177.8 30.48 0)
 			(effects
 				(font
@@
 		)
 		(property "Datasheet" "~"
-			(at 177.8 40.64 0)
+			(at 177.8 30.48 0)
 			(effects
 				(font
@@
 		)
 		(property "Description" "Mounting Hole without connection"
-			(at 177.8 40.64 0)
-			(effects
-				(font
+			(at 177.8 30.48 0)
+			(effects
+				(font

Commit message: Sent Mech Models Out to Fab
Parts:
- added R1, R2, R3: 1K, Thunderscope_Rev5:GEN_R_0402, symbol Thunderscope_Rev5:RES 1K OHM 1% 1/10W 0402
- D1: value GREEN -> RGB; symbol Thunderscope_Rev5:LED RGB 1204 APFA3010LSEEZGKQBKC -> Thunderscope_Rev5:LED RGB 1204 APFA3010LSEKJ3ZGKQBC; MANUFACTURER PART NUMBER APFA3010LSEEZGKQBKC -> APFA3010LSEKJ3ZGKQBC; SUPPLIER PART NUMBER 1 604-APFA3010LSEEZGKQ -> 604-APFA3010LSEKJ3ZG
- J8: footprint TE_M2_KEYM_2199230 -> Thunderscope_Rev5:TE_M2_KEYM_2199230
Connections:
- net GND: now also D1.2 (A), J10.2, J4.1, J5.6, J6.SH1, J6.SH2, J8.10, J8.16, J8.2, J8.22, J8.28, J8.34, J8.4, J8.40, J8.46, J8.52, J8.58, J8.70, J8.72, J8.74, J8.76, J8.77
- net at D1.1 (R): now also R3.2
- net at D1.3 (G): now also R2.2
- net at D1.4 (B): now also R1.2
- net M2_PET3_N: now reaches J8.12
- net +VUSB: now reaches J8.13
- net +VUSB: now also J10.1, J5.1, J8.15, J8.17, J8.19, J8.3, J8.5, J8.69, J8.71, J8.73
- net M2_PET3_P: now reaches J8.14
- net M2_PER2_N: now reaches J8.18
- net M2_PER2_P: now reaches J8.20
- net M2_PET2_N: now reaches J8.24
- net M2_PET2_P: now reaches J8.26
- net M2_PER1_N: now reaches J8.30
- net M2_PER1_P: now reaches J8.32
- net M2_PET1_N: now reaches J8.36
- net M2_PET1_P: now reaches J8.38
- net M2_PER0_N: now reaches J8.42
- net M2_PER0_P: now reaches J8.44
- net M2_PET0_N: now reaches J8.48
- net M2_PERST#: now reaches J8.49
- net M2_PET0_P: now reaches J8.50
- net M2_REFCLK_N: now reaches J8.54
- net M2_REFCLK_P: now reaches J8.56
- net M2_PER3_N: now reaches J8.6
- net M2_PER3_P: now reaches J8.8
- net LED_R: now reaches J5.3
- net LED_R: now also R3.1
- net LED_B: now reaches J5.4
- net LED_B: now also R1.1
- net LED_G: now reaches J5.5
- net LED_G: now also R2.1
- no-connect marks 0 -> 162
Other:
- note added: "Custom Pinout"
- note added: "Main Board"
- moved on the sheet: J10, J3, J5, J6

Commit message: Changed Mech Model to use M2 Mounting Hardware
Parts:
- added J11, J12: 009155002852006, Thunderscope_Rev5:KYO_009155002852006, symbol Thunderscope_Rev5:CONN SPRING 2 PIN
- added SO2, SO3: 2.5mm M2 SMT Standoff, ThunderScope:M2_SMT_Standoff_9774025243R, symbol ThunderScope:M2_2.5mm_SMT_Standoff_9774025243R
- J1, J1002A1, J1002B1, J1002C1, J1002D1, J2: footprint MOL_0731000105 -> Thunderscope_Rev5:MOL_0731000105
- J10: footprint KYO_009155002852006 -> Thunderscope_Rev5:KYO_009155002852006
- J3: footprint GEN_1.27mm_2x5_Pin_TH_RA -> Thunderscope_Rev5:GEN_1.27mm_2x5_Pin_TH_RA
- J4: footprint GEN_5.08mm_1x2_Pin_TH_RA -> Thunderscope_Rev5:GEN_5.08mm_1x2_Pin_TH_RA
- J5: footprint GEN_2.54mm_6_Pin_TH_RA -> Thunderscope_Rev5:GEN_2.54MM_6_PIN_TH_RA
- J7: renamed from J11; footprint KEY_7792 -> Thunderscope_Rev5:KEY_7792
- P1: footprint PCIeX4-GF-2D-1000-1K-O64 -> Thunderscope_Rev5:PCIeX4-GF-2D-1000-1K-O64; now left out of the parts list
- SO1: renamed from H1; value MountingHole -> 2.5mm M2 SMT Standoff; footprint (none) -> ThunderScope:M2_SMT_Standoff_9774025243R; symbol Mechanical:MountingHole -> ThunderScope:M2_2.5mm_SMT_Standoff_9774025243R; MANUFACTURER (none) -> Wurth Elektronik; MANUFACTURER PART NUMBER (none) -> 9774025243R; SUPPLIER 1 (none) -> Mouser; SUPPLIER PART NUMBER 1 (none) -> 710-9774025243R; now in the parts list
Connections:
- net GND: now also SO1.1, J11.2, J12.1, J12.2, SO2.1, SO3.1
- no-connect marks 162 -> 163
