File: Hardware/KiCad/Interposer_Board_JoneyTech/Interposer_Board_JoneyTech.kicad_sch (KiCad schematic)
At the start: 2 parts, among them J1 M.2 Key M, J2 M.2 Key M

Commit message: Interposer Board WIP
Parts:
- added H1, H2, H3, H4: MountingHole, Adaptor_Board_JoneyTech:M.2 Mounting Hole, symbol Mechanical:MountingHole_Pad
- J1, J2: footprint PCB EDGE M.2 Key M -> ThunderScope:PCB EDGE M.2 Key M
Connections:
- net GND: now also H1.1, H2.1, H3.1, H4.1

Commit message: Interposer Mech Changes
Moved adaptor back 0.5mm to align with board edge. Changed mounting holes to M2, and added exposed copper on edges.
Parts:
- H1, H2, H3, H4: footprint Adaptor_Board_JoneyTech:M.2 Mounting Hole -> ThunderScope:MountingHole_2.2mm_M2_Pad_Via
Changed lines of the file:
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@@
 			)
 		)
-		(property "Footprint" "Adaptor_Board_JoneyTech:M.2 Mounting Hole"
+		(property "Footprint" "ThunderScope:MountingHole_2.2mm_M2_Pad_Via"
 			(at 180.34 33.02 0)
 			(effects
@@
 			)
 		)
-		(property "Footprint" "Adaptor_Board_JoneyTech:M.2 Mounting Hole"
+		(property "Footprint" "ThunderScope:MountingHole_2.2mm_M2_Pad_Via"
 			(at 195.58 20.32 0)
 			(effects
@@
 			)
 		)
-		(property "Footprint" "Adaptor_Board_JoneyTech:M.2 Mounting Hole"
+		(property "Footprint" "ThunderScope:MountingHole_2.2mm_M2_Pad_Via"
 			(at 109.22 33.02 0)
 			(effects
@@
 			)
 		)
-		(property "Footprint" "Adaptor_Board_JoneyTech:M.2 Mounting Hole"
+		(property "Footprint" "ThunderScope:MountingHole_2.2mm_M2_Pad_Via"
 			(at 165.1 20.32 0)
 			(effects
