File: Hardware/KiCad/Interposer_Board_JoneyTech/Interposer_Board_JoneyTech.kicad_pcb (KiCad board)
At the start: 2 copper layers, 80 x 60 mm, 4 parts, among them J1 M.2 Key M, J2 M.2 Key M

Commit message: Moved Fan Board Edge Down 0.9mm
Parts:
- added H1: MountingHole, Adaptor_Board_JoneyTech:M.2 Mounting Hole, F.Cu at (79.8, 91.8)
- added H1: MountingHole, Adaptor_Board_JoneyTech:M.2 Mounting Hole, F.Cu at (79.8, 48.5)
Other:
- board size 80 x 60 mm -> 123 x 99.5 mm

Commit message: Reduced Board Length from 123mm to 122.5mm
Other:
- board size 123 x 99.5 mm -> 122.5 x 99.5 mm
Changed lines of the file:
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@@
 	)
 	(gr_arc
-		(start 192.2761 46.2786)
-		(mid 192.629653 46.425047)
-		(end 192.7761 46.7786)
+		(start 191.7761 46.2786)
+		(mid 192.129653 46.425047)
+		(end 192.2761 46.7786)
 		(stroke
 			(width 0.05)
@@
 			(width 0.05)
 			(type solid)
-		)
-		(layer "Edge.Cuts")
-	)
-	(gr_line
-		(start 192.7761 90.8536)
-		(end 192.7761 119.3786)
-		(stroke
-			(width 0.05)
-			(type default)
 		)
 		(layer "Edge.Cuts")
@@
 	)
 	(gr_arc
-		(start 192.7761 119.3786)
-		(mid 192.629653 119.732153)
-		(end 192.2761 119.878601)
+		(start 192.2761 119.3786)
+		(mid 192.129653 119.732153)
+		(end 191.7761 119.878601)
 		(stroke
 			(width 0.05)
@@
 		(layer "Edge.Cuts")
 	)
+	(gr_arc
+		(start 70.2761 119.8786)
+		(mid 69.922547 119.732153)
+		(end 69.7761 119.3786)
+		(stroke
+			(width 0.05)
+			(type default)
+		)
+		(layer "Edge.Cuts")
+	)
 	(gr_line
 		(start 109.9511 91.903601)
@@
 			(width 0.05)
 			(type default)
-		)
-		(layer "Edge.Cuts")
-	)
-	(gr_arc
-		(start 70.2761 119.8786)
-		(mid 69.922546 119.732153)
-		(end 69.7761 119.378599)
-		(stroke
-			(width 0.05)
-			(type solid)
 		)
 		(layer "Edge.Cuts")
@@
 	(gr_line
 		(start 179.7761 46.2786)
-		(end 192.2761 46.278599)
+		(end 191.7761 46.2786)
 		(stroke
 			(width 0.05)
@@
 	)
 	(gr_line
-		(start 192.7761 80.3536)
-		(end 192.7761 90.8536)
-		(stroke
-			(width 0.05)
-			(type default)
-		)
-		(layer "Edge.Cuts")
-	)
-	(gr_line
 		(start 106.4511 74.8786)
 		(end 106.4511 90.1536)
@@
 	)
 	(gr_line
-		(start 192.7761 80.3536)
-		(end 192.7761 46.7786)
-		(stroke
-			(width 0.05)
-			(type default)
-		)
-		(layer "Edge.Cuts")
-	)
-	(gr_line
-		(start 192.2761 119.878601)
+		(start 191.7761 119.8786)
 		(end 70.2761 119.8786)
 		(stroke
@@
 	(gr_line
 		(start 69.7761 119.3786)
-		(end 69.776105 20.8786)
+		(end 69.7761 20.8786)
 		(stroke
 			(width 0.05)
@@
 		)
 		(layer "Edge.Cuts")
+	)
+	(gr_line
+		(start 192.2761 119.3786)
+		(end 192.2761 46.7786)
+		(stroke
+			(width 0.05)
+			(type default)
+		)
+		(layer "Edge.Cuts")

Commit message: Interposer Board WIP
Parts:
- H1, H2: renamed from REF**; value M.2 Mounting Hole -> MountingHole
- J1, J2: footprint DSO.PcbLib:PCB EDGE M.2 Key M -> ThunderScope:PCB EDGE M.2 Key M
- renumbered H1 to H3, H1 to H4
Routing:
- added copper zone on In1.Cu, net GND
- added copper zone on In2.Cu, net GND
Other:
- copper layers 2 -> 4
- board text added: "1"
- board text added: "2"
- board text added: "3"
- board text added: "4"
- board text added: "THIS SIDE TOWARDS ADAPTOR BOARD"
- board text added: "THIS SIDE TOWARDS MAIN BOARD"
- board text added: "TS-USB4-INTERPOSER-JONEYTECH"
- board text added: "You live like this, sheltered, in a delicate world, and you believe you are living. Then you read a book… or you take a trip… and you discover that you are not living, that you are hibernating. The symptoms of hibernating are easily detectable: first, restlessness. The second symptom (when hibernating becomes dangerous and might degenerate into death): absence of pleasure. That is all. It appears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"
- board text removed: "Interposer Board for JoneyTech TB3 Adaptor"
Changed lines of the file:
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@@
 	(layers
 		(0 "F.Cu" signal "Top Layer")
+		(4 "In1.Cu" signal)
+		(6 "In2.Cu" signal)
 		(2 "B.Cu" signal "Bottom Layer")
 		(9 "F.Adhes" user "F.Adhesive")
@@
 			)
 			(layer "dielectric 1"
+				(type "prepreg")
+				(color "FR4 natural")
+				(thickness 0.1)
+				(material "FR4")
+				(epsilon_r 4.74)
+				(loss_tangent 0.02)
+			)
+			(layer "In1.Cu"
+				(type "copper")
+				(thickness 0.035)
+			)
+			(layer "dielectric 2"
 				(type "core")
-				(thickness 0.69)
-				(material "PP-006")
-				(epsilon_r 4.29)
+				(thickness 0.42)
+				(material "FR4")
+				(epsilon_r 4.6)
+				(loss_tangent 0.02)
+			)
+			(layer "In2.Cu"
+				(type "copper")
+				(thickness 0.035)
+			)
+			(layer "dielectric 3"
+				(type "prepreg")
+				(color "FR4 natural")
+				(thickness 0.1)
+				(material "FR4")
+				(epsilon_r 4.74)
 				(loss_tangent 0.02)
 			)
@@
 			)
 			(copper_finish "None")
-			(dielectric_constraints no)
+			(dielectric_constraints yes)
 		)
 		(pad_to_mask_clearance 0)
@@
 	(net 69 "unconnected-(J1-Pad20)")
 	(net 70 "unconnected-(J1-Pad56)")
-	(footprint "DSO.PcbLib:PCB EDGE M.2 Key M"
+	(footprint "ThunderScope:PCB EDGE M.2 Key M"
 		(layer "F.Cu")
 		(at 110.6386 69.3036 -90)
@@
 		)
 		(property "Datasheet" ""
-			(at 0 0 90)
+			(at 0 0 270)
 			(layer "F.Fab")
 			(hide yes)
@@
 		)
 		(property "Description" ""
-			(at 0 0 90)
+			(at 0 0 270)
 			(layer "F.Fab")
 			(hide yes)
@@
 		(layer "F.Cu")
 		(at 167.2511 42.3536)
-		(property "Reference" "REF**"
+		(property "Reference" "H2"
 			(at 0 -0.5 0)
 			(unlocked yes)
@@
 			)
 		)
-		(property "Value" "M.2 Mounting Hole"
+		(property "Value" "MountingHole"
 			(at 0 1 0)
 			(unlocked yes)
@@
 			)
 		)
-		(property "Description" ""
+		(property "Description" "Mounting Hole with connection"
 			(at 0 0 0)
 			(unlocked yes)
@@
 			)
 		)
-		(attr through_hole)
+		(property ki_fp_filters "MountingHole*Pad*")
+		(sheetname "/")
+		(sheetfile "Interposer_Board_JoneyTech.kicad_sch")
+		(attr through_hole exclude_from_bom)
 		(fp_text user "${REFERENCE}"
 			(at 0 2.5 0)
@@
 			)
 		)
-		(pad "MOUNTING-HOLE" thru_hole circle
+		(pad "1" thru_hole circle
 			(at 0 0)
 			(size 5.5 5.5)
@@
 			(remove_unused_layers no)
 			(net 1 "GND")
+			(pinfunction "1")
+			(pintype "input")
 			(solder_mask_margin 0.1016)
 		)
@@
 		(layer "F.Cu")
 		(at 79.7761 91.7786)
-		(property "Reference" "H1"
+		(property "Reference" "H4"
 			(at 0 -0.5 0)
 			(unlocked yes)
@@
 			)
 		)
-		(property "Description" "Mounting Hole without connection"
+		(property "Description" "Mounting Hole with connection"
 			(at 0 0 0)
 			(unlocked yes)
@@
 			)
 		)
+		(property ki_fp_filters "MountingHole*Pad*")
+		(sheetname "/")
+		(sheetfile "Interposer_Board_JoneyTech.kicad_sch")
 		(attr through_hole exclude_from_bom)
 		(fp_text user "${REFERENCE}"
@@
 			)
 		)
-		(pad "MOUNTING-HOLE" thru_hole circle
+		(pad "1" thru_hole circle
 			(at 0 0)
 			(size 5.5 5.5)
@@
 			(layers "*.Cu" "*.Mask")
 			(remove_unused_layers no)
+			(net 1 "GND")
+			(pinfunction "1")
+			(pintype "input")
 			(solder_mask_margin 0.1016)
 		)
@@
 		(layer "F.Cu")
 		(at 186.4511 80.3536)
-		(property "Reference" "REF**"
+		(property "Reference" "H1"
 			(at 0 -0.5 0)
 			(unlocked yes)
@@
 			)
 		)
-		(property "Value" "M.2 Mounting Hole"
+		(property "Value" "MountingHole"
 			(at 0 1 0)
 			(unlocked yes)
@@
 			)
 		)
-		(property "Description" ""
+		(property "Description" "Mounting Hole with connection"
 			(at 0 0 0)
 			(unlocked yes)
@@
 			)
 		)
-		(attr through_hole)
+		(property ki_fp_filters "MountingHole*Pad*")
+		(sheetname "/")
+		(sheetfile "Interposer_Board_JoneyTech.kicad_sch")
+		(attr through_hole exclude_from_bom)
 		(fp_text user "${REFERENCE}"
 			(at 0 2.5 0)
@@
 			)
 		)
-		(pad "MOUNTING-HOLE" thru_hole circle
+		(pad "1" thru_hole circle
 			(at 0 0)
 			(size 5.5 5.5)
@@
 			(remove_unused_layers no)
 			(net 1 "GND")
+			(pinfunction "1")
+			(pintype "input")
 			(solder_mask_margin 0.1016)
 		)
@@
 		(layer "F.Cu")
 		(at 79.7511 48.4786)
-		(property "Reference" "H1"
+		(property "Reference" "H3"
 			(at 0 -0.5 0)
 			(unlocked yes)
@@
 			)
 		)
-		(property "Description" "Mounting Hole without connection"
+		(property "Description" "Mounting Hole with connection"
 			(at 0 0 0)
 			(unlocked yes)
@@
 			)
 		)
+		(property ki_fp_filters "MountingHole*Pad*")
+		(sheetname "/")
+		(sheetfile "Interposer_Board_JoneyTech.kicad_sch")
 		(attr through_hole exclude_from_bom)
 		(fp_text user "${REFERENCE}"
@@
 			)
 		)
-		(pad "MOUNTING-HOLE" thru_hole circle
+		(pad "1" thru_hole circle
 			(at 0 0)
 			(size 5.5 5.5)
@@
 			(layers "*.Cu" "*.Mask")
 			(remove_unused_layers no)
+			(net 1 "GND")
+			(pinfunction "1")
+			(pintype "input")
 			(solder_mask_margin 0.1016)
 		)
 		(embedded_fonts no)
 	)
-	(footprint "DSO.PcbLib:PCB EDGE M.2 Key M"
+	(footprint "ThunderScope:PCB EDGE M.2 Key M"
 		(layer "B.Cu")
 		(at 178.2511 94.1536 180)
 		(property "Reference" "J2"
-			(at 15.93511 -11.704398 180)
+			(at 1.48647 1.491898 0)
 			(unlocked yes)
 			(layer "B.SilkS")
@@
 		)
 		(property "Value" "M.2 Key M"
-			(at 10.729795 13.390802 180)
+			(at 16.520205 -17.040802 0)
 			(unlocked yes)
 			(layer "B.SilkS")
@@
 		(property "Datasheet" ""
 			(at 0 0 0)
-			(layer "F.Fab")
+			(layer "B.Fab")
 			(hide yes)
 			(effects
@@
 					(thickness 0.15)
 				)
+				(justify mirror)
 			)
 		)
 		(property "Description" ""
 			(at 0 0 0)
-			(layer "F.Fab")
+			(layer "B.Fab")
 			(hide yes)
 			(effects
@@
 					(thickness 0.15)
 				)
+				(justify mirror)
 			)
 		)
@@
 		)
 		(fp_line
-			(start 20.95 -0.7)
-			(end 20.95 -4)
+			(start 20.95 -4)
+			(end 20.95 -0.7)
 			(stroke
 				(width 0.05)
@@
 		)
 		(fp_line
-			(start 5.475 -1.3)
-			(end 5.475 -4.2)
+			(start 5.475 -4.2)
+			(end 16 -4.2)
 			(stroke
 				(width 0.05)
@@
 		(fp_line
 			(start 5.475 -4.2)
-			(end 16 -4.2)
+			(end 5.475 -1.3)
 			(stroke
 				(width 0.05)
@@
 		)
 		(fp_line
-			(start 4.275 -1.3)
-			(end 4.275 -4.2)
+			(start 4.275 -4.2)
+			(end 4.275 -1.3)
 			(stroke
 				(width 0.05)
@@
 		(layer "Edge.Cuts")
 	)
-	(gr_text "Interposer Board for JoneyTech TB3 Adaptor"
-		(at 72.7761 24.8786 0)
+	(gr_text "You live like this, sheltered, in a delicate world, and you believe you are living.\nThen you read a book… or you take a trip… and you discover that you are not living, that you are hibernating.\nThe symptoms of hibernating are easily detectable: first, restlessness.\nThe second symptom (when hibernating becomes dangerous and might degenerate into death): absence of pleasure.\nThat is all. It appears like an innocuous illness. Monotony, boredom, death.\nMillions live like this (or die like this) without knowing it.\nThey work in offices. They drive a car. They picnic with their families. They raise children.\nAnd then some shock treatment takes place, a person, a book, a song, and it awakens them and saves them from death.\nSome never awaken.\n\n-Anaïs Nin"
+		(at 73.7761 24.3786 0)
+		(layer "F.Mask")
+		(effects
+			(font
+				(size 1 1)
+				(thickness 0.125)
+			)
+			(justify left top)
+		)
+	)
+	(gr_text "TS-USB4-INTERPOSER-JONEYTECH"
+		(at 131.0261 112.3786 0)
 		(layer "F.SilkS")
 		(effects
 			(font
-				(size 1 1)
-				(thickness 0.2)
-				(bold yes)
-			)
-			(justify left bottom)
+				(size 1.5 1.5)
+				(thickness 0.25)
+			)
+			(justify bottom)
+		)
+	)
+	(gr_text "THIS SIDE TOWARDS MAIN BOARD"
+		(at 131.0261 115.8786 0)
+		(layer "F.SilkS")
+		(effects
+			(font
+				(size 1.5 1.5)
+				(thickness 0.25)
+			)
+			(justify bottom)
+		)
+	)
+	(gr_text "1"
+		(at 186.4511 84.8786 0)
+		(layer "F.SilkS")
+		(effects
+			(font
+				(size 2 2)
+				(thickness 0.3)
+			)
+			(justify top)
+		)
+	)
+	(gr_text "2"
+		(at 167.2511 46.8786 0)
+		(layer "B.SilkS")
+		(effects
+			(font
+				(size 2 2)
+				(thickness 0.3)
+			)
+			(justify top mirror)
+		)
+	)
+	(gr_text "TS-USB4-INTERPOSER-JONEYTECH"
+		(at 131.0261 112.3786 0)
+		(layer "B.SilkS")
+		(effects
+			(font
+				(size 1.5 1.5)
+				(thickness 0.25)
+			)
+			(justify bottom mirror)
+		)
+	)
+	(gr_text "4"
+		(at 79.7761 96.3036 0)
+		(layer "B.SilkS")
+		(effects
+			(font
+				(size 2 2)
+				(thickness 0.3)
+			)
+			(justify top mirror)
+		)
+	)
+	(gr_text "THIS SIDE TOWARDS ADAPTOR BOARD"
+		(at 131.0261 115.8786 0)
+		(layer "B.SilkS")
+		(effects
+			(font
+				(size 1.5 1.5)
+				(thickness 0.25)
+			)
+			(justify bottom mirror)
+		)
+	)
+	(gr_text "3"
+		(at 79.7511 53.0036 0)
+		(layer "B.SilkS")
+		(effects
+			(font
+				(size 2 2)
+				(thickness 0.3)
+			)
+			(justify top mirror)
 		)
 	)
@@
 		(net 1)
 		(net_name "GND")
-		(layer "F.Cu")
+		(layers "F.Cu" "In1.Cu" "In2.Cu")
 		(hatch edge 0.5)
 		(connect_pads
@@
 		(min_thickness 0.2032)
 		(filled_areas_thickness no)
-		(fill yes
+		(fill
 			(thermal_gap 0.254)
 			(thermal_bridge_width 0.254)

Commit message: Interposer Mech Changes
Moved adaptor back 0.5mm to align with board edge. Changed mounting holes to M2, and added exposed copper on edges.
Parts:
- H1, H2, H3, H4: footprint Adaptor_Board_JoneyTech:M.2 Mounting Hole -> ThunderScope:MountingHole_2.2mm_M2_Pad_Via
- moved H1 0.50 mm to (186.0, 80.4)
- moved J1 0.50 mm to (110.1, 69.3)
Routing:
- net GND: track 1.86 -> 0.00 mm, vias 1 -> 0
- added copper zone on In2.Cu, net +3V3
- added copper zone on B.Cu, net GND
- removed copper zone on B.Cu, net +3V3
- removed copper zone on In2.Cu, net GND
Other:
- outline, holes or cut-outs redrawn

Commit message: JoneyTech Interposer Board Ready For Fab
Routing:
- net /PERST#: track 0.00 -> 85.3 mm, vias 0 -> 2
- net /REFCLK_P: track 0.00 -> 77.7 mm
- net /REFCLK_N: track 0.00 -> 77.1 mm
- net /RX0_P: track 0.00 -> 75.2 mm
- net /RX0_N: track 0.00 -> 74.6 mm
- net /TX0_P: track 0.00 -> 72.7 mm
- net /TX0_N: track 0.00 -> 72.2 mm
- net /RX1_P: track 0.00 -> 70.2 mm
- net /RX1_N: track 0.00 -> 69.7 mm
- net /TX1_P: track 0.00 -> 67.7 mm
- net /TX1_N: track 0.00 -> 67.2 mm
- net /RX2_P: track 0.00 -> 65.2 mm
- net /RX2_N: track 0.00 -> 64.7 mm
- net /TX2_P: track 0.00 -> 62.8 mm
- net /TX2_N: track 0.00 -> 62.2 mm
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- added copper zone on B.Cu, net +3V3
- added copper zone on In2.Cu, net GND
- removed copper zone on In2.Cu, net +3V3

Commit message: JoneyTech Interposer Diff Pairs Skew Matched
Routing:
- net /RX3_N: track 59.7 -> 60.2 mm
- net /RX0_N: track 74.6 -> 75.1 mm
- net /TX3_N: track 57.2 -> 57.8 mm
- net /RX1_N: track 69.7 -> 70.2 mm
- net /REFCLK_N: track 77.1 -> 77.6 mm
- net /TX1_N: track 67.2 -> 67.7 mm
- net /RX2_N: track 64.7 -> 65.2 mm
- net /TX2_N: track 62.2 -> 62.7 mm
- net /TX0_N: track 72.2 -> 72.7 mm

Commit message: Fixed Hole Spacing on IOCrest Interposer
Also added clearance holes for heatsink push pins and grounding lug
Parts:
- added HS1: HSB30-373710, ThunderScope:SSKY_HSB30-373710_MountingHoles, F.Cu at (151.3, 70.1)
- added J11: 7793, ThunderScope:KEY_7792_ClearenceHoles, F.Cu at (185.0, 106.5)
Routing:
- net GND: vias 1191 -> 1187
Other:
- board text added: "Differential trace width is 0.17644 mm and spacing is 0.127mm target impedance is 85 Ohm differential and tolerance is 10% traces are on top copper and reference is on inner layer 1"
