File: Hardware/KiCad/Interposer_Board_IOCrest/Interposer_Board_IOCrest.kicad_pcb (KiCad board)
At the start: 4 copper layers, 122.5 x 99.5 mm, 6 parts, among them J1 M.2 Key M, J2 M.2 Key M

Commit message: IOCrest Interposer WIP
Routing:
- net /PERST#: track 0.00 -> 99.4 mm, vias 0 -> 2
- net /REFCLK_P: track 0.00 -> 91.8 mm
- net /REFCLK_N: track 0.00 -> 91.3 mm
- net /RX0_P: track 0.00 -> 89.3 mm
- net /RX0_N: track 0.00 -> 88.8 mm
- net /TX0_P: track 0.00 -> 86.8 mm
- net /TX0_N: track 0.00 -> 86.3 mm
- net /RX1_P: track 0.00 -> 84.3 mm
- net /RX1_N: track 0.00 -> 83.8 mm
- net /TX1_P: track 0.00 -> 81.9 mm
- net /TX1_N: track 0.00 -> 81.3 mm
- net /RX2_P: track 0.00 -> 79.4 mm
- net /RX2_N: track 0.00 -> 78.8 mm
- net /TX2_P: track 0.00 -> 76.9 mm
- net /TX2_N: track 0.00 -> 76.4 mm
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
Commit message: IOCrest Interposer Ready to Fab
Routing:
- net GND: vias 1245 -> 1249

Commit message: Fixed Hole Spacing on IOCrest Interposer
Also added clearance holes for heatsink push pins and grounding lug
Parts:
- added HS1: HSB30-373710, ThunderScope:SSKY_HSB30-373710_MountingHoles, F.Cu at (151.3, 70.1)
- added J11: 7793, ThunderScope:KEY_7792_ClearenceHoles, F.Cu at (185.0, 106.5)
- moved J1 0.90 mm to (104.9, 51.2)
- moved H1 0.10 mm to (179.7, 62.3)
Routing:
- net /PERST#: track 99.8 -> 99.0 mm
- net GND: vias 1249 -> 1235
Other:
- outline, holes or cut-outs redrawn
- board text added: "Differential trace width is 0.17644 mm and spacing is 0.127mm target impedance is 85 Ohm differential and tolerance is 10% traces are on top copper and reference is on inner layer 1"

Commit message: Updated Interposer Boards
Used PCBway's trace/space on diff pairs, fixed bottom soldermask on edge connectors, and board outline tweaks
Parts:
- removed J11: 7793, ThunderScope:KEY_7792_ClearenceHoles
- moved J1 0.10 mm to (105.0, 51.2)
- moved H1 0.10 mm to (179.8, 62.3)
Routing:
- net /TX1_N: track 81.8 -> 80.8 mm
- net /TX1_P: track 81.9 -> 80.8 mm
- net /RX1_N: track 84.3 -> 83.3 mm
- net /RX1_P: track 84.3 -> 83.3 mm
- net /RX3_N: track 74.4 -> 73.4 mm
- net /TX0_N: track 86.8 -> 85.8 mm
- net /RX3_P: track 74.4 -> 73.4 mm
- net /TX0_P: track 86.8 -> 85.8 mm
- net /RX0_N: track 89.3 -> 88.3 mm
- net /TX2_N: track 76.8 -> 75.9 mm
- net /TX3_N: track 71.9 -> 70.9 mm
- net /RX0_P: track 89.3 -> 88.3 mm
- net /TX3_P: track 71.9 -> 70.9 mm
- net /TX2_P: track 76.9 -> 75.9 mm
- net /REFCLK_N: track 91.8 -> 90.8 mm
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Other:
- outline, holes or cut-outs redrawn
- board text added: "Differential trace width is 0.188 mm and spacing is 0.1397mm target impedance is 85 Ohm differential and tolerance is 10% traces are on top copper and reference is on inner layer 1"
- board text removed: "Differential trace width is 0.17644 mm and spacing is 0.127mm target impedance is 85 Ohm differential and tolerance is 10% traces are on top copper and reference is on inner layer 1"
