File: Hardware/KiCad/TS_Back_Endcap/TS_Back_Endcap.kicad_sch (KiCad schematic)
At the start: 8 parts

Commit message: Swapped pinout of fan pads
Connections:
- net GND: now also TP1.2; no longer TP1.1
- net VUSB: now also TP1.1; no longer TP1.2
Other:
- moved on the sheet: TP1
Changed lines of the file:
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@@
 (kicad_sch
-	(version 20241209)
+	(version 20250114)
 	(generator "eeschema")
 	(generator_version "9.0")
@@
 	(symbol
 		(lib_id "ThunderScope:009155002852006_PCB_Pads")
-		(at 116.84 96.52 180)
+		(at 116.84 93.98 0)
+		(mirror y)
 		(unit 1)
 		(exclude_from_sim no)
@@
 		)
 		(property "Footprint" "ThunderScope:009155002852006_PCB_Pads"
-			(at 116.84 96.52 0)
+			(at 116.84 93.98 0)
 			(effects
 				(font
@@
 		)
 		(property "Datasheet" ""
-			(at 116.84 96.52 0)
+			(at 116.84 93.98 0)
 			(effects
 				(font
@@
 		)
 		(property "Description" ""
-			(at 116.84 96.52 0)
-			(effects
-				(font
+			(at 116.84 93.98 0)
+			(effects
+				(font
