File: Hardware/KiCad/Thunderscope_Rev5.1/FPGA.kicad_sch (KiCad schematic)
At the start: 29 parts, among them J12 009155002852006, J13 009155002852006, J5 2.54mm 6 Pin TH, J9 F300-1B7H1-11036-E100, U1 SN74LVC1G17, U10 FIN1019MTCX, Y2 25MHz

Commit message: Fixed #310
Swapped Labels, Swapped P15 and P14, Swapped TP42 and TP25. No Copper Change
Changed lines of the file:
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@@
+		)
+	)
+	(hierarchical_label "PGA_SCLK"
+		(shape output)
+		(at 144.78 55.88 0)
+		(effects
+			(font
+				(size 1.27 1.27)
+			)
+			(justify left)
 		)
 	)
@@
 		)
 	)
+	(hierarchical_label "PGA_SDIO"
+		(shape output)
+		(at 144.78 58.42 0)
+		(effects
+			(font
+				(size 1.27 1.27)
+			)
+			(justify left)
+		)
+	)
 	(hierarchical_label "TERM_[4..1]"
 		(shape output)
@@
 		)
 	)
-	(hierarchical_label "PGA_SCLK"
-		(shape output)
-		(at 144.78 58.42 0)
-		(effects
-			(font
-				(size 1.27 1.27)
-			)
-			(justify left)
-		)
-	)
 	(hierarchical_label "FE_EN"
 		(shape output)
@@
 		(effects
 			(font
-				(size 1.27 1.27)
-			)
-			(justify left)
-		)
-	)
-	(hierarchical_label "PGA_SDIO"
-		(shape output)
-		(at 144.78 55.88 0)
-		(effects
-			(font
