File: Hardware/KiCad/Thunderscope_Rev5.1/FE_Channel.kicad_sch (KiCad schematic)
At the start: 93 parts, among them J1002_4 BNC, J3_4 UFL, J4_4 UFL, K1000_4 FTR-B3SA4.5Z, K1001_4 FTR-B3SA4.5Z, Q1002_4 DMN62D0UW, Q1003_4 DMN62D0UW, Q1004_4 DMN62D0UW, U1008_4 LMH6518, U1009_4 BUF802, U1010_4 TS12A4516, U1011_4 OPA140AIDR

Commit message: Swapped Relay PNs, Implements #337
Also removed ground pour from CH1
Parts:
- K1000_4, K1001_4: value FTR-B3SA4.5Z -> UD2-4.5NUN-L; footprint Thunderscope_Rev5:FUJ_FTR-B3SA -> Thunderscope_Rev5:KEMET_UD2-4.5NUN-L; symbol Thunderscope_Rev5:RELAY DPDT-NO FTR-B3SA4.5Z -> Thunderscope_Rev5:RELAY DPDT-NO UD2-4.5NUN-L; MANUFACTURER Fujitsu -> KEMET; MANUFACTURER PART NUMBER FTR-B3SA4.5Z -> UD2-4.5NUN-L; SUPPLIER PART NUMBER 1 817-FTR-B3SA4.5Z -> 80-UD2-4.5NUN-L
Changed lines of the file:
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@@
 	)
 	(symbol
-		(lib_id "Thunderscope_Rev5:RELAY DPDT-NO FTR-B3SA4.5Z")
+		(lib_id "Thunderscope_Rev5:RELAY DPDT-NO UD2-4.5NUN-L")
 		(at 81.28 35.56 0)
 		(unit 1)
@@
 			)
 		)
-		(property "Value" "FTR-B3SA4.5Z"
+		(property "Value" "UD2-4.5NUN-L"
 			(at 81.28 35.56 0)
 			(effects
@@
 			)
 		)
-		(property "Footprint" "Thunderscope_Rev5:FUJ_FTR-B3SA"
+		(property "Footprint" "Thunderscope_Rev5:KEMET_UD2-4.5NUN-L"
 			(at 81.28 35.56 0)
 			(effects
@@
 			)
 		)
-		(property "MANUFACTURER" "Fujitsu"
+		(property "MANUFACTURER" "KEMET"
 			(at 81.28 35.56 0)
 			(effects
@@
 			)
 		)
-		(property "MANUFACTURER PART NUMBER" "FTR-B3SA4.5Z"
+		(property "MANUFACTURER PART NUMBER" "UD2-4.5NUN-L"
 			(at 81.28 35.56 0)
 			(effects
@@
 			)
 		)
-		(property "SUPPLIER PART NUMBER 1" "817-FTR-B3SA4.5Z"
+		(property "SUPPLIER PART NUMBER 1" "80-UD2-4.5NUN-L"
 			(at 81.28 35.56 0)
 			(effects
@@
 	)
 	(symbol
-		(lib_id "Thunderscope_Rev5:RELAY DPDT-NO FTR-B3SA4.5Z")
+		(lib_id "Thunderscope_Rev5:RELAY DPDT-NO UD2-4.5NUN-L")
 		(at 81.28 73.66 0)
 		(unit 3)
@@
 			)
 		)
-		(property "Value" "FTR-B3SA4.5Z"
+		(property "Value" "UD2-4.5NUN-L"
 			(at 81.28 77.47 0)
 			(effects
@@
 			)
 		)
-		(property "Footprint" "Thunderscope_Rev5:FUJ_FTR-B3SA"
+		(property "Footprint" "Thunderscope_Rev5:KEMET_UD2-4.5NUN-L"
 			(at 81.28 73.66 0)
 			(effects
@@
 			)
 		)
-		(property "MANUFACTURER" "Fujitsu"
+		(property "MANUFACTURER" "KEMET"
 			(at 81.28 73.66 0)
 			(effects
@@
 			)
 		)
-		(property "MANUFACTURER PART NUMBER" "FTR-B3SA4.5Z"
+		(property "MANUFACTURER PART NUMBER" "UD2-4.5NUN-L"
 			(at 81.28 73.66 0)
 			(effects
@@
 			)
 		)
-		(property "SUPPLIER PART NUMBER 1" "817-FTR-B3SA4.5Z"
+		(property "SUPPLIER PART NUMBER 1" "80-UD2-4.5NUN-L"
 			(at 81.28 73.66 0)
 			(effects
@@
 	)
 	(symbol
-		(lib_id "Thunderscope_Rev5:RELAY DPDT-NO FTR-B3SA4.5Z")
+		(lib_id "Thunderscope_Rev5:RELAY DPDT-NO UD2-4.5NUN-L")
 		(at 187.96 35.56 0)
 		(unit 2)
@@
 			)
 		)
-		(property "Value" "FTR-B3SA4.5Z"
+		(property "Value" "UD2-4.5NUN-L"
 			(at 187.96 35.56 0)
 			(effects
@@
 			)
 		)
-		(property "Footprint" "Thunderscope_Rev5:FUJ_FTR-B3SA"
+		(property "Footprint" "Thunderscope_Rev5:KEMET_UD2-4.5NUN-L"
 			(at 187.96 35.56 0)
 			(effects
@@
 			)
 		)
-		(property "MANUFACTURER" "Fujitsu"
+		(property "MANUFACTURER" "KEMET"
 			(at 187.96 35.56 0)
 			(effects
@@
 			)
 		)
-		(property "MANUFACTURER PART NUMBER" "FTR-B3SA4.5Z"
+		(property "MANUFACTURER PART NUMBER" "UD2-4.5NUN-L"
 			(at 187.96 35.56 0)
 			(effects
@@
 			)
 		)
-		(property "SUPPLIER PART NUMBER 1" "817-FTR-B3SA4.5Z"
+		(property "SUPPLIER PART NUMBER 1" "80-UD2-4.5NUN-L"
 			(at 187.96 35.56 0)
 			(effects
@@
 	)
 	(symbol
-		(lib_id "Thunderscope_Rev5:RELAY DPDT-NO FTR-B3SA4.5Z")
+		(lib_id "Thunderscope_Rev5:RELAY DPDT-NO UD2-4.5NUN-L")
 		(at 226.06 73.66 0)
 		(unit 3)
@@
 			)
 		)
-		(property "Value" "FTR-B3SA4.5Z"
+		(property "Value" "UD2-4.5NUN-L"
 			(at 226.06 77.47 0)
 			(effects
@@
 			)
 		)
-		(property "Footprint" "Thunderscope_Rev5:FUJ_FTR-B3SA"
+		(property "Footprint" "Thunderscope_Rev5:KEMET_UD2-4.5NUN-L"
 			(at 226.06 73.66 0)
 			(effects
@@
 			)
 		)
-		(property "MANUFACTURER" "Fujitsu"
+		(property "MANUFACTURER" "KEMET"
 			(at 226.06 73.66 0)
 			(effects
@@
 			)
 		)
-		(property "MANUFACTURER PART NUMBER" "FTR-B3SA4.5Z"
+		(property "MANUFACTURER PART NUMBER" "UD2-4.5NUN-L"
 			(at 226.06 73.66 0)
 			(effects
@@
 			)
 		)
-		(property "SUPPLIER PART NUMBER 1" "817-FTR-B3SA4.5Z"
+		(property "SUPPLIER PART NUMBER 1" "80-UD2-4.5NUN-L"
 			(at 226.06 73.66 0)
 			(effects
@@
 	)
 	(symbol
-		(lib_id "Thunderscope_Rev5:RELAY DPDT-NO FTR-B3SA4.5Z")
+		(lib_id "Thunderscope_Rev5:RELAY DPDT-NO UD2-4.5NUN-L")
 		(at 337.82 35.56 0)
 		(unit 2)
@@
 			)
 		)
-		(property "Value" "FTR-B3SA4.5Z"
+		(property "Value" "UD2-4.5NUN-L"
 			(at 337.82 35.56 0)
 			(effects
@@
 			)
 		)
-		(property "Footprint" "Thunderscope_Rev5:FUJ_FTR-B3SA"
+		(property "Footprint" "Thunderscope_Rev5:KEMET_UD2-4.5NUN-L"
 			(at 337.82 35.56 0)
 			(effects
@@
 			)
 		)
-		(property "MANUFACTURER" "Fujitsu"
+		(property "MANUFACTURER" "KEMET"
 			(at 337.82 35.56 0)
 			(effects
@@
 			)
 		)
-		(property "MANUFACTURER PART NUMBER" "FTR-B3SA4.5Z"
+		(property "MANUFACTURER PART NUMBER" "UD2-4.5NUN-L"
 			(at 337.82 35.56 0)
 			(effects
@@
 			)
 		)
-		(property "SUPPLIER PART NUMBER 1" "817-FTR-B3SA4.5Z"
+		(property "SUPPLIER PART NUMBER 1" "80-UD2-4.5NUN-L"
 			(at 337.82 35.56 0)
 			(effects
@@
 	)
 	(symbol
-		(lib_id "Thunderscope_Rev5:RELAY DPDT-NO FTR-B3SA4.5Z")
+		(lib_id "Thunderscope_Rev5:RELAY DPDT-NO UD2-4.5NUN-L")
 		(at 226.06 35.56 0)
 		(unit 1)
@@
 			)
 		)
-		(property "Value" "FTR-B3SA4.5Z"
+		(property "Value" "UD2-4.5NUN-L"
 			(at 226.06 35.56 0)
 			(effects
@@
 			)
 		)
-		(property "Footprint" "Thunderscope_Rev5:FUJ_FTR-B3SA"
+		(property "Footprint" "Thunderscope_Rev5:KEMET_UD2-4.5NUN-L"
 			(at 226.06 35.56 0)
 			(effects
@@
 			)
 		)
-		(property "MANUFACTURER" "Fujitsu"
+		(property "MANUFACTURER" "KEMET"
 			(at 226.06 35.56 0)
 			(effects
@@
 			)
 		)
-		(property "MANUFACTURER PART NUMBER" "FTR-B3SA4.5Z"
+		(property "MANUFACTURER PART NUMBER" "UD2-4.5NUN-L"
 			(at 226.06 35.56 0)
 			(effects
@@
 			)
 		)
-		(property "SUPPLIER PART NUMBER 1" "817-FTR-B3SA4.5Z"
+		(property "SUPPLIER PART NUMBER 1" "80-UD2-4.5NUN-L"
 			(at 226.06 35.56 0)
 			(effects

Commit message: Changed Relay Caps to 22uF 0805 as per #338
Parts:
- C1026_4, C1027_4, C1028_4, C1029_4: value 10uF -> 22uF; footprint Thunderscope_Rev5:GEN_C_0603 -> Thunderscope_Rev5:GEN_C_0805; symbol Thunderscope_Rev5:CAP 10uF 25V X5R 0603 -> Thunderscope_Rev5:CAP 22uF 25V X5R 0805; HOUSE PART NUMBER (none) -> C-22uF-0805-002; MANUFACTURER PART NUMBER GRM188R61E106MA73D -> GRM21BR61E226ME44L; PACKAGE 0402 -> 0805; SUPPLIER PART NUMBER 1 81-GRM188R61E106MA3D -> 81-GRM21BR61E226ME4L
Changed lines of the file:
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@@
 	)
 	(symbol
-		(lib_id "Thunderscope_Rev5:CAP 10uF 25V X5R 0603")
+		(lib_id "Thunderscope_Rev5:CAP 22uF 25V X5R 0805")
 		(at 58.42 81.28 0)
 		(unit 1)
@@
 			)
 		)
-		(property "Value" "10uF"
+		(property "Value" "22uF"
 			(at 60.96 83.82 0)
 			(effects
@@
 			)
 		)
-		(property "Footprint" "Thunderscope_Rev5:GEN_C_0603"
+		(property "Footprint" "Thunderscope_Rev5:GEN_C_0805"
 			(at 58.42 81.28 0)
 			(effects
@@
 			)
 		)
-		(property "PACKAGE" "0402"
+		(property "PACKAGE" "0805"
 			(at 41.292 92.71 0)
 			(effects
@@
 			)
 		)
-		(property "SUPPLIER PART NUMBER 1" "81-GRM188R61E106MA3D"
+		(property "SUPPLIER PART NUMBER 1" "81-GRM21BR61E226ME4L"
 			(at 56.166 75.692 0)
 			(effects
@@
 			)
 		)
-		(property "HOUSE PART NUMBER" ""
+		(property "HOUSE PART NUMBER" "C-22uF-0805-002"
 			(at 56.166 75.692 0)
 			(effects
@@
 			)
 		)
-		(property "MANUFACTURER PART NUMBER" "GRM188R61E106MA73D"
+		(property "MANUFACTURER PART NUMBER" "GRM21BR61E226ME44L"
 			(at 56.166 75.692 0)
 			(effects
@@
 	)
 	(symbol
-		(lib_id "Thunderscope_Rev5:CAP 10uF 25V X5R 0603")
+		(lib_id "Thunderscope_Rev5:CAP 22uF 25V X5R 0805")
 		(at 187.96 81.28 0)
 		(unit 1)
@@
 			)
 		)
-		(property "Value" "10uF"
+		(property "Value" "22uF"
 			(at 190.5 83.82 0)
 			(effects
@@
 			)
 		)
-		(property "Footprint" "Thunderscope_Rev5:GEN_C_0603"
+		(property "Footprint" "Thunderscope_Rev5:GEN_C_0805"
 			(at 187.96 81.28 0)
 			(effects
@@
 			)
 		)
-		(property "PACKAGE" "0402"
+		(property "PACKAGE" "0805"
 			(at 170.832 92.71 0)
 			(effects
@@
 			)
 		)
-		(property "SUPPLIER PART NUMBER 1" "81-GRM188R61E106MA3D"
+		(property "SUPPLIER PART NUMBER 1" "81-GRM21BR61E226ME4L"
 			(at 185.706 75.692 0)
 			(effects
@@
 			)
 		)
-		(property "HOUSE PART NUMBER" ""
+		(property "HOUSE PART NUMBER" "C-22uF-0805-002"
 			(at 185.706 75.692 0)
 			(effects
@@
 			)
 		)
-		(property "MANUFACTURER PART NUMBER" "GRM188R61E106MA73D"
+		(property "MANUFACTURER PART NUMBER" "GRM21BR61E226ME44L"
 			(at 185.706 75.692 0)
 			(effects
@@
 	)
 	(symbol
-		(lib_id "Thunderscope_Rev5:CAP 10uF 25V X5R 0603")
+		(lib_id "Thunderscope_Rev5:CAP 22uF 25V X5R 0805")
 		(at 203.2 81.28 0)
 		(unit 1)
@@
 			)
 		)
-		(property "Value" "10uF"
+		(property "Value" "22uF"
 			(at 205.74 83.82 0)
 			(effects
@@
 			)
 		)
-		(property "Footprint" "Thunderscope_Rev5:GEN_C_0603"
+		(property "Footprint" "Thunderscope_Rev5:GEN_C_0805"
 			(at 203.2 81.28 0)
 			(effects
@@
 			)
 		)
-		(property "PACKAGE" "0402"
+		(property "PACKAGE" "0805"
 			(at 186.072 92.71 0)
 			(effects
@@
 			)
 		)
-		(property "SUPPLIER PART NUMBER 1" "81-GRM188R61E106MA3D"
+		(property "SUPPLIER PART NUMBER 1" "81-GRM21BR61E226ME4L"
 			(at 200.946 75.692 0)
 			(effects
@@
 			)
 		)
-		(property "HOUSE PART NUMBER" ""
+		(property "HOUSE PART NUMBER" "C-22uF-0805-002"
 			(at 200.946 75.692 0)
 			(effects
@@
 			)
 		)
-		(property "MANUFACTURER PART NUMBER" "GRM188R61E106MA73D"
+		(property "MANUFACTURER PART NUMBER" "GRM21BR61E226ME44L"
 			(at 200.946 75.692 0)
 			(effects
@@
 	)
 	(symbol
-		(lib_id "Thunderscope_Rev5:CAP 10uF 25V X5R 0603")
+		(lib_id "Thunderscope_Rev5:CAP 22uF 25V X5R 0805")
 		(at 43.18 81.28 0)
 		(unit 1)
@@
 			)
 		)
-		(property "Value" "10uF"
+		(property "Value" "22uF"
 			(at 45.72 83.82 0)
 			(effects
@@
 			)
 		)
-		(property "Footprint" "Thunderscope_Rev5:GEN_C_0603"
+		(property "Footprint" "Thunderscope_Rev5:GEN_C_0805"
 			(at 43.18 81.28 0)
 			(effects
@@
 			)
 		)
-		(property "PACKAGE" "0402"
+		(property "PACKAGE" "0805"
 			(at 26.052 92.71 0)
 			(effects
@@
 			)
 		)
-		(property "SUPPLIER PART NUMBER 1" "81-GRM188R61E106MA3D"
+		(property "SUPPLIER PART NUMBER 1" "81-GRM21BR61E226ME4L"
 			(at 40.926 75.692 0)
 			(effects
@@
 			)
 		)
-		(property "HOUSE PART NUMBER" ""
+		(property "HOUSE PART NUMBER" "C-22uF-0805-002"
 			(at 40.926 75.692 0)
 			(effects
@@
 			)
 		)
-		(property "MANUFACTURER PART NUMBER" "GRM188R61E106MA73D"
+		(property "MANUFACTURER PART NUMBER" "GRM21BR61E226ME44L"
 			(at 40.926 75.692 0)
 			(effects

Commit message: Changed trimpot to 2kOhm, as per #313
Parts:
- R1049_4: value 5K TRIMPOT -> 2K TRIMPOT; symbol Thunderscope_Rev5:TRIMMER 5K OHM 0.1W J LEAD TOP -> Thunderscope_Rev5:TRIMMER 2K OHM 0.1W J LEAD TOP; MANUFACTURER PART NUMBER TC33X-2-502E -> TC33X-2-202E; SUPPLIER PART NUMBER 1 652-TC33X-2-502E -> 652-TC33X-2-202E
Changed lines of the file:
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@@
 	)
 	(symbol
-		(lib_id "Thunderscope_Rev5:TRIMMER 5K OHM 0.1W J LEAD TOP")
+		(lib_id "Thunderscope_Rev5:TRIMMER 2K OHM 0.1W J LEAD TOP")
 		(at 248.92 215.9 0)
 		(unit 1)
@@
 			)
 		)
-		(property "Value" "5K TRIMPOT"
+		(property "Value" "2K TRIMPOT"
 			(at 249.976 217.98 0)
 			(effects
@@
 			)
 		)
-		(property "SUPPLIER PART NUMBER 1" "652-TC33X-2-502E"
+		(property "SUPPLIER PART NUMBER 1" "652-TC33X-2-202E"
 			(at 243.332 210.312 0)
 			(effects
@@
 			)
 		)
-		(property "MANUFACTURER PART NUMBER" "TC33X-2-502E"
+		(property "MANUFACTURER PART NUMBER" "TC33X-2-202E"
 			(at 243.332 210.312 0)
 			(effects

Commit message: Schematic changes for #339
Parts:
- added R1001_4: 9.09, Thunderscope_Rev5:GEN_R_0402, symbol Thunderscope_Rev5:RES 9.09 OHM 1% 1/10W 0402
- added R1002_4: 300K, Thunderscope_Rev5:GEN_R_0402, symbol Thunderscope_Rev5:RES 300K OHM 1% 1/10W 0402
- C1021_4: value 8pF -> 12pF; symbol Thunderscope_Rev5:CAP 8pF 50V C0G 0402 -> Thunderscope_Rev5:CAP 12pF 50V C0G 0402; MANUFACTURER PART NUMBER CBR04C809B5GAC -> CBR04C120F5GAC; SUPPLIER PART NUMBER 1 80-CBR04C809B5GAC -> 80-CBR04C120F5G
- C1022_4: value 5pF -> DNP; footprint Thunderscope_Rev5:GEN_C_0603 -> Thunderscope_Rev5:GEN_C_0402; symbol Thunderscope_Rev5:CAP 5pF 250V C0G 0603 -> Thunderscope_Rev5:CAP DNP 0402; MANUFACTURER KEMET -> (none); MANUFACTURER PART NUMBER CBR06C509BAGAC -> (none); PACKAGE 0603 -> 0402; SUPPLIER 1 Mouser -> (none); SUPPLIER PART NUMBER 1 80-CBR06C509BAGAC -> (none); VOLTAGE RATING 250V -> (none); now not fitted; now left out of the parts list
- C1023_4: value 2.4pF -> 4.3pF; symbol Thunderscope_Rev5:CAP 2.4pF 250V C0G 0603 -> Thunderscope_Rev5:CAP 4.3pF 250V C0G 0603; MANUFACTURER PART NUMBER CBR06C249BAGAC -> CBR06C439BAGAC; SUPPLIER PART NUMBER 1 80-CBR06C249BAGAC -> 80-CBR06C439BAGAC
- C1024_4: value 2.4pF -> 1.5pF; symbol Thunderscope_Rev5:CAP 2.4pF 250V C0G 0603 -> Thunderscope_Rev5:CAP 1.5pF 250V C0G 0603; MANUFACTURER PART NUMBER CBR06C249BAGAC -> CBR06C159BAGAC; SUPPLIER PART NUMBER 1 80-CBR06C249BAGAC -> 80-CBR06C159BAG
- C1025_4: value 12pF -> 7pF; symbol Thunderscope_Rev5:CAP 12pF 50V C0G 0402 -> Thunderscope_Rev5:CAP 7pF 50V C0G 0402; MANUFACTURER PART NUMBER CBR04C120F5GAC -> CBR04C709B5GAC; SUPPLIER PART NUMBER 1 80-CBR04C120F5G -> 80-CBR04C709B5GAC
- R1021_4: value 30 -> 15; symbol Thunderscope_Rev5:RES 30 OHM 1% 1/3W 0603 -> Thunderscope_Rev5:RES 15 OHM 1% 1/3W 0603; MANUFACTURER PART NUMBER SG73P1JTTD30R0F -> SG73P1JTTD15R0F; SUPPLIER PART NUMBER 1 660-SG73P1JTTD30R0F -> 660-SG73P1JTTD15R0F
- R1022_4: value 10 -> 22; symbol Thunderscope_Rev5:RES 10 OHM 1% 1/3W 0603 -> Thunderscope_Rev5:RES 22 OHM 1% 1/3W 0603; MANUFACTURER PART NUMBER SG73P1JTTD10R0F -> SG73P1JTTD22R0F; SUPPLIER PART NUMBER 1 660-SG73P1JTTD10R0F -> 660-SG73P1JTTD22R0F
- R1024_4: value 976k -> 680K; footprint Thunderscope_Rev5:GEN_R_0603 -> Thunderscope_Rev5:GEN_R_0402; symbol Thunderscope_Rev5:RES 976k OHM 1% 1/10W 0603 -> Thunderscope_Rev5:RES 680K OHM 1% 1/16W 0402; MANUFACTURER KOA Speer -> Yageo; MANUFACTURER PART NUMBER RK73H1JTTD9763F -> RC0402FR-07681KL; PACKAGE 0603 -> 0402; SUPPLIER PART NUMBER 1 660-RK73H1JTTD9763F -> 603-RC0402FR-07680KL
Connections:
- net ATTEN_50X_R: now also C1023_4.2, R1001_4.2; no longer C1021_4.2, C1024_4.1, C1059_4.1, K1001_4.7, R1026_4.2
- net GND: now also C1022_4.1; no longer C1022_4.2
- net TERM_1M_R: now also C1022_4.2; no longer C1022_4.1
- net TERM_50Z: now also R1021_4.2; no longer R1021_4.1
- net TERM_50Z_R: now also R1021_4.1; no longer R1021_4.2
- removed net ATTEN_50X: C1023_4.2, K1001_4.2, R1024_4.1
- new net: R1002_4.2, R1024_4.1
- new net ATTEN_50X_IN: K1001_4.2, R1001_4.1
- new net ATTEN_50X_OUT: C1021_4.2, C1024_4.1, C1059_4.1, K1001_4.7, R1002_4.1, R1026_4.2
Other:
- note removed: "(GRM21B5C2A223JA01L)"
- note removed: "DONE: Change 8pF cap to 5pF"
- note removed: "DONE: Change Coupling Cap to 0805 C0G"
- note removed: "DONE: Change Relays to 4.5V Parts as we are now powering them w/ +VUSB"
- note removed: "DONE: Change second 12pF to something lower and add trimcap in parallel"
- note removed: "DONE: Remove FB4 and FB6"
- note removed: "DONE: Revert back to non-latched relays to avoid indeterminate state when powered off"
- note removed: "DONE: Revert to Mechanical Trimpot"
- note removed: "DONE: add cap + resistor across 30 Ohm resistor in 50Z path"
- note removed: "DONE: change to 1.2nF"
- note removed: "DONE: change to 220pF"
- note removed: "DONE: change to 35.7k"
- note removed: "DONE: change to 50 ohm 0508"
- note removed: "DONE: change to 50Ohm"
- note removed: "DONE: change upper R to 976k"
- note removed: "DONE: connect CLL directly to GND"
- note removed: "DONE: remove ferrites on +/-5V to make planes easier to keep away from signal"
- note removed: "WK73R2ATTD49R9F"
- moved on the sheet: C1021_4, C1023_4, C1024_4, C1025_4, C1026_4, C1027_4, C1028_4, C1029_4, C1058_4, C1059_4, D1000_4, D1001_4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

Commit message: Finished layout for #339
Also added new attenuator gnd cutouts with fewer cutouts on CH3 and no cutouts on CH4
Parts:
- C1022_4: footprint Thunderscope_Rev5:GEN_C_0402 -> Thunderscope_Rev5:GEN_C_0603; symbol Thunderscope_Rev5:CAP DNP 0402 -> Thunderscope_Rev5:CAP DNP 0603; PACKAGE 0402 -> 0603
- C1024_4: footprint Thunderscope_Rev5:GEN_C_0603 -> Thunderscope_Rev5:GEN_C_0402; symbol Thunderscope_Rev5:CAP 1.5pF 250V C0G 0603 -> Thunderscope_Rev5:CAP 1.5pF 50V C0G 0402; MANUFACTURER PART NUMBER CBR06C159BAGAC -> CBR04C159A5GAC; PACKAGE 0603 -> 0402; SUPPLIER PART NUMBER 1 80-CBR06C159BAG -> 80-CBR04C159A5GAC; VOLTAGE RATING 250V -> 50V
Changed lines of the file:
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@@
 	)
 	(symbol
-		(lib_id "Thunderscope_Rev5:CAP 1.5pF 250V C0G 0603")
+		(lib_id "Thunderscope_Rev5:CAP 1.5pF 50V C0G 0402")
 		(at 284.48 43.18 0)
 		(unit 1)
@@
 			)
 		)
-		(property "Footprint" "Thunderscope_Rev5:GEN_C_0603"
+		(property "Footprint" "Thunderscope_Rev5:GEN_C_0402"
 			(at 284.48 43.18 0)
 			(effects
@@
 			)
 		)
-		(property "PACKAGE" "0603"
+		(property "PACKAGE" "0402"
 			(at 281.94 52.07 0)
 			(effects
@@
 			)
 		)
-		(property "SUPPLIER PART NUMBER 1" "80-CBR06C159BAG"
+		(property "SUPPLIER PART NUMBER 1" "80-CBR04C159A5GAC"
 			(at 278.892 40.926 0)
 			(effects
@@
 			)
 		)
-		(property "VOLTAGE RATING" "250V"
+		(property "VOLTAGE RATING" "50V"
 			(at 281.94 54.61 0)
 			(effects
@@
 			)
 		)
-		(property "MANUFACTURER PART NUMBER" "CBR06C159BAGAC"
+		(property "MANUFACTURER PART NUMBER" "CBR04C159A5GAC"
 			(at 282.226 37.592 0)
 			(effects
@@
 	)
 	(symbol
-		(lib_id "Thunderscope_Rev5:CAP DNP 0402")
+		(lib_id "Thunderscope_Rev5:CAP DNP 0603")
 		(at 101.6 45.72 0)
 		(unit 1)
@@
 			)
 		)
-		(property "Footprint" "Thunderscope_Rev5:GEN_C_0402"
+		(property "Footprint" "Thunderscope_Rev5:GEN_C_0603"
 			(at 101.6 45.72 0)
 			(effects
@@
 			)
 		)
-		(property "PACKAGE" "0402"
+		(property "PACKAGE" "0603"
 			(at 99.346 40.132 0)
 			(effects

Commit message: Schematic Changes for #340
Parts:
- removed Q1004_4: DMN62D0UW, Thunderscope_Rev5:GEN_SOT_323, symbol Thunderscope_Rev5:NMOS DMN62D0UW
- removed R1050_4, R1051_4: 10K, Thunderscope_Rev5:GEN_R_0402, symbol Thunderscope_Rev5:RES 10K OHM 1% 1/10W 0402
- removed U1010_4: TS12A4516, Thunderscope_Rev5:GEN_SOT23_5_950_2900X1600X1450, symbol Thunderscope_Rev5:IC SWITCH SPST TS12A4516DBVR
- added C1035_?: 27pF, Thunderscope_Rev5:GEN_C_0402, symbol Thunderscope_Rev5:CAP 27pF 50V C0G 0402
- added C?: 150pF, Thunderscope_Rev5:GEN_C_0402, symbol Thunderscope_Rev5:CAP 150pF 50V C0G 0402
- added R1047_?: 10M, Thunderscope_Rev5:GEN_R_0603, symbol Thunderscope_Rev5:RES 10M OHM 1% 1/10W 0603
- added U?: TMUX4053, Thunderscope_Rev5:TI_TSOT-23-16_DYY0016A, symbol Thunderscope_Rev5:IC SWITCH 3X SPDT TMUX4053
- C1030_4: value 1.2nF -> 1nF; symbol Thunderscope_Rev5:CAP 1.2nF 100V C0G 0603 -> Thunderscope_Rev5:CAP 1nF 100V C0G 0603; MANUFACTURER PART NUMBER GCM1885C2A122FA16D -> GCM1885C2A102FA16D; SUPPLIER PART NUMBER 1 81-GCM1885C2A122FA6D -> 81-GCM1885C2A102FA6D
- C1031_4: value 22nF -> 10nF; footprint Thunderscope_Rev5:GEN_C_0805 -> Thunderscope_Rev5:GEN_C_0603; symbol Thunderscope_Rev5:CAP 22nF 100V C0G 0805 -> Thunderscope_Rev5:CAP 10nF 50V C0G 0603; MANUFACTURER PART NUMBER GRM21B5C2A223JA01L -> GRM1885C1H103JA01J; PACKAGE 0805 -> 0603; SUPPLIER PART NUMBER 1 81-GRM21B5C2A223JA1L -> 81-GRM1885C1H103JA1J; VOLTAGE RATING 100V -> 50V
- C1035_4: value 220pF -> 100pF; symbol Thunderscope_Rev5:CAP 220pF 50V C0G 0402 -> Thunderscope_Rev5:CAP 100pF 50V C0G 0402; MANUFACTURER PART NUMBER GCM1555C1H221FA16J -> GCM1555C1H101FA16D; SUPPLIER PART NUMBER 1 81-GCM1555C1H221FA6J -> 81-GCM1555C1H101FA6D
- R1038_4: value 909k -> 10M; footprint Thunderscope_Rev5:GEN_R_0402 -> Thunderscope_Rev5:GEN_R_0603; symbol Thunderscope_Rev5:RES 909K OHM 1% 1/16W 0402 -> Thunderscope_Rev5:RES 10M OHM 1% 1/10W 0603; MANUFACTURER Yageo -> KOA Speer; MANUFACTURER PART NUMBER RC0402FR-07909KL -> RK73H1JTTD1005F; PACKAGE 0402 -> 0603; SUPPLIER PART NUMBER 1 603-RC0402FR-07909KL -> 660-RK73H1JTTD1005F
Connections:
- net +5V: now also U?.16 (VDD)
- net -5V: now also U?.7 (VSS)
- net DC_CPL: now also U?.10 (SEL2), U?.11 (SEL1), U?.9 (SEL3)
- net DC_FB: now also U?.15 (D2)
- net GND: now also R1047_?.2, U?.6 (~{EN}), U?.8 (GND)
- net OPA_OUT: now also U?.4 (D3)
- net SW_COM: no longer names the net of C1031_4.2, U1011_4.3 (+)
- net SW_COM: now also R1047_?.1, U?.13 (S1B); no longer R1047_4.1
- net SW_NO: no longer names the net of C1031_4.1, R1039_4.2
- net SW_NO: now also R1047_4.1, U?.14 (D1)
- new net: C1035_?.1, U?.5 (S3A)
- new net: C1035_?.2, U?.2 (S2A)
- new net: C?.2, U?.1 (S2B)
- new net: C?.1, U?.3 (S3B)
- no-connect marks 5 -> 6
Other:
- note added: "This cap is switched in during AC coupling"
- note added: "This cap is switched in during DC coupling"
- note removed: "80uA @ V+ and 80uA @ V-"
- moved on the sheet: C1030_4, C1031_4, C1035_4, C1044_4, C1045_4, C1046_4, C1047_4, C1048_4, C1049_4, C1050_4, C1052_4, C1053_4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
