File: Hardware/KiCad/Thunderscope_Rev5.1/FE_Channel.kicad_sch (KiCad schematic)
At the start: 95 parts, among them J1002_4 BNC, J3_4 UFL, J4_4 UFL, K1000_4 UD2-4.5NUN-L, K1001_4 UD2-4.5NUN-L, Q1002_4 DMN62D0UW, Q1003_4 DMN62D0UW, U1008_4 LMH6518, U1009_4 BUF802, U1011_4 OPA140AIDR

Commit message: Annotated Schematic Changes For #340
Parts:
- gave numbers to parts that had none: 4
Other:
- moved on the sheet: C1030_4
Changed lines of the file:
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@@
 	(wire
 		(pts
-			(xy 124.46 167.64) (xy 134.62 167.64)
+			(xy 127 167.64) (xy 134.62 167.64)
 		)
 		(stroke
@@
 	(wire
 		(pts
-			(xy 93.98 167.64) (xy 114.3 167.64)
+			(xy 93.98 167.64) (xy 116.84 167.64)
 		)
 		(stroke
@@
 		(on_board yes)
 		(dnp no)
-		(property "Reference" "R?"
+		(property "Reference" "R1003_4"
 			(at 76.2 193.04 0)
 			(effects
@@
 			(project "Thunderscope_Rev5.1"
 				(path "/031d3e2c-42e0-4016-8c32-579d45c83e09/02e7ff63-3631-4d05-9bcb-1390e77ff703"
-					(reference "R1047_?")
+					(reference "R1003_3")
 					(unit 1)
 				)
 				(path "/031d3e2c-42e0-4016-8c32-579d45c83e09/d4ceb53c-d7d3-49f3-84e4-450b713426dc"
-					(reference "R?")
+					(reference "R1003_4")
 					(unit 1)
 				)
 				(path "/031d3e2c-42e0-4016-8c32-579d45c83e09/da233e23-d1b0-4723-86d8-4ec9b143e851"
-					(reference "R1047_?")
+					(reference "R1003_2")
 					(unit 1)
 				)
 				(path "/031d3e2c-42e0-4016-8c32-579d45c83e09/f35774a1-d397-4f7e-9c64-3142469f9c73"
-					(reference "R1047_?")
+					(reference "R1003_1")
 					(unit 1)
 				)
@@
 		(on_board yes)
 		(dnp no)
-		(property "Reference" "C?"
+		(property "Reference" "C1001_4"
 			(at 78.74 232.41 90)
 			(effects
@@
 			(project "Thunderscope_Rev5.1"
 				(path "/031d3e2c-42e0-4016-8c32-579d45c83e09/02e7ff63-3631-4d05-9bcb-1390e77ff703"
-					(reference "C1035_?")
+					(reference "C1001_3")
 					(unit 1)
 				)
 				(path "/031d3e2c-42e0-4016-8c32-579d45c83e09/d4ceb53c-d7d3-49f3-84e4-450b713426dc"
-					(reference "C?")
+					(reference "C1001_4")
 					(unit 1)
 				)
 				(path "/031d3e2c-42e0-4016-8c32-579d45c83e09/da233e23-d1b0-4723-86d8-4ec9b143e851"
-					(reference "C1035_?")
+					(reference "C1001_2")
 					(unit 1)
 				)
 				(path "/031d3e2c-42e0-4016-8c32-579d45c83e09/f35774a1-d397-4f7e-9c64-3142469f9c73"
-					(reference "C1035_?")
+					(reference "C1001_1")
 					(unit 1)
 				)
@@
 	(symbol
 		(lib_id "Thunderscope_Rev5:CAP 1nF 100V C0G 0603")
-		(at 119.38 167.64 0)
+		(at 121.92 167.64 0)
 		(unit 1)
 		(exclude_from_sim no)
@@
 		(dnp no)
 		(property "Reference" "C1030_4"
-			(at 116.586 165.386 0)
+			(at 119.126 165.386 0)
 			(effects
 				(font
@@
 		)
 		(property "Value" "1nF"
-			(at 121.92 170.18 0)
+			(at 124.46 170.18 0)
 			(effects
 				(font
@@
 		)
 		(property "Footprint" "Thunderscope_Rev5:GEN_C_0603"
-			(at 119.38 167.64 0)
+			(at 121.92 167.64 0)
 			(effects
 				(font
@@
 		)
 		(property "Datasheet" ""
-			(at 119.38 167.64 0)
+			(at 121.92 167.64 0)
 			(effects
 				(font
@@
 		)
 		(property "Description" ""
-			(at 119.38 167.64 0)
+			(at 121.92 167.64 0)
 			(effects
 				(font
@@
 		)
 		(property "PACKAGE" "0603"
-			(at 113.792 165.386 0)
+			(at 116.332 165.386 0)
 			(effects
 				(font
@@
 		)
 		(property "VOLTAGE RATING" "100V"
-			(at 121.92 172.72 0)
+			(at 124.46 172.72 0)
 			(effects
 				(font
@@
 		)
 		(property "SUPPLIER 1" "Mouser"
-			(at 113.792 165.386 0)
+			(at 116.332 165.386 0)
 			(effects
 				(font
@@
 		)
 		(property "SUPPLIER PART NUMBER 1" "81-GCM1885C2A102FA6D"
-			(at 113.792 165.386 0)
+			(at 116.332 165.386 0)
 			(effects
 				(font
@@
 		)
 		(property "HOUSE PART NUMBER" ""
-			(at 113.792 162.846 0)
+			(at 116.332 162.846 0)
 			(effects
 				(font
@@
 		)
 		(property "MANUFACTURER" "Murata"
-			(at 113.792 162.846 0)
+			(at 116.332 162.846 0)
 			(effects
 				(font
@@
 		)
 		(property "MANUFACTURER PART NUMBER" "GCM1885C2A102FA16D"
-			(at 113.792 162.846 0)
+			(at 116.332 162.846 0)
 			(effects
 				(font
@@
 		)
 		(property "TEMPERATURE COEFFICIENT" "C0G"
-			(at 117.126 175.768 0)
+			(at 119.666 175.768 0)
 			(effects
 				(font
@@
 		)
 		(property "ALTIUM_VALUE" ""
-			(at 119.38 167.64 0)
+			(at 121.92 167.64 0)
 			(effects
 				(font
@@
 		(on_board yes)
 		(dnp no)
-		(property "Reference" "U?"
-			(at 45.72 212.09 0)
+		(property "Reference" "U1001_4"
+			(at 59.69 212.09 0)
 			(effects
 				(font
@@
 		)
 		(instances
-			(project ""
+			(project "Thunderscope_Rev5.1"
+				(path "/031d3e2c-42e0-4016-8c32-579d45c83e09/02e7ff63-3631-4d05-9bcb-1390e77ff703"
+					(reference "U1001_3")
+					(unit 1)
+				)
 				(path "/031d3e2c-42e0-4016-8c32-579d45c83e09/d4ceb53c-d7d3-49f3-84e4-450b713426dc"
-					(reference "U?")
+					(reference "U1001_4")
+					(unit 1)
+				)
+				(path "/031d3e2c-42e0-4016-8c32-579d45c83e09/da233e23-d1b0-4723-86d8-4ec9b143e851"
+					(reference "U1001_2")
+					(unit 1)
+				)
+				(path "/031d3e2c-42e0-4016-8c32-579d45c83e09/f35774a1-d397-4f7e-9c64-3142469f9c73"
+					(reference "U1001_1")
 					(unit 1)
 				)
@@
 		(on_board yes)
 		(dnp no)
-		(property "Reference" "C?"
+		(property "Reference" "C1002_4"
 			(at 78.74 245.11 90)
 			(effects
@@
 			(project "Thunderscope_Rev5.1"
 				(path "/031d3e2c-42e0-4016-8c32-579d45c83e09/02e7ff63-3631-4d05-9bcb-1390e77ff703"
-					(reference "C?")
+					(reference "C1002_3")
 					(unit 1)
 				)
 				(path "/031d3e2c-42e0-4016-8c32-579d45c83e09/d4ceb53c-d7d3-49f3-84e4-450b713426dc"
-					(reference "C?")
+					(reference "C1002_4")
 					(unit 1)
 				)
 				(path "/031d3e2c-42e0-4016-8c32-579d45c83e09/da233e23-d1b0-4723-86d8-4ec9b143e851"
-					(reference "C?")
+					(reference "C1002_2")
 					(unit 1)
 				)
 				(path "/031d3e2c-42e0-4016-8c32-579d45c83e09/f35774a1-d397-4f7e-9c64-3142469f9c73"
-					(reference "C?")
+					(reference "C1002_1")
 					(unit 1)
 				)

Commit message: Schematic Changes for #341 and #342
Parts:
- added C1003_4, C1004_4, C1005_4, C1006_4, C1007_4, C1008_4: 10uF, Thunderscope_Rev5:GEN_C_0603, symbol Thunderscope_Rev5:CAP 10uF 25V X5R 0603
- R1037_4: value 49.9 -> 0; symbol Thunderscope_Rev5:RES 49.9 OHM 1% 1/10W 0402 -> Thunderscope_Rev5:RES 0 OHM 1/16W 0402; MANUFACTURER PART NUMBER RC0402FR-0749R9L -> RC0402JR-070RL; SUPPLIER PART NUMBER 1 603-RC0402FR-0749R9L -> 603-RC0402JR-070RL
Connections:
- net +5V: now also C1004_4.2, C1006_4.2, C1008_4.2
- net -5V: now also C1003_4.1, C1005_4.1, C1007_4.1
- net GND: now also C1003_4.2, C1004_4.1, C1005_4.2, C1006_4.1, C1007_4.2, C1008_4.1
Other:
- moved on the sheet: C1044_4, C1045_4, C1046_4, C1047_4, C1048_4, C1049_4, C1050_4, C1052_4, C1053_4, C1054_4, C1055_4, C1056_4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
