File: Hardware/KiCad/Thunderscope_Rev5.1/CON_PCIe_X4.kicad_sch (KiCad schematic)
At the start: 47 parts, among them J3 1.27mm 6 Pin TH, J4 TSW-101-16-G-Q-RA, P1 PCIeX4-GF-2D-1000-1K-O64, U11 TPS563203DRLR

Commit message: New +VUSB Buck WIP
Just need to add some poly pours
Parts:
- removed C82: 100nF, Thunderscope_Rev5:GEN_C_0402, symbol Thunderscope_Rev5:CAP 100nF 16V X7R 0402
- removed C85: 12pF, Thunderscope_Rev5:GEN_C_0402, symbol Thunderscope_Rev5:CAP 12pF 50V C0G 0402
- removed L6: 4.7uH, Thunderscope_Rev5:IND_SRN6045TA-100M, symbol Thunderscope_Rev5:IND 4.7uH 4.5A 26 MOHM 6x6mm
- removed U11: TPS563203DRLR, Thunderscope_Rev5:TI_SOT563_DRL0006A, symbol Thunderscope_Rev5:IC BUCK TPS563203DRL
- added C12, C22: 22uF, Thunderscope_Rev5:GEN_C_0805, symbol Thunderscope_Rev5:CAP 22uF 25V X5R 0805
- added C13: 100nF, Thunderscope_Rev5:GEN_C_0402, symbol Thunderscope_Rev5:CAP 100nF 16V X7R 0402
- added R87, R92: 10K, Thunderscope_Rev5:GEN_R_0402, symbol Thunderscope_Rev5:RES 10K OHM 1% 1/10W 0402
- added R88: 35.7k, Thunderscope_Rev5:GEN_R_0402, symbol Thunderscope_Rev5:RES 35.7K OHM 1% 1/16W 0402
- added R95: 1K, Thunderscope_Rev5:GEN_R_0402, symbol Thunderscope_Rev5:RES 1K OHM 1% 1/10W 0402
- added SYM1: SYM_ESD_Large, Symbol:ESD-Logo_6.6x6mm_SilkScreen, symbol Graphic:SYM_ESD_Large
- added TP86: PCB, Thunderscope_Rev5:GEN_TP_PCB, symbol Thunderscope_Rev5:TP PCB 1mm
- added U11: TPSM82913, Thunderscope_Rev5:TI_B0QFN_RDU0028A, symbol Thunderscope_Rev5:IC BUCK MODULE TPSM82913
- R73: value 280K -> 4.7K; symbol Thunderscope_Rev5:RES 280K OHM 1% 1/16W 0402 -> Thunderscope_Rev5:RES 4.7K OHM 1% 1/10W 0402; MANUFACTURER Yageo -> Panasonic; MANUFACTURER PART NUMBER AC0402FR-07280KL -> ERJ-2RKF4701X; SUPPLIER PART NUMBER 1 603-AC0402FR-07280KL -> 667-ERJ-2RKF4701X
- R74: value 35.7k -> 1K; symbol Thunderscope_Rev5:RES 35.7K OHM 1% 1/16W 0402 -> Thunderscope_Rev5:RES 1K OHM 1% 1/10W 0402; HOUSE PART NUMBER (none) -> R-1K-0402-1%-001; MANUFACTURER PART NUMBER RC0402FR-0735K7L -> RC0402FR-071KL; SUPPLIER PART NUMBER 1 603-RC0402FR-0735K7L -> 603-RC0402FR-071KL
Connections:
- net +12V_PCIe_R: now also C12.2, R87.2, U11.18 (VIN)
- net +VUSB: now also C22.2, R92.1, U11.10 (VOUT), U11.11 (VOUT), U11.12 (VOUT), U11.13 (VOUT), U11.14 (VOUT), U11.15 (VOUT), U11.27 (VOUT)
- net GND: now also C12.1, C13.1, C22.1, R88.2, U11.1 (PGND), U11.16 (PGND), U11.17 (PGND), U11.2 (PGND), U11.20 (PSNS), U11.25 (PGND), U11.26 (PGND), U11.28 (PGND), U11.3 (PGND), U11.5 (PGND), U11.6 (PGND), U11.7 (PGND), U11.8 (PGND), U11.9 (PGND)
- net at R73.1: now also R95.1; no longer R74.1
- new net: R92.2, TP86.1, U11.19 (PG)
- new net: R74.1, R95.2, U11.22 (FB)
- new net: C13.2, U11.21 (NR/SS)
- new net: R88.1, U11.23 (S-CONF)
- new net: R87.1, U11.24 (EN/SYNC)
Other:
- note added: "Vout = 0.8V*(5.7+1)/1"
- note added: "Vout = 0.8V*(R1+R2)/R2"
- note added: "Vout = 5.36V"
- note removed: "Vout = 0.6 * (280/35.7 + 1)"
- note removed: "Vout = 0.6 * (R1/R2 + 1)"
- note removed: "Vout = 5.31V"
- moved on the sheet: C28, C29, C32, C33, C36, C37, C40, C41, C44, C45, C80, C81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

Commit message: Added 1uF at -5V output as per #354
Also added net label to +VUSB PG output
Connections:
- net +VUSB_PG: now reaches R92.2, TP86.1, U11.19 (PG)
Other:
- moved on the sheet: TP86
Changed lines of the file:
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@@
 	)
 	(junction
-		(at 139.7 160.02)
-		(diameter 0)
-		(color 0 0 0 0)
-	)
-	(junction
 		(at 276.86 154.94)
 		(diameter 0)
@@
 	)
 	(junction
+		(at 139.7 157.48)
+		(diameter 0)
+		(color 0 0 0 0)
+	)
+	(junction
 		(at 129.54 142.24)
 		(diameter 0)
@@
 	(wire
 		(pts
+			(xy 139.7 157.48) (xy 139.7 165.1)
+		)
+		(stroke
+			(width 0)
+			(type default)
+		)
+	)
+	(wire
+		(pts
 			(xy 93.98 170.18) (xy 93.98 172.72)
 		)
@@
 	(wire
 		(pts
-			(xy 139.7 152.4) (xy 139.7 160.02)
+			(xy 139.7 152.4) (xy 139.7 157.48)
 		)
 		(stroke
@@
 		)
 	)
-	(wire
-		(pts
-			(xy 139.7 160.02) (xy 139.7 165.1)
-		)
-		(stroke
-			(width 0)
-			(type default)
-		)
-	)
 	(bus
 		(pts
@@
 		)
 	)
+	(label "+VUSB_PG"
+		(at 137.16 165.1 180)
+		(effects
+			(font
+				(size 1.27 1.27)
+			)
+			(justify right bottom)
+		)
+	)
 	(label "GND"
 		(at 109.22 93.98 180)
@@
 	(symbol
 		(lib_id "Thunderscope_Rev5:TP PCB 1mm")
-		(at 139.7 160.02 180)
+		(at 139.7 157.48 180)
 		(unit 1)
 		(exclude_from_sim no)
@@
 		(dnp no)
 		(property "Reference" "TP86"
-			(at 135.89 162.56 0)
+			(at 135.89 160.02 0)
 			(effects
 				(font
@@
 		)
 		(property "Value" "PCB"
-			(at 140.97 165.1 0)
+			(at 140.97 162.56 0)
 			(effects
 				(font
@@
 		)
 		(property "Footprint" "Thunderscope_Rev5:GEN_TP_PCB"
-			(at 139.7 160.02 0)
+			(at 139.7 157.48 0)
 			(effects
 				(font
@@
 		)
 		(property "Datasheet" ""
-			(at 139.7 160.02 0)
+			(at 139.7 157.48 0)
 			(effects
 				(font
@@
 		)
 		(property "Description" ""
-			(at 139.7 160.02 0)
+			(at 139.7 157.48 0)
 			(effects
 				(font
@@
 		)
 		(property "HOUSE PART NUMBER" ""
-			(at 140.97 167.64 0)
+			(at 140.97 165.1 0)
 			(effects
 				(font
@@
 		)
 		(property "MANUFACTURER" ""
-			(at 140.97 167.64 0)
+			(at 140.97 165.1 0)
 			(effects
 				(font
@@
 		)
 		(property "MANUFACTURER PART NUMBER" ""
-			(at 140.97 167.64 0)
+			(at 140.97 165.1 0)
 			(effects
 				(font
@@
 		)
 		(property "ALTIUM_VALUE" ""
-			(at 139.7 160.02 0)
+			(at 139.7 157.48 0)
 			(effects
 				(font
