File: Hardware/KiCad/Thunderscope_Rev5.1/FE.kicad_sch (KiCad schematic)
At the start: 25 parts, among them Q1 DMN62D0UW, Q2 DMN62D0UW, U2 MCP4452-104E, U3 MCP4728, U4 REF2025, U5 OPA140AIDR

Commit message: Finished FE Support Component Changes from #333, #334
Parts:
- added C82: 100nF, Thunderscope_Rev5:GEN_C_0402, symbol Thunderscope_Rev5:CAP 100nF 16V X7R 0402
- added C85, C93, C94, C95, C96: 10uF, Thunderscope_Rev5:GEN_C_0603, symbol Thunderscope_Rev5:CAP 10uF 25V X5R 0603
- added R107: 100, Thunderscope_Rev5:GEN_R_0402, symbol Thunderscope_Rev5:RES 100 OHM 1% 1/10W 0402
- C4: value 100nF -> 100pF; symbol Thunderscope_Rev5:CAP 100nF 16V X7R 0402 -> Thunderscope_Rev5:CAP 100pF 50V C0G 0402; MANUFACTURER PART NUMBER GCM155R71C104KA55D -> GCM1555C1H101FA16D; SUPPLIER PART NUMBER 1 81-GCM155R71C104KA5D -> 81-GCM1555C1H101FA6D; TEMPERATURE COEFFICIENT (none) -> C0G; VOLTAGE RATING 16V -> 50V
Connections:
- net +5V: now also C85.2, C94.2, C95.2, C96.2
- net -5V: now also C93.1
- net -VBIAS: now also C82.2, R107.1; no longer C4.2, R13.4, U5.6 (OUT)
- net GND: now also C82.1, C85.1, C93.2, C94.1, C95.1, C96.1
- new net: C4.2, R107.2, R13.4, U5.6 (OUT)
Other:
- moved on the sheet: C11, C2, C3, C8, Q1, Q2, R10, R11, R12, R9, TP59, TP6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

Commit message: Changed opamp package and did layout for #344
Parts:
- U5: value OPA140AIDR -> OPA140AIDBVR; footprint Thunderscope_Rev5:TI_SOIC8_D0008A -> Thunderscope_Rev5:GEN_SOT23_5_950_2900X1600X1450; MANUFACTURER PART NUMBER OPA140AIDR -> OPA140AIDBVR; SUPPLIER PART NUMBER 1 OPA140AIDR -> OPA140AIDBVR
Connections:
- net +5V: now also U5.5 (V+); no longer U5.7 (V+)
- net -5V: now also U5.2 (V-); no longer U5.4 (V-)
- net U5-: now also U5.4 (-); no longer U5.2 (-)
- net at C4.2, R107.2, R13.4: now also U5.1 (OUT); no longer U5.6 (OUT)
- no-connect marks 3 -> 1
Changed lines of the file:
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@@
 	)
 	(no_connect
-		(at 182.88 139.7)
-	)
-	(no_connect
 		(at 116.84 66.04)
 	)
-	(no_connect
-		(at 187.96 142.24)
-	)
 	(wire
 		(pts
@@
 			)
 		)
-		(property "Value" "OPA140AIDR"
+		(property "Value" "OPA140AIDBVR"
 			(at 184.15 160.02 0)
 			(effects
@@
 			)
 		)
-		(property "Footprint" "Thunderscope_Rev5:TI_SOIC8_D0008A"
+		(property "Footprint" "Thunderscope_Rev5:GEN_SOT23_5_950_2900X1600X1450"
 			(at 182.88 152.4 0)
 			(effects
@@
 			)
 		)
-		(property "SUPPLIER PART NUMBER 1" "OPA140AIDR"
+		(property "SUPPLIER PART NUMBER 1" "OPA140AIDBVR"
 			(at 164.592 168.148 0)
 			(effects
@@
 			)
 		)
-		(property "MANUFACTURER PART NUMBER" "OPA140AIDR"
+		(property "MANUFACTURER PART NUMBER" "OPA140AIDBVR"
 			(at 164.592 168.148 0)
 			(effects
@@
 		(pin "3"
 		)
-		(pin "6"
-		)
 		(pin "2"
 		)
-		(pin "7"
-		)
-		(pin "8"
+		(pin "5"
 		)
 		(pin "4"

Commit message: Changed DAC PN, Closes #373
Parts:
- U3: MANUFACTURER PART NUMBER MCP4728 -> MCP4728T-E/UN; SUPPLIER PART NUMBER 1 579-MCP4728A1T-E/UN -> 579-MCP4728T-E/UN
Changed lines of the file:
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@@
 			)
 		)
-		(property "SUPPLIER PART NUMBER 1" "579-MCP4728A1T-E/UN"
+		(property "SUPPLIER PART NUMBER 1" "579-MCP4728T-E/UN"
 			(at 135.89 59.69 0)
 			(effects
@@
 			)
 		)
-		(property "MANUFACTURER PART NUMBER" "MCP4728"
+		(property "MANUFACTURER PART NUMBER" "MCP4728T-E/UN"
 			(at 116.332 45.72 0)
 			(effects
