File: Hardware/KiCad/Thunderscope_Rev5.1/FPGA_Bank_IO.kicad_sch (KiCad schematic)
At the start: 18 parts, among them U18 IC FPGA XC7A50T-2CSG325C

Commit message: Fixed #310
Swapped Labels, Swapped P15 and P14, Swapped TP42 and TP25. No Copper Change
Connections:
- net PGA_SCLK: now also TP25.1, U18.N14 (IO_L8N_T1_D12_14); no longer TP42.1, U18.P15 (IO_L11P_T1_SRCC_14)
- net PGA_SDIO: now also TP42.1, U18.P15 (IO_L11P_T1_SRCC_14); no longer TP25.1, U18.N14 (IO_L8N_T1_D12_14)
Other:
- moved on the sheet: TP25
Changed lines of the file:
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@@
 	)
 	(junction
+		(at 99.06 78.74)
+		(diameter 0)
+		(color 0 0 0 0)
+	)
+	(junction
 		(at 99.06 127)
 		(diameter 0)
@@
 		(color 0 0 0 0)
 	)
-	(junction
-		(at 88.9 78.74)
-		(diameter 0)
-		(color 0 0 0 0)
-	)
 	(no_connect
 		(at 274.32 63.5)
@@
 	(wire
 		(pts
-			(xy 88.9 78.74) (xy 93.98 78.74)
-		)
-		(stroke
-			(width 0)
-			(type default)
-		)
-	)
-	(wire
-		(pts
 			(xy 66.04 124.46) (xy 83.82 124.46)
 		)
@@
 	(wire
 		(pts
+			(xy 99.06 78.74) (xy 104.14 78.74)
+		)
+		(stroke
+			(width 0)
+			(type default)
+		)
+	)
+	(wire
+		(pts
 			(xy 66.04 121.92) (xy 83.82 121.92)
 		)
@@
 	(wire
 		(pts
+			(xy 99.06 91.44) (xy 104.14 91.44)
+		)
+		(stroke
+			(width 0)
+			(type default)
+		)
+	)
+	(wire
+		(pts
 			(xy 180.34 40.64) (xy 182.88 40.64)
 		)
@@
 	(wire
 		(pts
-			(xy 66.04 91.44) (xy 99.06 91.44)
-		)
-		(stroke
-			(width 0)
-			(type default)
-		)
-	)
-	(wire
-		(pts
 			(xy 104.14 124.46) (xy 104.14 129.54)
 		)
@@
 	(wire
 		(pts
-			(xy 99.06 91.44) (xy 104.14 91.44)
+			(xy 66.04 78.74) (xy 99.06 78.74)
 		)
 		(stroke
@@
 		)
 	)
-	(wire
-		(pts
-			(xy 66.04 78.74) (xy 88.9 78.74)
-		)
-		(stroke
-			(width 0)
-			(type default)
-		)
-	)
 	(bus
 		(pts
@@
 	(wire
 		(pts
+			(xy 66.04 91.44) (xy 99.06 91.44)
+		)
+		(stroke
+			(width 0)
+			(type default)
+		)
+	)
+	(wire
+		(pts
 			(xy 73.66 185.42) (xy 76.2 185.42)
 		)
@@
 		)
 	)
-	(label "PGA_SCLK"
-		(at 81.28 91.44 180)
-		(effects
-			(font
-				(size 1.27 1.27)
-			)
-			(justify right bottom)
-		)
-	)
 	(label "CLK25"
 		(at 81.28 101.6 180)
@@
 		)
 	)
+	(label "PGA_SDIO"
+		(at 81.28 91.44 180)
+		(effects
+			(font
+				(size 1.27 1.27)
+			)
+			(justify right bottom)
+		)
+	)
 	(label "D3A_P"
 		(at 198.12 76.2 180)
@@
 		)
 	)
+	(label "PGA_SCLK"
+		(at 81.28 78.74 180)
+		(effects
+			(font
+				(size 1.27 1.27)
+			)
+			(justify right bottom)
+		)
+	)
 	(label "LCLK_N"
 		(at 198.12 99.06 180)
@@
 		)
 	)
-	(label "PGA_SDIO"
-		(at 81.28 78.74 180)
-		(effects
-			(font
-				(size 1.27 1.27)
-			)
-			(justify right bottom)
-		)
-	)
 	(label "ATTEN_3"
 		(at 81.28 58.42 180)
@@
 	(hierarchical_label "PGA_SCLK"
 		(shape output)
-		(at 104.14 91.44 0)
+		(at 104.14 78.74 0)
 		(effects
 			(font
@@
 		)
 	)
+	(hierarchical_label "PGA_SDIO"
+		(shape output)
+		(at 104.14 91.44 0)
+		(effects
+			(font
+				(size 1.27 1.27)
+			)
+			(justify left)
+		)
+	)
 	(hierarchical_label "CLK25"
 		(shape input)
@@
 		)
 	)
-	(hierarchical_label "PGA_SDIO"
-		(shape output)
-		(at 93.98 78.74 0)
-		(effects
-			(font
-				(size 1.27 1.27)
-			)
-			(justify left)
-		)
-	)
 	(symbol
 		(lib_id "Thunderscope_Rev5:TP PCB 1mm")
@@
 	(symbol
 		(lib_id "Thunderscope_Rev5:TP PCB 1mm")
-		(at 88.9 78.74 90)
+		(at 99.06 78.74 90)
 		(unit 1)
 		(exclude_from_sim no)
@@
 		(dnp no)
 		(property "Reference" "TP25"
-			(at 91.44 71.12 90)
+			(at 101.6 71.12 90)
 			(effects
 				(font
@@
 		)
 		(property "Value" "PCB"
-			(at 83.82 80.01 0)
+			(at 93.98 80.01 0)
 			(effects
 				(font
@@
 		)
 		(property "Footprint" "Thunderscope_Rev5:GEN_TP_PCB"
-			(at 88.9 78.74 0)
+			(at 99.06 78.74 0)
 			(effects
 				(font
@@
 		)
 		(property "Datasheet" ""
-			(at 88.9 78.74 0)
+			(at 99.06 78.74 0)
 			(effects
 				(font
@@
 		)
 		(property "Description" ""
-			(at 88.9 78.74 0)
+			(at 99.06 78.74 0)
 			(effects
 				(font
@@
 		)
 		(property "HOUSE PART NUMBER" ""
-			(at 83.82 80.01 0)
+			(at 93.98 80.01 0)
 			(effects
 				(font
@@
 		)
 		(property "MANUFACTURER" ""
-			(at 83.82 80.01 0)
+			(at 93.98 80.01 0)
 			(effects
 				(font
@@
 		)
 		(property "MANUFACTURER PART NUMBER" ""
-			(at 83.82 80.01 0)
+			(at 93.98 80.01 0)
 			(effects
 				(font
@@
 		)
 		(property "ALTIUM_VALUE" ""
-			(at 88.9 78.74 0)
+			(at 99.06 78.74 0)
 			(effects
 				(font
@@
 		)
 		(instances
-			(project "Thunderscope_Rev5"
+			(project "Thunderscope_Rev5.1"
 				(path "/031d3e2c-42e0-4016-8c32-579d45c83e09/0f922f52-a6e9-41f0-8991-df4889546a95/3dc749f1-bb54-4961-a356-74c6bb9263ea"
 					(reference "TP25")
@@
 		)
 		(instances
-			(project "Thunderscope_Rev5"
+			(project "Thunderscope_Rev5.1"
 				(path "/031d3e2c-42e0-4016-8c32-579d45c83e09/0f922f52-a6e9-41f0-8991-df4889546a95/3dc749f1-bb54-4961-a356-74c6bb9263ea"
 					(reference "TP42")

Commit message: Updated Version Resistor DNPs, Closes #371
Parts:
- R75: now fitted
- R76: now not fitted
Changed lines of the file:
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@@
 		(in_bom yes)
 		(on_board yes)
-		(dnp yes)
+		(dnp no)
 		(property "Reference" "R75"
 			(at 68.58 182.88 0)
@@
 		(in_bom yes)
 		(on_board yes)
-		(dnp no)
+		(dnp yes)
 		(property "Reference" "R76"
 			(at 68.58 187.96 0)
