File: Hardware/KiCad/ThunderScope MUXboard/Connectors.kicad_sch (KiCad schematic)
At the start: 35 parts, among them J1 Conn_02x30_Odd_Even, J2 Conn_02x30_Odd_Even, J3 Conn_02x22_Odd_Even, J4 Conn_02x22_Odd_Even, J5 RED V+, J6 BLUE V-, U21 Seeeduino XIAO SAMD21, U22 TLV77333PDBVR

Commit message: Test fixture boards out to fab
Parts:
- J5, J6: footprint Connector:CalTest_CT3151 -> ThunderScope:CT3151
Connections:
- no-connect marks 132 -> 133
Changed lines of the file:
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@@
+	)
+	(no_connect
+		(at 77.47 107.95)
 	)
 	(no_connect
@@
 			)
 		)
-		(property "Footprint" "Connector:CalTest_CT3151"
+		(property "Footprint" "ThunderScope:CT3151"
 			(at 35.56 29.21 0)
 			(effects
@@
 			)
 		)
-		(property "Footprint" "Connector:CalTest_CT3151"
+		(property "Footprint" "ThunderScope:CT3151"
 			(at 35.56 41.91 0)
 			(effects
