File: Hardware/KiCad/ThunderScope MUXboard/ThunderScope Muxboard.kicad_sch (KiCad schematic)
At the start: 46 parts, among them U1 MC74HC238ADTR2G, U10 SN74HC32DR, U11 SN74HC32DR, U12 SN74HC32DR, U13 SN74HC32DR, U14 SN74HC32DR, U15 SN74HC32DR, U16 SN74HC32DR, U17 SN74HC32DR, U18 SN74HC32DR, U19 SN74HC32DR, U2 MC74HC238ADTR2G, U3 MC74HC238ADTR2G, U4 MC74HC238ADTR2G, U5 MC74HC238ADTR2G, U6 MC74HC238ADTR2G, U7 MC74HC238ADTR2G, U8 SN74HC32DR, U9 SN74HC32DR

Commit message: Test fixture boards out to fab
Parts:
- U1, U2, U3, U4, U5, U6, U7: symbol 74xx:74HC238 -> ThunderScope:MC74HC238ADTR2G; LCSC (none) -> C904037
- U10, U11, U12, U13, U14, U15, U16, U17, U18, U19, U8, U9: footprint PCM_JLCPCB:SOIC-14_L8.7-W3.9-P1.27-LS6.0-BL -> ThunderScope:SOIC-14_L8.7-W3.9-P1.27-LS6.0-BL; symbol PCM_JLCPCB-ICs:Gate, AND, 4 Channel, 74HC08D,653 -> ThunderScope:SN74HC32DR; LCSC (none) -> C6838
Connections:
- net GND: no longer U15.10 (3B), U15.12 (4A)
