File: Hardware/KiCad/ThunderScope MUXboard/relays.kicad_sch (KiCad schematic)
At the start: 86 parts, among them U101 VO1400AEF, U102 VO1400AEF, U105 VO1400AEF, U106 VO1400AEF, U107 VO1400AEF, U108 VO1400AEF, U109 VO1400AEF, U110 VO1400AEF, U111 VO1400AEF, U112 VO1400AEF, U113 VO1400AEF, U114 VO1400AEF, U115 VO1400AEF, U116 VO1400AEF, U117 VO1400AEF, U118 VO1400AEF, U119 VO1400AEF, U120 VO1400AEF, U121 VO1400AEF, U122 VO1400AEF, U123 VO1400AEF, U124 VO1400AEF, U125 VO1400AEF, U126 VO1400AEF, U127 VO1400AEF, U128 VO1400AEF, U129 VO1400AEF, U130 VO1400AEF, U133 VO1400AEF, U134 VO1400AEF, U139 VO1400AEF, U142 VO1400AEF, U143 VO1400AEF, U144 VO1400AEF, U145 VO1400AEF, U146 VO1400AEF, U147 VO1400AEF, U149 VO1400AEF, U154 VO1400AEF, U157 VO1400AEF, U159 VO1400AEF, U161 VO1400AEF, U162 VO1400AEF

Commit message: Test fixture boards out to fab
Parts:
- U101, U102, U105, U106, U107, U108, U109, U110, U111, U112, U113, U114, U115, U116, U117, U118, U119, U120, U121, U122, U123, U124, U125, U126, U127, U128, U129, U130, U133, U134, U139, U142, U143, U144, U145, U146, U147, U149, U154, U157, U159, U161, U162: value VO1400AEF -> CPC1017N; symbol Relay_SolidState:CPC1017N -> ThunderScope:CPC1017N; LCSC (none) -> C81521
