File: Hardware/KiCad/Thunderscope Digital Test Fixture/Thunderscope Digital Test/Thunderscope Digital Test.kicad_pcb (KiCad board)
At the start: 4 copper layers, 142.5 x 136.3 mm, 65 parts, among them J1 Conn_02x30_Odd_Even, J2 Conn_02x30_Odd_Even, J3 Conn_ARM_JTAG_SWD_10, J9 USB_C_Receptacle_USB2.0_14P, U12 USBLC6-2P6, U2 JTAG-HS2-Header, U3 STM32H743ZGT6, U4 SN74LV1T34DCK, U5 SN74LV1T34DCK, U6 SN74LV1T34DCK, U8 TPS62A02, X1 X322512MSB4SI

Commit message: Test fixture boards out to fab
Other:
- board text added: "JTAG for DUT"
- board text removed: "DUT for JTAG"
Changed lines of the file:
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@@
 			(psa4output no)
 			(plot_black_and_white yes)
-			(plotinvisibletext no)
 			(sketchpadsonfab no)
 			(plotpadnumbers no)
@@
 			(layer "B.Fab")
 		)
-		(fp_text user "${REFERENCE}"
-			(at 0 0.25 90)
-			(layer "B.Fab")
-			(hide yes)
-			(effects
-				(font
-					(size 0.25 0.25)
-					(thickness 0.04)
-				)
-				(justify mirror)
-			)
-		)
 		(pad "1" smd roundrect
 			(at -0.5 0 90)
@@
 			(layer "B.Fab")
 		)
-		(fp_text user "${REFERENCE}"
-			(at 0 0.25 90)
-			(layer "B.Fab")
-			(hide yes)
-			(effects
-				(font
-					(size 0.25 0.25)
-					(thickness 0.04)
-				)
-				(justify mirror)
-			)
-		)
 		(pad "1" smd roundrect
 			(at -0.5 0 270)
@@
 			(layer "B.Fab")
 		)
-		(fp_text user "${REFERENCE}"
-			(at 0 0.25 180)
-			(layer "B.Fab")
-			(hide yes)
-			(effects
-				(font
-					(size 0.25 0.25)
-					(thickness 0.04)
-				)
-				(justify mirror)
-			)
-		)
 		(pad "1" smd roundrect
 			(at -0.5 0)
@@
 			(layer "B.Fab")
 		)
-		(fp_text user "${REFERENCE}"
-			(at 0 0.25 90)
-			(layer "B.Fab")
-			(hide yes)
-			(effects
-				(font
-					(size 0.25 0.25)
-					(thickness 0.04)
-				)
-				(justify mirror)
-			)
-		)
 		(pad "1" smd roundrect
 			(at -0.5 0 270)
@@
 			(layer "B.Fab")
 		)
-		(fp_text user "${REFERENCE}"
-			(at 0 0.25 0)
-			(layer "B.Fab")
-			(hide yes)
-			(effects
-				(font
-					(size 0.25 0.25)
-					(thickness 0.04)
-				)
-				(justify mirror)
-			)
-		)
 		(pad "1" smd roundrect
 			(at -0.5 0)
@@
 			(layer "B.Fab")
 		)
-		(fp_text user "${REFERENCE}"
-			(at 0 0.25 0)
-			(layer "B.Fab")
-			(hide yes)
-			(effects
-				(font
-					(size 0.25 0.25)
-					(thickness 0.04)
-				)
-				(justify mirror)
-			)
-		)
 		(pad "1" smd roundrect
 			(at -0.5 0 180)
@@
 			(layer "B.Fab")
 		)
-		(fp_text user "${REFERENCE}"
-			(at 0 0.25 0)
-			(layer "B.Fab")
-			(hide yes)
-			(effects
-				(font
-					(size 0.25 0.25)
-					(thickness 0.04)
-				)
-				(justify mirror)
-			)
-		)
 		(pad "1" smd roundrect
 			(at -0.5 0 180)
@@
 			(layer "B.Fab")
 		)
-		(fp_text user "${REFERENCE}"
-			(at 0 0.25 0)
-			(layer "B.Fab")
-			(hide yes)
-			(effects
-				(font
-					(size 0.25 0.25)
-					(thickness 0.04)
-				)
-				(justify mirror)
-			)
-		)
 		(pad "1" smd roundrect
 			(at -0.5 0)
@@
 			(layer "B.Fab")
 		)
-		(fp_text user "${REFERENCE}"
-			(at 0 0.25 0)
-			(layer "B.Fab")
-			(hide yes)
-			(effects
-				(font
-					(size 0.25 0.25)
-					(thickness 0.04)
-				)
-				(justify mirror)
-			)
-		)
 		(pad "1" smd roundrect
 			(at -0.5 0 180)
@@
 			(layer "B.Fab")
 		)
-		(fp_text user "${REFERENCE}"
-			(at 0 0.25 90)
-			(layer "B.Fab")
-			(hide yes)
-			(effects
-				(font
-					(size 0.25 0.25)
-					(thickness 0.04)
-				)
-				(justify mirror)
-			)
-		)
 		(pad "1" smd roundrect
 			(at -0.5 0 270)
@@
 			(layer "B.Fab")
 		)
-		(fp_text user "${REFERENCE}"
-			(at 0 0.25 0)
-			(layer "B.Fab")
-			(hide yes)
-			(effects
-				(font
-					(size 0.25 0.25)
-					(thickness 0.04)
-				)
-				(justify mirror)
-			)
-		)
 		(pad "1" smd roundrect
 			(at -0.5 0)
@@
 			(layer "B.Fab")
 		)
-		(fp_text user "${REFERENCE}"
-			(at 0 0.25 0)
-			(layer "B.Fab")
-			(hide yes)
-			(effects
-				(font
-					(size 0.25 0.25)
-					(thickness 0.04)
-				)
-				(justify mirror)
-			)
-		)
 		(pad "1" smd roundrect
 			(at -0.5 0 180)
@@
 			(layer "B.Fab")
 		)
-		(fp_text user "${REFERENCE}"
-			(at 0 0.25 0)
-			(layer "B.Fab")
-			(hide yes)
-			(effects
-				(font
-					(size 0.25 0.25)
-					(thickness 0.04)
-				)
-				(justify mirror)
-			)
-		)
 		(pad "1" smd roundrect
 			(at -0.5 0)
@@
 		)
 	)
-	(gr_text "DUT\nfor\nJTAG\n"
+	(gr_text "JTAG\nfor\nDUT\n"
 		(at 221.8 -2.25 180)
 		(layer "F.SilkS")
