File: Hardware/KiCad/Thunderscope Digital Test Fixture/Thunderscope Digital Test/Thunderscope Digital Test.kicad_sch (KiCad schematic)
At the start: 65 parts, among them J1 Conn_02x30_Odd_Even, J2 Conn_02x30_Odd_Even, J3 Conn_ARM_JTAG_SWD_10, J9 USB_C_Receptacle_USB2.0_14P, U12 USBLC6-2P6, U2 JTAG-HS2-Header, U3 STM32H743ZGT6, U4 SN74LV1T34DCK, U5 SN74LV1T34DCK, U6 SN74LV1T34DCK, U8 TPS62A02, X1 X322512MSB4SI

Commit message: Digital Test Controller Rev 2 Release
Parts:
- added D1, D2: TPD1E1B04, Thunderscope_Rev5:TI_X1SON_DPY0002A, symbol Thunderscope_Rev5:TVS TPD1E1B04
- added J4: 1.27mm 6 Pin TH, Thunderscope_Rev5:GEN_1.27mm_2x5_Pin_TH_RA, symbol Thunderscope_Rev5:CONN 1.27mm 2x5 Pin TH RA
Connections:
- net GND: now also D1.2 (A), D2.2 (A), J4.1, J4.10, J4.2, J4.4, J4.5, J4.6, J4.8, J4.9
- net REFINOUT: now reaches U3.110 (PA15)
- net REFINOUT: now also D1.1 (K), J4.3
- net SYNC: now reaches U3.111 (PC10)
- net SYNC: now also D2.1 (K), J4.7
- no-connect marks 55 -> 53
Other:
- note added: "REFCLK and SYNC Connector"
- note added: "Uses JLC04161H-3313 stackup"
- note removed: "???"
- note removed: "JLC04161H-3313"
- moved on the sheet: C10, C13, U2, X1
