File: Hardware/KiCad/Thunderscope_Rev5.3/FE_Channel.kicad_sch (KiCad schematic)
At the start: 105 parts, among them J1002_4 BNC, J3_4 UFL, J4_4 UFL, K1000_4 UD2-4.5NUN-L, K1001_4 UD2-4.5NUN-L, Q1002_4 DMN62D0UW, Q1003_4 DMN62D0UW, U1001_4 TMUX4053, U1008_4 LMH6518, U1009_4 BUF802, U1011_4 OPA140AIDBVR

Commit message: Changed C1021 to 4pF, closes #412
Parts:
- C1021_4: value 5pF -> 4pF; symbol Thunderscope_Rev5:CAP 5pF 50V C0G 0402 -> Thunderscope_Rev5:CAP 4pF 50V C0G 0402; MANUFACTURER PART NUMBER CBR04C509B5GAC -> CBR04C409B5GAC; SUPPLIER PART NUMBER 1 80-CBR04C509B5G -> 80-CBR04C409B5G
Changed lines of the file:
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@@
 	)
 	(symbol
-		(lib_id "Thunderscope_Rev5:CAP 5pF 50V C0G 0402")
+		(lib_id "Thunderscope_Rev5:CAP 4pF 50V C0G 0402")
 		(at 320.04 45.72 0)
 		(unit 1)
@@
 			)
 		)
-		(property "Value" "5pF"
+		(property "Value" "4pF"
 			(at 326.39 45.72 90)
 			(effects
@@
 			)
 		)
-		(property "SUPPLIER PART NUMBER 1" "80-CBR04C509B5G"
+		(property "SUPPLIER PART NUMBER 1" "80-CBR04C409B5G"
 			(at 317.786 41.212 0)
 			(effects
@@
 			)
 		)
-		(property "MANUFACTURER PART NUMBER" "CBR04C509B5GAC"
+		(property "MANUFACTURER PART NUMBER" "CBR04C409B5GAC"
 			(at 317.786 40.132 0)
 			(effects

Commit message: Changed C1011 to 3pF, closes #409
Parts:
- C1011_4: value 2.5pF -> 3pF; symbol Thunderscope_Rev5:CAP 2.5pF 200V C0G 0402 -> Thunderscope_Rev5:CAP 3pF 200V C0G 0402; MANUFACTURER PART NUMBER CBR04C259B2GAC -> CBR04C309B2GAC; SUPPLIER PART NUMBER 1 80-CBR04C259B2GAC -> 80-CBR04C309B2GAC
Changed lines of the file:
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@@
 	)
 	(symbol
-		(lib_id "Thunderscope_Rev5:CAP 2.5pF 200V C0G 0402")
+		(lib_id "Thunderscope_Rev5:CAP 3pF 200V C0G 0402")
 		(at 233.68 58.42 270)
 		(unit 1)
@@
 			)
 		)
-		(property "Value" "2.5pF"
+		(property "Value" "3pF"
 			(at 236.22 59.69 90)
 			(effects
@@
 			)
 		)
-		(property "SUPPLIER PART NUMBER 1" "80-CBR04C259B2GAC"
+		(property "SUPPLIER PART NUMBER 1" "80-CBR04C309B2GAC"
 			(at 235.934 52.832 0)
 			(effects
@@
 			)
 		)
-		(property "MANUFACTURER PART NUMBER" "CBR04C259B2GAC"
+		(property "MANUFACTURER PART NUMBER" "CBR04C309B2GAC"
 			(at 239.268 56.166 0)
 			(effects

Commit message: Changed R1002 to 976k as per #408
Parts:
- R1002_4: value 2M -> 976k; symbol Thunderscope_Rev5:RES 2M OHM 1% 1/10W 0402 -> Thunderscope_Rev5:RES 976k OHM 1% 1/10W 0402; MANUFACTURER PART NUMBER RK73H1ETTP2004F -> RK73H1ETTP9763F; SUPPLIER PART NUMBER 1 660-RK73H1ETTP2004F -> 660-RK73H1ETTP9763F
Other:
- moved on the sheet: R1002_4
Changed lines of the file:
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@@
 	)
 	(symbol
-		(lib_id "Thunderscope_Rev5:RES 2M OHM 1% 1/10W 0402")
-		(at 269.24 48.26 180)
+		(lib_id "Thunderscope_Rev5:RES 976k OHM 1% 1/10W 0402")
+		(at 269.24 48.26 0)
 		(unit 1)
 		(exclude_from_sim no)
@@
 			)
 		)
-		(property "Value" "2M"
+		(property "Value" "976k"
 			(at 269.24 48.26 0)
 			(effects
@@
 			)
 		)
-		(property "SUPPLIER PART NUMBER 1" "660-RK73H1ETTP2004F"
+		(property "SUPPLIER PART NUMBER 1" "660-RK73H1ETTP9763F"
 			(at 269.24 48.26 0)
 			(effects
@@
 			)
 		)
-		(property "MANUFACTURER PART NUMBER" "RK73H1ETTP2004F"
+		(property "MANUFACTURER PART NUMBER" "RK73H1ETTP9763F"
 			(at 269.24 48.26 0)
 			(effects

Commit message: Changed C1012 to thin film part for #408
Parts:
- C1012_4: symbol Thunderscope_Rev5:CAP 0.3pF 250V C0G 0402 -> Thunderscope_Rev5:CAP 0.3pF 100V Thin Film 0402; MANUFACTURER Johanson Technology -> KYOCERA AVX; MANUFACTURER PART NUMBER QSCF251Q0R3A1GV001T -> 04021J0R3ZBSTR; SUPPLIER PART NUMBER 1 609-QSCF251Q0R3A1GV0 -> 581-04021J0R3ZBSTR; VOLTAGE RATING 250V -> 100V
Changed lines of the file:
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@@
 	)
 	(symbol
-		(lib_id "Thunderscope_Rev5:CAP 0.3pF 250V C0G 0402")
+		(lib_id "Thunderscope_Rev5:CAP 0.3pF 100V Thin Film 0402")
 		(at 256.54 48.26 0)
 		(unit 1)
@@
 			)
 		)
-		(property "SUPPLIER PART NUMBER 1" "609-QSCF251Q0R3A1GV0"
+		(property "SUPPLIER PART NUMBER 1" "581-04021J0R3ZBSTR"
 			(at 250.952 46.006 0)
 			(effects
@@
 			)
 		)
-		(property "VOLTAGE RATING" "250V"
+		(property "VOLTAGE RATING" "100V"
 			(at 254 59.69 0)
 			(effects
@@
 			)
 		)
-		(property "MANUFACTURER" "Johanson Technology"
+		(property "MANUFACTURER" "KYOCERA AVX"
 			(at 254.286 42.672 0)
 			(effects
@@
 			)
 		)
-		(property "MANUFACTURER PART NUMBER" "QSCF251Q0R3A1GV001T"
+		(property "MANUFACTURER PART NUMBER" "04021J0R3ZBSTR"
 			(at 254.286 42.672 0)
 			(effects

Commit message: Changed C1021 to 3pF, closes #412
Parts:
- C1021_4: value 4pF -> 3pF; symbol Thunderscope_Rev5:CAP 4pF 50V C0G 0402 -> Thunderscope_Rev5:CAP 3pF 200V C0G 0402; MANUFACTURER PART NUMBER CBR04C409B5GAC -> CBR04C309B2GAC; SUPPLIER PART NUMBER 1 80-CBR04C409B5G -> 80-CBR04C309B2GAC; VOLTAGE RATING 50V -> 200V
Other:
- moved on the sheet: C1021_4
Changed lines of the file:
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@@
 	)
 	(symbol
-		(lib_id "Thunderscope_Rev5:CAP 4pF 50V C0G 0402")
-		(at 320.04 45.72 0)
+		(lib_id "Thunderscope_Rev5:CAP 3pF 200V C0G 0402")
+		(at 320.04 45.72 270)
 		(unit 1)
 		(exclude_from_sim no)
@@
 		(dnp no)
 		(property "Reference" "C1021_4"
-			(at 322.58 49.53 90)
-			(effects
-				(font
-					(size 1.27 1.27)
-				)
-				(justify left top)
-			)
-		)
-		(property "Value" "4pF"
-			(at 326.39 45.72 90)
-			(effects
-				(font
-					(size 1.27 1.27)
-				)
-				(justify bottom)
+			(at 316.23 45.72 0)
+			(effects
+				(font
+					(size 1.27 1.27)
+				)
+			)
+		)
+		(property "Value" "3pF"
+			(at 323.85 45.72 0)
+			(effects
+				(font
+					(size 1.27 1.27)
+				)
 			)
 		)
@@
 		)
 		(property "PACKAGE" "0402"
-			(at 302.912 57.15 0)
-			(effects
-				(font
-					(size 1.27 1.27)
-				)
-				(justify left bottom)
+			(at 320.04 45.72 0)
+			(effects
+				(font
+					(size 1.27 1.27)
+				)
 				(hide yes)
 			)
 		)
 		(property "SUPPLIER 1" "Mouser"
-			(at 317.786 41.212 0)
-			(effects
-				(font
-					(size 1.27 1.27)
-				)
-				(justify left bottom)
-				(hide yes)
-			)
-		)
-		(property "SUPPLIER PART NUMBER 1" "80-CBR04C409B5G"
-			(at 317.786 41.212 0)
-			(effects
-				(font
-					(size 1.27 1.27)
-				)
-				(justify left bottom)
-				(hide yes)
-			)
-		)
-		(property "VOLTAGE RATING" "50V"
-			(at 322.58 50.8 0)
-			(effects
-				(font
-					(size 1.27 1.27)
-				)
-				(justify left)
+			(at 320.04 45.72 0)
+			(effects
+				(font
+					(size 1.27 1.27)
+				)
+				(hide yes)
+			)
+		)
+		(property "SUPPLIER PART NUMBER 1" "80-CBR04C309B2GAC"
+			(at 320.04 45.72 0)
+			(effects
+				(font
+					(size 1.27 1.27)
+				)
+				(hide yes)
+			)
+		)
+		(property "VOLTAGE RATING" "200V"
+			(at 320.04 45.72 0)
+			(effects
+				(font
+					(size 1.27 1.27)
+				)
 				(hide yes)
 			)
 		)
 		(property "TEMPERATURE COEFFICIENT" "C0G"
-			(at 317.786 40.132 0)
+			(at 325.628 43.466 0)
 			(effects
 				(font
@@
 		)
 		(property "MANUFACTURER" "KEMET"
-			(at 317.786 40.132 0)
-			(effects
-				(font
-					(size 1.27 1.27)
-				)
-				(justify left bottom)
+			(at 320.04 45.72 0)
+			(effects
+				(font
+					(size 1.27 1.27)
+				)
 				(hide yes)
 			)
 		)
 		(property "HOUSE PART NUMBER" ""
-			(at 317.786 40.132 0)
-			(effects
-				(font
-					(size 1.27 1.27)
-				)
-				(justify left bottom)
-				(hide yes)
-			)
-		)
-		(property "MANUFACTURER PART NUMBER" "CBR04C409B5GAC"
-			(at 317.786 40.132 0)
-			(effects
-				(font
-					(size 1.27 1.27)
-				)
-				(justify left bottom)
+			(at 320.04 45.72 0)
+			(effects
+				(font
+					(size 1.27 1.27)
+				)
+				(hide yes)
+			)
+		)
+		(property "MANUFACTURER PART NUMBER" "CBR04C309B2GAC"
+			(at 320.04 45.72 0)
+			(effects
+				(font
+					(size 1.27 1.27)
+				)
 				(hide yes)
 			)
@@
 		(dnp no)
 		(property "Reference" "R1026_4"
-			(at 312.42 45.72 90)
-			(effects
-				(font
+			(at 307.34 45.72 90)
+			(effects
+				(font

Commit message: Changed R1037 to 50R, closes #415
Parts:
- R1037_4: value 0 -> 49.9; symbol Thunderscope_Rev5:RES 0 OHM 1/16W 0402 -> Thunderscope_Rev5:RES 49.9 OHM 1% 1/10W 0402; MANUFACTURER PART NUMBER RC0402JR-070RL -> RC0402FR-0749R9L; SUPPLIER PART NUMBER 1 603-RC0402JR-070RL -> 603-RC0402FR-0749R9L
Changed lines of the file:
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@@
 	)
 	(symbol
-		(lib_id "Thunderscope_Rev5:RES 0 OHM 1/16W 0402")
+		(lib_id "Thunderscope_Rev5:RES 49.9 OHM 1% 1/10W 0402")
 		(at 251.46 167.64 0)
 		(unit 1)
@@
 			)
 		)
-		(property "Value" "0"
+		(property "Value" "49.9"
 			(at 251.46 167.64 0)
 			(effects
@@
 		)
 		(property "PACKAGE" "0402"
-			(at 248.412 176.276 0)
+			(at 251.46 167.64 0)
 			(effects
 				(font
@@
 		)
 		(property "SUPPLIER 1" "Mouser"
-			(at 245.872 166.664 0)
+			(at 251.46 167.64 0)
 			(effects
 				(font
 					(size 1.27 1.27)
 				)
-				(justify left bottom)
 				(hide yes)
 			)
 		)
-		(property "SUPPLIER PART NUMBER 1" "603-RC0402JR-070RL"
-			(at 245.872 166.664 0)
+		(property "SUPPLIER PART NUMBER 1" "603-RC0402FR-0749R9L"
+			(at 251.46 167.64 0)
 			(effects
 				(font
 					(size 1.27 1.27)
 				)
-				(justify left bottom)
 				(hide yes)
 			)
 		)
 		(property "MANUFACTURER" "Yageo"
-			(at 245.872 164.124 0)
+			(at 251.46 167.64 0)
 			(effects
 				(font
 					(size 1.27 1.27)
 				)
-				(justify left bottom)
 				(hide yes)
 			)
 		)
 		(property "HOUSE PART NUMBER" ""
-			(at 245.872 164.124 0)
+			(at 251.46 167.64 0)
 			(effects
 				(font
 					(size 1.27 1.27)
 				)
-				(justify left bottom)
 				(hide yes)
 			)
 		)
-		(property "MANUFACTURER PART NUMBER" "RC0402JR-070RL"
-			(at 245.872 164.124 0)
+		(property "MANUFACTURER PART NUMBER" "RC0402FR-0749R9L"
+			(at 251.46 167.64 0)
 			(effects
 				(font
 					(size 1.27 1.27)
 				)
-				(justify left bottom)
 				(hide yes)
 			)
 		)
 		(property "TOLERANCE" "1%"
-			(at 245.872 166.664 0)
+			(at 251.46 167.64 0)
 			(effects
 				(font
 					(size 1.27 1.27)
 				)
-				(justify left bottom)
 				(hide yes)
 			)

Commit message: Changed R1021 & C1058 per #423
Parts:
- C1058_4: value 12pF -> 18pF; symbol Thunderscope_Rev5:CAP 12pF 50V C0G 0402 -> Thunderscope_Rev5:CAP 18pF 50V C0G 0402; MANUFACTURER PART NUMBER CBR04C120F5GAC -> CBR04C180F5GAC; SUPPLIER PART NUMBER 1 80-CBR04C120F5G -> 80-CBR04C180F5G
- R1021_4: value 16 -> 15; symbol Thunderscope_Rev5:RES 16 OHM 1% 1/3W 0603 -> Thunderscope_Rev5:RES 15 OHM 1% 1/3W 0603; MANUFACTURER PART NUMBER SG73P1JTTD16R0F -> SG73P1JTTD15R0F; SUPPLIER PART NUMBER 1 660-SG73P1JTTD16R0F -> 660-SG73P1JTTD15R0F
Changed lines of the file:
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@@
 	)
 	(symbol
-		(lib_id "Thunderscope_Rev5:RES 16 OHM 1% 1/3W 0603")
+		(lib_id "Thunderscope_Rev5:RES 15 OHM 1% 1/3W 0603")
 		(at 137.16 33.02 0)
 		(unit 1)
@@
 			)
 		)
-		(property "Value" "16"
+		(property "Value" "15"
 			(at 137.16 33.02 0)
 			(effects
@@
 		)
 		(property "TOLERANCE" "1%"
-			(at 134.112 41.656 0)
+			(at 137.16 33.02 0)
 			(effects
 				(font
@@
 		)
 		(property "PACKAGE" "0603"
-			(at 134.62 35.56 0)
+			(at 137.16 33.02 0)
 			(effects
 				(font
@@
 		)
 		(property "SUPPLIER 1" "Mouser"
-			(at 131.572 29.504 0)
+			(at 137.16 33.02 0)
 			(effects
 				(font
 					(size 1.27 1.27)
 				)
-				(justify left bottom)
 				(hide yes)
 			)
 		)
-		(property "SUPPLIER PART NUMBER 1" "660-SG73P1JTTD16R0F"
-			(at 131.572 29.504 0)
+		(property "SUPPLIER PART NUMBER 1" "660-SG73P1JTTD15R0F"
+			(at 137.16 33.02 0)
 			(effects
 				(font
 					(size 1.27 1.27)
 				)
-				(justify left bottom)
 				(hide yes)
 			)
 		)
 		(property "HOUSE PART NUMBER" ""
-			(at 131.572 29.21 0)
+			(at 137.16 33.02 0)
 			(effects
 				(font
 					(size 1.27 1.27)
 				)
-				(justify left bottom)
 				(hide yes)
 			)
 		)
 		(property "MANUFACTURER" "KOA Speer"
-			(at 131.572 29.21 0)
+			(at 137.16 33.02 0)
 			(effects
 				(font
 					(size 1.27 1.27)
 				)
-				(justify left bottom)
 				(hide yes)
 			)
 		)
-		(property "MANUFACTURER PART NUMBER" "SG73P1JTTD16R0F"
-			(at 131.572 29.21 0)
+		(property "MANUFACTURER PART NUMBER" "SG73P1JTTD15R0F"
+			(at 137.16 33.02 0)
 			(effects
 				(font
 					(size 1.27 1.27)
 				)
-				(justify left bottom)
 				(hide yes)
 			)
@@
 	)
 	(symbol
-		(lib_id "Thunderscope_Rev5:CAP 12pF 50V C0G 0402")
+		(lib_id "Thunderscope_Rev5:CAP 18pF 50V C0G 0402")
 		(at 129.54 27.94 90)
 		(unit 1)
@@
 			)
 		)
-		(property "Value" "12pF"
+		(property "Value" "18pF"
 			(at 130.81 29.21 90)
 			(effects
@@
 			)
 		)
-		(property "SUPPLIER PART NUMBER 1" "80-CBR04C120F5G"
+		(property "SUPPLIER PART NUMBER 1" "80-CBR04C180F5G"
 			(at 125.032 30.194 0)
 			(effects
@@
 			)
 		)
-		(property "MANUFACTURER PART NUMBER" "CBR04C120F5GAC"
+		(property "MANUFACTURER PART NUMBER" "CBR04C180F5GAC"
 			(at 123.952 30.194 0)
 			(effects

Commit message: DNP'd Keystone TPs and Excluded PCIe Bracket and Shield LID from BOM
Parts:
- SHLD1000_4: now left out of the parts list
Changed lines of the file:
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@@
 		(unit 1)
 		(exclude_from_sim no)
-		(in_bom yes)
+		(in_bom no)
 		(on_board no)
 		(dnp no)
