File: Hardware/KiCad/Thunderscope_Rev5.3/Thunderscope_Rev5.3.kicad_sch (KiCad schematic)
At the start: 16 parts

Commit message: Schematic Changes for #424
Other:
- added sheet ADC Driver 1 (ADC_Driver.kicad_sch)
- added sheet ADC Driver 2 (ADC_Driver.kicad_sch)
- added sheet ADC Driver 3 (ADC_Driver.kicad_sch)
- added sheet ADC Driver 4 (ADC_Driver.kicad_sch)
- moved on the sheet: EMI1, EMI2, HS1

Commit message: DNP'd Keystone TPs and Excluded PCIe Bracket and Shield LID from BOM
Parts:
- TP2, TP3, TP45, TP73, TP74: now not fitted
Changed lines of the file:
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@@
 		(in_bom yes)
 		(on_board yes)
-		(dnp no)
+		(dnp yes)
 		(property "Reference" "TP2"
 			(at 246.38 163.83 0)
@@
 		(in_bom yes)
 		(on_board yes)
-		(dnp no)
+		(dnp yes)
 		(property "Reference" "TP73"
 			(at 269.24 163.83 0)
@@
 		(in_bom yes)
 		(on_board yes)
-		(dnp no)
+		(dnp yes)
 		(property "Reference" "TP45"
 			(at 261.62 163.83 0)
@@
 		(in_bom yes)
 		(on_board yes)
-		(dnp no)
+		(dnp yes)
 		(property "Reference" "TP3"
 			(at 254 163.83 0)
@@
 		(in_bom yes)
 		(on_board yes)
-		(dnp no)
+		(dnp yes)
 		(property "Reference" "TP74"
 			(at 276.86 163.83 0)

Commit message: Exclude Heatsink From BOM
Parts:
- HS1: now left out of the parts list
Changed lines of the file:
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@@
 		(unit 1)
 		(exclude_from_sim no)
-		(in_bom yes)
+		(in_bom no)
 		(on_board yes)
 		(dnp no)
