File: Hardware/KiCad/Thunderscope_Rev5.3/M2_KEY_M.kicad_sch (KiCad schematic)
At the start: 50 parts, among them J1 BNC, J10 009155002852006, J11 7793, J2 BNC, J8 M.2 Key M, U17 TPS61023

Commit message: Changed PCIe caps to 220nF, closes #420
Parts:
- C30, C31, C34, C35, C38, C39, C42, C43: value 100nF -> 220nF; symbol Thunderscope_Rev5:CAP 100nF 16V X7R 0402 -> Thunderscope_Rev5:CAP 220nF 16V X7R 0402; MANUFACTURER PART NUMBER GCM155R71C104KA55D -> GCM155R71C224KE02D; SUPPLIER PART NUMBER 1 81-GCM155R71C104KA5D -> 81-GCM155R71C224KE2D
Changed lines of the file:
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@@
 	)
 	(symbol
-		(lib_id "Thunderscope_Rev5:CAP 100nF 16V X7R 0402")
+		(lib_id "Thunderscope_Rev5:CAP 220nF 16V X7R 0402")
 		(at 88.9 38.1 270)
 		(mirror x)
@@
 			)
 		)
-		(property "Value" "100nF"
+		(property "Value" "220nF"
 			(at 87.63 39.37 90)
 			(effects
@@
 			)
 		)
-		(property "SUPPLIER PART NUMBER 1" "81-GCM155R71C104KA5D"
+		(property "SUPPLIER PART NUMBER 1" "81-GCM155R71C224KE2D"
 			(at 91.154 43.688 0)
 			(effects
@@
 			)
 		)
-		(property "MANUFACTURER PART NUMBER" "GCM155R71C104KA55D"
+		(property "MANUFACTURER PART NUMBER" "GCM155R71C224KE02D"
 			(at 91.44 45.72 0)
 			(effects
@@
 	)
 	(symbol
-		(lib_id "Thunderscope_Rev5:CAP 100nF 16V X7R 0402")
+		(lib_id "Thunderscope_Rev5:CAP 220nF 16V X7R 0402")
 		(at 93.98 50.8 270)
 		(mirror x)
@@
 			)
 		)
-		(property "Value" "100nF"
+		(property "Value" "220nF"
 			(at 95.25 52.07 90)
 			(effects
@@
 			)
 		)
-		(property "SUPPLIER PART NUMBER 1" "81-GCM155R71C104KA5D"
+		(property "SUPPLIER PART NUMBER 1" "81-GCM155R71C224KE2D"
 			(at 96.234 56.388 0)
 			(effects
@@
 			)
 		)
-		(property "MANUFACTURER PART NUMBER" "GCM155R71C104KA55D"
+		(property "MANUFACTURER PART NUMBER" "GCM155R71C224KE02D"
 			(at 96.52 58.42 0)
 			(effects
@@
 	)
 	(symbol
-		(lib_id "Thunderscope_Rev5:CAP 100nF 16V X7R 0402")
+		(lib_id "Thunderscope_Rev5:CAP 220nF 16V X7R 0402")
 		(at 88.9 68.58 270)
 		(mirror x)
@@
 			)
 		)
-		(property "Value" "100nF"
+		(property "Value" "220nF"
 			(at 87.63 69.85 90)
 			(effects
@@
 			)
 		)
-		(property "SUPPLIER PART NUMBER 1" "81-GCM155R71C104KA5D"
+		(property "SUPPLIER PART NUMBER 1" "81-GCM155R71C224KE2D"
 			(at 91.154 74.168 0)
 			(effects
@@
 			)
 		)
-		(property "MANUFACTURER PART NUMBER" "GCM155R71C104KA55D"
+		(property "MANUFACTURER PART NUMBER" "GCM155R71C224KE02D"
 			(at 91.44 76.2 0)
 			(effects
@@
 	)
 	(symbol
-		(lib_id "Thunderscope_Rev5:CAP 100nF 16V X7R 0402")
+		(lib_id "Thunderscope_Rev5:CAP 220nF 16V X7R 0402")
 		(at 93.98 66.04 270)
 		(mirror x)
@@
 			)
 		)
-		(property "Value" "100nF"
+		(property "Value" "220nF"
 			(at 95.25 67.31 90)
 			(effects
@@
 			)
 		)
-		(property "SUPPLIER PART NUMBER 1" "81-GCM155R71C104KA5D"
+		(property "SUPPLIER PART NUMBER 1" "81-GCM155R71C224KE2D"
 			(at 96.234 71.628 0)
 			(effects
@@
 			)
 		)
-		(property "MANUFACTURER PART NUMBER" "GCM155R71C104KA55D"
+		(property "MANUFACTURER PART NUMBER" "GCM155R71C224KE02D"
 			(at 96.52 73.66 0)
 			(effects
@@
 	)
 	(symbol
-		(lib_id "Thunderscope_Rev5:CAP 100nF 16V X7R 0402")
+		(lib_id "Thunderscope_Rev5:CAP 220nF 16V X7R 0402")
 		(at 88.9 53.34 270)
 		(mirror x)
@@
 			)
 		)
-		(property "Value" "100nF"
+		(property "Value" "220nF"
 			(at 87.63 54.61 90)
 			(effects
@@
 			)
 		)
-		(property "SUPPLIER PART NUMBER 1" "81-GCM155R71C104KA5D"
+		(property "SUPPLIER PART NUMBER 1" "81-GCM155R71C224KE2D"
 			(at 91.154 58.928 0)
 			(effects
@@
 			)
 		)
-		(property "MANUFACTURER PART NUMBER" "GCM155R71C104KA55D"
+		(property "MANUFACTURER PART NUMBER" "GCM155R71C224KE02D"
 			(at 91.44 60.96 0)
 			(effects
@@
 	)
 	(symbol
-		(lib_id "Thunderscope_Rev5:CAP 100nF 16V X7R 0402")
+		(lib_id "Thunderscope_Rev5:CAP 220nF 16V X7R 0402")
 		(at 88.9 83.82 270)
 		(mirror x)
@@
 			)
 		)
-		(property "Value" "100nF"
+		(property "Value" "220nF"
 			(at 87.63 85.09 90)
 			(effects
@@
 			)
 		)
-		(property "SUPPLIER PART NUMBER 1" "81-GCM155R71C104KA5D"
+		(property "SUPPLIER PART NUMBER 1" "81-GCM155R71C224KE2D"
 			(at 91.154 89.408 0)
 			(effects
@@
 			)
 		)
-		(property "MANUFACTURER PART NUMBER" "GCM155R71C104KA55D"
+		(property "MANUFACTURER PART NUMBER" "GCM155R71C224KE02D"
 			(at 91.44 91.44 0)
 			(effects
@@
 	)
 	(symbol
-		(lib_id "Thunderscope_Rev5:CAP 100nF 16V X7R 0402")
+		(lib_id "Thunderscope_Rev5:CAP 220nF 16V X7R 0402")
 		(at 93.98 35.56 270)
 		(mirror x)
@@
 			)
 		)
-		(property "Value" "100nF"
+		(property "Value" "220nF"
 			(at 95.25 36.83 90)
 			(effects
@@
 			)
 		)
-		(property "SUPPLIER PART NUMBER 1" "81-GCM155R71C104KA5D"
+		(property "SUPPLIER PART NUMBER 1" "81-GCM155R71C224KE2D"
 			(at 96.234 41.148 0)
 			(effects
@@
 			)
 		)
-		(property "MANUFACTURER PART NUMBER" "GCM155R71C104KA55D"
+		(property "MANUFACTURER PART NUMBER" "GCM155R71C224KE02D"
 			(at 96.52 43.18 0)
 			(effects
@@
 	)
 	(symbol
-		(lib_id "Thunderscope_Rev5:CAP 100nF 16V X7R 0402")
+		(lib_id "Thunderscope_Rev5:CAP 220nF 16V X7R 0402")
 		(at 93.98 81.28 270)
 		(mirror x)
@@
 			)
 		)
-		(property "Value" "100nF"
+		(property "Value" "220nF"
 			(at 95.25 82.55 90)
 			(effects
@@
 			)
 		)
-		(property "SUPPLIER PART NUMBER 1" "81-GCM155R71C104KA5D"
+		(property "SUPPLIER PART NUMBER 1" "81-GCM155R71C224KE2D"
 			(at 96.234 86.868 0)
 			(effects
@@
 			)
 		)
-		(property "MANUFACTURER PART NUMBER" "GCM155R71C104KA55D"
+		(property "MANUFACTURER PART NUMBER" "GCM155R71C224KE02D"
 			(at 96.52 88.9 0)
 			(effects

Commit message: Schematic Changes for #421
Also changed sch note re: pcie coupling caps
Other:
- note added: "AC Couple PER Lines with 220nF"
- note removed: "AC Couple PER Lines with 100nF"
Changed lines of the file:
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@@
 		)
 	)
-	(text "AC Couple PER Lines with 100nF"
+	(text "AC Couple PER Lines with 220nF"
 		(exclude_from_sim no)
 		(at 76.2 114.3 0)

Commit message: Cleaned up unused layers
Some footprints had assembly outline on random user layers
Parts:
- SO1, SO2, SO3: footprint ThunderScope:M2_SMT_Standoff_9774025243R -> Thunderscope_Rev5:STANDOFF_M2_9774025243R; symbol ThunderScope:M2_2.5mm_SMT_Standoff_9774025243R -> Thunderscope_Rev5:STANDOFF_M2_9774025243R
Changed lines of the file:
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@@
 	)
 	(symbol
-		(lib_id "ThunderScope:M2_2.5mm_SMT_Standoff_9774025243R")
+		(lib_id "Thunderscope_Rev5:STANDOFF_M2_9774025243R")
 		(at 38.1 185.42 0)
 		(unit 1)
@@
 			)
 		)
-		(property "Footprint" "ThunderScope:M2_SMT_Standoff_9774025243R"
+		(property "Footprint" "Thunderscope_Rev5:STANDOFF_M2_9774025243R"
 			(at 38.1 185.42 0)
 			(effects
@@
 	)
 	(symbol
-		(lib_id "ThunderScope:M2_2.5mm_SMT_Standoff_9774025243R")
+		(lib_id "Thunderscope_Rev5:STANDOFF_M2_9774025243R")
 		(at 99.06 185.42 0)
 		(unit 1)
@@
 			)
 		)
-		(property "Footprint" "ThunderScope:M2_SMT_Standoff_9774025243R"
+		(property "Footprint" "Thunderscope_Rev5:STANDOFF_M2_9774025243R"
 			(at 99.06 185.42 0)
 			(effects
@@
 	)
 	(symbol
-		(lib_id "ThunderScope:M2_2.5mm_SMT_Standoff_9774025243R")
+		(lib_id "Thunderscope_Rev5:STANDOFF_M2_9774025243R")
 		(at 68.58 185.42 0)
 		(unit 1)
@@
 			)
 		)
-		(property "Footprint" "ThunderScope:M2_SMT_Standoff_9774025243R"
+		(property "Footprint" "Thunderscope_Rev5:STANDOFF_M2_9774025243R"
 			(at 68.58 185.42 0)
 			(effects

Commit message: DNP'd Keystone TPs and Excluded PCIe Bracket and Shield LID from BOM
Parts:
- TP19, TP20: now not fitted
Changed lines of the file:
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@@
 		(in_bom yes)
 		(on_board yes)
-		(dnp no)
+		(dnp yes)
 		(property "Reference" "TP19"
 			(at 60.96 146.05 0)
@@
 		(in_bom yes)
 		(on_board yes)
-		(dnp no)
+		(dnp yes)
 		(property "Reference" "TP20"
 			(at 81.28 146.05 0)

Commit message: Changed C100 to 18pF from 12pF for BOM consolidation
Parts:
- C100: value 12pF -> 18pF; symbol Thunderscope_Rev5:CAP 12pF 50V C0G 0402 -> Thunderscope_Rev5:CAP 18pF 50V C0G 0402; MANUFACTURER PART NUMBER CBR04C120F5GAC -> CBR04C180F5GAC; SUPPLIER PART NUMBER 1 80-CBR04C120F5G -> 80-CBR04C180F5G
Changed lines of the file:
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@@
 	)
 	(symbol
-		(lib_id "Thunderscope_Rev5:CAP 12pF 50V C0G 0402")
+		(lib_id "Thunderscope_Rev5:CAP 18pF 50V C0G 0402")
 		(at 246.38 147.32 0)
 		(unit 1)
@@
 			)
 		)
-		(property "Value" "12pF"
+		(property "Value" "18pF"
 			(at 248.92 148.59 0)
 			(effects
@@
 			)
 		)
-		(property "SUPPLIER PART NUMBER 1" "80-CBR04C120F5G"
+		(property "SUPPLIER PART NUMBER 1" "80-CBR04C180F5G"
 			(at 244.126 142.812 0)
 			(effects
@@
 			)
 		)
-		(property "MANUFACTURER PART NUMBER" "CBR04C120F5GAC"
+		(property "MANUFACTURER PART NUMBER" "CBR04C180F5GAC"
 			(at 244.126 141.732 0)
 			(effects
