File: Hardware/KiCad/Thunderscope_Rev5.3/CON_PCIe_X4.kicad_sch (KiCad schematic)
At the start: 53 parts, among them J3 1.27mm 6 Pin TH, J4 TSW-101-16-G-Q-RA, P1 PCIeX4-GF-2D-1000-1K-O64, U11 TPSM82913

Commit message: Changed PCIe caps to 220nF, closes #420
Parts:
- C28, C29, C32, C33, C36, C37, C40, C41: value 100nF -> 220nF; symbol Thunderscope_Rev5:CAP 100nF 16V X7R 0402 -> Thunderscope_Rev5:CAP 220nF 16V X7R 0402; MANUFACTURER PART NUMBER GCM155R71C104KA55D -> GCM155R71C224KE02D; SUPPLIER PART NUMBER 1 81-GCM155R71C104KA5D -> 81-GCM155R71C224KE2D
Changed lines of the file:
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@@
 	)
 	(symbol
-		(lib_id "Thunderscope_Rev5:CAP 100nF 16V X7R 0402")
+		(lib_id "Thunderscope_Rev5:CAP 220nF 16V X7R 0402")
 		(at 172.72 83.82 270)
 		(mirror x)
@@
 			)
 		)
-		(property "Value" "100nF"
+		(property "Value" "220nF"
 			(at 173.99 85.09 90)
 			(effects
@@
 			)
 		)
-		(property "SUPPLIER PART NUMBER 1" "81-GCM155R71C104KA5D"
+		(property "SUPPLIER PART NUMBER 1" "81-GCM155R71C224KE2D"
 			(at 174.974 89.408 0)
 			(effects
@@
 			)
 		)
-		(property "MANUFACTURER PART NUMBER" "GCM155R71C104KA55D"
+		(property "MANUFACTURER PART NUMBER" "GCM155R71C224KE02D"
 			(at 175.26 91.44 0)
 			(effects
@@
 	)
 	(symbol
-		(lib_id "Thunderscope_Rev5:CAP 100nF 16V X7R 0402")
+		(lib_id "Thunderscope_Rev5:CAP 220nF 16V X7R 0402")
 		(at 167.64 101.6 270)
 		(mirror x)
@@
 			)
 		)
-		(property "Value" "100nF"
+		(property "Value" "220nF"
 			(at 166.37 102.87 90)
 			(effects
@@
 			)
 		)
-		(property "SUPPLIER PART NUMBER 1" "81-GCM155R71C104KA5D"
+		(property "SUPPLIER PART NUMBER 1" "81-GCM155R71C224KE2D"
 			(at 169.894 107.188 0)
 			(effects
@@
 			)
 		)
-		(property "MANUFACTURER PART NUMBER" "GCM155R71C104KA55D"
+		(property "MANUFACTURER PART NUMBER" "GCM155R71C224KE02D"
 			(at 170.18 109.22 0)
 			(effects
@@
 	)
 	(symbol
-		(lib_id "Thunderscope_Rev5:CAP 100nF 16V X7R 0402")
+		(lib_id "Thunderscope_Rev5:CAP 220nF 16V X7R 0402")
 		(at 172.72 99.06 270)
 		(mirror x)
@@
 			)
 		)
-		(property "Value" "100nF"
+		(property "Value" "220nF"
 			(at 173.99 100.33 90)
 			(effects
@@
 			)
 		)
-		(property "SUPPLIER PART NUMBER 1" "81-GCM155R71C104KA5D"
+		(property "SUPPLIER PART NUMBER 1" "81-GCM155R71C224KE2D"
 			(at 174.974 104.648 0)
 			(effects
@@
 			)
 		)
-		(property "MANUFACTURER PART NUMBER" "GCM155R71C104KA55D"
+		(property "MANUFACTURER PART NUMBER" "GCM155R71C224KE02D"
 			(at 175.26 106.68 0)
 			(effects
@@
 	)
 	(symbol
-		(lib_id "Thunderscope_Rev5:CAP 100nF 16V X7R 0402")
+		(lib_id "Thunderscope_Rev5:CAP 220nF 16V X7R 0402")
 		(at 167.64 93.98 270)
 		(mirror x)
@@
 			)
 		)
-		(property "Value" "100nF"
+		(property "Value" "220nF"
 			(at 166.37 95.25 90)
 			(effects
@@
 			)
 		)
-		(property "SUPPLIER PART NUMBER 1" "81-GCM155R71C104KA5D"
+		(property "SUPPLIER PART NUMBER 1" "81-GCM155R71C224KE2D"
 			(at 169.894 99.568 0)
 			(effects
@@
 			)
 		)
-		(property "MANUFACTURER PART NUMBER" "GCM155R71C104KA55D"
+		(property "MANUFACTURER PART NUMBER" "GCM155R71C224KE02D"
 			(at 170.18 101.6 0)
 			(effects
@@
 	)
 	(symbol
-		(lib_id "Thunderscope_Rev5:CAP 100nF 16V X7R 0402")
+		(lib_id "Thunderscope_Rev5:CAP 220nF 16V X7R 0402")
 		(at 172.72 91.44 270)
 		(mirror x)
@@
 			)
 		)
-		(property "Value" "100nF"
+		(property "Value" "220nF"
 			(at 173.99 92.71 90)
 			(effects
@@
 			)
 		)
-		(property "SUPPLIER PART NUMBER 1" "81-GCM155R71C104KA5D"
+		(property "SUPPLIER PART NUMBER 1" "81-GCM155R71C224KE2D"
 			(at 174.974 97.028 0)
 			(effects
@@
 			)
 		)
-		(property "MANUFACTURER PART NUMBER" "GCM155R71C104KA55D"
+		(property "MANUFACTURER PART NUMBER" "GCM155R71C224KE02D"
 			(at 175.26 99.06 0)
 			(effects
@@
 	)
 	(symbol
-		(lib_id "Thunderscope_Rev5:CAP 100nF 16V X7R 0402")
+		(lib_id "Thunderscope_Rev5:CAP 220nF 16V X7R 0402")
 		(at 172.72 76.2 270)
 		(mirror x)
@@
 			)
 		)
-		(property "Value" "100nF"
+		(property "Value" "220nF"
 			(at 173.99 77.47 90)
 			(effects
@@
 			)
 		)
-		(property "SUPPLIER PART NUMBER 1" "81-GCM155R71C104KA5D"
+		(property "SUPPLIER PART NUMBER 1" "81-GCM155R71C224KE2D"
 			(at 174.974 81.788 0)
 			(effects
@@
 			)
 		)
-		(property "MANUFACTURER PART NUMBER" "GCM155R71C104KA55D"
+		(property "MANUFACTURER PART NUMBER" "GCM155R71C224KE02D"
 			(at 175.26 83.82 0)
 			(effects
@@
 	)
 	(symbol
-		(lib_id "Thunderscope_Rev5:CAP 100nF 16V X7R 0402")
+		(lib_id "Thunderscope_Rev5:CAP 220nF 16V X7R 0402")
 		(at 167.64 86.36 270)
 		(mirror x)
@@
 			)
 		)
-		(property "Value" "100nF"
+		(property "Value" "220nF"
 			(at 166.37 87.63 90)
 			(effects
@@
 			)
 		)
-		(property "SUPPLIER PART NUMBER 1" "81-GCM155R71C104KA5D"
+		(property "SUPPLIER PART NUMBER 1" "81-GCM155R71C224KE2D"
 			(at 169.894 91.948 0)
 			(effects
@@
 			)
 		)
-		(property "MANUFACTURER PART NUMBER" "GCM155R71C104KA55D"
+		(property "MANUFACTURER PART NUMBER" "GCM155R71C224KE02D"
 			(at 170.18 93.98 0)
 			(effects
@@
 	)
 	(symbol
-		(lib_id "Thunderscope_Rev5:CAP 100nF 16V X7R 0402")
+		(lib_id "Thunderscope_Rev5:CAP 220nF 16V X7R 0402")
 		(at 167.64 78.74 270)
 		(mirror x)
@@
 			)
 		)
-		(property "Value" "100nF"
+		(property "Value" "220nF"
 			(at 166.37 80.01 90)
 			(effects
@@
 			)
 		)
-		(property "SUPPLIER PART NUMBER 1" "81-GCM155R71C104KA5D"
+		(property "SUPPLIER PART NUMBER 1" "81-GCM155R71C224KE2D"
 			(at 169.894 84.328 0)
 			(effects
@@
 			)
 		)
-		(property "MANUFACTURER PART NUMBER" "GCM155R71C104KA55D"
+		(property "MANUFACTURER PART NUMBER" "GCM155R71C224KE02D"
 			(at 170.18 86.36 0)
 			(effects

Commit message: Schematic Changes for #421
Also changed sch note re: pcie coupling caps
Parts:
- added Q3: DMN62D0UW, Thunderscope_Rev5:GEN_SOT_323, symbol Thunderscope_Rev5:NMOS DMN62D0UW
- added R108: 10K, Thunderscope_Rev5:GEN_R_0402, symbol Thunderscope_Rev5:RES 10K OHM 1% 1/10W 0402
Connections:
- net +VUSB_PG: now also Q3.2 (G), R108.1
- net GND: now also Q3.3 (S), R108.2
- net CLKREQ#: now reaches P1.B12
- net CLKREQ#: now also Q3.1 (D)
- net PWRBRK#: now reaches P1.B30
- no-connect marks 17 -> 16
Other:
- note added: "AC Couple PER Lines with 220nF"
- note removed: "AC Couple PER Lines with 100nF"

Commit message: DNP'd Keystone TPs and Excluded PCIe Bracket and Shield LID from BOM
Parts:
- SHLD1: now left out of the parts list
- TP14, TP15: now not fitted
Changed lines of the file:
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@@
 		(unit 1)
 		(exclude_from_sim no)
-		(in_bom yes)
+		(in_bom no)
 		(on_board no)
 		(dnp no)
@@
 		(in_bom yes)
 		(on_board yes)
-		(dnp no)
+		(dnp yes)
 		(property "Reference" "TP14"
 			(at 30.48 146.05 0)
@@
 		(in_bom yes)
 		(on_board yes)
-		(dnp no)
+		(dnp yes)
 		(property "Reference" "TP15"
 			(at 45.72 146.05 0)

Commit message: Removed old schematic notes
Other:
- note removed: "DONE: 12V to VUSB Buck Regulator"
Changed lines of the file:
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@@
-		)
-	)
-	(text "DONE: 12V to VUSB Buck Regulator"
-		(exclude_from_sim no)
-		(at 35.56 190.5 0)
-		(effects
-			(font
-				(size 1.27 1.27)
-				(thickness 0.254)
-				(bold yes)
-				(color 0 194 194 1)
-			)
 		)
 	)
