File: Hardware/KiCad/Thunderscope_Rev5.3/PLL.kicad_sch (KiCad schematic)
At the start: 47 parts, among them J6 UFL, J7 UFL, U7 ZL30260LDG1, Y1 10MHz

Commit message: Changed C65 to 100nF, closes #422
Parts:
- C65: value 0 -> 100nF; footprint Thunderscope_Rev5:GEN_R_0402 -> Thunderscope_Rev5:GEN_C_0402; symbol Thunderscope_Rev5:RES 0 OHM 1/16W 0402 -> Thunderscope_Rev5:CAP 100nF 16V X7R 0402; HOUSE PART NUMBER (none) -> C-100nF-0402-002; MANUFACTURER Yageo -> Murata; MANUFACTURER PART NUMBER RC0402JR-070RL -> GCM155R71C104KA55D; SUPPLIER PART NUMBER 1 603-RC0402JR-070RL -> 81-GCM155R71C104KA5D; VOLTAGE RATING (none) -> 16V
Changed lines of the file:
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@@
 	)
 	(symbol
-		(lib_id "Thunderscope_Rev5:RES 0 OHM 1/16W 0402")
-		(at 119.38 91.44 0)
+		(lib_id "Thunderscope_Rev5:CAP 100nF 16V X7R 0402")
+		(at 119.38 91.44 270)
 		(unit 1)
 		(exclude_from_sim no)
@@
 		(dnp no)
 		(property "Reference" "C65"
-			(at 119.38 93.98 0)
+			(at 120.65 90.17 90)
 			(effects
 				(font
 					(size 1.27 1.27)
 				)
+				(justify left)
 			)
 		)
-		(property "Value" "0"
-			(at 119.38 91.44 0)
+		(property "Value" "100nF"
+			(at 120.65 92.71 90)
 			(effects
 				(font
 					(size 1.27 1.27)
 				)
+				(justify left)
 			)
 		)
-		(property "Footprint" "Thunderscope_Rev5:GEN_R_0402"
+		(property "Footprint" "Thunderscope_Rev5:GEN_C_0402"
 			(at 119.38 91.44 0)
 			(effects
@@
 		)
 		(property "PACKAGE" "0402"
-			(at 113.792 90.384 0)
+			(at 119.38 91.44 0)
 			(effects
 				(font
 					(size 1.27 1.27)
 				)
-				(justify left bottom)
 				(hide yes)
 			)
 		)
 		(property "SUPPLIER 1" "Mouser"
-			(at 113.792 90.384 0)
+			(at 119.38 91.44 0)
 			(effects
 				(font
 					(size 1.27 1.27)
 				)
-				(justify left bottom)
 				(hide yes)
 			)
 		)
-		(property "SUPPLIER PART NUMBER 1" "603-RC0402JR-070RL"
-			(at 113.792 90.384 0)
+		(property "SUPPLIER PART NUMBER 1" "81-GCM155R71C104KA5D"
+			(at 119.38 91.44 0)
 			(effects
 				(font
 					(size 1.27 1.27)
 				)
-				(justify left bottom)
 				(hide yes)
 			)
 		)
-		(property "MANUFACTURER" "Yageo"
-			(at 113.792 90.384 0)
+		(property "MANUFACTURER" "Murata"
+			(at 119.38 91.44 0)
 			(effects
 				(font
 					(size 1.27 1.27)
 				)
-				(justify left bottom)
 				(hide yes)
 			)
 		)
-		(property "HOUSE PART NUMBER" ""
-			(at 113.792 90.384 0)
+		(property "HOUSE PART NUMBER" "C-100nF-0402-002"
+			(at 119.38 91.44 0)
 			(effects
 				(font
 					(size 1.27 1.27)
 				)
-				(justify left bottom)
 				(hide yes)
 			)
 		)
-		(property "MANUFACTURER PART NUMBER" "RC0402JR-070RL"
-			(at 113.792 90.384 0)
+		(property "MANUFACTURER PART NUMBER" "GCM155R71C104KA55D"
+			(at 119.38 91.44 0)
 			(effects
 				(font
 					(size 1.27 1.27)
 				)
-				(justify left bottom)
 				(hide yes)
 			)
@@
 			)
 		)
+		(property "VOLTAGE RATING" "16V"
+			(at 119.38 91.44 0)
+			(effects
+				(font
+					(size 1.27 1.27)
+				)
+				(hide yes)
+			)
+		)

Commit message: Removed Clock Test Ports, Closing #406
Parts:
- removed C69, C70: 0, Thunderscope_Rev5:GEN_R_0402, symbol Thunderscope_Rev5:RES 0 OHM 1/16W 0402
- removed J6, J7: UFL, Thunderscope_Rev5:TE_2334884-1, symbol Thunderscope_Rev5:UFL Jack SMD
Connections:
- net ADC_CLK_R_N is gone; now on net ADC_CLK_N: U7.48 (OC6N)
- net ADC_CLK_R_P is gone; now on net ADC_CLK_P: U7.47 (OC6P)

Commit message: Removed old schematic notes
Other:
- note removed: "DONE: Replace with 50 ohm"
Changed lines of the file:
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@@
-		)
-	)
-	(text "DONE: Replace with 50 ohm"
-		(exclude_from_sim no)
-		(at 193.04 83.82 0)
-		(effects
-			(font
-				(size 1.27 1.27)
-				(thickness 0.254)
-				(bold yes)
-				(color 0 194 194 1)
-			)
 		)
 	)
