File: Hardware/KiCad/Thunderscope_Rev5.3/ADC_Driver.kicad_sch (KiCad schematic)
At the start: 12 parts, among them U12_4 ADA4930-1YCPZ

Commit message: Added PACKAGE field to symbols without it
Parts:
- U12_4: PACKAGE (none) -> 16-QFN (3x3mm)
Changed lines of the file:
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@@
+			)
+		)
+		(property "PACKAGE" "16-QFN (3x3mm)"
+			(at 160.02 109.22 0)
+			(effects
+				(font
+					(size 1.27 1.27)
+				)
+				(hide yes)
 			)
 		)

Commit message: Added Substitutions Policy Field
Parts:
- C104_4, C105_4, C69_4, C70_4, R131_4, R136_4, R137_4: Substitutions Policy (none) -> Any Parametric Equivalent
- R132_4, R133_4, R134_4, R135_4: Substitutions Policy (none) -> ECO Required for Substitution
- U12_4: Substitutions Policy (none) -> No Substitutions
Changed lines of the file:
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@@
+			)
+		)
+		(property "Substitutions Policy" "Any Parametric Equivalent"
+			(at 177.8 111.76 0)
+			(effects
+				(font
+					(size 1.27 1.27)
+				)
+				(hide yes)
 			)
 		)
@@
 			)
 		)
+		(property "Substitutions Policy" "Any Parametric Equivalent"
+			(at 109.22 86.36 0)
+			(effects
+				(font
+					(size 1.27 1.27)
+				)
+				(hide yes)
+			)
+		)
 		(pin "1"
 		)
@@
 			)
 		)
+		(property "Substitutions Policy" "No Substitutions"
+			(at 160.02 109.22 0)
+			(effects
+				(font
+					(size 1.27 1.27)
+				)
+				(hide yes)
+			)
+		)
 		(pin "4"
 		)
@@
 			)
 		)
+		(property "Substitutions Policy" "Any Parametric Equivalent"
+			(at 134.62 86.36 0)
+			(effects
+				(font
+					(size 1.27 1.27)
+				)
+				(hide yes)
+			)
+		)
 		(pin "2"
 		)
@@
 			)
 		)
+		(property "Substitutions Policy" "Any Parametric Equivalent"
+			(at 116.84 109.22 0)
+			(effects
+				(font
+					(size 1.27 1.27)
+				)
+				(hide yes)
+			)
+		)
 		(pin "2"
 		)
@@
 			)
 		)
+		(property "Substitutions Policy" "Any Parametric Equivalent"
+			(at 177.8 106.68 0)
+			(effects
+				(font
+					(size 1.27 1.27)
+				)
+				(hide yes)
+			)
+		)
 		(pin "1"
 		)
@@
 			)
 		)
+		(property "Substitutions Policy" "ECO Required for Substitution"
+			(at 127 114.3 0)
+			(effects
+				(font
+					(size 1.27 1.27)
+				)
+				(hide yes)
+			)
+		)
 		(pin "1"
 		)
@@
 			)
 		)
+		(property "Substitutions Policy" "Any Parametric Equivalent"
+			(at 180.34 124.46 0)
+			(effects
+				(font
+					(size 1.27 1.27)
+				)
+				(hide yes)
+			)
+		)
 		(pin "2"
 		)
@@
 			)
 		)
+		(property "Substitutions Policy" "ECO Required for Substitution"
+			(at 142.24 116.84 0)
+			(effects
+				(font
+					(size 1.27 1.27)
+				)
+				(hide yes)
+			)
+		)
 		(pin "1"
 		)
@@
 			)
 		)
+		(property "Substitutions Policy" "ECO Required for Substitution"
+			(at 127 104.14 0)
+			(effects
+				(font
+					(size 1.27 1.27)
+				)
+				(hide yes)
+			)
+		)
 		(pin "1"
 		)
@@
 			)
 		)
+		(property "Substitutions Policy" "ECO Required for Substitution"
+			(at 142.24 101.6 0)
+			(effects
+				(font
+					(size 1.27 1.27)
+				)
+				(hide yes)
+			)
+		)
 		(pin "1"
 		)
@@
 				(hide yes)
 			)
+		)
+		(property "Substitutions Policy" "Any Parametric Equivalent"
+			(at 121.92 86.36 0)
+			(effects
+				(font
+					(size 1.27 1.27)
+				)
+				(hide yes)
+			)
