File: Hardware/KiCad/Thunderscope_Rev5.3/FPGA_PWR.kicad_sch (KiCad schematic)
At the start: 44 parts, among them U18 IC FPGA XC7A50T-2CSG325C

Commit message: Added PACKAGE field to symbols without it
Parts:
- FB12, FB13: PACKAGE (none) -> 0402
- U18: PACKAGE (none) -> 324-BGA (15x15mm)
Changed lines of the file:
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@@
 			)
 		)
+		(property "PACKAGE" "324-BGA (15x15mm)"
+			(at 144.78 170.18 0)
+			(effects
+				(font
+					(size 1.27 1.27)
+				)
+				(hide yes)
+			)
+		)
 		(pin "H10"
 		)
@@
 			)
 		)
+		(property "PACKAGE" "324-BGA (15x15mm)"
+			(at 142.24 66.04 0)
+			(effects
+				(font
+					(size 1.27 1.27)
+				)
+				(hide yes)
+			)
+		)
 		(pin "D8"
 		)
@@
 			)
 		)
+		(property "PACKAGE" "0402"
+			(at 203.2 160.02 0)
+			(effects
+				(font
+					(size 1.27 1.27)
+				)
+				(hide yes)
+			)
+		)
 		(pin "1"
 		)
@@
 			)
 		)
+		(property "PACKAGE" "0402"
+			(at 101.6 119.38 0)
+			(effects
+				(font
+					(size 1.27 1.27)
+				)
+				(hide yes)
+			)
+		)
 		(pin "1"
 		)
@@
 			)
 		)
+		(property "PACKAGE" "324-BGA (15x15mm)"
+			(at 144.78 134.62 0)
+			(effects
+				(font
+					(size 1.27 1.27)
+				)
+				(hide yes)
+			)
+		)
 		(pin "D8"
 		)
@@
 			)
 		)
+		(property "PACKAGE" "324-BGA (15x15mm)"
+			(at 274.32 165.1 0)
+			(effects
+				(font
+					(size 1.27 1.27)
+				)
+				(hide yes)
+			)
+		)

Commit message: Added Substitutions Policy Field
Parts:
- C138, C139, C140, C141, C142, C143, C144, C145, C146, C147, C148, C149, C150, C151, C152, C153, C154, C155, C156, C157, C158, C159, C160, C161, C162, C163, C164, C165, C166, C167, C168, C169, C170, C171, C172, C173, C189, C190, C191, C86, C87: Substitutions Policy (none) -> Any Parametric Equivalent
- FB12, FB13, U18: Substitutions Policy (none) -> No Substitutions
