File: Hardware/KiCad/Thunderscope_Rev5.3/ACQ_FE_VREG.kicad_sch (KiCad schematic)
At the start: 66 parts, among them U13 LM27761, U14 TPS7A9101, U15 TPS7A9101, U16 TPS7A2033, U9 TPS7A2033

Commit message: Added PACKAGE field to symbols without it
Parts:
- U13: PACKAGE (none) -> 8-WFDFN (2x2mm)
- U14, U15: PACKAGE (none) -> 10-DFN (2.5x2.5mm)
- U16, U9: PACKAGE (none) -> SOT-23-5
Changed lines of the file:
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@@
 			)
 		)
+		(property "PACKAGE" "10-DFN (2.5x2.5mm)"
+			(at 86.36 106.68 0)
+			(effects
+				(font
+					(size 1.27 1.27)
+				)
+				(hide yes)
+			)
+		)
 		(pin "10"
 		)
@@
 			)
 		)
+		(property "PACKAGE" "SOT-23-5"
+			(at 93.98 38.1 0)
+			(effects
+				(font
+					(size 1.27 1.27)
+				)
+				(hide yes)
+			)
+		)
 		(pin "3"
 		)
@@
 			)
 		)
+		(property "PACKAGE" "10-DFN (2.5x2.5mm)"
+			(at 220.98 40.64 0)
+			(effects
+				(font
+					(size 1.27 1.27)
+				)
+				(hide yes)
+			)
+		)
 		(pin "3"
 		)
@@
 			)
 		)
+		(property "PACKAGE" "SOT-23-5"
+			(at 83.82 175.26 0)
+			(effects
+				(font
+					(size 1.27 1.27)
+				)
+				(hide yes)
+			)
+		)
 		(pin "3"
 		)
@@
 			)
 		)
+		(property "PACKAGE" "8-WFDFN (2x2mm)"
+			(at 205.74 114.3 0)
+			(effects
+				(font
+					(size 1.27 1.27)
+				)
+				(hide yes)
+			)
+		)

Commit message: Added Substitutions Policy Field
Parts:
- C103, C106, C107, C108, C109, C110, C111, C112, C114, C115, C116, C117, C118, C119, C120, C121, C122, C123, C124, C125, C126, C76, C77, C97, C98, R100, R101, R102, R103, R104, R105, R106, R111, R86, R89, R90, R93, R94, R96, R97, R98, R99: Substitutions Policy (none) -> Any Parametric Equivalent
- R91, U13, U14, U15, U16, U9: Substitutions Policy (none) -> No Substitutions

Commit message: Changed 10k,4.7k,280k resistors MPNs to RC0402FR series
Parts:
- R101, R111, R86, R94: symbol Thunderscope_Rev5:RES 10K OHM 1% 1/10W 0402 -> Thunderscope_Rev5:RES 10K OHM 1% 1/16W 0402; MANUFACTURER Panasonic -> Yageo; MANUFACTURER PART NUMBER ERJ-2RKF1002X -> RC0402FR-0710KL; SUPPLIER PART NUMBER 1 667-ERJ-2RKF1002X -> 603-RC0402FR-0710KL
- R102, R104, R99: symbol Thunderscope_Rev5:RES 4.7K OHM 1% 1/10W 0402 -> Thunderscope_Rev5:RES 4.7K OHM 1% 1/16W 0402; MANUFACTURER Panasonic -> Yageo; MANUFACTURER PART NUMBER ERJ-2RKF4701X -> RC0402FR-074K7L; SUPPLIER PART NUMBER 1 667-ERJ-2RKF4701X -> 603-RC0402FR-074K7L
- R93: MANUFACTURER PART NUMBER AC0402FR-07280KL -> RC0402FR-07280KL; SUPPLIER PART NUMBER 1 603-AC0402FR-07280KL -> 603-RC0402FR-07280KL
Changed lines of the file:
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@@
 	)
 	(symbol
-		(lib_id "Thunderscope_Rev5:RES 10K OHM 1% 1/10W 0402")
+		(lib_id "Thunderscope_Rev5:RES 10K OHM 1% 1/16W 0402")
 		(at 190.5 45.72 90)
 		(unit 1)
@@
 			)
 		)
-		(property "Description" "10 kOhms ±1% 0.1W, 1/10W Chip Resistor 0402 (1005 Metric) Automotive AEC-Q200 Thick Film"
+		(property "Description" "10 kOhms ±1% 0.063W, 1/16W Chip Resistor 0402 (1005 Metric) Moisture Resistant Thick Film"
 			(at 190.5 45.72 0)
 			(effects
@@
 			)
 		)
-		(property "SUPPLIER PART NUMBER 1" "667-ERJ-2RKF1002X"
+		(property "SUPPLIER PART NUMBER 1" "603-RC0402FR-0710KL"
 			(at 184.912 46.776 0)
 			(effects
@@
 			)
 		)
-		(property "MANUFACTURER" "Panasonic"
+		(property "MANUFACTURER" "Yageo"
 			(at 184.912 46.776 0)
 			(effects
@@
 			)
 		)
-		(property "MANUFACTURER PART NUMBER" "ERJ-2RKF1002X"
+		(property "MANUFACTURER PART NUMBER" "RC0402FR-0710KL"
 			(at 184.912 46.776 0)
 			(effects
@@
 	)
 	(symbol
-		(lib_id "Thunderscope_Rev5:RES 4.7K OHM 1% 1/10W 0402")
+		(lib_id "Thunderscope_Rev5:RES 4.7K OHM 1% 1/16W 0402")
 		(at 251.46 58.42 90)
 		(unit 1)
@@
 			)
 		)
-		(property "Description" "4.7 kOhms ±1% 0.1W, 1/10W Chip Resistor 0402 (1005 Metric) Automotive AEC-Q200 Thick Film"
+		(property "Description" "4.7 kOhms ±1% 0.063W, 1/16W Chip Resistor 0402 (1005 Metric) Moisture Resistant Thick Film"
 			(at 251.46 58.42 0)
 			(effects
@@
 			)
 		)
-		(property "SUPPLIER PART NUMBER 1" "667-ERJ-2RKF4701X"
+		(property "SUPPLIER PART NUMBER 1" "603-RC0402FR-074K7L"
 			(at 245.872 59.476 0)
 			(effects
@@
 			)
 		)
-		(property "MANUFACTURER" "Panasonic"
+		(property "MANUFACTURER" "Yageo"
 			(at 245.872 59.476 0)
 			(effects
@@
 			)
 		)
-		(property "MANUFACTURER PART NUMBER" "ERJ-2RKF4701X"
+		(property "MANUFACTURER PART NUMBER" "RC0402FR-074K7L"
 			(at 245.872 59.476 0)
 			(effects
@@
 	)
 	(symbol
-		(lib_id "Thunderscope_Rev5:RES 4.7K OHM 1% 1/10W 0402")
+		(lib_id "Thunderscope_Rev5:RES 4.7K OHM 1% 1/16W 0402")
 		(at 254 40.64 90)
 		(unit 1)
@@
 			)
 		)
-		(property "Description" "4.7 kOhms ±1% 0.1W, 1/10W Chip Resistor 0402 (1005 Metric) Automotive AEC-Q200 Thick Film"
+		(property "Description" "4.7 kOhms ±1% 0.063W, 1/16W Chip Resistor 0402 (1005 Metric) Moisture Resistant Thick Film"
 			(at 254 40.64 0)
 			(effects
@@
 			)
 		)
-		(property "SUPPLIER PART NUMBER 1" "667-ERJ-2RKF4701X"
+		(property "SUPPLIER PART NUMBER 1" "603-RC0402FR-074K7L"
 			(at 248.412 41.696 0)
 			(effects
@@
 			)
 		)
-		(property "MANUFACTURER" "Panasonic"
+		(property "MANUFACTURER" "Yageo"
 			(at 248.412 41.696 0)
 			(effects
@@
 			)
 		)
-		(property "MANUFACTURER PART NUMBER" "ERJ-2RKF4701X"
+		(property "MANUFACTURER PART NUMBER" "RC0402FR-074K7L"
 			(at 248.412 41.696 0)
 			(effects
@@
 			)
 		)
-		(property "SUPPLIER PART NUMBER 1" "603-AC0402FR-07280KL"
+		(property "SUPPLIER PART NUMBER 1" "603-RC0402FR-07280KL"
 			(at 241.3 111.76 0)
 			(effects
@@
 			)
 		)
-		(property "MANUFACTURER PART NUMBER" "AC0402FR-07280KL"
+		(property "MANUFACTURER PART NUMBER" "RC0402FR-07280KL"
 			(at 241.3 111.76 0)
 			(effects
@@
 	)
 	(symbol
-		(lib_id "Thunderscope_Rev5:RES 4.7K OHM 1% 1/10W 0402")
+		(lib_id "Thunderscope_Rev5:RES 4.7K OHM 1% 1/16W 0402")
 		(at 116.84 124.46 90)
 		(unit 1)
@@
 			)
 		)
-		(property "Description" "4.7 kOhms ±1% 0.1W, 1/10W Chip Resistor 0402 (1005 Metric) Automotive AEC-Q200 Thick Film"
+		(property "Description" "4.7 kOhms ±1% 0.063W, 1/16W Chip Resistor 0402 (1005 Metric) Moisture Resistant Thick Film"
 			(at 116.84 124.46 0)
 			(effects
@@
 			)
 		)
-		(property "SUPPLIER PART NUMBER 1" "667-ERJ-2RKF4701X"
+		(property "SUPPLIER PART NUMBER 1" "603-RC0402FR-074K7L"
 			(at 111.252 125.516 0)
 			(effects
@@
 			)
 		)
-		(property "MANUFACTURER" "Panasonic"
+		(property "MANUFACTURER" "Yageo"
 			(at 111.252 125.516 0)
 			(effects
@@
 			)
 		)
-		(property "MANUFACTURER PART NUMBER" "ERJ-2RKF4701X"
+		(property "MANUFACTURER PART NUMBER" "RC0402FR-074K7L"
 			(at 111.252 125.516 0)
 			(effects
@@
 	)
 	(symbol
-		(lib_id "Thunderscope_Rev5:RES 10K OHM 1% 1/10W 0402")
+		(lib_id "Thunderscope_Rev5:RES 10K OHM 1% 1/16W 0402")
 		(at 182.88 63.5 90)
 		(unit 1)
@@
 			)
 		)
-		(property "Description" "10 kOhms ±1% 0.1W, 1/10W Chip Resistor 0402 (1005 Metric) Automotive AEC-Q200 Thick Film"
+		(property "Description" "10 kOhms ±1% 0.063W, 1/16W Chip Resistor 0402 (1005 Metric) Moisture Resistant Thick Film"
 			(at 182.88 63.5 0)
 			(effects
@@
 			)
 		)
-		(property "SUPPLIER PART NUMBER 1" "667-ERJ-2RKF1002X"
+		(property "SUPPLIER PART NUMBER 1" "603-RC0402FR-0710KL"
 			(at 182.88 63.5 0)
 			(effects
@@
 			)
 		)
-		(property "MANUFACTURER" "Panasonic"
+		(property "MANUFACTURER" "Yageo"
 			(at 182.88 63.5 0)
 			(effects
@@
 			)
 		)
-		(property "MANUFACTURER PART NUMBER" "ERJ-2RKF1002X"
+		(property "MANUFACTURER PART NUMBER" "RC0402FR-0710KL"
 			(at 182.88 63.5 0)
 			(effects
@@
 	)
 	(symbol
-		(lib_id "Thunderscope_Rev5:RES 10K OHM 1% 1/10W 0402")
+		(lib_id "Thunderscope_Rev5:RES 10K OHM 1% 1/16W 0402")
 		(at 50.8 129.54 90)
 		(unit 1)
@@
 			)
 		)
-		(property "Description" "10 kOhms ±1% 0.1W, 1/10W Chip Resistor 0402 (1005 Metric) Automotive AEC-Q200 Thick Film"
+		(property "Description" "10 kOhms ±1% 0.063W, 1/16W Chip Resistor 0402 (1005 Metric) Moisture Resistant Thick Film"
 			(at 50.8 129.54 0)
 			(effects
@@
 			)
 		)
-		(property "SUPPLIER PART NUMBER 1" "667-ERJ-2RKF1002X"
+		(property "SUPPLIER PART NUMBER 1" "603-RC0402FR-0710KL"
 			(at 45.212 130.596 0)
 			(effects
@@
 			)
 		)
-		(property "MANUFACTURER" "Panasonic"
+		(property "MANUFACTURER" "Yageo"
 			(at 45.212 130.596 0)
 			(effects
@@
 			)
 		)
-		(property "MANUFACTURER PART NUMBER" "ERJ-2RKF1002X"
+		(property "MANUFACTURER PART NUMBER" "RC0402FR-0710KL"
 			(at 45.212 130.596 0)
 			(effects
@@
 	)
 	(symbol
-		(lib_id "Thunderscope_Rev5:RES 10K OHM 1% 1/10W 0402")
+		(lib_id "Thunderscope_Rev5:RES 10K OHM 1% 1/16W 0402")
 		(at 71.12 40.64 90)
 		(unit 1)
@@
 			)
 		)
-		(property "Description" "10 kOhms ±1% 0.1W, 1/10W Chip Resistor 0402 (1005 Metric) Automotive AEC-Q200 Thick Film"
+		(property "Description" "10 kOhms ±1% 0.063W, 1/16W Chip Resistor 0402 (1005 Metric) Moisture Resistant Thick Film"
 			(at 71.12 40.64 0)
 			(effects
@@
 			)
 		)
-		(property "SUPPLIER PART NUMBER 1" "667-ERJ-2RKF1002X"
+		(property "SUPPLIER PART NUMBER 1" "603-RC0402FR-0710KL"
 			(at 65.532 41.696 0)
 			(effects
@@
 			)
 		)
-		(property "MANUFACTURER" "Panasonic"
+		(property "MANUFACTURER" "Yageo"
 			(at 65.532 41.696 0)
 			(effects
@@
 			)
 		)
-		(property "MANUFACTURER PART NUMBER" "ERJ-2RKF1002X"
+		(property "MANUFACTURER PART NUMBER" "RC0402FR-0710KL"
 			(at 65.532 41.696 0)
 			(effects
