File: Hardware/KiCad/Thunderscope_Rev5.3/ADC.kicad_sch (KiCad schematic)
At the start: 28 parts, among them U6 HMCAD1520

Commit message: Added PACKAGE field to symbols without it
Parts:
- FB1, FB2: PACKAGE (none) -> 0402
- U6: PACKAGE (none) -> 48-QFN (7x7mm)
Changed lines of the file:
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@@
+			)
+		)
+		(property "PACKAGE" "0402"
+			(at 208.28 30.48 0)
+			(effects
+				(font
+					(size 1.27 1.27)
+				)
+				(hide yes)
 			)
 		)
@@
 			)
 		)
+		(property "PACKAGE" "0402"
+			(at 66.04 30.48 0)
+			(effects
+				(font
+					(size 1.27 1.27)
+				)
+				(hide yes)
+			)
+		)
 		(pin "1"
 		)
@@
 			)
 		)
+		(property "PACKAGE" "48-QFN (7x7mm)"
+			(at 149.86 119.38 0)
+			(effects
+				(font
+					(size 1.27 1.27)
+				)
+				(hide yes)
+			)
+		)

Commit message: Added Substitutions Policy Field
Parts:
- C14, C15, C16, C17, C18, C19, C20, C21, C23, C24, C25, C26, C27, R15, R16, R17, R22: Substitutions Policy (none) -> Any Parametric Equivalent
- FB1, FB2, U6: Substitutions Policy (none) -> No Substitutions

Commit message: Changed 10k,4.7k,280k resistors MPNs to RC0402FR series
Parts:
- R15, R16, R17: symbol Thunderscope_Rev5:RES 10K OHM 1% 1/10W 0402 -> Thunderscope_Rev5:RES 10K OHM 1% 1/16W 0402; MANUFACTURER Panasonic -> Yageo; MANUFACTURER PART NUMBER ERJ-2RKF1002X -> RC0402FR-0710KL; SUPPLIER PART NUMBER 1 667-ERJ-2RKF1002X -> 603-RC0402FR-0710KL
Changed lines of the file:
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@@
 	)
 	(symbol
-		(lib_id "Thunderscope_Rev5:RES 10K OHM 1% 1/10W 0402")
+		(lib_id "Thunderscope_Rev5:RES 10K OHM 1% 1/16W 0402")
 		(at 93.98 68.58 90)
 		(unit 1)
@@
 			)
 		)
-		(property "Description" "10 kOhms ±1% 0.1W, 1/10W Chip Resistor 0402 (1005 Metric) Automotive AEC-Q200 Thick Film"
+		(property "Description" "10 kOhms ±1% 0.063W, 1/16W Chip Resistor 0402 (1005 Metric) Moisture Resistant Thick Film"
 			(at 93.98 68.58 0)
 			(effects
@@
 			)
 		)
-		(property "SUPPLIER PART NUMBER 1" "667-ERJ-2RKF1002X"
+		(property "SUPPLIER PART NUMBER 1" "603-RC0402FR-0710KL"
 			(at 88.392 69.636 0)
 			(effects
@@
 			)
 		)
-		(property "MANUFACTURER" "Panasonic"
+		(property "MANUFACTURER" "Yageo"
 			(at 88.392 69.85 0)
 			(effects
@@
 			)
 		)
-		(property "MANUFACTURER PART NUMBER" "ERJ-2RKF1002X"
+		(property "MANUFACTURER PART NUMBER" "RC0402FR-0710KL"
 			(at 88.392 69.85 0)
 			(effects
@@
 	)
 	(symbol
-		(lib_id "Thunderscope_Rev5:RES 10K OHM 1% 1/10W 0402")
+		(lib_id "Thunderscope_Rev5:RES 10K OHM 1% 1/16W 0402")
 		(at 78.74 76.2 0)
 		(unit 1)
@@
 			)
 		)
-		(property "Description" "10 kOhms ±1% 0.1W, 1/10W Chip Resistor 0402 (1005 Metric) Automotive AEC-Q200 Thick Film"
+		(property "Description" "10 kOhms ±1% 0.063W, 1/16W Chip Resistor 0402 (1005 Metric) Moisture Resistant Thick Film"
 			(at 78.74 76.2 0)
 			(effects
@@
 			)
 		)
-		(property "SUPPLIER PART NUMBER 1" "667-ERJ-2RKF1002X"
+		(property "SUPPLIER PART NUMBER 1" "603-RC0402FR-0710KL"
 			(at 73.152 75.224 0)
 			(effects
@@
 			)
 		)
-		(property "MANUFACTURER" "Panasonic"
+		(property "MANUFACTURER" "Yageo"
 			(at 73.152 72.684 0)
 			(effects
@@
 			)
 		)
-		(property "MANUFACTURER PART NUMBER" "ERJ-2RKF1002X"
+		(property "MANUFACTURER PART NUMBER" "RC0402FR-0710KL"
 			(at 73.152 72.684 0)
 			(effects
@@
 	)
 	(symbol
-		(lib_id "Thunderscope_Rev5:RES 10K OHM 1% 1/10W 0402")
+		(lib_id "Thunderscope_Rev5:RES 10K OHM 1% 1/16W 0402")
 		(at 88.9 68.58 90)
 		(unit 1)
@@
 			)
 		)
-		(property "Description" "10 kOhms ±1% 0.1W, 1/10W Chip Resistor 0402 (1005 Metric) Automotive AEC-Q200 Thick Film"
+		(property "Description" "10 kOhms ±1% 0.063W, 1/16W Chip Resistor 0402 (1005 Metric) Moisture Resistant Thick Film"
 			(at 88.9 68.58 0)
 			(effects
@@
 			)
 		)
-		(property "SUPPLIER PART NUMBER 1" "667-ERJ-2RKF1002X"
+		(property "SUPPLIER PART NUMBER 1" "603-RC0402FR-0710KL"
 			(at 83.312 69.636 0)
 			(effects
@@
 			)
 		)
-		(property "MANUFACTURER" "Panasonic"
+		(property "MANUFACTURER" "Yageo"
 			(at 83.312 69.85 0)
 			(effects
@@
 			)
 		)
-		(property "MANUFACTURER PART NUMBER" "ERJ-2RKF1002X"
+		(property "MANUFACTURER PART NUMBER" "RC0402FR-0710KL"
 			(at 83.312 69.85 0)
 			(effects
