File: Hardware/KiCad/Thunderscope_Rev5.3/FE.kicad_sch (KiCad schematic)
At the start: 32 parts, among them Q1 DMN62D0UW, Q2 DMN62D0UW, U2 MCP4452-104E, U3 MCP4728, U4 REF2025, U5 OPA140AIDBVR

Commit message: Added PACKAGE field to symbols without it
Parts:
- Q1, Q2: PACKAGE (none) -> SOT-323
- U2: PACKAGE (none) -> 14-TSSOP
- U3: PACKAGE (none) -> 10-MSOP
- U4, U5: PACKAGE (none) -> SOT-23-5
Changed lines of the file:
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@@
 			)
 		)
+		(property "PACKAGE" "SOT-23-5"
+			(at 182.88 152.4 0)
+			(effects
+				(font
+					(size 1.27 1.27)
+				)
+				(hide yes)
+			)
+		)
 		(pin "3"
 		)
@@
 			)
 		)
+		(property "PACKAGE" "SOT-323"
+			(at 68.58 68.58 0)
+			(effects
+				(font
+					(size 1.27 1.27)
+				)
+				(hide yes)
+			)
+		)
 		(pin "1"
 		)
@@
 			)
 		)
+		(property "PACKAGE" "10-MSOP"
+			(at 137.16 60.96 0)
+			(effects
+				(font
+					(size 1.27 1.27)
+				)
+				(hide yes)
+			)
+		)
 		(pin "4"
 		)
@@
 			)
 		)
+		(property "PACKAGE" "SOT-23-5"
+			(at 76.2 124.46 0)
+			(effects
+				(font
+					(size 1.27 1.27)
+				)
+				(hide yes)
+			)
+		)
 		(pin "1"
 		)
@@
 			)
 		)
+		(property "PACKAGE" "14-TSSOP"
+			(at 226.06 45.72 0)
+			(effects
+				(font
+					(size 1.27 1.27)
+				)
+				(hide yes)
+			)
+		)
 		(pin "6"
 		)
@@
 			)
 		)
+		(property "PACKAGE" "SOT-323"
+			(at 58.42 73.66 0)
+			(effects
+				(font
+					(size 1.27 1.27)
+				)
+				(hide yes)
+			)
+		)

Commit message: Added Substitutions Policy Field
Parts:
- C11, C2, C3, C4, C5, C6, C7, C8, C82, C85, C93, C94, C95, C96, R10, R107, R11, R12, R9: Substitutions Policy (none) -> Any Parametric Equivalent
- Q1, Q2, U2, U3: Substitutions Policy (none) -> ECO Required for Substitution
- R13, U4, U5: Substitutions Policy (none) -> No Substitutions

Commit message: Changed 10k,4.7k,280k resistors MPNs to RC0402FR series
Parts:
- R10, R11, R12, R9: symbol Thunderscope_Rev5:RES 4.7K OHM 1% 1/10W 0402 -> Thunderscope_Rev5:RES 4.7K OHM 1% 1/16W 0402; MANUFACTURER Panasonic -> Yageo; MANUFACTURER PART NUMBER ERJ-2RKF4701X -> RC0402FR-074K7L; SUPPLIER PART NUMBER 1 667-ERJ-2RKF4701X -> 603-RC0402FR-074K7L
Changed lines of the file:
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@@
 	)
 	(symbol
-		(lib_id "Thunderscope_Rev5:RES 4.7K OHM 1% 1/10W 0402")
+		(lib_id "Thunderscope_Rev5:RES 4.7K OHM 1% 1/16W 0402")
 		(at 81.28 63.5 90)
 		(unit 1)
@@
 			)
 		)
-		(property "Description" "4.7 kOhms ±1% 0.1W, 1/10W Chip Resistor 0402 (1005 Metric) Automotive AEC-Q200 Thick Film"
+		(property "Description" "4.7 kOhms ±1% 0.063W, 1/16W Chip Resistor 0402 (1005 Metric) Moisture Resistant Thick Film"
 			(at 81.28 63.5 0)
 			(effects
@@
 			)
 		)
-		(property "SUPPLIER PART NUMBER 1" "667-ERJ-2RKF4701X"
+		(property "SUPPLIER PART NUMBER 1" "603-RC0402FR-074K7L"
 			(at 75.692 64.476 0)
 			(effects
@@
 			)
 		)
-		(property "MANUFACTURER" "Panasonic"
+		(property "MANUFACTURER" "Yageo"
 			(at 75.692 64.77 0)
 			(effects
@@
 			)
 		)
-		(property "MANUFACTURER PART NUMBER" "ERJ-2RKF4701X"
+		(property "MANUFACTURER PART NUMBER" "RC0402FR-074K7L"
 			(at 75.692 64.77 0)
 			(effects
@@
 	)
 	(symbol
-		(lib_id "Thunderscope_Rev5:RES 4.7K OHM 1% 1/10W 0402")
+		(lib_id "Thunderscope_Rev5:RES 4.7K OHM 1% 1/16W 0402")
 		(at 50.8 63.5 90)
 		(unit 1)
@@
 			)
 		)
-		(property "Description" "4.7 kOhms ±1% 0.1W, 1/10W Chip Resistor 0402 (1005 Metric) Automotive AEC-Q200 Thick Film"
+		(property "Description" "4.7 kOhms ±1% 0.063W, 1/16W Chip Resistor 0402 (1005 Metric) Moisture Resistant Thick Film"
 			(at 50.8 63.5 0)
 			(effects
@@
 			)
 		)
-		(property "SUPPLIER PART NUMBER 1" "667-ERJ-2RKF4701X"
+		(property "SUPPLIER PART NUMBER 1" "603-RC0402FR-074K7L"
 			(at 45.212 64.476 0)
 			(effects
@@
 			)
 		)
-		(property "MANUFACTURER" "Panasonic"
+		(property "MANUFACTURER" "Yageo"
 			(at 45.212 64.77 0)
 			(effects
@@
 			)
 		)
-		(property "MANUFACTURER PART NUMBER" "ERJ-2RKF4701X"
+		(property "MANUFACTURER PART NUMBER" "RC0402FR-074K7L"
 			(at 45.212 64.77 0)
 			(effects
@@
 	)
 	(symbol
-		(lib_id "Thunderscope_Rev5:RES 4.7K OHM 1% 1/10W 0402")
+		(lib_id "Thunderscope_Rev5:RES 4.7K OHM 1% 1/16W 0402")
 		(at 76.2 63.5 90)
 		(unit 1)
@@
 			)
 		)
-		(property "Description" "4.7 kOhms ±1% 0.1W, 1/10W Chip Resistor 0402 (1005 Metric) Automotive AEC-Q200 Thick Film"
+		(property "Description" "4.7 kOhms ±1% 0.063W, 1/16W Chip Resistor 0402 (1005 Metric) Moisture Resistant Thick Film"
 			(at 76.2 63.5 0)
 			(effects
@@
 			)
 		)
-		(property "SUPPLIER PART NUMBER 1" "667-ERJ-2RKF4701X"
+		(property "SUPPLIER PART NUMBER 1" "603-RC0402FR-074K7L"
 			(at 70.612 64.476 0)
 			(effects
@@
 			)
 		)
-		(property "MANUFACTURER" "Panasonic"
+		(property "MANUFACTURER" "Yageo"
 			(at 70.612 64.77 0)
 			(effects
@@
 			)
 		)
-		(property "MANUFACTURER PART NUMBER" "ERJ-2RKF4701X"
+		(property "MANUFACTURER PART NUMBER" "RC0402FR-074K7L"
 			(at 70.612 64.77 0)
 			(effects
@@
 	)
 	(symbol
-		(lib_id "Thunderscope_Rev5:RES 4.7K OHM 1% 1/10W 0402")
+		(lib_id "Thunderscope_Rev5:RES 4.7K OHM 1% 1/16W 0402")
 		(at 45.72 63.5 90)
 		(unit 1)
@@
 			)
 		)
-		(property "Description" "4.7 kOhms ±1% 0.1W, 1/10W Chip Resistor 0402 (1005 Metric) Automotive AEC-Q200 Thick Film"
+		(property "Description" "4.7 kOhms ±1% 0.063W, 1/16W Chip Resistor 0402 (1005 Metric) Moisture Resistant Thick Film"
 			(at 45.72 63.5 0)
 			(effects
@@
 			)
 		)
-		(property "SUPPLIER PART NUMBER 1" "667-ERJ-2RKF4701X"
+		(property "SUPPLIER PART NUMBER 1" "603-RC0402FR-074K7L"
 			(at 40.132 64.476 0)
 			(effects
@@
 			)
 		)
-		(property "MANUFACTURER" "Panasonic"
+		(property "MANUFACTURER" "Yageo"
 			(at 40.132 64.77 0)
 			(effects
@@
 			)
 		)
-		(property "MANUFACTURER PART NUMBER" "ERJ-2RKF4701X"
+		(property "MANUFACTURER PART NUMBER" "RC0402FR-074K7L"
 			(at 40.132 64.77 0)
 			(effects
