File: Hardware/KiCad/Thunderscope_Rev5.3/FPGA.kicad_sch (KiCad schematic)
At the start: 29 parts, among them J12 009155002852006, J13 009155002852006, J5 2.54mm 6 Pin TH, J9 F300-1B7H1-11036-E100, U1 SN74LVC1G17, U10 FIN1019MTCX, Y2 25MHz

Commit message: Added PACKAGE field to symbols without it
Parts:
- D1: PACKAGE (none) -> 4-SMD
- J12, J13, J9: PACKAGE (none) -> Surface Mount
- J5: PACKAGE (none) -> Through Hole
- U1: PACKAGE (none) -> SC-70-5
- U10: PACKAGE (none) -> 14-TSSOP
- Y2: PACKAGE (none) -> 4-SMD (2.0x1.6mm)
Changed lines of the file:
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@@
 			)
 		)
+		(property "PACKAGE" "Surface Mount"
+			(at 276.86 167.64 0)
+			(effects
+				(font
+					(size 1.27 1.27)
+				)
+				(hide yes)
+			)
+		)
 		(pin "1"
 		)
@@
 			)
 		)
+		(property "PACKAGE" "Through Hole"
+			(at 78.74 149.86 0)
+			(effects
+				(font
+					(size 1.27 1.27)
+				)
+				(hide yes)
+			)
+		)
 		(pin "2"
 		)
@@
 			)
 		)
+		(property "PACKAGE" "4-SMD"
+			(at 271.78 38.1 0)
+			(effects
+				(font
+					(size 1.27 1.27)
+				)
+				(hide yes)
+			)
+		)
 		(pin "4"
 		)
@@
 			)
 		)
+		(property "PACKAGE" "Surface Mount"
+			(at 276.86 152.4 0)
+			(effects
+				(font
+					(size 1.27 1.27)
+				)
+				(hide yes)
+			)
+		)
 		(pin "1"
 		)
@@
 			)
 		)
+		(property "PACKAGE" "14-TSSOP"
+			(at 233.68 88.9 0)
+			(effects
+				(font
+					(size 1.27 1.27)
+				)
+				(hide yes)
+			)
+		)
 		(pin "9"
 		)
@@
 			)
 		)
+		(property "PACKAGE" "SC-70-5"
+			(at 223.52 157.48 0)
+			(effects
+				(font
+					(size 1.27 1.27)
+				)
+				(hide yes)
+			)
+		)
 		(pin "5"
 		)
@@
 			)
 		)
+		(property "PACKAGE" "Surface Mount"
+			(at 20.32 27.94 0)
+			(effects
+				(font
+					(size 1.27 1.27)
+				)
+				(hide yes)
+			)
+		)
 		(pin "10"
 		)
@@
 			)
 		)
+		(property "PACKAGE" "4-SMD (2.0x1.6mm)"
+			(at 208.28 38.1 0)
+			(effects
+				(font
+					(size 1.27 1.27)
+				)
+				(hide yes)
+			)
+		)

Commit message: Added Substitutions Policy Field
Parts:
- C1, C130, C78, C79, R6, R60, R61, R62, R63, R64, R65, R8, R85: Substitutions Policy (none) -> Any Parametric Equivalent
- D1, J5, U1, Y2: Substitutions Policy (none) -> ECO Required for Substitution
- J12, J13, J9, U10: Substitutions Policy (none) -> No Substitutions

Commit message: Changed 10k,4.7k,280k resistors MPNs to RC0402FR series
Parts:
- R61, R62, R8: symbol Thunderscope_Rev5:RES 10K OHM 1% 1/10W 0402 -> Thunderscope_Rev5:RES 10K OHM 1% 1/16W 0402; MANUFACTURER Panasonic -> Yageo; MANUFACTURER PART NUMBER ERJ-2RKF1002X -> RC0402FR-0710KL; SUPPLIER PART NUMBER 1 667-ERJ-2RKF1002X -> 603-RC0402FR-0710KL
Changed lines of the file:
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@@
 	)
 	(symbol
-		(lib_id "Thunderscope_Rev5:RES 10K OHM 1% 1/10W 0402")
+		(lib_id "Thunderscope_Rev5:RES 10K OHM 1% 1/16W 0402")
 		(at 246.38 119.38 270)
 		(mirror x)
@@
 			)
 		)
-		(property "Description" "10 kOhms ±1% 0.1W, 1/10W Chip Resistor 0402 (1005 Metric) Automotive AEC-Q200 Thick Film"
+		(property "Description" "10 kOhms ±1% 0.063W, 1/16W Chip Resistor 0402 (1005 Metric) Moisture Resistant Thick Film"
 			(at 246.38 119.38 0)
 			(effects
@@
 			)
 		)
-		(property "SUPPLIER PART NUMBER 1" "667-ERJ-2RKF1002X"
+		(property "SUPPLIER PART NUMBER 1" "603-RC0402FR-0710KL"
 			(at 251.968 120.356 0)
 			(effects
@@
 			)
 		)
-		(property "MANUFACTURER" "Panasonic"
+		(property "MANUFACTURER" "Yageo"
 			(at 251.968 120.65 0)
 			(effects
@@
 			)
 		)
-		(property "MANUFACTURER PART NUMBER" "ERJ-2RKF1002X"
+		(property "MANUFACTURER PART NUMBER" "RC0402FR-0710KL"
 			(at 251.968 120.65 0)
 			(effects
@@
 	)
 	(symbol
-		(lib_id "Thunderscope_Rev5:RES 10K OHM 1% 1/10W 0402")
+		(lib_id "Thunderscope_Rev5:RES 10K OHM 1% 1/16W 0402")
 		(at 246.38 88.9 270)
 		(mirror x)
@@
 			)
 		)
-		(property "Description" "10 kOhms ±1% 0.1W, 1/10W Chip Resistor 0402 (1005 Metric) Automotive AEC-Q200 Thick Film"
+		(property "Description" "10 kOhms ±1% 0.063W, 1/16W Chip Resistor 0402 (1005 Metric) Moisture Resistant Thick Film"
 			(at 246.38 88.9 0)
 			(effects
@@
 			)
 		)
-		(property "SUPPLIER PART NUMBER 1" "667-ERJ-2RKF1002X"
+		(property "SUPPLIER PART NUMBER 1" "603-RC0402FR-0710KL"
 			(at 251.968 89.876 0)
 			(effects
@@
 			)
 		)
-		(property "MANUFACTURER" "Panasonic"
+		(property "MANUFACTURER" "Yageo"
 			(at 251.968 90.17 0)
 			(effects
@@
 			)
 		)
-		(property "MANUFACTURER PART NUMBER" "ERJ-2RKF1002X"
+		(property "MANUFACTURER PART NUMBER" "RC0402FR-0710KL"
 			(at 251.968 90.17 0)
 			(effects
@@
 	)
 	(symbol
-		(lib_id "Thunderscope_Rev5:RES 10K OHM 1% 1/10W 0402")
+		(lib_id "Thunderscope_Rev5:RES 10K OHM 1% 1/16W 0402")
 		(at 193.04 165.1 270)
 		(mirror x)
@@
 			)
 		)
-		(property "Description" "10 kOhms ±1% 0.1W, 1/10W Chip Resistor 0402 (1005 Metric) Automotive AEC-Q200 Thick Film"
+		(property "Description" "10 kOhms ±1% 0.063W, 1/16W Chip Resistor 0402 (1005 Metric) Moisture Resistant Thick Film"
 			(at 193.04 165.1 0)
 			(effects
@@
 			)
 		)
-		(property "SUPPLIER PART NUMBER 1" "667-ERJ-2RKF1002X"
+		(property "SUPPLIER PART NUMBER 1" "603-RC0402FR-0710KL"
 			(at 198.628 166.076 0)
 			(effects
@@
 			)
 		)
-		(property "MANUFACTURER" "Panasonic"
+		(property "MANUFACTURER" "Yageo"
 			(at 198.628 166.37 0)
 			(effects
@@
 			)
 		)
-		(property "MANUFACTURER PART NUMBER" "ERJ-2RKF1002X"
+		(property "MANUFACTURER PART NUMBER" "RC0402FR-0710KL"
 			(at 198.628 166.37 0)
 			(effects
