File: Hardware/KiCad/Thunderscope_Rev5.3/FPGA_CFG_MGT.kicad_sch (KiCad schematic)
At the start: 21 parts, among them U18 IC FPGA XC7A50T-2CSG325C, U19 MX25L6433FZNI-08G

Commit message: Added PACKAGE field to symbols without it
Parts:
- FB11: PACKAGE (none) -> 0402
- U18: PACKAGE (none) -> 324-BGA (15x15mm)
- U19: PACKAGE (none) -> 8-WSON (6x5mm)
Changed lines of the file:
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@@
+			)
+		)
+		(property "PACKAGE" "8-WSON (6x5mm)"
+			(at 220.98 60.96 0)
+			(effects
+				(font
+					(size 1.27 1.27)
+				)
+				(hide yes)
 			)
 		)
@@
 			)
 		)
+		(property "PACKAGE" "324-BGA (15x15mm)"
+			(at 127 165.1 0)
+			(effects
+				(font
+					(size 1.27 1.27)
+				)
+				(hide yes)
+			)
+		)
 		(pin "A17"
 		)
@@
 					(size 1.27 1.27)
 				)
+			)
+		)
+		(property "PACKAGE" "0402"
+			(at 111.76 93.98 0)
+			(effects
+				(font
+					(size 1.27 1.27)
+				)
+				(hide yes)
 			)
 		)
@@
 			)
 		)
+		(property "PACKAGE" "324-BGA (15x15mm)"
+			(at 93.98 25.4 0)
+			(effects
+				(font
+					(size 1.27 1.27)
+				)
+				(hide yes)
+			)
+		)

Commit message: Added Substitutions Policy Field
Parts:
- C129, R113, R114, R115, R66, R67, R68: Substitutions Policy (none) -> Any Parametric Equivalent
- FB11, U18: Substitutions Policy (none) -> No Substitutions
- U19: Substitutions Policy (none) -> ECO Required for Substitution
Changed lines of the file:
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@@
 			)
 		)
+		(property "Substitutions Policy" "ECO Required for Substitution"
+			(at 220.98 60.96 0)
+			(effects
+				(font
+					(size 1.27 1.27)
+				)
+				(hide yes)
+			)
+		)
 		(pin "2"
 		)
@@
 			)
 		)
+		(property "Substitutions Policy" "Any Parametric Equivalent"
+			(at 185.42 45.72 0)
+			(effects
+				(font
+					(size 1.27 1.27)
+				)
+				(hide yes)
+			)
+		)
 		(pin "2"
 		)
@@
 			)
 		)
+		(property "Substitutions Policy" "No Substitutions"
+			(at 127 165.1 0)
+			(effects
+				(font
+					(size 1.27 1.27)
+				)
+				(hide yes)
+			)
+		)
 		(pin "A17"
 		)
@@
 			)
 		)
+		(property "Substitutions Policy" "Any Parametric Equivalent"
+			(at 111.76 55.88 0)
+			(effects
+				(font
+					(size 1.27 1.27)
+				)
+				(hide yes)
+			)
+		)
 		(pin "2"
 		)
@@
 			)
 		)
+		(property "Substitutions Policy" ""
+			(at 177.8 78.74 90)
+			(effects
+				(font
+					(size 1.27 1.27)
+				)
+				(hide yes)
+			)
+		)
 		(pin "1"
 		)
@@
 			)
 		)
+		(property "Substitutions Policy" ""
+			(at 121.92 53.34 0)
+			(effects
+				(font
+					(size 1.27 1.27)
+				)
+				(hide yes)
+			)
+		)
 		(pin "1"
 		)
@@
 			)
 		)
+		(property "Substitutions Policy" "Any Parametric Equivalent"
+			(at 175.26 45.72 0)
+			(effects
+				(font
+					(size 1.27 1.27)
+				)
+				(hide yes)
+			)
+		)
 		(pin "2"
 		)
@@
 			)
 		)
+		(property "Substitutions Policy" ""
+			(at 167.64 50.8 90)
+			(effects
+				(font
+					(size 1.27 1.27)
+				)
+				(hide yes)
+			)
+		)
 		(pin "1"
 		)
@@
 			)
 		)
+		(property "Substitutions Policy" "No Substitutions"
+			(at 111.76 93.98 0)
+			(effects
+				(font
+					(size 1.27 1.27)
+				)
+				(hide yes)
+			)
+		)
 		(pin "2"
 		)
@@
 			)
 		)
+		(property "Substitutions Policy" ""
+			(at 160.02 58.42 90)
+			(effects
+				(font
+					(size 1.27 1.27)
+				)
+				(hide yes)
+			)
+		)
 		(pin "1"
 		)
@@
 			)
 		)
+		(property "Substitutions Policy" ""
+			(at 182.88 78.74 90)
+			(effects
+				(font
+					(size 1.27 1.27)
+				)
+				(hide yes)
+			)
+		)
 		(pin "1"
 		)
@@
 			)
 		)
+		(property "Substitutions Policy" ""
+			(at 187.96 78.74 90)
+			(effects
+				(font
+					(size 1.27 1.27)
+				)
+				(hide yes)
+			)
+		)
 		(pin "1"
 		)
@@
 			)
 		)
+		(property "Substitutions Policy" ""
+			(at 124.46 25.4 90)
+			(effects
+				(font
+					(size 1.27 1.27)
+				)
+				(hide yes)
+			)
+		)
 		(pin "1"
 		)
@@
 			)
 		)
+		(property "Substitutions Policy" "Any Parametric Equivalent"
+			(at 243.84 60.96 0)
+			(effects
+				(font
+					(size 1.27 1.27)
+				)
+				(hide yes)
+			)
+		)
 		(pin "1"
 		)
@@
 			)
 		)
+		(property "Substitutions Policy" "No Substitutions"
+			(at 93.98 25.4 0)
+			(effects
+				(font
+					(size 1.27 1.27)
+				)
+				(hide yes)
+			)
+		)
 		(pin "K1"
 		)
@@
 			)
 		)
+		(property "Substitutions Policy" ""
+			(at 119.38 25.4 90)
+			(effects
+				(font
+					(size 1.27 1.27)
+				)
+				(hide yes)
+			)
+		)
 		(pin "1"
 		)
@@
 			)
 		)
+		(property "Substitutions Policy" ""
+			(at 114.3 25.4 90)
+			(effects
+				(font
+					(size 1.27 1.27)
+				)
+				(hide yes)
+			)
+		)
 		(pin "1"
 		)
@@
 			)
 		)
+		(property "Substitutions Policy" "Any Parametric Equivalent"
+			(at 193.04 162.56 0)
+			(effects
+				(font
+					(size 1.27 1.27)
+				)
+				(hide yes)
+			)
+		)
 		(pin "2"
 		)
@@
 			)
 		)
+		(property "Substitutions Policy" "Any Parametric Equivalent"
+			(at 180.34 45.72 0)
+			(effects
+				(font
+					(size 1.27 1.27)
+				)
+				(hide yes)
+			)
+		)
 		(pin "2"
 		)
@@
 			)
 		)
+		(property "Substitutions Policy" ""
+			(at 172.72 78.74 90)
+			(effects
+				(font
+					(size 1.27 1.27)
+				)
+				(hide yes)
+			)
+		)
 		(pin "1"
 		)
@@
 			)
 		)
+		(property "Substitutions Policy" ""
+			(at 109.22 25.4 90)
+			(effects
+				(font
+					(size 1.27 1.27)
+				)
+				(hide yes)
+			)
+		)
 		(pin "1"
 		)
@@
 			)
 		)
+		(property "Substitutions Policy" "Any Parametric Equivalent"
+			(at 111.76 60.96 0)
+			(effects
+				(font
+					(size 1.27 1.27)
+				)
+				(hide yes)
+			)
+		)

Commit message: Changed 10k,4.7k,280k resistors MPNs to RC0402FR series
Parts:
- R113, R114: symbol Thunderscope_Rev5:RES 4.7K OHM 1% 1/10W 0402 -> Thunderscope_Rev5:RES 4.7K OHM 1% 1/16W 0402; MANUFACTURER Panasonic -> Yageo; MANUFACTURER PART NUMBER ERJ-2RKF4701X -> RC0402FR-074K7L; SUPPLIER PART NUMBER 1 667-ERJ-2RKF4701X -> 603-RC0402FR-074K7L
- R66, R67, R68: symbol Thunderscope_Rev5:RES 10K OHM 1% 1/10W 0402 -> Thunderscope_Rev5:RES 10K OHM 1% 1/16W 0402; MANUFACTURER Panasonic -> Yageo; MANUFACTURER PART NUMBER ERJ-2RKF1002X -> RC0402FR-0710KL; SUPPLIER PART NUMBER 1 667-ERJ-2RKF1002X -> 603-RC0402FR-0710KL
Changed lines of the file:
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@@
 	)
 	(symbol
-		(lib_id "Thunderscope_Rev5:RES 10K OHM 1% 1/10W 0402")
+		(lib_id "Thunderscope_Rev5:RES 10K OHM 1% 1/16W 0402")
 		(at 185.42 45.72 270)
 		(unit 1)
@@
 			)
 		)
-		(property "Description" "10 kOhms ±1% 0.1W, 1/10W Chip Resistor 0402 (1005 Metric) Automotive AEC-Q200 Thick Film"
+		(property "Description" "10 kOhms ±1% 0.063W, 1/16W Chip Resistor 0402 (1005 Metric) Moisture Resistant Thick Film"
 			(at 185.42 45.72 0)
 			(effects
@@
 			)
 		)
-		(property "SUPPLIER PART NUMBER 1" "667-ERJ-2RKF1002X"
+		(property "SUPPLIER PART NUMBER 1" "603-RC0402FR-0710KL"
 			(at 191.008 44.664 0)
 			(effects
@@
 			)
 		)
-		(property "MANUFACTURER" "Panasonic"
+		(property "MANUFACTURER" "Yageo"
 			(at 191.008 44.664 0)
 			(effects
@@
 			)
 		)
-		(property "MANUFACTURER PART NUMBER" "ERJ-2RKF1002X"
+		(property "MANUFACTURER PART NUMBER" "RC0402FR-0710KL"
 			(at 191.008 44.664 0)
 			(effects
@@
 	)
 	(symbol
-		(lib_id "Thunderscope_Rev5:RES 4.7K OHM 1% 1/10W 0402")
+		(lib_id "Thunderscope_Rev5:RES 4.7K OHM 1% 1/16W 0402")
 		(at 111.76 55.88 0)
 		(unit 1)
@@
 			)
 		)
-		(property "Description" "4.7 kOhms ±1% 0.1W, 1/10W Chip Resistor 0402 (1005 Metric) Automotive AEC-Q200 Thick Film"
+		(property "Description" "4.7 kOhms ±1% 0.063W, 1/16W Chip Resistor 0402 (1005 Metric) Moisture Resistant Thick Film"
 			(at 111.76 55.88 0)
 			(effects
@@
 			)
 		)
-		(property "SUPPLIER PART NUMBER 1" "667-ERJ-2RKF4701X"
+		(property "SUPPLIER PART NUMBER 1" "603-RC0402FR-074K7L"
 			(at 106.172 54.824 0)
 			(effects
@@
 			)
 		)
-		(property "MANUFACTURER" "Panasonic"
+		(property "MANUFACTURER" "Yageo"
 			(at 102.936 53.34 0)
 			(effects
@@
 			)
 		)
-		(property "MANUFACTURER PART NUMBER" "ERJ-2RKF4701X"
+		(property "MANUFACTURER PART NUMBER" "RC0402FR-074K7L"
 			(at 102.936 53.34 0)
 			(effects
@@
 	)
 	(symbol
-		(lib_id "Thunderscope_Rev5:RES 10K OHM 1% 1/10W 0402")
+		(lib_id "Thunderscope_Rev5:RES 10K OHM 1% 1/16W 0402")
 		(at 175.26 45.72 90)
 		(unit 1)
@@
 			)
 		)
-		(property "Description" "10 kOhms ±1% 0.1W, 1/10W Chip Resistor 0402 (1005 Metric) Automotive AEC-Q200 Thick Film"
+		(property "Description" "10 kOhms ±1% 0.063W, 1/16W Chip Resistor 0402 (1005 Metric) Moisture Resistant Thick Film"
 			(at 175.26 45.72 0)
 			(effects
@@
 			)
 		)
-		(property "SUPPLIER PART NUMBER 1" "667-ERJ-2RKF1002X"
+		(property "SUPPLIER PART NUMBER 1" "603-RC0402FR-0710KL"
 			(at 169.672 46.776 0)
 			(effects
@@
 			)
 		)
-		(property "MANUFACTURER" "Panasonic"
+		(property "MANUFACTURER" "Yageo"
 			(at 169.672 46.776 0)
 			(effects
@@
 			)
 		)
-		(property "MANUFACTURER PART NUMBER" "ERJ-2RKF1002X"
+		(property "MANUFACTURER PART NUMBER" "RC0402FR-0710KL"
 			(at 169.672 46.776 0)
 			(effects
@@
 	)
 	(symbol
-		(lib_id "Thunderscope_Rev5:RES 10K OHM 1% 1/10W 0402")
+		(lib_id "Thunderscope_Rev5:RES 10K OHM 1% 1/16W 0402")
 		(at 180.34 45.72 90)
 		(unit 1)
@@
 			)
 		)
-		(property "Description" "10 kOhms ±1% 0.1W, 1/10W Chip Resistor 0402 (1005 Metric) Automotive AEC-Q200 Thick Film"
+		(property "Description" "10 kOhms ±1% 0.063W, 1/16W Chip Resistor 0402 (1005 Metric) Moisture Resistant Thick Film"
 			(at 180.34 45.72 0)
 			(effects
@@
 			)
 		)
-		(property "SUPPLIER PART NUMBER 1" "667-ERJ-2RKF1002X"
+		(property "SUPPLIER PART NUMBER 1" "603-RC0402FR-0710KL"
 			(at 174.752 46.776 0)
 			(effects
@@
 			)
 		)
-		(property "MANUFACTURER" "Panasonic"
+		(property "MANUFACTURER" "Yageo"
 			(at 174.752 46.776 0)
 			(effects
@@
 			)
 		)
-		(property "MANUFACTURER PART NUMBER" "ERJ-2RKF1002X"
+		(property "MANUFACTURER PART NUMBER" "RC0402FR-0710KL"
 			(at 174.752 46.776 0)
 			(effects
@@
 	)
 	(symbol
-		(lib_id "Thunderscope_Rev5:RES 4.7K OHM 1% 1/10W 0402")
+		(lib_id "Thunderscope_Rev5:RES 4.7K OHM 1% 1/16W 0402")
 		(at 111.76 60.96 0)
 		(unit 1)
@@
 			)
 		)
-		(property "Description" "4.7 kOhms ±1% 0.1W, 1/10W Chip Resistor 0402 (1005 Metric) Automotive AEC-Q200 Thick Film"
+		(property "Description" "4.7 kOhms ±1% 0.063W, 1/16W Chip Resistor 0402 (1005 Metric) Moisture Resistant Thick Film"
 			(at 111.76 60.96 0)
 			(effects
@@
 			)
 		)
-		(property "SUPPLIER PART NUMBER 1" "667-ERJ-2RKF4701X"
+		(property "SUPPLIER PART NUMBER 1" "603-RC0402FR-074K7L"
 			(at 106.172 59.904 0)
 			(effects
@@
 			)
 		)
-		(property "MANUFACTURER" "Panasonic"
+		(property "MANUFACTURER" "Yageo"
 			(at 103.008 58.42 0)
 			(effects
@@
 			)
 		)
-		(property "MANUFACTURER PART NUMBER" "ERJ-2RKF4701X"
+		(property "MANUFACTURER PART NUMBER" "RC0402FR-074K7L"
 			(at 103.008 58.42 0)
 			(effects
