File: Hardware/KiCad/Thunderscope_Rev5.3/FPGA_VREG.kicad_sch (KiCad schematic)
At the start: 66 parts, among them U20 TPS62A02, U21 TPS62A02, U22 TPS7A9101, U23 TPS62A02, U8 TPS62A02

Commit message: Added PACKAGE field to symbols without it
Parts:
- L2, L3, L4, L5: PACKAGE (none) -> 1210
- U20, U21, U23, U8: PACKAGE (none) -> SOT-563
- U22: PACKAGE (none) -> 10-DFN (2.5x2.5mm)
Changed lines of the file:
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@@
 			)
 		)
+		(property "PACKAGE" "SOT-563"
+			(at 203.2 88.9 0)
+			(effects
+				(font
+					(size 1.27 1.27)
+				)
+				(hide yes)
+			)
+		)
 		(pin "1"
 		)
@@
 			)
 		)
+		(property "PACKAGE" "SOT-563"
+			(at 58.42 38.1 0)
+			(effects
+				(font
+					(size 1.27 1.27)
+				)
+				(hide yes)
+			)
+		)
 		(pin "5"
 		)
@@
 			)
 		)
+		(property "PACKAGE" "1210"
+			(at 99.06 91.44 0)
+			(effects
+				(font
+					(size 1.27 1.27)
+				)
+				(hide yes)
+			)
+		)
 		(pin "2"
 		)
@@
 			)
 		)
+		(property "PACKAGE" "1210"
+			(at 236.22 40.64 0)
+			(effects
+				(font
+					(size 1.27 1.27)
+				)
+				(hide yes)
+			)
+		)
 		(pin "1"
 		)
@@
 			)
 		)
+		(property "PACKAGE" "SOT-563"
+			(at 66.04 88.9 0)
+			(effects
+				(font
+					(size 1.27 1.27)
+				)
+				(hide yes)
+			)
+		)
 		(pin "1"
 		)
@@
 			)
 		)
+		(property "PACKAGE" "1210"
+			(at 236.22 91.44 0)
+			(effects
+				(font
+					(size 1.27 1.27)
+				)
+				(hide yes)
+			)
+		)
 		(pin "2"
 		)
@@
 			)
 		)
+		(property "PACKAGE" "10-DFN (2.5x2.5mm)"
+			(at 86.36 149.86 0)
+			(effects
+				(font
+					(size 1.27 1.27)
+				)
+				(hide yes)
+			)
+		)
 		(pin "1"
 		)
@@
 			)
 		)
+		(property "PACKAGE" "SOT-563"
+			(at 203.2 38.1 0)
+			(effects
+				(font
+					(size 1.27 1.27)
+				)
+				(hide yes)
+			)
+		)
 		(pin "1"
 		)
@@
 			)
 		)
+		(property "PACKAGE" "1210"
+			(at 91.44 40.64 0)
+			(effects
+				(font
+					(size 1.27 1.27)
+				)
+				(hide yes)
+			)
+		)

Commit message: Added Substitutions Policy Field
Parts:
- C10, C174, C175, C176, C177, C178, C179, C180, C181, C182, C183, C184, C185, C186, C187, C188, C71, C72, C73, C74, C75, C9, R1, R116, R117, R118, R119, R120, R121, R122, R123, R124, R125, R126, R127, R128, R129, R130, R55, R56, R57, R69, R70: Substitutions Policy (none) -> Any Parametric Equivalent
- L2, L3, L4, L5: Substitutions Policy (none) -> ECO Required for Substitution
- U20, U21, U22, U23, U8: Substitutions Policy (none) -> No Substitutions

Commit message: Changed 10k,4.7k,280k resistors MPNs to RC0402FR series
Parts:
- R1, R117, R118, R121, R124, R128, R129, R130: symbol Thunderscope_Rev5:RES 10K OHM 1% 1/10W 0402 -> Thunderscope_Rev5:RES 10K OHM 1% 1/16W 0402; MANUFACTURER Panasonic -> Yageo; MANUFACTURER PART NUMBER ERJ-2RKF1002X -> RC0402FR-0710KL; SUPPLIER PART NUMBER 1 667-ERJ-2RKF1002X -> 603-RC0402FR-0710KL
- R119, R69, R70: symbol Thunderscope_Rev5:RES 4.7K OHM 1% 1/10W 0402 -> Thunderscope_Rev5:RES 4.7K OHM 1% 1/16W 0402; MANUFACTURER Panasonic -> Yageo; MANUFACTURER PART NUMBER ERJ-2RKF4701X -> RC0402FR-074K7L; SUPPLIER PART NUMBER 1 667-ERJ-2RKF4701X -> 603-RC0402FR-074K7L
